Commit message: Corrected the height of laser scanner

File: robots/mpo_500/xacros/sick_s300_laser.xacro (robot description, xacro)
@@ -15,5 +15,5 @@
       </inertial>
       <visual>
-        <origin xyz="0 0 0" rpy="0 0 -1.57" />
+        <origin xyz="0 0 -0.05" rpy="0 0 -1.57" />
         <geometry>
           <mesh filename="package://neo_simulation/robots/mpo_500/meshes/MPO-500-SICK.STL" />
