Commit message: Sensors in Robot model for mp-500 is updated

File: robots/mpo_500/xacros/sick_laser.xacro (robot description, xacro)
@@ -16,5 +16,5 @@
       <visual>
       <!-- SICK S3 sensor: Uncomment/Comment it out if required  -->
-<!--       <origin xyz="0 0 -0.12" rpy="-1.57 0 3.14" />
+      <origin xyz="0 0 -0.12" rpy="-1.57 0 3.14" />
         <geometry>
         <mesh filename="package://neo_simulation/robots/mpo_500/meshes/SICK-S300.dae" scale="0.001 0.001 0.001" />
@@ -26,7 +26,7 @@
         <mesh filename="package://neo_simulation/robots/mpo_500/meshes/SICK-S300.dae" scale="0.001 0.001 0.001" />
         </geometry>
-      </collision> -->
+      </collision>
       <!-- Microscan 3 sensor: Uncomment/Comment it out if required  -->
- <origin xyz="-0.0 0 -0.06" rpy="1.57 0 0" />
+<!--  <origin xyz="-0.0 0 -0.06" rpy="1.57 0 0" />
       <geometry>
       <mesh filename="package://neo_simulation/robots/mpo_500/meshes/SICK-MICROSCAN3.dae" scale="0.001 0.001 0.001" />
@@ -38,5 +38,5 @@
         <mesh filename="package://neo_simulation/robots/mp_500/meshes/SICK-MICROSCAN3.dae" scale="0.001 0.001 0.001" />
         </geometry>
-      </collision>
+      </collision> -->
     </link>
   </xacro:macro>
