Commit message: removed gazebo_ros plugin and transmission tag from mpo_500_gazebo.xacro

File: robots/mpo_500/xacros/mpo_500_gazebo.xacro (robot description, xacro)
@@ -26,40 +26,4 @@
     <material value="Gazebo/Black"/>
   </gazebo>
-  <transmission name="wheel_front_left_trans">
-	<type>transmission_interface/SimpleTransmission</type>
-	<actuator name="wheel_front_left_motor">
-		<mechanicalReduction>1</mechanicalReduction>
-	</actuator>
-	<joint name="wheel_front_left_joint">
-		<hardwareInterface>VelocityJointInterface</hardwareInterface>
-	</joint>
-  </transmission>
-  <transmission name="wheel_front_right_trans">
-	<type>transmission_interface/SimpleTransmission</type>
-	<actuator name="wheel_front_right_motor">
-		<mechanicalReduction>1</mechanicalReduction>
-	</actuator>
-	<joint name="wheel_front_right_joint">
-		<hardwareInterface>VelocityJointInterface</hardwareInterface>
-	</joint>
-  </transmission>
-  <transmission name="wheel_back_left_trans">
-	<type>transmission_interface/SimpleTransmission</type>
-	<actuator name="wheel_back_left_motor">
-		<mechanicalReduction>1</mechanicalReduction>
-	</actuator>
-	<joint name="wheel_back_left_joint">
-		<hardwareInterface>VelocityJointInterface</hardwareInterface>
-	</joint>
-  </transmission>
-  <transmission name="wheel_back_right_trans">
-	<type>transmission_interface/SimpleTransmission</type>
-	<actuator name="wheel_back_right_motor">
-		<mechanicalReduction>1</mechanicalReduction>
-	</actuator>
-	<joint name="wheel_back_right_joint">
-		<hardwareInterface>VelocityJointInterface</hardwareInterface>
-	</joint>
-  </transmission>
   <gazebo reference="sick_s300_laser_front_link">
       <material value="Gazebo/Yellow"/>

Commit message: changed frame names of MPO-500 and updated navigation parameters for MPO-500

File: robots/mpo_500/xacros/mpo_500_gazebo.xacro (robot description, xacro)
@@ -24,5 +24,5 @@
       <sensor type="ray" name="sick_laser_front_sensor">
           <pose>0 0 0 0 0 0</pose>
-          <visualize>true</visualize>
+          <visualize>false</visualize>
           <update_rate>40</update_rate>
           <ray>

File: robots/mpo_500/xacros/omni_wheel.xacro (robot description, xacro)
@@ -2,5 +2,5 @@
 <robot xmlns:xacro="http://www.ros.org/wiki/xacro" name="mpo_500">
   <xacro:macro name="omni_wheel_250" params="name parent *origin">
-   <joint name="${name}_joint" type="continuous">
+   <joint name="${name}_joint" type="fixed">
     <insert_block name="origin" />
     <axis xyz="0 1 0" />
