Commit message: change in mass and inertia values

File: robots/mpo_500/xacros/omni_wheel.xacro (robot description, xacro)
@@ -11,7 +11,7 @@
    <link name="${name}_link" type="wheel">
     <inertial>
-      <mass value="5" />
+      <mass value="0.1" />
       <origin xyz="0 0 0" rpy="0 0 0" />
-      <inertia ixx="0.022166" ixy="0" ixz="0" iyy="0.022166" iyz="0" izz="0.036" />
+      <inertia ixx="0.00044332" ixy="0" ixz="0" iyy="0.00044332" iyz="0" izz="0.00072" />
     </inertial>
     <visual>

Commit message: Collision model for MPO-500 is updated! Works in all the world!

File: robots/mpo_500/xacros/omni_wheel.xacro (robot description, xacro)
@@ -26,5 +26,5 @@
      <origin xyz="0 0 0" rpy="0 0 0" />
      <geometry>
-        <mesh filename="package://neo_simulation/robots/mpo_500/meshes/MPO-500-WHEEL.dae" scale="0.001 0.001 0.001"/>
+       <sphere radius="0.127"/>
      </geometry>
     </collision>
