Commit message: disabled scan visu in simulation and changed joint type

File: robots/mpo_700/xacros/mpo_700_gazebo.xacro (robot description, xacro)
@@ -8,5 +8,5 @@
       <sensor type="ray" name="sick_laser_front_sensor">
           <pose>0 0 0 0 0 0</pose>
-          <visualize>true</visualize>
+          <visualize>false</visualize>
           <update_rate>40</update_rate>
           <ray>

File: robots/mpo_700/xacros/mpo_700_wheel.xacro (robot description, xacro)
@@ -2,5 +2,5 @@
 <robot xmlns:xacro="http://www.ros.org/wiki/xacro" name="mpo_700">
   <xacro:macro name="mpo_700_wheel" params="name parent *origin">
-   <joint name="${name}_joint" type="revolute">
+   <joint name="${name}_joint" type="fixed">
     <insert_block name="origin" />
     <limit effort="1000.0" lower="-1e+16" upper="1e+16" velocity="3.5"/>
