Commit message: Collision for wheels are updated for better contact solution between the wheel and the ground

File: robots/mpo_700/xacros/mpo_700_wheel.xacro (robot description, xacro)
@@ -4,5 +4,5 @@
    <joint name="${name}_joint" type="revolute">
     <insert_block name="origin" />
-    <limit effort="1000.0" lower="-1e+16" upper="1e+16" velocity="20.5"/>
+    <limit effort="1000.0" lower="-1e+16" upper="1e+16" velocity="30.5"/>
     <axis xyz="0 -1 0" />
     <joint_properties damping="30" friction="110"/>
@@ -27,5 +27,6 @@
      <origin xyz="0 0 0" rpy="0 0 0" />
      <geometry>
-        <mesh filename="package://neo_simulation/robots/mpo_700/meshes/MPO-700-WHEEL.dae" scale="0.001 0.001 0.001"/>
+      <sphere radius="0.09" />
+        <!-- <mesh filename="package://neo_simulation/robots/mpo_700/meshes/MPO-700-WHEEL.dae" scale="0.001 0.001 0.001"/> -->
      </geometry>
     </collision>
