Commit message: mp_400 files are updated

File: robots/mp_400/mp_400.urdf.xacro (robot description, xacro)
@@ -14,20 +14,20 @@
   <!-- Wheel Macro -->
   <xacro:caster_wheel name="wheel_front_right" parent="base_link">
-    <origin xyz="0 0. -0.14" rpy="-1.57 0 -1.57" />
+    <origin xyz="0.2 0.155 -0.1" rpy="0 0 0" />
   </xacro:caster_wheel>
   <xacro:caster_wheel name="wheel_front_left" parent="base_link">
-    <origin xyz="-0. -0.32 -0.14" rpy="-1.57 0 -1.57" />
+    <origin xyz="0.2 -0.155 -0.1" rpy="0 0 0" />
   </xacro:caster_wheel>
   <xacro:caster_wheel name="wheel_back_right" parent="base_link">
-    <origin xyz="-0.4 0 -0.14" rpy="-1.57 0 -1.57" />
+    <origin xyz="-0.2 0.155 -0.1" rpy="0 0 0" />
   </xacro:caster_wheel>
    <xacro:caster_wheel name="wheel_back_left" parent="base_link">
-    <origin xyz="-0.4 -0.32  -0.14" rpy="-1.57 0 -1.57" />
+    <origin xyz="-0.2 -0.155  -0.1" rpy="0 0 0" />
   </xacro:caster_wheel>
   <xacro:fixed_wheel name="fixed_wheel_right" parent="base_link">
-    <origin xyz="0 0.0 0.0" rpy="1.57 0 1.57" />
+    <origin xyz="0 0.2 -0.1" rpy="0 0 0" />
   </xacro:fixed_wheel>
   <xacro:fixed_wheel name="fixed_wheel_left" parent="base_link">
-    <origin xyz="0 0.0 0.0" rpy="1.57 0 -1.57" />
+    <origin xyz="0 -0.2 -0.1" rpy="0 0 3.14" />
   </xacro:fixed_wheel>
   <!--+++++++++++++++++++laserscanner_link++++++++++++++++++++++++-->

File: robots/mp_400/xacros/mp_400_body.xacro (robot description, xacro)
@@ -10,5 +10,5 @@
     </inertial>
       <visual name='body'>
-      <origin xyz="0.0 0.0 -0.16" rpy="-1.57 0 1.57" /><!-- for stl -->
+      <origin xyz="0.0 0.0 -0.18" rpy="-1.57 0 1.57" /><!-- for stl -->
         <geometry>
             <mesh filename="package://neo_simulation/robots/mp_400/meshes/MP-400-BODY.dae" scale="0.001 0.001 0.001"/>

File: robots/mp_400/xacros/mp_400_caster_wheel.xacro (robot description, xacro)
@@ -16,10 +16,10 @@
       <inertia ixx="13.177588678963057" ixy="-0.00000019386313414965295" ixz="-0.0000007636494859403484" iyy="8.48847991205267" iyz="-2.366298925984707" izz="7.157972023102095" />
     </inertial>
-      <visual name='castor_wheel'>
-    <origin xyz="0. 0.012 0." rpy="0 0 0" /><!-- for STL -->
-        <geometry>
+      <visual name='caster_wheel'>
+    <origin xyz="-0.2 -0.16 -0.07" rpy="-1.57 0 -1.57" />
+    <geometry>
             <mesh filename="package://neo_simulation/robots/mp_400/meshes/MP-400-WHEEL.dae" scale="0.001 0.001 0.001"/>
-        </geometry>
-      </visual>
+    </geometry>
+    </visual>
     <collision>
       <origin xyz="0 0. 0" rpy="0 0 0" />
@@ -28,5 +28,5 @@
       </geometry>
     </collision>
-</link>
+    </link>
   </xacro:macro>
 </robot>

File: robots/mp_400/xacros/mp_400_fixed_wheel.xacro (robot description, xacro)
@@ -17,5 +17,5 @@
     </inertial>
       <visual name='fixed_wheel'>
-    <origin xyz="0 0.0 0" rpy=" 0 0 0" />
+    <origin xyz="-0. -0.2 0.074" rpy="1.57 0 1.57" />
         <geometry>
             <mesh filename="package://neo_simulation/robots/mp_400/meshes/MP-400-FIXED-WHEEL.dae" scale="0.001 0.001 0.001"/>

Commit message: Further modifications for Mp 400

File: robots/mp_400/mp_400.urdf.xacro (robot description, xacro)
@@ -34,6 +34,6 @@
    <!-- SENSORS -->
   <xacro:include filename="$(find neo_simulation)/robots/mp_400/xacros/sick_laser.xacro" />
-  <xacro:sick_laser_v0 name="laserscanner_link" parent="base_link" ros_topic="sick_300/scan">
-    <origin xyz="0.230 0 0.11" rpy="0 0 0" />
+  <xacro:sick_laser_v0 name="laserscanner" parent="base_link" ros_topic="sick_300/scan">
+    <origin xyz="0.230 0 0.110" rpy="0 3.14 3.14" />
   </xacro:sick_laser_v0>
 </robot>

File: robots/mp_400/xacros/mp_400_body.xacro (robot description, xacro)
@@ -10,5 +10,5 @@
     </inertial>
       <visual name='body'>
-      <origin xyz="0.0 0.0 -0.18" rpy="-1.57 0 1.57" /><!-- for stl -->
+      <origin xyz="0.0 0.0 -0.19" rpy="-1.57 0 1.57" /><!-- for stl -->
         <geometry>
             <mesh filename="package://neo_simulation/robots/mp_400/meshes/MP-400-BODY.dae" scale="0.001 0.001 0.001"/>

File: robots/mp_400/xacros/mp_400_gazebo.xacro (robot description, xacro)
@@ -13,6 +13,6 @@
     <self_collide>false</self_collide>
   </gazebo>
-  <gazebo reference="laserscanner_front_link">
-      <sensor type="ray" name="laserscanner_front_link">
+  <gazebo reference="laserscanner_link">
+      <sensor type="ray" name="laserscanner_link">
           <pose>0 0 0 0 0 0</pose>
           <visualize>false</visualize>
@@ -42,7 +42,7 @@
             </noise>
           </ray>
-          <plugin name="laserscanner_front_link" filename="libgazebo_ros_laser.so">
+          <plugin name="laserscanner_link" filename="libgazebo_ros_laser.so">
             <topicName>sick_s300_front/scan</topicName>
-            <frameName>laserscanner_front_link</frameName>
+            <frameName>laserscanner_link</frameName>
           </plugin>
         </sensor>

File: robots/mp_400/xacros/sick_laser.xacro (robot description, xacro)
@@ -16,5 +16,5 @@
       <visual>
       <!-- SICK S3 sensor: Uncomment/Comment it out if required  -->
-      <origin xyz="0 0 0." rpy="1.57 0 3.14" />
+      <origin xyz="0 0 0.08" rpy="-1.57 0 3.14" />
         <geometry>
         <mesh filename="package://neo_simulation/robots/mp_400/meshes/SICK-S300.dae" scale="0.001 0.001 0.001" />
@@ -22,5 +22,5 @@
       </visual>
       <collision>
-        <origin xyz="0 0 0" rpy="1.57 0 3.14" />
+        <origin xyz="0 0 0" rpy="-1.57 0 3.14" />
         <geometry>
         <mesh filename="package://neo_simulation/robots/mp_400/meshes/SICK-S300.dae" scale="0.001 0.001 0.001" />

Commit message: Robot model for mp-400 is updated

File: robots/mp_400/mp_400.urdf.xacro (robot description, xacro)
@@ -13,26 +13,26 @@
   </xacro:mp_400_base>
   <!-- Wheel Macro -->
+  <xacro:caster_wheel name="wheel_front_left" parent="base_link">
+    <origin xyz="0.165 0.155 0.036" rpy="0 0 1.57" />
+  </xacro:caster_wheel>
+  <xacro:caster_wheel name="wheel_back_left" parent="base_link">
+    <origin xyz="-0.220 0.155 0.036" rpy="0 0 1.57" />
+  </xacro:caster_wheel>
   <xacro:caster_wheel name="wheel_front_right" parent="base_link">
-    <origin xyz="0.2 0.155 -0.1" rpy="0 0 0" />
+    <origin xyz="0.165 -0.155 0.036" rpy="0 0 1.57" />
   </xacro:caster_wheel>
-  <xacro:caster_wheel name="wheel_front_left" parent="base_link">
-    <origin xyz="0.2 -0.155 -0.1" rpy="0 0 0" />
-  </xacro:caster_wheel>
-  <xacro:caster_wheel name="wheel_back_right" parent="base_link">
-    <origin xyz="-0.2 0.155 -0.1" rpy="0 0 0" />
-  </xacro:caster_wheel>
-   <xacro:caster_wheel name="wheel_back_left" parent="base_link">
-    <origin xyz="-0.2 -0.155  -0.1" rpy="0 0 0" />
+   <xacro:caster_wheel name="wheel_back_right" parent="base_link">
+    <origin xyz="-0.220 -0.155 0.036" rpy="0 0 1.57" />
   </xacro:caster_wheel>
   <xacro:fixed_wheel name="fixed_wheel_right" parent="base_link">
-    <origin xyz="0 0.2 -0.1" rpy="0 0 0" />
+    <origin xyz="0. -0.26 0.075" rpy="0 0 -1.57" />
   </xacro:fixed_wheel>
   <xacro:fixed_wheel name="fixed_wheel_left" parent="base_link">
-    <origin xyz="0 -0.2 -0.1" rpy="0 0 3.14" />
+    <origin xyz="-0. 0.26 0.075" rpy="0 0 1.57" />
   </xacro:fixed_wheel>
   <!--+++++++++++++++++++laserscanner_link++++++++++++++++++++++++-->
    <!-- SENSORS -->
   <xacro:include filename="$(find neo_simulation)/robots/mp_400/xacros/sick_laser.xacro" />
-  <xacro:sick_laser_v0 name="laserscanner" parent="base_link" ros_topic="sick_300/scan">
+  <xacro:sick_laser_v0 name="laserscanner_1" parent="base_link" ros_topic="sick/scan">
     <origin xyz="0.230 0 0.110" rpy="0 3.14 3.14" />
   </xacro:sick_laser_v0>

File: robots/mp_400/xacros/mp_400_body.xacro (robot description, xacro)
@@ -4,11 +4,12 @@
     <link name="${name}">
     <inertial>
-      <mass value="5.67" />
-        <origin xyz="0 0 0.0" rpy="0 0 0"/>
-        <inertia ixx="0.07" ixy="0.0" ixz="0.0"
-                 iyy="0.08" iyz="0.0" izz="0.1" />
+        <mass value="30" />
+        <origin xyz="0 0 0" rpy="0 0 0"/>
+        <inertia ixx="1.71402" ixy="0.0" ixz="0.0"
+                 iyy="0.8856" iyz="0.0"
+                 izz="2.5725" />
     </inertial>
       <visual name='body'>
-      <origin xyz="0.0 0.0 -0.19" rpy="-1.57 0 1.57" /><!-- for stl -->
+      <origin xyz="0.0 0.0 0." rpy="0 0 1.57" />
         <geometry>
             <mesh filename="package://neo_simulation/robots/mp_400/meshes/MP-400-BODY.dae" scale="0.001 0.001 0.001"/>
@@ -18,5 +19,5 @@
       </visual>
       <collision name='body_collision'>
-        <origin xyz="0.0 0.0 0.0" rpy="-1.57 0 1.57" />
+        <origin xyz="0.0 0.0 0.0" rpy="0 0 1.57" />
         <geometry>
           <mesh filename="package://neo_simulation/robots/mp_400/meshes/MP-400-BODY.dae" scale="0.001 0.001 0.001"/>

File: robots/mp_400/xacros/mp_400_caster_wheel.xacro (robot description, xacro)
@@ -17,7 +17,7 @@
     </inertial>
       <visual name='caster_wheel'>
-    <origin xyz="-0.2 -0.16 -0.07" rpy="-1.57 0 -1.57" />
+    <origin xyz="0 0 0" rpy="0 0 0" />
     <geometry>
-            <mesh filename="package://neo_simulation/robots/mp_400/meshes/MP-400-WHEEL.dae" scale="0.001 0.001 0.001"/>
+            <mesh filename="package://neo_simulation/robots/mp_400/meshes/MP-400-CASTER-WHEEL.dae" scale="0.001 0.001 0.001"/>
     </geometry>
     </visual>
@@ -25,5 +25,5 @@
       <origin xyz="0 0. 0" rpy="0 0 0" />
       <geometry>
-            <mesh filename="package://neo_simulation/robots/mp_400/meshes/MP-400-WHEEL.dae" scale="0.001 0.001 0.001"/>
+            <mesh filename="package://neo_simulation/robots/mp_400/meshes/MP-400-CASTER-WHEEL.dae" scale="0.001 0.001 0.001"/>
       </geometry>
     </collision>

File: robots/mp_400/xacros/mp_400_fixed_wheel.xacro (robot description, xacro)
@@ -17,5 +17,5 @@
     </inertial>
       <visual name='fixed_wheel'>
-    <origin xyz="-0. -0.2 0.074" rpy="1.57 0 1.57" />
+    <origin xyz="0 0 0.0" rpy="0 0 0" />
         <geometry>
             <mesh filename="package://neo_simulation/robots/mp_400/meshes/MP-400-FIXED-WHEEL.dae" scale="0.001 0.001 0.001"/>

File: robots/mp_400/xacros/mp_400_gazebo.xacro (robot description, xacro)
@@ -13,6 +13,6 @@
     <self_collide>false</self_collide>
   </gazebo>
-  <gazebo reference="laserscanner_link">
-      <sensor type="ray" name="laserscanner_link">
+  <gazebo reference="laserscanner_1_link">
+      <sensor type="ray" name="laserscanner_1_link">
           <pose>0 0 0 0 0 0</pose>
           <visualize>false</visualize>
@@ -42,7 +42,7 @@
             </noise>
           </ray>
-          <plugin name="laserscanner_link" filename="libgazebo_ros_laser.so">
-            <topicName>sick_s300_front/scan</topicName>
-            <frameName>laserscanner_link</frameName>
+          <plugin name="laserscanner_1_link" filename="libgazebo_ros_laser.so">
+            <topicName>sick/scan</topicName>
+            <frameName>laserscanner_1_link</frameName>
           </plugin>
         </sensor>
@@ -53,4 +53,5 @@
       <odometryTopic>odom</odometryTopic>
       <odometryFrame>odom</odometryFrame>
+      <odometryRate>20.0</odometryRate>
       <robotBaseFrame>base_link</robotBaseFrame>
     </plugin>

File: robots/mp_400/xacros/sick_laser.xacro (robot description, xacro)
@@ -16,5 +16,5 @@
       <visual>
       <!-- SICK S3 sensor: Uncomment/Comment it out if required  -->
-      <origin xyz="0 0 0.08" rpy="-1.57 0 3.14" />
+<!--       <origin xyz="0 0 -0.11" rpy="-1.57 0 3.14" />
         <geometry>
         <mesh filename="package://neo_simulation/robots/mp_400/meshes/SICK-S300.dae" scale="0.001 0.001 0.001" />
@@ -22,11 +22,11 @@
       </visual>
       <collision>
-        <origin xyz="0 0 0" rpy="-1.57 0 3.14" />
+        <origin xyz="0 0 -0.11" rpy="-1.57 0 3.14" />
         <geometry>
         <mesh filename="package://neo_simulation/robots/mp_400/meshes/SICK-S300.dae" scale="0.001 0.001 0.001" />
         </geometry>
-      </collision>
+      </collision> -->
       <!-- Microscan 3 sensor: Uncomment/Comment it out if required  -->
-<!--  <origin xyz="-0.0 0 0.06" rpy="-1.57 0 0" />
+ <origin xyz="-0.0 0 -0.06" rpy="1.57 0 0" />
       <geometry>
       <mesh filename="package://neo_simulation/robots/mp_400/meshes/SICK-MICROSCAN3.dae" scale="0.001 0.001 0.001" />
@@ -34,9 +34,9 @@
       </visual>
       <collision>
- <origin xyz="-0.0 0 0.06" rpy="-1.57 0 0" />
+ <origin xyz="-0.0 0 -0.06" rpy="1.57 0 0" />
       <geometry>
         <mesh filename="package://neo_simulation/robots/mp_400/meshes/SICK-MICROSCAN3.dae" scale="0.001 0.001 0.001" />
         </geometry>
-      </collision> -->
+      </collision>
     </link>
   </xacro:macro>
