Commit message: Models updated and works well on eband-local planner

File: robots/mp_400/mp_400.urdf.xacro (robot description, xacro)
@@ -9,5 +9,7 @@
 <xacro:include filename="$(find neo_simulation)/robots/mp_400/xacros/mp_400_caster_wheel.xacro" />
 <!--+++++++++++++++++++left_wheel_link++++++++++++++++++++++++-->
-<xacro:include filename="$(find neo_simulation)/robots/mp_400/xacros/mp_400_fixed_wheel.xacro" />
+<xacro:include filename="$(find neo_simulation)/robots/mp_400/xacros/mp_400_fixed_wheel_left.xacro" />
+<!--+++++++++++++++++++right_wheel_link++++++++++++++++++++++++-->
+<xacro:include filename="$(find neo_simulation)/robots/mp_400/xacros/mp_400_fixed_wheel_right.xacro" />
   <xacro:mp_400_base name="base_link">
   </xacro:mp_400_base>
@@ -25,10 +27,10 @@
     <origin xyz="-0.220 -0.155 0.036" rpy="0 0 1.57" />
   </xacro:caster_wheel>
-  <xacro:fixed_wheel name="fixed_wheel_right" parent="base_link">
-    <origin xyz="0. -0.26 0.075" rpy="0 0 -1.57" />
-  </xacro:fixed_wheel>
-  <xacro:fixed_wheel name="fixed_wheel_left" parent="base_link">
-    <origin xyz="-0. 0.26 0.075" rpy="0 0 1.57" />
-  </xacro:fixed_wheel>
+  <xacro:fixed_wheel_right name="fixed_wheel_right" parent="base_link">
+    <origin xyz="0. -0.26 0.074" rpy="0 0 1.57" />
+  </xacro:fixed_wheel_right>
+  <xacro:fixed_wheel_left name="fixed_wheel_left" parent="base_link">
+    <origin xyz="-0. 0.26 0.074" rpy="0 0 1.57" />
+  </xacro:fixed_wheel_left>
   <!--+++++++++++++++++++laserscanner_link++++++++++++++++++++++++-->
    <!-- SENSORS -->

File: robots/mp_400/xacros/mp_400_body.xacro (robot description, xacro)
@@ -3,5 +3,5 @@
   <xacro:macro name="mp_400_base" params="name">
     <link name="${name}">
-    <inertial>
+  <inertial>
         <mass value="30" />
         <origin xyz="0 0 0" rpy="0 0 0"/>
@@ -9,5 +9,5 @@
                  iyy="0.8856" iyz="0.0"
                  izz="2.5725" />
-    </inertial>
+</inertial>
       <visual name='body'>
       <origin xyz="0.0 0.0 0." rpy="0 0 1.57" />
@@ -26,4 +26,13 @@
       </collision>
     </link>
+  <gazebo reference="${name}">
+    <kp>10000.0</kp>
+    <kd>10.0</kd>
+    <mu1>1.5</mu1>
+    <mu2>1.5</mu2>
+    <fdir1>.1 0 0</fdir1>
+    <maxVel>10.0</maxVel>
+    <minDepth>0.0005</minDepth>
+</gazebo>
   </xacro:macro>
 </robot>

File: robots/mp_400/xacros/mp_400_caster_wheel.xacro (robot description, xacro)
@@ -4,6 +4,6 @@
    <joint name="${name}_joint" type="fixed">
     <insert_block name="origin" />
-    <axis xyz="0 1 0" />
-    <joint_properties damping="1" friction="1" />
+    <axis xyz="-1 0 0" />
+    <joint_properties damping="1." friction="1.0" />
     <limit effort="1000.0" lower="-1e+16" upper="1e+16" velocity="3.5"/>
     <parent link="${parent}" />
@@ -11,9 +11,10 @@
    </joint>
    <link name="${name}_link" type="wheel">
-    <inertial>
-      <mass value="3.5" />
-      <origin xyz="0.000000010 -0.045437214 -0.073569633" rpy="0 0 0" />
-      <inertia ixx="13.177588678963057" ixy="-0.00000019386313414965295" ixz="-0.0000007636494859403484" iyy="8.48847991205267" iyz="-2.366298925984707" izz="7.157972023102095" />
-    </inertial>
+   <inertial>
+        <mass value="1.4"/>
+        <inertia ixx="0.00499743171" ixy="0.00000004464" ixz="-0.00000002245"
+                 iyy="0.00499741733" iyz="-0.00000000164"
+                 izz="0.00839239692"/>
+</inertial>
       <visual name='caster_wheel'>
     <origin xyz="0 0 0" rpy="0 0 0" />
@@ -29,4 +30,14 @@
     </collision>
     </link>
+<gazebo reference="${name}_link">
+      <kp>10000.0</kp>
+      <kd>10.0</kd>
+      <mu1>0.5</mu1>
+      <mu2>0.2</mu2>
+      <fdir1>.5 0 0</fdir1>
+      <maxVel>3.0</maxVel>
+      <minDepth>0.00</minDepth>
+      <implicitSpringDamper>3</implicitSpringDamper>
+</gazebo>
   </xacro:macro>
 </robot>

File: robots/mp_400/xacros/mp_400_gazebo.xacro (robot description, xacro)
@@ -49,11 +49,31 @@
   </gazebo>
   <gazebo>
-    <plugin name="mp_400_controller" filename="libgazebo_ros_planar_move.so">
-      <commandTopic>cmd_vel</commandTopic>
-      <odometryTopic>odom</odometryTopic>
-      <odometryFrame>odom</odometryFrame>
-      <odometryRate>20.0</odometryRate>
-      <robotBaseFrame>base_link</robotBaseFrame>
+    <plugin name="diff_dirve_controller" filename="libgazebo_ros_diff_drive.so">
+        <alwaysOn>true</alwaysOn>
+        <updateRate>40</updateRate>
+        <legacyMode>false</legacyMode>
+        <torque>5</torque>
+        <leftJoint>fixed_wheel_left_joint</leftJoint>
+        <rightJoint>fixed_wheel_right_joint</rightJoint>
+        <wheelSeparation>0.529</wheelSeparation>
+        <wheelDiameter>0.15</wheelDiameter>
+        <commandTopic>cmd_vel</commandTopic>
+        <rosDebugLevel>na</rosDebugLevel>
+        <odometryTopic>odom</odometryTopic>
+        <odometryFrame>odom</odometryFrame>
+        <robotBaseFrame>base_link</robotBaseFrame>
+        <publishWheelTF>true</publishWheelTF>
+        <publishWheelJointState>true</publishWheelJointState>
+        <wheelAcceleration>6.0</wheelAcceleration>
+        <wheelTorque>5</wheelTorque>
+        <odometrySource>world</odometrySource>
+        <publishTf>1</publishTf>
+        <publishOdomTF>true</publishOdomTF>
     </plugin>
   </gazebo>
+<!-- <gazebo>
+  <plugin name="gazebo_ros_control" filename="libgazebo_ros_control.so">
+    <robotNamespace>/mp_400</robotNamespace>
+  </plugin>
+</gazebo> -->
 </robot>

File: robots/mp_400/xacros/sick_laser.xacro (robot description, xacro)
@@ -10,5 +10,5 @@
     <link name="${name}_link" type="laser">
       <inertial>
-        <mass value="0.001" />
+        <mass value="0.0001" />
         <origin xyz="0 0 0" rpy="0 0 0" />
         <inertia ixx="0.0001" ixy="0" ixz="0" iyy="0.000001" iyz="0" izz="0.0001" />

File: robots/mp_500/mp_500.urdf.xacro (robot description, xacro)
@@ -14,11 +14,11 @@
   <!-- Wheel Macro -->
   <xacro:caster_wheel name="caster_wheel" parent="base_link">
-    <origin xyz="-0.43 0. 0.171" rpy="-1.570796 0 1.570796 " />
+    <origin xyz="-0.43 0. 0.176" rpy="-1.570796 0 1.570796 " />
   </xacro:caster_wheel>
   <xacro:fixed_wheel name="wheel_right" parent="base_link">
-    <origin xyz="0. -0.25 0.125" rpy="0 0 1.570796" />
+    <origin xyz="0. -0.25 0.13" rpy="0 0 -1.570796" />
   </xacro:fixed_wheel>
   <xacro:fixed_wheel name="wheel_left" parent="base_link">
-    <origin xyz="0. 0.25 0.125" rpy="0 0 -1.570796" />
+    <origin xyz="0. 0.25 0.13" rpy="0 0 -1.570796" />
   </xacro:fixed_wheel>
  <!--+++++++++++++++++++laserscanner_front_link++++++++++++++++++++++++-->

File: robots/mp_500/xacros/mp_500_body.xacro (robot description, xacro)
@@ -4,10 +4,10 @@
     <link name="${name}">
   <inertial>
-  <mass value="56.4" />
-  <origin xyz="0.000122063 0.106046383 0.229559509" rpy="0 0 0"/>
-  <inertia ixx="1934.300108107" ixy="-1.1189088783480243" ixz="-0.40794571883788144"
-           iyy="1331.584507173302" iyz="-53.61566974072236"
-           izz="2565.65991901786" />
-  </inertial>
+        <mass value="5" />
+        <origin xyz="0 0 0" rpy="0 0 0"/>
+        <inertia ixx="1.71402" ixy="0.0" ixz="0.0"
+                 iyy="0.8856" iyz="0.0"
+                 izz="2.5725" />
+</inertial>
   <visual name='body'>
   <origin xyz="0.0 0.0 0" rpy="0 0 1.570796" />
@@ -23,4 +23,13 @@
   </collision>
   </link>
+<gazebo reference="${name}_link">
+    <kp>1000.0</kp>
+    <kd>10.0</kd>
+    <mu1>200</mu1>
+    <mu2>100</mu2>
+    <fdir1>0.5 0 0</fdir1>
+    <maxVel>10.0</maxVel>
+    <minDepth>0.0005</minDepth>
+    </gazebo>
   </xacro:macro>
 </robot>

File: robots/mp_500/xacros/mp_500_caster_wheel.xacro (robot description, xacro)
@@ -4,15 +4,17 @@
    <joint name="${name}_joint" type="fixed">
     <insert_block name="origin" />
+        <axis xyz="0 -1 0" />
       <limit effort="1000.0" lower="-1e+16" upper="1e+16" velocity="3.5"/>
       <parent link="${parent}" />
       <child link="${name}_link" />
-      <joint_properties damping="1" friction="1" />
+      <joint_properties damping="1.0" friction="1.0" />
    </joint>
    <link name="${name}_link" type="wheel">
     <inertial>
-      <mass value="3.5" />
-      <origin xyz="0.000000010 -0.045437214 -0.073569633" rpy="0 0 0" />
-      <inertia ixx="13.177588678963057" ixy="-0.00000019386313414965295" ixz="-0.0000007636494859403484" iyy="8.48847991205267" iyz="-2.366298925984707" izz="7.157972023102095" />
-    </inertial>
+        <mass value="1.82362"/>
+        <inertia ixx="0.00499743171" ixy="0.00000004464" ixz="-0.00000002245"
+                 iyy="0.00499741733" iyz="0.00000000164"
+izz="0.00839239692"/>
+</inertial>
       <visual name='castor_wheel'>
     <origin xyz="0 0 0" rpy="0 0 0" />
@@ -28,4 +30,13 @@
     </collision>
 </link>
+<gazebo reference="${name}_link">
+      <kp>8000.0</kp>
+      <kd>1460.0</kd>
+      <mu1>0.5</mu1>
+      <mu2>0.2</mu2>
+      <fdir1>1 0 0</fdir1>
+      <maxVel>3.0</maxVel>
+      <minDepth>0.00</minDepth>
+</gazebo>
   </xacro:macro>
 </robot>

File: robots/mp_500/xacros/mp_500_fixed_wheel.xacro (robot description, xacro)
@@ -2,8 +2,9 @@
 <robot xmlns:xacro="http://www.ros.org/wiki/xacro" name="mp_500">
   <xacro:macro name="fixed_wheel" params="name parent *origin">
-   <joint name="${name}_joint" type="fixed">
+   <joint name="${name}_joint" type="revolute">
     <insert_block name="origin" />
-    <axis xyz="0 1 0" />
-    <joint_properties damping="1" friction="1" />
+    <limit effort="1000.0" lower="-1e+16" upper="1e+16" velocity="3.5"/>
+    <axis xyz="-1 0 0" />
+    <joint_properties damping="0" friction="0.0" />
     <parent link="${parent}" />
     <child link="${name}_link" />
@@ -11,9 +12,10 @@
    <link name="${name}_link" type="wheel">
     <inertial>
-      <mass value="5.3" />
-      <origin xyz="0.000000143 -0.04248127 0.073712479" rpy="0 0 0" />
-      <inertia ixx="46.639251649513" ixy="0.0000023227242816" ixz="-0.000001619382358553578" iyy="25.926276619468705" iyz="-0.0000008220581770145895" izz="25.78086321479202" />
-    </inertial>
-      <visual>
+        <mass value="1.82362"/>
+        <inertia ixx="0.00399743171" ixy="0.00000004464" ixz="-0.00000002245"
+                 iyy="0.00399741733" iyz="-0.00000000164"
+                 izz="0.00739239692"/>
+</inertial>
+    <visual>
     <origin xyz="0 0 0" rpy="0 0 0" />
         <geometry>
@@ -28,4 +30,11 @@
     </collision>
 </link>
+  <gazebo reference="${name}_link">
+      <mu1 value = "300.0"/>
+      <mu2 value = "100.0"/>
+      <kp value="8000.0" />
+      <kd value="1460.0" />
+      <fdir1 value="0.5 0 0"/>
+</gazebo>
   </xacro:macro>
 </robot>

File: robots/mp_500/xacros/mp_500_gazebo.xacro (robot description, xacro)
@@ -45,10 +45,25 @@
   </gazebo>
   <gazebo>
-    <plugin name="mp_500_controller" filename="libgazebo_ros_planar_move.so">
-      <commandTopic>cmd_vel</commandTopic>
-      <odometryTopic>odom</odometryTopic>
-      <odometryFrame>odom</odometryFrame>
-      <odometryRate>20.0</odometryRate>
-      <robotBaseFrame>base_link</robotBaseFrame>
+    <plugin name="diff_dirve_controller" filename="libgazebo_ros_diff_drive.so">
+        <alwaysOn>true</alwaysOn>
+        <updateRate>100</updateRate>
+        <legacyMode>false</legacyMode>
+        <torque>2.5</torque>
+        <leftJoint>wheel_left_joint</leftJoint>
+        <rightJoint>wheel_right_joint</rightJoint>
+        <wheelSeparation>0.592</wheelSeparation>
+        <wheelDiameter>0.260</wheelDiameter>
+        <commandTopic>cmd_vel</commandTopic>
+        <rosDebugLevel>na</rosDebugLevel>
+        <odometryTopic>odom</odometryTopic>
+        <odometryFrame>odom</odometryFrame>
+        <robotBaseFrame>base_link</robotBaseFrame>
+        <publishWheelTF>true</publishWheelTF>
+        <publishWheelJointState>true</publishWheelJointState>
+        <wheelAcceleration>0</wheelAcceleration>
+        <wheelTorque>200</wheelTorque>
+        <odometrySource>world</odometrySource>
+        <publishTf>1</publishTf>
+        <publishOdomTF>true</publishOdomTF>
     </plugin>
   </gazebo>

File: robots/mp_500/xacros/sick_laser.xacro (robot description, xacro)
@@ -10,5 +10,5 @@
     <link name="${name}_link" type="laser">
       <inertial>
-        <mass value="0.001" />
+        <mass value="0.0001" />
         <origin xyz="0 0 0" rpy="0 0 0" />
         <inertia ixx="0.0001" ixy="0" ixz="0" iyy="0.000001" iyz="0" izz="0.0001" />
