Commit message: Ur10 for MMO 500 has been updated

File: robots/mmo_500/urdf/ur10.urdf.xacro (robot description, xacro)
@@ -85,5 +85,5 @@
         <limit lower="${shoulder_pan_lower_limit}" upper="${shoulder_pan_upper_limit}" effort="330.0" velocity="2.16"/>
       </xacro:if>
-      <dynamics damping="0.5" friction="0.0"/>
+      <dynamics damping="0.5" friction="10.0"/>
     </joint>
     <link name="shoulder_link">
@@ -113,5 +113,5 @@
         <limit lower="${shoulder_lift_lower_limit}" upper="${shoulder_lift_upper_limit}" effort="330.0" velocity="2.16"/>
       </xacro:if>
-      <dynamics damping="0.5" friction="0.0"/>
+      <dynamics damping="0.5" friction="10.0"/>
     </joint>
     <link name="upper_arm_link">
@@ -141,5 +141,5 @@
         <limit lower="${elbow_joint_lower_limit}" upper="${elbow_joint_upper_limit}" effort="150.0" velocity="3.15"/>
       </xacro:if>
-      <dynamics damping="0.5" friction="0.0"/>
+      <dynamics damping="0.5" friction="10.0"/>
     </joint>
     <link name="forearm_link">
@@ -169,5 +169,5 @@
         <limit lower="${wrist_1_lower_limit}" upper="${wrist_1_upper_limit}" effort="54.0" velocity="3.2"/>
       </xacro:if>
-      <dynamics damping="0.5" friction="0.0"/>
+      <dynamics damping="0.5" friction="10.0"/>
     </joint>
     <link name="wrist_1_link">
@@ -197,5 +197,5 @@
         <limit lower="${wrist_2_lower_limit}" upper="${wrist_2_upper_limit}" effort="54.0" velocity="3.2"/>
       </xacro:if>
-      <dynamics damping="0.5" friction="0.0"/>
+      <dynamics damping="0.5" friction="10.0"/>
     </joint>
     <link name="wrist_2_link">
@@ -225,5 +225,5 @@
         <limit lower="${wrist_3_lower_limit}" upper="${wrist_3_upper_limit}" effort="54.0" velocity="3.2"/>
       </xacro:if>
-      <dynamics damping="0.5" friction="0.0"/>
+      <dynamics damping="0.5" friction="10.0"/>
     </joint>
     <link name="wrist_3_link">
@@ -508,5 +508,5 @@
     <child link="H1_F1_palm_link"/>
   </joint>
-  <joint name="H1_F1J1" type="revolute">
+  <joint name="H1_F1J1" type="fixed">
     <origin rpy="-8.8818E-16 -1.0061E-16 0.022402" xyz="0 0 0.00016528"/>
     <axis xyz="0 0 1"/>
@@ -514,7 +514,7 @@
     <child link="H1_F1_ur10_base_link"/>
     <limit effort="50" lower="-0.785398163397" upper="0.785398163397" velocity="1.0"/>
-    <dynamics damping="0.0" friction="0.0"/>
-  </joint>
-  <joint name="H1_F1J2" type="revolute">
+    <dynamics damping="0.0" friction="10.0"/>
+  </joint>
+  <joint name="H1_F1J2" type="fixed">
     <origin rpy="0.070695 6.9389E-16 2.0947E-16" xyz="0 0.035 0.11683"/>
     <axis xyz="1 0 0"/>
@@ -522,5 +522,5 @@
     <child link="H1_F1_link_1"/>
     <limit effort="50" lower="-1.3962634016" upper="1.0471975512" velocity="1.0"/>
-    <dynamics damping="0.0" friction="0.0"/>
+    <dynamics damping="0.0" friction="10.0"/>
   </joint>
   <joint name="H1_F1J3" type="revolute">
@@ -530,24 +530,6 @@
     <child link="H1_F1_link_2"/>
     <limit effort="50" lower="-1.0471975512" upper="1.57079632679" velocity="1.0"/>
-    <dynamics damping="0.0" friction="0.0"/>
-  </joint>
-  <transmission name="H1_F1J1_transmission">
-    <type>transmission_interface/SimpleTransmission</type>
-    <actuator name="H1_F1J1">
-      <mechanicalReduction>1</mechanicalReduction>
-    </actuator>
-    <joint name="H1_F1J1">
-      <hardwareInterface>hardware_interface/PositionJointInterface</hardwareInterface>
-    </joint>
-  </transmission>
-  <transmission name="H1_F1J2_transmission">
-    <type>transmission_interface/SimpleTransmission</type>
-    <actuator name="H1_F1J2">
-      <mechanicalReduction>1</mechanicalReduction>
-    </actuator>
-    <joint name="H1_F1J2">
-      <hardwareInterface>hardware_interface/PositionJointInterface</hardwareInterface>
-    </joint>
-  </transmission>
+    <dynamics damping="0.0" friction="10.0"/>
+  </joint>
   <transmission name="H1_F1J3_transmission">
     <type>transmission_interface/SimpleTransmission</type>
@@ -696,5 +678,5 @@
     <child link="H1_F2_palm_link"/>
   </joint>
-  <joint name="H1_F2J1" type="revolute">
+  <joint name="H1_F2J1" type="fixed">
     <origin rpy="-8.8818E-16 -1.0061E-16 0.022402" xyz="0 0 0.00016528"/>
     <axis xyz="0 0 1"/>
@@ -702,7 +684,7 @@
     <child link="H1_F2_ur10_base_link"/>
     <limit effort="30" lower="-0.785398163397" upper="0.785398163397" velocity="1.0"/>
-    <dynamics damping="0.0" friction="0.0"/>
-  </joint>
-  <joint name="H1_F2J2" type="revolute">
+    <dynamics damping="0.0" friction="10.0"/>
+  </joint>
+  <joint name="H1_F2J2" type="fixed">
     <origin rpy="0.070695 6.9389E-16 2.0947E-16" xyz="0 0.035 0.11683"/>
     <axis xyz="1 0 0"/>
@@ -710,5 +692,5 @@
     <child link="H1_F2_link_1"/>
     <limit effort="30" lower="-1.3962634016" upper="1.0471975512" velocity="1.0"/>
-    <dynamics damping="0.0" friction="0.0"/>
+    <dynamics damping="0.0" friction="10.0"/>
   </joint>
   <joint name="H1_F2J3" type="revolute">
@@ -718,24 +700,6 @@
     <child link="H1_F2_link_2"/>
     <limit effort="30" lower="-1.0471975512" upper="1.57079632679" velocity="1.0"/>
-    <dynamics damping="0.0" friction="0.0"/>
-  </joint>
-  <transmission name="H1_F2J1_transmission">
-    <type>transmission_interface/SimpleTransmission</type>
-    <actuator name="H1_F2J1">
-      <mechanicalReduction>1</mechanicalReduction>
-    </actuator>
-    <joint name="H1_F2J1">
-      <hardwareInterface>hardware_interface/PositionJointInterface</hardwareInterface>
-    </joint>
-  </transmission>
-  <transmission name="H1_F2J2_transmission">
-    <type>transmission_interface/SimpleTransmission</type>
-    <actuator name="H1_F2J2">
-      <mechanicalReduction>1</mechanicalReduction>
-    </actuator>
-    <joint name="H1_F2J2">
-      <hardwareInterface>hardware_interface/PositionJointInterface</hardwareInterface>
-    </joint>
-  </transmission>
+    <dynamics damping="0.0" friction="10.0"/>
+  </joint>
   <transmission name="H1_F2J3_transmission">
     <type>transmission_interface/SimpleTransmission</type>
@@ -884,5 +848,5 @@
     <child link="H1_F3_palm_link"/>
   </joint>
-  <joint name="H1_F3J1" type="revolute">
+  <joint name="H1_F3J1" type="fixed">
     <origin rpy="-8.8818E-16 -1.0061E-16 0.022402" xyz="0 0 0.00016528"/>
     <axis xyz="0 0 1"/>
@@ -890,7 +854,7 @@
     <child link="H1_F3_ur10_base_link"/>
     <limit effort="30" lower="-0.785398163397" upper="0.785398163397" velocity="1.0"/>
-    <dynamics damping="0.0" friction="0.0"/>
-  </joint>
-  <joint name="H1_F3J2" type="revolute">
+    <dynamics damping="0.0" friction="10.0"/>
+  </joint>
+  <joint name="H1_F3J2" type="fixed">
     <origin rpy="0.070695 6.9389E-16 2.0947E-16" xyz="0 0.035 0.11683"/>
     <axis xyz="1 0 0"/>
@@ -898,5 +862,5 @@
     <child link="H1_F3_link_1"/>
     <limit effort="30" lower="-1.3962634016" upper="1.0471975512" velocity="1.0"/>
-    <dynamics damping="0.0" friction="0.0"/>
+    <dynamics damping="0.0" friction="10.0"/>
   </joint>
   <joint name="H1_F3J3" type="revolute">
@@ -906,24 +870,6 @@
     <child link="H1_F3_link_2"/>
     <limit effort="30" lower="-1.0471975512" upper="1.57079632679" velocity="1.0"/>
-    <dynamics damping="0.0" friction="0.0"/>
-  </joint>
-  <transmission name="H1_F3J1_transmission">
-    <type>transmission_interface/SimpleTransmission</type>
-    <actuator name="H1_F3J1">
-      <mechanicalReduction>1</mechanicalReduction>
-    </actuator>
-    <joint name="H1_F3J1">
-      <hardwareInterface>hardware_interface/PositionJointInterface</hardwareInterface>
-    </joint>
-  </transmission>
-  <transmission name="H1_F3J2_transmission">
-    <type>transmission_interface/SimpleTransmission</type>
-    <actuator name="H1_F3J2">
-      <mechanicalReduction>1</mechanicalReduction>
-    </actuator>
-    <joint name="H1_F3J2">
-      <hardwareInterface>hardware_interface/PositionJointInterface</hardwareInterface>
-    </joint>
-  </transmission>
+    <dynamics damping="0.0" friction="10.0"/>
+  </joint>
   <transmission name="H1_F3J3_transmission">
     <type>transmission_interface/SimpleTransmission</type>
@@ -1006,9 +952,9 @@
     <kp>1000000.0</kp>
     <kd>100.0</kd>
-    <mu1>1.5</mu1>
-    <mu2>1.5</mu2>
-    <fdir1>1 0 0</fdir1>
-    <maxVel>1.0</maxVel>
-    <minDepth>0.002</minDepth>
+    <mu1>100000</mu1>
+    <mu2>100000</mu2>
+    <fdir1>1 0 0</fdir1>
+    <maxVel>1.0</maxVel>
+    <minDepth>0.001</minDepth>
     <material>Gazebo/DarkGrey</material>
   </gazebo>
@@ -1016,146 +962,146 @@
     <kp>1000000.0</kp>
     <kd>100.0</kd>
-    <mu1>1.5</mu1>
-    <mu2>1.5</mu2>
-    <fdir1>1 0 0</fdir1>
-    <maxVel>1.0</maxVel>
-    <minDepth>0.002</minDepth>
+    <mu1>100000</mu1>
+    <mu2>100000</mu2>
+    <fdir1>1 0 0</fdir1>
+    <maxVel>1.0</maxVel>
+    <minDepth>0.001</minDepth>
     <material>Gazebo/DarkGrey</material>
   </gazebo><gazebo reference="H1_F1_tip">
     <kp>1000000.0</kp>
-    <kd>100.0</kd>
-    <mu1>1.5</mu1>
-    <mu2>1.5</mu2>
-    <fdir1>1 0 0</fdir1>
-    <maxVel>1.0</maxVel>
-    <minDepth>0.002</minDepth>
+    <kd>10.0</kd>
+    <mu1>100000</mu1>
+    <mu2>100000</mu2>
+    <fdir1>1 0 0</fdir1>
+    <maxVel>1.0</maxVel>
+    <minDepth>0.001</minDepth>
     <material>Gazebo/DarkGrey</material>
   </gazebo>
   <gazebo reference="H1_F2_link_1">
     <kp>1000000.0</kp>
-    <kd>100.0</kd>
-    <mu1>1.5</mu1>
-    <mu2>1.5</mu2>
-    <fdir1>1 0 0</fdir1>
-    <maxVel>1.0</maxVel>
-    <minDepth>0.002</minDepth>
+    <kd>10.0</kd>
+    <mu1>100000</mu1>
+    <mu2>100000</mu2>
+    <fdir1>1 0 0</fdir1>
+    <maxVel>1.0</maxVel>
+    <minDepth>0.001</minDepth>
     <material>Gazebo/DarkGrey</material>
   </gazebo>
   <gazebo reference="H1_F2_link_2">
     <kp>1000000.0</kp>
-    <kd>100.0</kd>
-    <mu1>1.5</mu1>
-    <mu2>1.5</mu2>
-    <fdir1>1 0 0</fdir1>
-    <maxVel>1.0</maxVel>
-    <minDepth>0.002</minDepth>
+    <kd>10.0</kd>
+    <mu1>100000</mu1>
+    <mu2>100000</mu2>
+    <fdir1>1 0 0</fdir1>
+    <maxVel>1.0</maxVel>
+    <minDepth>0.001</minDepth>
     <material>Gazebo/DarkGrey</material>
   </gazebo><gazebo reference="H1_F2_tip">
     <kp>1000000.0</kp>
-    <kd>100.0</kd>
-    <mu1>1.5</mu1>
-    <mu2>1.5</mu2>
-    <fdir1>1 0 0</fdir1>
-    <maxVel>1.0</maxVel>
-    <minDepth>0.002</minDepth>
+    <kd>10.0</kd>
+    <mu1>100000</mu1>
+    <mu2>100000</mu2>
+    <fdir1>1 0 0</fdir1>
+    <maxVel>1.0</maxVel>
+    <minDepth>0.001</minDepth>
     <material>Gazebo/DarkGrey</material>
   </gazebo>
   <gazebo reference="H1_F3_link_1">
     <kp>1000000.0</kp>
-    <kd>100.0</kd>
-    <mu1>1.5</mu1>
-    <mu2>1.5</mu2>
-    <fdir1>1 0 0</fdir1>
-    <maxVel>1.0</maxVel>
-    <minDepth>0.002</minDepth>
+    <kd>10.0</kd>
+    <mu1>100000</mu1>
+    <mu2>100000</mu2>
+    <fdir1>1 0 0</fdir1>
+    <maxVel>1.0</maxVel>
+    <minDepth>0.001</minDepth>
     <material>Gazebo/DarkGrey</material>
   </gazebo>
   <gazebo reference="H1_F3_link_2">
     <kp>1000000.0</kp>
-    <kd>100.0</kd>
-    <mu1>1.5</mu1>
-    <mu2>1.5</mu2>
-    <fdir1>1 0 0</fdir1>
-    <maxVel>1.0</maxVel>
-    <minDepth>0.002</minDepth>
+    <kd>10.0</kd>
+    <mu1>100000</mu1>
+    <mu2>100000</mu2>
+    <fdir1>1 0 0</fdir1>
+    <maxVel>1.0</maxVel>
+    <minDepth>0.001</minDepth>
     <material>Gazebo/DarkGrey</material>
   </gazebo><gazebo reference="H1_F3_tip">
     <kp>1000000.0</kp>
-    <kd>100.0</kd>
-    <mu1>1.5</mu1>
-    <mu2>1.5</mu2>
-    <fdir1>1 0 0</fdir1>
-    <maxVel>1.0</maxVel>
-    <minDepth>0.002</minDepth>
+    <kd>10.0</kd>
+    <mu1>100000</mu1>
+    <mu2>100000</mu2>
+    <fdir1>1 0 0</fdir1>
+    <maxVel>1.0</maxVel>
+    <minDepth>0.001</minDepth>
     <material>Gazebo/DarkGrey</material>
   </gazebo>
   <gazebo reference="H1_F1_ur10_base_link">
     <kp>1000000.0</kp>
-    <kd>100.0</kd>
-    <mu1>1.5</mu1>
-    <mu2>1.5</mu2>
-    <fdir1>1 0 0</fdir1>
-    <maxVel>1.0</maxVel>
-    <minDepth>0.002</minDepth>
+    <kd>10.0</kd>
+    <mu1>1000</mu1>
+    <mu2>1000</mu2>
+    <fdir1>1 0 0</fdir1>
+    <maxVel>1.0</maxVel>
+    <minDepth>0.001</minDepth>
     <material>Gazebo/DarkGrey</material>
   </gazebo>
   <gazebo reference="H1_F2_ur10_base_link">
     <kp>1000000.0</kp>
-    <kd>100.0</kd>
-    <mu1>1.5</mu1>
-    <mu2>1.5</mu2>
-    <fdir1>1 0 0</fdir1>
-    <maxVel>1.0</maxVel>
-    <minDepth>0.002</minDepth>
+    <kd>10.0</kd>
+    <mu1>100000</mu1>
+    <mu2>100000</mu2>
+    <fdir1>1 0 0</fdir1>
+    <maxVel>1.0</maxVel>
+    <minDepth>0.001</minDepth>
     <material>Gazebo/DarkGrey</material>
   </gazebo>
   <gazebo reference="H1_F3_ur10_base_link">
     <kp>1000000.0</kp>
-    <kd>100.0</kd>
-    <mu1>1.5</mu1>
-    <mu2>1.5</mu2>
-    <fdir1>1 0 0</fdir1>
-    <maxVel>1.0</maxVel>
-    <minDepth>0.002</minDepth>
+    <kd>10.0</kd>
+    <mu1>100000</mu1>
+    <mu2>100000</mu2>
+    <fdir1>1 0 0</fdir1>
+    <maxVel>1.0</maxVel>
+    <minDepth>0.001</minDepth>
     <material>Gazebo/DarkGrey</material>
   </gazebo>
   <gazebo reference="H1_F1_palm_link">
     <kp>1000000.0</kp>
-    <kd>100.0</kd>
-    <mu1>1.5</mu1>
-    <mu2>1.5</mu2>
-    <fdir1>1 0 0</fdir1>
-    <maxVel>1.0</maxVel>
-    <minDepth>0.002</minDepth>
+    <kd>10.0</kd>
+    <mu1>100000</mu1>
+    <mu2>100000</mu2>
+    <fdir1>1 0 0</fdir1>
+    <maxVel>1.0</maxVel>
+    <minDepth>0.001</minDepth>
     <material>Gazebo/DarkGrey</material>
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
File: robots/mmo_500/urdf/xacros/common.gazebo.xacro (robot description, xacro)
@@ -1,9 +1,38 @@
 <?xml version="1.0"?>
-<robot xmlns:xacro="http://ros.org/wiki/xacro" name="mmo_500">
-  <gazebo>
-    <plugin name="ros_control" filename="libgazebo_ros_control.so">
+<robot xmlns:xacro="http://www.ros.org/wiki/xacro" name="mmo_500">
+<gazebo>
+  <plugin name="ros_control" filename="libgazebo_ros_control.so">
     <legacyModeNS>false</legacyModeNS>
-	<updateRate>1000.0</updateRate>
+    <robotSimType>gazebo_ros_control/DefaultRobotHWSim</robotSimType>
+  </plugin>
+</gazebo>
+<gazebo>
+	<plugin filename="libgazebo_ros_moveit_planning_scene.so" name="gazebo_ros_moveit_planning_scene">
+		<topicName>/planning_scene</topicName>
+ 		<sceneName>laboratory</sceneName>
+		<robotName>mmo_500</robotName>
+		<updatePeriod>0.5</updatePeriod>
+	</plugin>
+</gazebo>
+<gazebo>
+   <plugin name="gazebo_grasp_fix" filename="libgazebo_grasp_fix.so">
+        <arm>
+           <arm_name>arm</arm_name>
+           <palm_link>wrist_3_link</palm_link>
+           <gripper_link>H1_F1_link_1</gripper_link>
+           <gripper_link>H1_F2_link_1</gripper_link>
+           <gripper_link>H1_F3_link_1</gripper_link>
+           <gripper_link>H1_F1_link_2</gripper_link>
+           <gripper_link>H1_F2_link_2</gripper_link>
+           <gripper_link>H1_F3_link_2</gripper_link>
+       </arm>
+       <forces_angle_tolerance>100</forces_angle_tolerance>
+       <update_rate>4</update_rate>
+       <grip_count_threshold>4</grip_count_threshold>
+       <max_grip_count>20</max_grip_count>
+       <release_tolerance>0.005</release_tolerance>
+       <disable_collisions_on_attach>false</disable_collisions_on_attach>
+       <contact_topic>__default_topic__</contact_topic>
     </plugin>
-  </gazebo>
+</gazebo>
 </robot>

File: robots/mmo_500/urdf/xacros/mpo_500_body.xacro (robot description, xacro)
@@ -4,5 +4,5 @@
     <link name="${name}">
       <inertial>
-        <mass value="215"/>
+        <mass value="200"/>
         <origin xyz="0 0 0" />
          <inertia ixx="5.652232699207" ixy="0.009719934438" ixz="1.293988226423"

File: robots/mmo_500/urdf/xacros/omni_wheel.xacro (robot description, xacro)
@@ -31,6 +31,6 @@
    </link>
   <gazebo reference="${name}_link">
-    <mu1 value="2.5"/>
-    <mu2 value="2.5"/>
+    <mu1 value="2.6"/>
+    <mu2 value="2.6"/>
     <kp value="100000.0" />
     <kd value="10.0" />
