Commit message: Model for MM-400 updated

File: robots/mm_400/urdf/prbt_macro.xacro (robot description, xacro)
@@ -17,5 +17,5 @@
       <parent link="${parent}" />
       <child link = "pilzbase_link" />
-      <origin xyz="0.1 0.0 0.12" rpy="0.0 0.0 0.0" />
+      <origin xyz="-0.05 0.0 0.12" rpy="0.0 0.0 0.0" />
     </joint>
     <!-- Height of Foot -->

File: robots/mm_400/urdf/xacros/mp_400_body.xacro (robot description, xacro)
@@ -4,5 +4,5 @@
     <link name="${name}">
   <inertial>
-        <mass value="30" />
+        <mass value="125" />
         <origin xyz="0 0 0" rpy="0 0 0"/>
         <inertia ixx="1.71402" ixy="0.0" ixz="0.0"
@@ -26,13 +26,4 @@
       </collision>
     </link>
-  <gazebo reference="${name}">
-    <kp>10000.0</kp>
-    <kd>10.0</kd>
-    <mu1>1.5</mu1>
-    <mu2>1.5</mu2>
-    <fdir1>.1 0 0</fdir1>
-    <maxVel>10.0</maxVel>
-    <minDepth>0.0005</minDepth>
-</gazebo>
   </xacro:macro>
 </robot>

File: robots/mm_400/urdf/xacros/mp_400_caster_wheel.xacro (robot description, xacro)
@@ -13,6 +13,6 @@
  <inertial>
       <origin rpy="0 0 0" xyz="0 0 0" />
-      <mass value="1.4" />
-      <inertia ixx="0.0000045" ixy="0" ixz="0" iyy="0.000005" iyz="0" izz="0.0000045" />
+      <mass value="0.08" />
+      <inertia ixx="0.00000045" ixy="0" ixz="0" iyy="0.0000005" iyz="0" izz="0.00000045" />
 </inertial>
       <visual name='caster_wheel'>
@@ -30,8 +30,8 @@
     </link>
 <gazebo reference="${name}_link">
-      <kp>10000.0</kp>
-      <kd>50.0</kd>
-      <mu1>0.08</mu1>
-      <mu2>0.05</mu2>
+      <kp>50000.0</kp>
+      <kd>500.0</kd>
+      <mu1>0.02</mu1>
+      <mu2>0.01</mu2>
       <implicitSpringDamper>1</implicitSpringDamper>
 </gazebo>

File: robots/mm_400/urdf/xacros/mp_400_fixed_wheel_left.xacro (robot description, xacro)
@@ -12,8 +12,8 @@
    <link name="${name}_link" type="wheel">
    <inertial>
-        <mass value="1.82362"/>
-        <inertia ixx="0.00399743171" ixy="0.00000004464" ixz="-0.00000002245"
-                 iyy="0.00399741733" iyz="-0.00000000164"
-                 izz="0.00739239692"/>
+        <mass value="1."/>
+        <inertia ixx="0.000399743171" ixy="0.000000004464" ixz="-0.000000002245"
+                 iyy="0.000399741733" iyz="-0.000000000164"
+                 izz="0.000739239692"/>
 </inertial>
       <visual name='fixed_wheel_left'>
@@ -31,11 +31,9 @@
 </link>
 <gazebo reference="${name}_link">
-      <kp>10000.0</kp>
-      <kd>10.0</kd>
-      <mu1>50</mu1>
+      <kp>100000.0</kp>
+      <kd>50.0</kd>
+      <mu1>20</mu1>
       <mu2>10</mu2>
       <fdir1>1 0 0</fdir1>
-      <maxVel>3.0</maxVel>
-      <minDepth>0.00</minDepth>
       <implicitSpringDamper>1</implicitSpringDamper>
 </gazebo>

File: robots/mm_400/urdf/xacros/mp_400_fixed_wheel_right.xacro (robot description, xacro)
@@ -12,8 +12,8 @@
    <link name="${name}_link" type="wheel">
    <inertial>
-        <mass value="1.82362"/>
-        <inertia ixx="0.00399743171" ixy="0.00000004464" ixz="-0.00000002245"
-                 iyy="0.00399741733" iyz="-0.00000000164"
-                 izz="0.00739239692"/>
+        <mass value="1."/>
+        <inertia ixx="0.000399743171" ixy="0.00000004464" ixz="-0.00000002245"
+                 iyy="0.000399741733" iyz="-0.00000000164"
+                 izz="0.000739239692"/>
 </inertial>
       <visual name='fixed_wheel_right'>
@@ -31,11 +31,9 @@
 </link>
 <gazebo reference="${name}_link">
-      <kp>10000.0</kp>
-      <kd>10.0</kd>
+      <kp>100000.0</kp>
+      <kd>50.0</kd>
       <mu1>20</mu1>
       <mu2>10</mu2>
       <fdir1>1 0 0</fdir1>
-      <maxVel>3.0</maxVel>
-      <minDepth>0.00</minDepth>
       <implicitSpringDamper>1</implicitSpringDamper>
 </gazebo>
