Commit message: MMO-500 is working

File: robots/mmo_500/urdf/xacros/mpo_500_body.xacro (robot description, xacro)
@@ -4,9 +4,9 @@
     <link name="${name}">
       <inertial>
-        <mass value="200"/>
-        <origin xyz="0 0 0" />
-         <inertia ixx="5.652232699207" ixy="0.009719934438" ixz="1.293988226423"
-                 iyy="5.669473158652" iyz="0.007379583694"
-                 izz="5.683196351726" />
+        <mass value="80"/>
+        <origin xyz="0 0.0 0.0" />
+         <inertia ixx="2.8" ixy="0.0" ixz="0.0"
+                 iyy="2.8" iyz="0.0"
+                 izz="2.8" />
       </inertial>
       <visual>

File: robots/mmo_500/urdf/xacros/omni_wheel.xacro (robot description, xacro)
@@ -2,8 +2,8 @@
 <robot xmlns:xacro="http://www.ros.org/wiki/xacro" name="mpo_500">
   <xacro:macro name="omni_wheel_250" params="name parent *origin">
-   <joint name="${name}_joint" type="fixed">
+   <joint name="${name}_joint" type="continuous">
     <insert_block name="origin" />
     <axis xyz="0 1 0" />
-    <joint_properties damping="1" friction="1" />
+    <joint_properties damping="100" friction="100" />
     <parent link="${parent}" />
     <child link="${name}_link" />
@@ -11,9 +11,9 @@
    <link name="${name}_link" type="wheel">
     <inertial>
-      <mass value="8.9" />
+      <mass value="4.2" />
       <origin xyz="0 0 0" rpy="0 0 0" />
-        <inertia  ixx="0.04" ixy="0.0007" ixz="0.0"
-                  iyy="0.02" iyz="0.004"
-                  izz="0.05" />
+        <inertia  ixx="0.0338" ixy="0.0" ixz="0.0"
+                  iyy="0.0338" iyz="0.0"
+                  izz="0.0338" />
     </inertial>
     <visual>
@@ -24,16 +24,14 @@
     </visual>
     <collision>
-     <origin xyz="0 0 0" rpy="0 0 0" />
+     <origin xyz="0 0 0" rpy="1.57 0 0" />
      <geometry>
-        <mesh filename="package://neo_simulation/robots/mmo_500/meshes/MPO-500-WHEEL.dae" scale="0.001 0.001 0.001"/>
+       <sphere radius="0.127" />
      </geometry>
     </collision>
    </link>
-  <gazebo reference="${name}_link">
-    <mu1 value="2.6"/>
-    <mu2 value="2.6"/>
-    <kp value="100000.0" />
-    <kd value="10.0" />
-  </gazebo>
+<gazebo reference="${name}_link">
+      <mu1>0.045</mu1>
+      <mu2>0.045</mu2>
+</gazebo>
   </xacro:macro>
 </robot>
