Commit message: updated mmo_500 model

File: robots/mmo_500/mmo_500.urdf.xacro (robot description, xacro)
@@ -3,47 +3,43 @@
   <!--GAZEBO REFERENCES
   MPO_500-->
-  <xacro:include filename="$(find neo_simulation)/robots/mmo_500/urdf/mpo_500/xacros/mpo_500_gazebo.xacro" />
- <!--CABINET-->
-  <xacro:include filename="$(find neo_simulation)/robots/mmo_500/urdf/cabinet/cabinet_gazebo.xacro" />
+  <xacro:include filename="$(find neo_simulation)/robots/mmo_500/urdf/xacros/mpo_500_gazebo.xacro" />
   <!--ur10 -->
-  <xacro:include filename="$(find neo_simulation)/robots/mmo_500/urdf/ur10/common.gazebo.xacro" />
-  <!-- MATERIALS -->
-  <xacro:include filename="$(find neo_simulation)/robots/mmo_500/urdf/mpo_500/xacros/mpo_500_materials.xacro" />
+  <xacro:include filename="$(find neo_simulation)/robots/mmo_500/urdf/xacros/common.gazebo.xacro" />
   <!-- BODY -->
-  <xacro:include filename="$(find neo_simulation)/robots/mmo_500/urdf/mpo_500/xacros/mpo_500_body.xacro" />
+  <xacro:include filename="$(find neo_simulation)/robots/mmo_500/urdf/xacros/mpo_500_body.xacro" />
   <!-- WHEELS -->
-  <xacro:include filename="$(find neo_simulation)/robots/mmo_500/urdf/mpo_500/xacros/omni_wheel.xacro" />
+  <xacro:include filename="$(find neo_simulation)/robots/mmo_500/urdf/xacros/omni_wheel.xacro" />
   <!-- SENSORS -->
-  <xacro:include filename="$(find neo_simulation)/robots/mmo_500/urdf/mpo_500/xacros/sick_s300_laser.xacro" />
+  <xacro:include filename="$(find neo_simulation)/robots/mmo_500/urdf/xacros/sick_laser.xacro" />
   <!-- CABINET -->
-  <xacro:include filename="$(find neo_simulation)/robots/mmo_500/urdf/cabinet/cabinet.xacro" />
+  <xacro:include filename="$(find neo_simulation)/robots/mmo_500/urdf/xacros/cabinet.xacro" />
   <!--ur10 -->
-  <xacro:include filename="$(find neo_simulation)/robots/mmo_500/urdf/ur10/ur10.urdf.xacro" />
+  <xacro:include filename="$(find neo_simulation)/robots/mmo_500/urdf/ur10.urdf.xacro" />
   <!-- Base Macro-->
   <xacro:mpo_500_base name="base_link">
   </xacro:mpo_500_base>
   <!-- Wheel Macro -->
-  <xacro:omni_wheel_250 name="wheel_front_left" parent="base_link" suffix="links">
+  <xacro:omni_wheel_250 name="wheel_front_left" parent="base_link">
   	<origin xyz="0.25 0.28 0.13" rpy="0 0 0" />
   </xacro:omni_wheel_250>
-  <xacro:omni_wheel_250 name="wheel_front_right" parent="base_link" suffix="rechts">
+  <xacro:omni_wheel_250 name="wheel_front_right" parent="base_link" >
   	<origin xyz="0.25 -0.28 0.13" rpy="0 0 0" />
   </xacro:omni_wheel_250>
-  <xacro:omni_wheel_250 name="wheel_back_left" parent="base_link" suffix="links">
+  <xacro:omni_wheel_250 name="wheel_back_left" parent="base_link">
   	<origin xyz="-0.25 0.28 0.13" rpy="0 0 0" />
   </xacro:omni_wheel_250>
-  <xacro:omni_wheel_250 name="wheel_back_right" parent="base_link" suffix="rechts">
+  <xacro:omni_wheel_250 name="wheel_back_right" parent="base_link" >
   	<origin xyz="-0.25 -0.28 0.13" rpy="0 0 0" />
   </xacro:omni_wheel_250>
   <!-- Sensors -->
-  <xacro:sick_s300_laser_v0 name="sick_s300_laser_front" parent="base_link" ros_topic="sick_s300_front/scan">
+  <xacro:sick_laser_v0 name="sick_s300_laser_front" parent="base_link" ros_topic="sick_s300_front/scan">
   	<origin xyz="0.442 0 0.420" rpy="0 0 0" />
-  </xacro:sick_s300_laser_v0>
-  <xacro:sick_s300_laser_v0 name="sick_s300_laser_back" parent="base_link" ros_topic="sick_s300_back/scan">
+  </xacro:sick_laser_v0>
+  <xacro:sick_laser_v0 name="sick_s300_laser_back" parent="base_link" ros_topic="sick_s300_back/scan">
   	<origin xyz="-0.442 0 0.420" rpy="0 0 3.14" />
-  </xacro:sick_s300_laser_v0>
+  </xacro:sick_laser_v0>
   <!--cabinet-->
   <xacro:mmo_500_cabinet name="cabinet" parent="base_link">
-  	<origin xyz="0.072 0 0.386" rpy="0 0 0" />-->
+  	<origin xyz="0.072 0 0.386" rpy="0 0 0" />
   </xacro:mmo_500_cabinet>
   <!--ur10-->

Commit message: Controller files, config files and launch files are added for MMO-500 and MMO-700

File: robots/mmo_500/mmo_500.urdf.xacro (robot description, xacro)
@@ -33,8 +33,8 @@
   </xacro:omni_wheel_250>
   <!-- Sensors -->
-  <xacro:sick_laser_v0 name="sick_s300_laser_front" parent="base_link" ros_topic="sick_s300_front/scan">
+  <xacro:sick_laser_v0 name="sick_laser_front" parent="base_link" ros_topic="sick_s300_front/scan">
   	<origin xyz="0.442 0 0.420" rpy="0 0 0" />
   </xacro:sick_laser_v0>
-  <xacro:sick_laser_v0 name="sick_s300_laser_back" parent="base_link" ros_topic="sick_s300_back/scan">
+  <xacro:sick_laser_v0 name="sick_laser_back" parent="base_link" ros_topic="sick_s300_back/scan">
   	<origin xyz="-0.442 0 0.420" rpy="0 0 3.14" />
   </xacro:sick_laser_v0>

File: robots/mmo_500/urdf/xacros/cabinet.xacro (robot description, xacro)
@@ -10,5 +10,5 @@
     <link name="${name}_link">
       <inertial>
-        <mass value="8" />
+        <mass value="2" />
         <origin xyz="0 0 0" rpy="0 0 0"/>
         <inertia ixx="0.457072" ixy="0.0" ixz="0.0"

File: robots/mmo_700/urdf/ur10.urdf.xacro (robot description, xacro)
@@ -90,5 +90,5 @@
         <limit lower="${shoulder_pan_lower_limit}" upper="${shoulder_pan_upper_limit}" effort="330.0" velocity="2.16"/>
       </xacro:if>
-      <dynamics damping="0.0" friction="0.0"/>
+      <dynamics damping="0.5" friction="0.0"/>
     </joint>
     <link name="${prefix}shoulder_link">
@@ -118,5 +118,5 @@
         <limit lower="${shoulder_lift_lower_limit}" upper="${shoulder_lift_upper_limit}" effort="330.0" velocity="2.16"/>
       </xacro:if>
-      <dynamics damping="0.0" friction="0.0"/>
+      <dynamics damping="0.5" friction="0.0"/>
     </joint>
     <link name="${prefix}upper_arm_link">
@@ -146,5 +146,5 @@
         <limit lower="${elbow_joint_lower_limit}" upper="${elbow_joint_upper_limit}" effort="150.0" velocity="3.15"/>
       </xacro:if>
-      <dynamics damping="0.0" friction="0.0"/>
+      <dynamics damping="0.5" friction="0.0"/>
     </joint>
     <link name="${prefix}forearm_link">
@@ -174,5 +174,5 @@
         <limit lower="${wrist_1_lower_limit}" upper="${wrist_1_upper_limit}" effort="54.0" velocity="3.2"/>
       </xacro:if>
-      <dynamics damping="0.0" friction="0.0"/>
+      <dynamics damping="0.5" friction="0.0"/>
     </joint>
     <link name="${prefix}wrist_1_link">
@@ -202,5 +202,5 @@
         <limit lower="${wrist_2_lower_limit}" upper="${wrist_2_upper_limit}" effort="54.0" velocity="3.2"/>
       </xacro:if>
-      <dynamics damping="0.0" friction="0.0"/>
+      <dynamics damping="0.5" friction="0.0"/>
     </joint>
     <link name="${prefix}wrist_2_link">
@@ -230,5 +230,5 @@
         <limit lower="${wrist_3_lower_limit}" upper="${wrist_3_upper_limit}" effort="54.0" velocity="3.2"/>
       </xacro:if>
-      <dynamics damping="0.0" friction="0.0"/>
+      <dynamics damping="0.5" friction="0.0"/>
     </joint>
     <link name="${prefix}wrist_3_link">

File: robots/mmo_700/urdf/xacros/cabinet.xacro (robot description, xacro)
@@ -10,5 +10,5 @@
     <link name="${name}_link">
       <inertial>
-        <mass value="8" />
+        <mass value="2" />
         <origin xyz="0 0 0" rpy="0 0 0"/>
         <inertia ixx="0.457072" ixy="0.0" ixz="0.0"

File: robots/mmo_700/urdf/xacros/common.gazebo.xacro (robot description, xacro)
@@ -3,6 +3,6 @@
   <gazebo>
     <plugin name="ros_control" filename="libgazebo_ros_control.so">
-            <robotNamespace>/</robotNamespace>
-        <alwaysOn>true</alwaysOn>
+  <robotNamespace>/</robotNamespace>
+  <alwaysOn>true</alwaysOn>
 	<updateRate>1000.0</updateRate>
   <legacyModeNS>false</legacyModeNS>

File: robots/mmo_700/urdf/xacros/mpo_700_body.xacro (robot description, xacro)
@@ -4,5 +4,5 @@
     <link name="${name}">
       <inertial>
-        <mass value="30" />
+        <mass value="40" />
         <origin xyz="0 0 0" rpy="0 0 0"/>
         <inertia ixx="1.71402" ixy="0.0" ixz="0.0"

File: robots/mmo_700/urdf/xacros/ur.transmission.xacro (robot description, xacro)
@@ -5,8 +5,7 @@
       <type>transmission_interface/SimpleTransmission</type>
       <joint name="${prefix}shoulder_pan_joint">
-        <hardwareInterface>PositionJointInterface</hardwareInterface>
+        <hardwareInterface>hardware_interface/PositionJointInterface</hardwareInterface>
       </joint>
       <actuator name="${prefix}shoulder_pan_motor">
-        <hardwareInterface>PositionJointInterface</hardwareInterface>
         <mechanicalReduction>1</mechanicalReduction>
       </actuator>
@@ -15,8 +14,7 @@
       <type>transmission_interface/SimpleTransmission</type>
       <joint name="${prefix}shoulder_lift_joint">
-        <hardwareInterface>PositionJointInterface</hardwareInterface>
+        <hardwareInterface>hardware_interface/PositionJointInterface</hardwareInterface>
       </joint>
       <actuator name="${prefix}shoulder_lift_motor">
-        <hardwareInterface>PositionJointInterface</hardwareInterface>
         <mechanicalReduction>1</mechanicalReduction>
       </actuator>
@@ -25,8 +23,7 @@
       <type>transmission_interface/SimpleTransmission</type>
       <joint name="${prefix}elbow_joint">
-        <hardwareInterface>PositionJointInterface</hardwareInterface>
+        <hardwareInterface>hardware_interface/PositionJointInterface</hardwareInterface>
       </joint>
       <actuator name="${prefix}elbow_motor">
-        <hardwareInterface>PositionJointInterface</hardwareInterface>
         <mechanicalReduction>1</mechanicalReduction>
       </actuator>
@@ -35,8 +32,7 @@
       <type>transmission_interface/SimpleTransmission</type>
       <joint name="${prefix}wrist_1_joint">
-        <hardwareInterface>PositionJointInterface</hardwareInterface>
+        <hardwareInterface>hardware_interface/PositionJointInterface</hardwareInterface>
       </joint>
       <actuator name="${prefix}wrist_1_motor">
-        <hardwareInterface>PositionJointInterface</hardwareInterface>
         <mechanicalReduction>1</mechanicalReduction>
       </actuator>
@@ -45,8 +41,7 @@
       <type>transmission_interface/SimpleTransmission</type>
       <joint name="${prefix}wrist_2_joint">
-        <hardwareInterface>PositionJointInterface</hardwareInterface>
+        <hardwareInterface>hardware_interface/PositionJointInterface</hardwareInterface>
       </joint>
       <actuator name="${prefix}wrist_2_motor">
-        <hardwareInterface>PositionJointInterface</hardwareInterface>
         <mechanicalReduction>1</mechanicalReduction>
       </actuator>
@@ -55,8 +50,7 @@
       <type>transmission_interface/SimpleTransmission</type>
       <joint name="${prefix}wrist_3_joint">
-        <hardwareInterface>PositionJointInterface</hardwareInterface>
+        <hardwareInterface>hardware_interface/PositionJointInterface</hardwareInterface>
       </joint>
       <actuator name="${prefix}wrist_3_motor">
-        <hardwareInterface>PositionJointInterface</hardwareInterface>
         <mechanicalReduction>1</mechanicalReduction>
       </actuator>

Commit message: Added Pilz arm

File: robots/mmo_500/mmo_500.urdf.xacro (robot description, xacro)
@@ -15,5 +15,7 @@
   <xacro:include filename="$(find neo_simulation)/robots/mmo_500/urdf/xacros/cabinet.xacro" />
   <!--ur10 -->
-  <xacro:include filename="$(find neo_simulation)/robots/mmo_500/urdf/ur10.urdf.xacro" />
+  <!-- <xacro:include filename="$(find neo_simulation)/robots/mmo_500/urdf/ur10.urdf.xacro" /> -->
+  <!-- Pilz -->
+  <xacro:include filename="$(find neo_simulation)/robots/mmo_500/urdf/prbt_macro.xacro" />
   <!-- Base Macro-->
   <xacro:mpo_500_base name="base_link">
@@ -44,5 +46,5 @@
   </xacro:mmo_500_cabinet>
   <!--ur10-->
-  <xacro:ur10_robot parent="cabinet_link" prefix="ur10" joint_limited="true"
+<!--   <xacro:ur10_robot parent="cabinet_link" prefix="ur10" joint_limited="true"
 		 shoulder_pan_lower_limit="${-pi}" shoulder_pan_upper_limit="${pi}"
 		 shoulder_lift_lower_limit="${-pi}" shoulder_lift_upper_limit="${pi}"
@@ -51,4 +53,8 @@
 		 wrist_2_lower_limit="${-pi}" wrist_2_upper_limit="${pi}"
 		 wrist_3_lower_limit="${-pi}" wrist_3_upper_limit="${pi}">
-  </xacro:ur10_robot>
+  </xacro:ur10_robot> -->
+  <!-- Pilz arm -->
+    <xacro:prbt parent="cabinet_link" prefix="pilz">
+    <origin xyz="0 0 0." rpy="0 0 0" />
+  </xacro:prbt>
 </robot>

Commit message: Position of the wheels of mpo-500 wheels are corrected

File: robots/mmo_500/mmo_500.urdf.xacro (robot description, xacro)
@@ -25,12 +25,12 @@
   	<origin xyz="0.25 0.28 0.13" rpy="0 0 0" />
   </xacro:omni_wheel_250>
-  <xacro:omni_wheel_250 name="wheel_front_right" parent="base_link" >
-  	<origin xyz="0.25 -0.28 0.13" rpy="0 0 0" />
+  <xacro:omni_wheel_250 name="wheel_front_right" parent="base_link">
+  	<origin xyz="0.25 -0.28 0.13" rpy="0 0 3.14" />
   </xacro:omni_wheel_250>
   <xacro:omni_wheel_250 name="wheel_back_left" parent="base_link">
   	<origin xyz="-0.25 0.28 0.13" rpy="0 0 0" />
   </xacro:omni_wheel_250>
-  <xacro:omni_wheel_250 name="wheel_back_right" parent="base_link" >
-  	<origin xyz="-0.25 -0.28 0.13" rpy="0 0 0" />
+  <xacro:omni_wheel_250 name="wheel_back_right" parent="base_link">
+  	<origin xyz="-0.25 -0.28 0.13" rpy="0 0 3.14" />
   </xacro:omni_wheel_250>
   <!-- Sensors -->

File: robots/mpo_500/mpo_500.urdf.xacro (robot description, xacro)
@@ -17,5 +17,5 @@
   </xacro:omni_wheel_250>
   <xacro:omni_wheel_250 name="wheel_front_right" parent="base_link">
-  	<origin xyz="0.25 -0.28 0.13" rpy="0 0 0" />
+  	<origin xyz="0.25 -0.28 0.13" rpy="0 0 3.14" />
   </xacro:omni_wheel_250>
   <xacro:omni_wheel_250 name="wheel_back_left" parent="base_link">
@@ -23,5 +23,5 @@
   </xacro:omni_wheel_250>
   <xacro:omni_wheel_250 name="wheel_back_right" parent="base_link">
-  	<origin xyz="-0.25 -0.28 0.13" rpy="0 0 0" />
+  	<origin xyz="-0.25 -0.28 0.13" rpy="0 0 3.14" />
   </xacro:omni_wheel_250>
   <!-- Sensors -->
