Commit message: Robot models for MPO-700, MPO-500, MMO-700, MMO-500 are updated

File: robots/mmo_500/mmo_500.urdf.xacro (robot description, xacro)
@@ -11,13 +11,16 @@
   <xacro:include filename="$(find neo_simulation)/robots/mmo_500/urdf/xacros/omni_wheel.xacro" />
   <!-- SENSORS -->
-  <xacro:include filename="$(find neo_simulation)/robots/mmo_500/urdf/xacros/sick_laser.xacro" />
-  <xacro:include filename="$(find neo_simulation)/robots/mmo_500/urdf/xacros/imu.xacro" />
-  <xacro:include filename="$(find neo_simulation)/robots/mmo_500/urdf/xacros/ultrasonic.xacro" />
+  <!-- Sick-S300 -->
+  <!-- <xacro:include filename="$(find neo_simulation)/robots/mmo_500/xacros/sick_S300.xacro" /> -->
+  <!--Sick Micro-scan  -->
+  <xacro:include filename="$(find neo_simulation)/robots/mmo_500/urdf/xacros/micro_scan.xacro" />
+  <!-- <xacro:include filename="$(find neo_simulation)/robots/mmo_500/urdf/xacros/imu.xacro" />
+  <xacro:include filename="$(find neo_simulation)/robots/mmo_500/urdf/xacros/ultrasonic.xacro" /> -->
   <!-- CABINET -->
   <xacro:include filename="$(find neo_simulation)/robots/mmo_500/urdf/xacros/cabinet.xacro" />
   <!--ur10 -->
-  <!-- <xacro:include filename="$(find neo_simulation)/robots/mmo_500/urdf/ur10.urdf.xacro" /> -->
+  <xacro:include filename="$(find neo_simulation)/robots/mmo_500/urdf/ur10.urdf.xacro" />
   <!-- Pilz -->
-  <xacro:include filename="$(find neo_simulation)/robots/mmo_500/urdf/prbt_macro.xacro" />
+  <!-- <xacro:include filename="$(find neo_simulation)/robots/mmo_500/urdf/prbt_macro.xacro" /> -->
   <!-- Base Macro-->
   <xacro:mpo_500_base name="base_link">
@@ -123,5 +126,5 @@
   </xacro:mmo_500_cabinet>
   <!--ur10-->
-<!--   <xacro:ur10_robot parent="cabinet_link" prefix="ur10" joint_limited="true"
+  <xacro:ur10_robot parent="cabinet_link" prefix="ur10" joint_limited="true"
 		 shoulder_pan_lower_limit="${-pi}" shoulder_pan_upper_limit="${pi}"
 		 shoulder_lift_lower_limit="${-pi}" shoulder_lift_upper_limit="${pi}"
@@ -130,8 +133,9 @@
 		 wrist_2_lower_limit="${-pi}" wrist_2_upper_limit="${pi}"
 		 wrist_3_lower_limit="${-pi}" wrist_3_upper_limit="${pi}">
-  </xacro:ur10_robot> -->
+  </xacro:ur10_robot>
   <!-- Pilz arm -->
-    <xacro:prbt parent="cabinet_link" prefix="pilz">
+<!--     <xacro:prbt parent="cabinet_link" prefix="pilz">
     <origin xyz="0 0 0." rpy="0 0 0" />
   </xacro:prbt>
+ -->
 </robot>

File: robots/mmo_500/urdf/xacros/camera.xacro (robot description, xacro)
@@ -1,4 +1,4 @@
 <?xml version="1.0"?>
-<robot xmlns:xacro="http://www.ros.org/wiki/xacro" name="mm_400">
+<robot xmlns:xacro="http://www.ros.org/wiki/xacro" name="mpo_500">
   <xacro:macro name="camera" params="name parent *origin">
     <xacro:property name="camera_link" value="0.05" />

File: robots/mmo_500/urdf/xacros/imu.xacro (robot description, xacro)
@@ -1,4 +1,4 @@
 <?xml version="1.0"?>
-<robot xmlns:xacro="http://www.ros.org/wiki/xacro" name="mp_400">
+<robot xmlns:xacro="http://www.ros.org/wiki/xacro" name="mpo_500">
   <xacro:macro name="imu" params="name parent *origin">
     <joint name="${name}_joint" type="fixed">

File: robots/mmo_500/urdf/xacros/micro_scan.xacro (robot description, xacro)
@@ -1,4 +1,4 @@
 <?xml version="1.0"?>
-<robot xmlns:xacro="http://www.ros.org/wiki/xacro" name="mpo_700">
+<robot xmlns:xacro="http://www.ros.org/wiki/xacro" name="mpo_500">
   <xacro:macro name="sick_laser_v0" params="name parent *origin ros_topic">
     <joint name="${name}_joint" type="fixed">
@@ -17,5 +17,5 @@
         <origin xyz="0 0 -0.06" rpy="1.57 0 0" />
       <geometry>
-        <mesh filename="package://neo_simulation/robots/mpo_700/meshes/SICK-MICROSCAN3.dae" scale="0.001 0.001 0.001" />
+        <mesh filename="package://neo_simulation/robots/mmo_500/meshes/SICK-MICROSCAN3.dae" scale="0.001 0.001 0.001" />
         </geometry>
       </visual>
@@ -23,5 +23,5 @@
         <origin xyz="0 0 -0.06" rpy="1.57 0 0" />
         <geometry>
-          <mesh filename="package://neo_simulation/robots/mpo_700/meshes/SICK-MICROSCAN3.dae" scale="0.001 0.001 0.001" />
+          <mesh filename="package://neo_simulation/robots/mmo_500/meshes/SICK-MICROSCAN3.dae" scale="0.001 0.001 0.001" />
         </geometry>
       </collision>

File: robots/mmo_500/urdf/xacros/sick_S300.xacro (robot description, xacro)
@@ -15,6 +15,5 @@
       </inertial>
       <visual>
-      <!-- SICK S3 sensor: Uncomment/Comment it out if required  -->
-      <origin xyz="0 0 -0.12" rpy="-1.57 0 3.14" />
+        <origin xyz="0 0 -0.12" rpy="-1.57 0 3.14" />
         <geometry>
         <mesh filename="package://neo_simulation/robots/mmo_500/meshes/SICK-S300.dae" scale="0.001 0.001 0.001" />
@@ -22,21 +21,9 @@
       </visual>
       <collision>
-        <origin xyz="0 0 0" rpy="-1.57 0 3.14" />
+        <origin xyz="0 0 -0.12" rpy="-1.57 0 3.14" />
         <geometry>
         <mesh filename="package://neo_simulation/robots/mmo_500/meshes/SICK-S300.dae" scale="0.001 0.001 0.001" />
         </geometry>
       </collision>
-      <!-- Microscan 3 sensor: Uncomment/Comment it out if required  -->
-<!--  <origin xyz="-0.0 0 -0.06" rpy="1.57 0 0" />
-      <geometry>
-      <mesh filename="package://neo_simulation/robots/mpo_500/meshes/SICK-MICROSCAN3.dae" scale="0.001 0.001 0.001" />
-      </geometry>
-      </visual>
-      <collision>
- <origin xyz="-0.0 0 -0.06" rpy="1.57 0 0" />
-      <geometry>
-        <mesh filename="package://neo_simulation/robots/mp_500/meshes/SICK-MICROSCAN3.dae" scale="0.001 0.001 0.001" />
-        </geometry>
-      </collision> -->
     </link>
   </xacro:macro>

File: robots/mmo_700/mmo_700.urdf.xacro (robot description, xacro)
@@ -10,11 +10,14 @@
   <xacro:include filename="$(find neo_simulation)/robots/mmo_700/urdf/xacros/mpo_700_body.xacro" />
   <!-- SENSORS -->
-  <xacro:include filename="$(find neo_simulation)/robots/mmo_700/urdf/xacros/sick_laser.xacro" />
-  <xacro:include filename="$(find neo_simulation)/robots/mmo_700/urdf/xacros/imu.xacro" />
-  <xacro:include filename="$(find neo_simulation)/robots/mmo_700/urdf/xacros/ultrasonic.xacro" />
+  <!-- Sick-S300 -->
+  <!-- <xacro:include filename="$(find neo_simulation)/robots/mmo_700/xacros/sick_S300.xacro" /> -->
+  <!--Sick Micro-scan  -->
+  <xacro:include filename="$(find neo_simulation)/robots/mmo_700/urdf/xacros/micro_scan.xacro" />
+  <!--   <xacro:include filename="$(find neo_simulation)/robots/mmo_700/urdf/xacros/imu.xacro" />
+  <xacro:include filename="$(find neo_simulation)/robots/mmo_700/urdf/xacros/ultrasonic.xacro" /> -->
   <!-- Gazebo -->
   <xacro:include filename="$(find neo_simulation)/robots/mmo_700/urdf/xacros/mpo_700_gazebo.xacro" />
   <!-- Head -->
-  <xacro:include filename="$(find neo_simulation)/robots/mmo_700/urdf/xacros/mpo_700_head.xacro" />
+  <xacro:include filename="$(find neo_simulation)/robots/mmo_700/urdf/xacros/mpo_700_caster.xacro" />
   <!-- Wheel -->
   <xacro:include filename="$(find neo_simulation)/robots/mmo_700/urdf/xacros/mpo_700_wheel.xacro" />
@@ -22,35 +25,39 @@
   <xacro:mpo_700_base name="base_link">
   </xacro:mpo_700_base>
-<xacro:mmo_700_head_0 name="mmo_700_head_0" parent="base_link">
+<xacro:mpo_700_caster_0 name="mpo_700_caster_front_left" parent="base_link">
     <origin xyz="0.24 0.18 0.27" rpy="3.14 0 -1.57" />
-  </xacro:mmo_700_head_0>
-<xacro:mmo_700_head_1 name="mmo_700_head_1" parent="base_link">
+  </xacro:mpo_700_caster_0>
+<!-- Casters -->
+<xacro:mpo_700_caster_1 name="mpo_700_caster_front_right" parent="base_link">
     <origin xyz="0.24 -0.18 0.27" rpy="3.14 0 1.57" />
-  </xacro:mmo_700_head_1>
-<xacro:mmo_700_head_2 name="mmo_700_head_2" parent="base_link">
+  </xacro:mpo_700_caster_1>
+<xacro:mpo_700_caster_2 name="mpo_700_caster_back_left" parent="base_link">
     <origin xyz="-0.24 0.18 0.27" rpy="3.14 0 -1.57" />
-  </xacro:mmo_700_head_2>
-<xacro:mmo_700_head_3 name="mmo_700_head_3" parent="base_link">
+  </xacro:mpo_700_caster_2>
+<xacro:mpo_700_caster_3 name="mpo_700_caster_back_right" parent="base_link">
     <origin xyz="-0.24 -0.18 0.27" rpy="3.14 0 1.57" />
-  </xacro:mmo_700_head_3>
-<xacro:mmo_700_wheel name="wheel_0" parent="mmo_700_head_0_link">
+  </xacro:mpo_700_caster_3>
+<!-- wheels -->
+<xacro:mpo_700_wheel name="mpo_700_wheel_front_left" parent="mpo_700_caster_front_left_link">
     <origin xyz="-0.05 0. 0.18" rpy="0 0 0" />
-  </xacro:mmo_700_wheel>
-<xacro:mmo_700_wheel name="wheel_1" parent="mmo_700_head_1_link">
+  </xacro:mpo_700_wheel>
+<xacro:mpo_700_wheel name="mpo_700_wheel_front_right" parent="mpo_700_caster_front_right_link">
     <origin xyz="-0.05 0. 0.18" rpy="0 0 0" />
-  </xacro:mmo_700_wheel>
-<xacro:mmo_700_wheel name="wheel_2" parent="mmo_700_head_2_link">
+  </xacro:mpo_700_wheel>
+<xacro:mpo_700_wheel name="mpo_700_wheel_back_left" parent="mpo_700_caster_back_left_link">
     <origin xyz="-0.05 0. 0.18" rpy="0 0 0" />
-  </xacro:mmo_700_wheel>
-<xacro:mmo_700_wheel name="wheel_3" parent="mmo_700_head_3_link">
+  </xacro:mpo_700_wheel>
+<xacro:mpo_700_wheel name="mpo_700_wheel_back_right" parent="mpo_700_caster_back_right_link">
     <origin xyz="-0.05 0. 0.18" rpy="0 0 0" />
-  </xacro:mmo_700_wheel>
+  </xacro:mpo_700_wheel>
 <!-- Sensors -->
-  <xacro:sick_v0 name="lidar_1" parent="base_link" ros_topic="lidar_1/scan_filtered">
-    <origin xyz="0.360 0 0.181" rpy="3.14 0 0 " />
-  </xacro:sick_v0>
-  <xacro:sick_v0 name="lidar_2" parent="base_link" ros_topic="lidar_2/scan_filtered">
-    <origin xyz="-0.360 0 0.181" rpy="3.14 0 3.14" />
-  </xacro:sick_v0>
+  <xacro:sick_laser_v0 name="lidar_1" parent="base_link" ros_topic="lidar_1/scan_filtered">
+  <!--<origin xyz="0.360 0 0.181" rpy="3.14 0 0" />-->
+    <origin xyz="0.338 0.288 0.223" rpy="3.14 0 0.79" /> <!-- Scanners on the side -->
+  </xacro:sick_laser_v0>
+  <xacro:sick_laser_v0 name="lidar_2" parent="base_link" ros_topic="lidar_2/scan_filtered">
+  <!--<origin xyz="-0.360 0 0.181" rpy="3.14 0 3.14" />-->
+    <origin xyz="-0.338 -0.288 0.223" rpy="3.14 0 3.93" /> <!-- Scanners on the side -->
+  </xacro:sick_laser_v0>
      <!--+++++++++++++++++++ IMU ++++++++++++++++++++++++-->
  <!-- Comment or uncomment based on your requirement -->

File: robots/mmo_700/urdf/xacros/mpo_700_caster.xacro (robot description, xacro)
@@ -1,5 +1,5 @@
 <?xml version="1.0"?>
 <robot xmlns:xacro="http://www.ros.org/wiki/xacro" name="mpo_700">
-  <xacro:macro name="mpo_700_head_0" params="name parent *origin">
+  <xacro:macro name="mpo_700_caster_0" params="name parent *origin">
    <joint name="${name}_joint" type="fixed">
     <insert_block name="origin" />
@@ -19,5 +19,5 @@
      <origin xyz="0 0 0.10" rpy="0 0 0"/>
      <geometry>
-        <mesh filename="package://neo_simulation/robots/mpo_700/meshes/MPO-700-HEAD.dae" scale="0.001 0.001 0.001"/>
+        <mesh filename="package://neo_simulation/robots/mmo_700/meshes/MPO-700-HEAD.dae" scale="0.001 0.001 0.001"/>
      </geometry>
     </visual>
@@ -25,10 +25,10 @@
      <origin xyz="0 0 0.10" rpy="0 0 0" />
      <geometry>
-        <mesh filename="package://neo_simulation/robots/mpo_700/meshes/MPO-700-HEAD.dae" scale="0.001 0.001 0.001"/>
+        <mesh filename="package://neo_simulation/robots/mmo_700/meshes/MPO-700-HEAD.dae" scale="0.001 0.001 0.001"/>
      </geometry>
     </collision>
    </link>
   </xacro:macro>
-  <xacro:macro name="mpo_700_head_1" params="name parent *origin">
+  <xacro:macro name="mpo_700_caster_1" params="name parent *origin">
    <joint name="${name}_joint" type="fixed">
     <insert_block name="origin" />
@@ -47,5 +47,5 @@
      <origin xyz="0 0 0.10" rpy="0 0 0"/>
      <geometry>
-        <mesh filename="package://neo_simulation/robots/mpo_700/meshes/MPO-700-HEAD.dae" scale="0.001 0.001 0.001"/>
+        <mesh filename="package://neo_simulation/robots/mmo_700/meshes/MPO-700-HEAD.dae" scale="0.001 0.001 0.001"/>
      </geometry>
     </visual>
@@ -53,10 +53,10 @@
      <origin xyz="0 0 0.10" rpy="0 0 0" />
      <geometry>
-        <mesh filename="package://neo_simulation/robots/mpo_700/meshes/MPO-700-HEAD.dae" scale="0.001 0.001 0.001"/>
+        <mesh filename="package://neo_simulation/robots/mmo_700/meshes/MPO-700-HEAD.dae" scale="0.001 0.001 0.001"/>
      </geometry>
     </collision>
    </link>
   </xacro:macro>
-  <xacro:macro name="mpo_700_head_2" params="name parent *origin">
+  <xacro:macro name="mpo_700_caster_2" params="name parent *origin">
    <joint name="${name}_joint" type="fixed">
     <insert_block name="origin" />
@@ -75,5 +75,5 @@
      <origin xyz="0 0 0.10" rpy="0 0 0"/>
      <geometry>
-        <mesh filename="package://neo_simulation/robots/mpo_700/meshes/MPO-700-HEAD.dae" scale="0.001 0.001 0.001"/>
+        <mesh filename="package://neo_simulation/robots/mmo_700/meshes/MPO-700-HEAD.dae" scale="0.001 0.001 0.001"/>
      </geometry>
     </visual>
@@ -81,10 +81,10 @@
      <origin xyz="0 0 0.10" rpy="0 0 0" />
      <geometry>
-        <mesh filename="package://neo_simulation/robots/mpo_700/meshes/MPO-700-HEAD.dae" scale="0.001 0.001 0.001"/>
+        <mesh filename="package://neo_simulation/robots/mmo_700/meshes/MPO-700-HEAD.dae" scale="0.001 0.001 0.001"/>
      </geometry>
     </collision>
    </link>
   </xacro:macro>
-  <xacro:macro name="mpo_700_head_3" params="name parent *origin">
+  <xacro:macro name="mpo_700_caster_3" params="name parent *origin">
    <joint name="${name}_joint" type="fixed">
     <insert_block name="origin" />
@@ -103,5 +103,5 @@
      <origin xyz="0 0 0.10" rpy="0 0 0"/>
      <geometry>
-        <mesh filename="package://neo_simulation/robots/mpo_700/meshes/MPO-700-HEAD.dae" scale="0.001 0.001 0.001"/>
+        <mesh filename="package://neo_simulation/robots/mmo_700/meshes/MPO-700-HEAD.dae" scale="0.001 0.001 0.001"/>
      </geometry>
     </visual>
@@ -109,5 +109,5 @@
      <origin xyz="0 0 0.10" rpy="0 0 0" />
      <geometry>
-        <mesh filename="package://neo_simulation/robots/mpo_700/meshes/MPO-700-HEAD.dae" scale="0.001 0.001 0.001"/>
+        <mesh filename="package://neo_simulation/robots/mmo_700/meshes/MPO-700-HEAD.dae" scale="0.001 0.001 0.001"/>
      </geometry>
     </collision>

File: robots/mmo_700/urdf/xacros/mpo_700_wheel.xacro (robot description, xacro)
@@ -1,5 +1,5 @@
 <?xml version="1.0"?>
 <robot xmlns:xacro="http://www.ros.org/wiki/xacro" name="mpo_700">
-  <xacro:macro name="mmo_700_wheel" params="name parent *origin">
+  <xacro:macro name="mpo_700_wheel" params="name parent *origin">
    <joint name="${name}_joint" type="fixed">
     <insert_block name="origin" />

File: robots/mmo_700/urdf/xacros/sick_S300.xacro (robot description, xacro)
@@ -10,18 +10,18 @@
     <link name="${name}_link" type="laser">
       <inertial>
-        <mass value="0.0001" />
+        <mass value="0.001" />
         <origin xyz="0 0 0" rpy="0 0 0" />
         <inertia ixx="0.0001" ixy="0" ixz="0" iyy="0.000001" iyz="0" izz="0.0001" />
       </inertial>
       <visual>
-        <origin xyz="0 0 -0.06" rpy="1.57 0 0" />
-      <geometry>
-        <mesh filename="package://neo_simulation/robots/mpo_700/meshes/SICK-MICROSCAN3.dae" scale="0.001 0.001 0.001" />
+        <origin xyz="0 0 -0.12" rpy="-1.57 0 3.14" />
+        <geometry>
+        <mesh filename="package://neo_simulation/robots/mpo_700/meshes/SICK-S300.dae" scale="0.001 0.001 0.001" />
         </geometry>
       </visual>
       <collision>
-        <origin xyz="0 0 -0.06" rpy="1.57 0 0" />
+        <origin xyz="0 0 -0.12" rpy="-1.57 0 3.14" />
         <geometry>
-          <mesh filename="package://neo_simulation/robots/mpo_700/meshes/SICK-MICROSCAN3.dae" scale="0.001 0.001 0.001" />
+        <mesh filename="package://neo_simulation/robots/mpo_700/meshes/SICK-S300.dae" scale="0.001 0.001 0.001" />
         </geometry>
       </collision>

File: robots/mpo_700/mpo_700.urdf.xacro (robot description, xacro)
@@ -16,26 +16,26 @@
   <xacro:mpo_700_base name="base_link">
   </xacro:mpo_700_base>
-<xacro:mpo_700_caster_0 name="mpo_700_caster_0" parent="base_link">
+<xacro:mpo_700_caster_0 name="mpo_700_caster_front_left" parent="base_link">
     <origin xyz="0.24 0.18 0.27" rpy="3.14 0 -1.57" />
   </xacro:mpo_700_caster_0>
-<xacro:mpo_700_caster_1 name="mpo_700_caster_1" parent="base_link">
+<xacro:mpo_700_caster_1 name="mpo_700_caster_front_right" parent="base_link">
     <origin xyz="0.24 -0.18 0.27" rpy="3.14 0 1.57" />
   </xacro:mpo_700_caster_1>
-<xacro:mpo_700_caster_2 name="mpo_700_caster_2" parent="base_link">
+<xacro:mpo_700_caster_2 name="mpo_700_caster_back_left" parent="base_link">
     <origin xyz="-0.24 0.18 0.27" rpy="3.14 0 -1.57" />
   </xacro:mpo_700_caster_2>
-<xacro:mpo_700_caster_3 name="mpo_700_caster_3" parent="base_link">
+<xacro:mpo_700_caster_3 name="mpo_700_caster_back_right" parent="base_link">
     <origin xyz="-0.24 -0.18 0.27" rpy="3.14 0 1.57" />
   </xacro:mpo_700_caster_3>
-<xacro:mpo_700_wheel name="wheel_0" parent="mpo_700_caster_0_link">
+<xacro:mpo_700_wheel name="mpo_700_wheel_front_left" parent="mpo_700_caster_front_left_link">
     <origin xyz="-0.05 0. 0.18" rpy="0 0 0" />
   </xacro:mpo_700_wheel>
-<xacro:mpo_700_wheel name="wheel_1" parent="mpo_700_caster_1_link">
+<xacro:mpo_700_wheel name="mpo_700_wheel_front_right" parent="mpo_700_caster_front_right_link">
     <origin xyz="-0.05 0. 0.18" rpy="0 0 0" />
   </xacro:mpo_700_wheel>
-<xacro:mpo_700_wheel name="wheel_2" parent="mpo_700_caster_2_link">
+<xacro:mpo_700_wheel name="mpo_700_wheel_back_left" parent="mpo_700_caster_back_left_link">
     <origin xyz="-0.05 0. 0.18" rpy="0 0 0" />
   </xacro:mpo_700_wheel>
-<xacro:mpo_700_wheel name="wheel_3" parent="mpo_700_caster_3_link">
+<xacro:mpo_700_wheel name="mpo_700_wheel_back_right" parent="mpo_700_caster_back_right_link">
     <origin xyz="-0.05 0. 0.18" rpy="0 0 0" />
   </xacro:mpo_700_wheel>

File: robots/mpo_700/xacros/mpo_700_body.xacro (robot description, xacro)
@@ -4,9 +4,9 @@
     <link name="${name}">
       <inertial>
-        <mass value="30" />
+        <mass value="0.01" />
         <origin xyz="0 0 0" rpy="0 0 0"/>
-        <inertia ixx="1.71402" ixy="0.0" ixz="0.0"
-                 iyy="0.8856" iyz="0.0"
-                 izz="2.5725" />
+        <inertia ixx="0.0008" ixy="0.0" ixz="0.0"
+                 iyy="0.0008" iyz="0.0"
+                 izz="0.0008" />
       </inertial>
       <visual>

File: robots/mpo_700/xacros/mpo_700_caster.xacro (robot description, xacro)
@@ -12,7 +12,7 @@
    <link name="${name}_link">
     <inertial>
-      <mass value="9" />
+  <mass value="0.0008" />
       <origin xyz="0 0 0" rpy="0 0 0" />
-      <inertia ixx="0.00044332" ixy="0" ixz="0" iyy="0.00044332" iyz="0" izz="0.00072" />
+      <inertia ixx="0.000044332" ixy="0" ixz="0" iyy="0.000044332" iyz="0" izz="0.000044332" />
     </inertial>
     <visual>
@@ -40,7 +40,7 @@
    <link name="${name}_link">
     <inertial>
-      <mass value="9" />
-      <origin xyz="0 0 0." rpy="0 0 0" />
-      <inertia ixx="0.00044332" ixy="0" ixz="0" iyy="0.00044332" iyz="0" izz="0.00072" />
+  <mass value="0.0008" />
+      <origin xyz="0 0 0" rpy="0 0 0" />
+      <inertia ixx="0.000044332" ixy="0" ixz="0" iyy="0.000044332" iyz="0" izz="0.000044332" />
     </inertial>
     <visual>
@@ -68,7 +68,7 @@
    <link name="${name}_link">
     <inertial>
-      <mass value="9" />
-      <origin xyz="0 0 0." rpy="0 0 0" />
-      <inertia ixx="0.00044332" ixy="0" ixz="0" iyy="0.00044332" iyz="0" izz="0.00072" />
+  <mass value="0.0008" />
+      <origin xyz="0 0 0" rpy="0 0 0" />
+      <inertia ixx="0.000044332" ixy="0" ixz="0" iyy="0.000044332" iyz="0" izz="0.000044332" />
     </inertial>
     <visual>
@@ -96,7 +96,7 @@
    <link name="${name}_link">
     <inertial>
-      <mass value="9" />
+  <mass value="0.0008" />
       <origin xyz="0 0 0" rpy="0 0 0" />
-      <inertia ixx="0.00044332" ixy="0" ixz="0" iyy="0.00044332" iyz="0" izz="0.00072" />
+      <inertia ixx="0.000044332" ixy="0" ixz="0" iyy="0.000044332" iyz="0" izz="0.000044332" />
     </inertial>
     <visual>

File: robots/mpo_700/xacros/mpo_700_wheel.xacro (robot description, xacro)
@@ -12,7 +12,9 @@
    <link name="${name}_link" type="wheel">
     <inertial>
-      <mass value="2" />
+      <mass value="0.0006" />
       <origin xyz="0 0 0" rpy="0 0 0" />
-      <inertia ixx="0.00044332" ixy="0" ixz="0" iyy="0.00044332" iyz="0" izz="0.00072" />
+        <inertia  ixx="0.04" ixy="0.000" ixz="0.0"
+                  iyy="0.02" iyz="0.00"
+                  izz="0.05" />
     </inertial>
     <visual>
