Commit message: changes in laser scanner position(z)

File: robots/mpo_500/mpo_500.urdf.xacro (robot description, xacro)
@@ -29,8 +29,8 @@
   <!-- Sensors -->
   <xacro:sick_s300_laser_v0 name="sick_s300_laser_front" parent="base_link" ros_topic="sick_s300_laser/front/scan">
-  	<origin xyz="0.442 0 0.362" rpy="0 0 0" />
+  	<origin xyz="0.442 0 0.420" rpy="0 0 0" />
   </xacro:sick_s300_laser_v0>
   <xacro:sick_s300_laser_v0 name="sick_s300_laser_back" parent="base_link" ros_topic="sick_s300_laser/back/scan">
-  	<origin xyz="-0.442 0 0.362" rpy="0 0 3.14" />
+  	<origin xyz="-0.442 0 0.420" rpy="0 0 3.14" />
   </xacro:sick_s300_laser_v0>
 </robot>

Commit message: Robot models have been added

File: robots/mpo_500/mpo_500.urdf.xacro (robot description, xacro)
@@ -3,6 +3,4 @@
   <!--GAZEBO REFERENCES -->
   <xacro:include filename="$(find neo_simulation)/robots/mpo_500/xacros/mpo_500_gazebo.xacro" />
-  <!-- MATERIALS -->
-  <xacro:include filename="$(find neo_simulation)/robots/mpo_500/xacros/mpo_500_materials.xacro" />
   <!-- BODY -->
   <xacro:include filename="$(find neo_simulation)/robots/mpo_500/xacros/mpo_500_body.xacro" />
@@ -10,5 +8,5 @@
   <xacro:include filename="$(find neo_simulation)/robots/mpo_500/xacros/omni_wheel.xacro" />
   <!-- SENSORS -->
-  <xacro:include filename="$(find neo_simulation)/robots/mpo_500/xacros/sick_s300_laser.xacro" />
+  <xacro:include filename="$(find neo_simulation)/robots/mpo_500/xacros/sick_laser.xacro" />
   <!-- Base Macro-->
   <xacro:mpo_500_base name="base_link">
@@ -28,9 +26,9 @@
   </xacro:omni_wheel_250>
   <!-- Sensors -->
-  <xacro:sick_s300_laser_v0 name="sick_s300_laser_front" parent="base_link" ros_topic="sick_s300_front/scan">
-  	<origin xyz="0.442 0 0.420" rpy="0 0 0" />
-  </xacro:sick_s300_laser_v0>
-  <xacro:sick_s300_laser_v0 name="sick_s300_laser_back" parent="base_link" ros_topic="sick_s300_back/scan">
-  	<origin xyz="-0.442 0 0.420" rpy="0 0 3.14" />
-  </xacro:sick_s300_laser_v0>
+  <xacro:sick_laser_v0 name="sick_laser_front" parent="base_link" ros_topic="sick_front/scan">
+  	<origin xyz="0.442 0 0.372" rpy="0 0 0" />
+  </xacro:sick_laser_v0>
+  <xacro:sick_laser_v0 name="sick_laser_back" parent="base_link" ros_topic="sick_back/scan">
+  	<origin xyz="-0.442 0 0.372" rpy="0 0 3.14" />
+  </xacro:sick_laser_v0>
 </robot>

File: robots/mpo_500/xacros/mpo_500_body.xacro (robot description, xacro)
@@ -11,15 +11,14 @@
       </inertial>
       <visual>
-        <origin xyz="0. 0. 0.215" rpy="0 0 1.571" />
+        <origin xyz="0. 0. 0" rpy="-1.571 0 1.571" />
         <geometry>
-            <mesh filename="package://neo_simulation/robots/mpo_500/meshes/MPO-500-BODY.STL"/>
+            <mesh filename="package://neo_simulation/robots/mpo_500/meshes/MPO-500-BODY.dae" scale="0.001 0.001 0.001"/>
         </geometry>
-        <material name="Neobotix/Grey" />
       </visual>
       <collision>
-        <origin xyz="0. 0. 0.2" rpy="0 0 0" />
+        <origin xyz="0. 0. 0.0" rpy="-1.571 0 1.571" />
         <geometry>
           <!--<box size="0.68 0.41 0.25"/> -->
-          <box size="0.769 0.51 0.307" />
+           <mesh filename="package://neo_simulation/robots/mpo_500/meshes/MPO-500-BODY.dae" scale="0.001 0.001 0.001"/>
         </geometry>
       </collision>

File: robots/mpo_500/xacros/mpo_500_gazebo.xacro (robot description, xacro)
@@ -4,28 +4,22 @@
     <gravity>true</gravity>
     <self_collide>false</self_collide>
-    <material value="Gazebo/Grey"/>
   </gazebo>
    <gazebo reference="wheel_front_left_link">
     <gravity>true</gravity>
     <self_collide>false</self_collide>
-    <material value="Gazebo/Black"/>
   </gazebo>
   <gazebo reference="wheel_front_right_link">
     <gravity>true</gravity>
     <self_collide>false</self_collide>
-    <material value="Gazebo/Black"/>
   </gazebo>
   <gazebo reference="wheel_back_left_link">
     <gravity>true</gravity>
     <self_collide>false</self_collide>
-    <material value="Gazebo/Black"/>
   </gazebo>
   <gazebo reference="wheel_back_right_link">
     <gravity>true</gravity>
     <self_collide>false</self_collide>
-    <material value="Gazebo/Black"/>
   </gazebo>
-  <gazebo reference="sick_s300_laser_front_link">
-      <material value="Gazebo/Yellow"/>
+  <gazebo reference="sick_laser_front_link">
       <sensor type="ray" name="sick_s300_laser_front_sensor">
           <pose>0 0 0 0 0 0</pose>
@@ -37,6 +31,6 @@
                 <samples>720</samples>
                 <resolution>1</resolution>
-                <min_angle>-2.35619</min_angle>
-                <max_angle>2.35619</max_angle>
+                <min_angle>-1.48353</min_angle>
+                <max_angle>1.48353</max_angle>
               </horizontal>
             </scan>
@@ -56,13 +50,12 @@
             </noise>
           </ray>
-          <plugin name="sick_s300_laser_front" filename="libgazebo_ros_laser.so">
-            <topicName>sick_s300_front/scan</topicName>
-            <frameName>sick_s300_laser_front_link</frameName>
+          <plugin name="sick_laser_front" filename="libgazebo_ros_laser.so">
+            <topicName>sick_front/scan</topicName>
+            <frameName>sick_laser_front_link</frameName>
           </plugin>
         </sensor>
   </gazebo>
-  <gazebo reference="sick_s300_laser_back_link">
-      <material value="Gazebo/Yellow"/>
-      <sensor type="ray" name="sick_s300_laser_back_sensor">
+  <gazebo reference="sick_laser_back_link">
+      <sensor type="ray" name="sick_laser_back_sensor">
           <pose>0 0 0 0 0 0</pose>
           <visualize>false</visualize>
@@ -73,6 +66,6 @@
                 <samples>720</samples>
                 <resolution>1</resolution>
-                <min_angle>-2.35619</min_angle>
-                <max_angle>2.35619</max_angle>
+                <min_angle>-1.48353</min_angle>
+                <max_angle>1.48353</max_angle>
               </horizontal>
             </scan>
@@ -92,7 +85,7 @@
             </noise>
           </ray>
-          <plugin name="sick_s300_laser_back" filename="libgazebo_ros_laser.so">
-            <topicName>sick_s300_back/scan</topicName>
-            <frameName>sick_s300_laser_back_link</frameName>
+          <plugin name="sick_laser_back" filename="libgazebo_ros_laser.so">
+            <topicName>sick_back/scan</topicName>
+            <frameName>sick_laser_back_link</frameName>
           </plugin>
         </sensor>
@@ -101,8 +94,4 @@
     <plugin name="mpo_500_controller" filename="libgazebo_ros_planar_move.so">
       <commandTopic>cmd_vel</commandTopic>
-      <leftFrontJoint>wheel_front_left_joint</leftFrontJoint>
-      <rightFrontJoint>wheel_front_right_joint</rightFrontJoint>
-      <leftRearJoint>wheel_back_left_joint</leftRearJoint>
-      <rightRearJoint>wheel_back_right_joint</rightRearJoint>
       <odometryTopic>odom</odometryTopic>
       <odometryFrame>odom</odometryFrame>

File: robots/mpo_500/xacros/omni_wheel.xacro (robot description, xacro)
@@ -11,19 +11,18 @@
    <link name="${name}_link" type="wheel">
     <inertial>
-      <mass value="0.1" />
+      <mass value="9" />
       <origin xyz="0 0 0" rpy="0 0 0" />
       <inertia ixx="0.00044332" ixy="0" ixz="0" iyy="0.00044332" iyz="0" izz="0.00072" />
     </inertial>
     <visual>
-     <origin xyz="0 0 0" rpy="0 0 1.571" />
+     <origin xyz="0 0 0" rpy="0 0 0"/>
      <geometry>
-        <mesh filename="package://neo_simulation/robots/mpo_500/meshes/MPO-500-WHEEL.STL"/>
+        <mesh filename="package://neo_simulation/robots/mpo_500/meshes/MPO-500-WHEEL.dae" scale="0.001 0.001 0.001"/>
      </geometry>
-     <material name="Neobotix/Black" />
     </visual>
     <collision>
-     <origin xyz="0 0 0" rpy="1.59 0 0" />
+     <origin xyz="0 0 0" rpy="0 0 0" />
      <geometry>
-        <cylinder radius="0.12" length="0.1"/>
+        <mesh filename="package://neo_simulation/robots/mpo_500/meshes/MPO-500-WHEEL.dae" scale="0.001 0.001 0.001"/>
      </geometry>
     </collision>

File: robots/mpo_700/mpo_700.urdf.xacro (robot description, xacro)
@@ -1,20 +1,52 @@
 <?xml version="1.0" ?>
 <robot name="mpo_700" xmlns:xacro="http://www.ros.org/wiki/xacro">
-  <!-- MATERIALS -->
-  <xacro:include filename="$(find neo_simulation)/robots/mpo_700/xacros/mpo_700_materials.xacro" />
   <!-- BODY -->
   <xacro:include filename="$(find neo_simulation)/robots/mpo_700/xacros/mpo_700_body.xacro" />
   <!-- SENSORS -->
-  <xacro:include filename="$(find neo_simulation)/robots/mpo_700/xacros/sick_s300_laser.xacro" />
+  <xacro:include filename="$(find neo_simulation)/robots/mpo_700/xacros/sick_laser.xacro" />
   <xacro:include filename="$(find neo_simulation)/robots/mpo_700/xacros/mpo_700_gazebo.xacro" />
+  <xacro:include filename="$(find neo_simulation)/robots/mpo_700/xacros/mpo_700_head.xacro" />
+  <xacro:include filename="$(find neo_simulation)/robots/mpo_700/xacros/mpo_700_wheel.xacro" />
   <!-- Base Macro-->
   <xacro:mpo_700_base name="base_link">
   </xacro:mpo_700_base>
-  <!-- Sensors -->
-  <xacro:sick_s300_laser_v0 name="sick_s300_laser_front" parent="base_link" ros_topic="sick_s300_front/scan">
-  	<origin xyz="0.360 0 0.223" rpy="3.14 0 1.57" />
-  </xacro:sick_s300_laser_v0>
-  <xacro:sick_s300_laser_v0 name="sick_s300_laser_back" parent="base_link" ros_topic="sick_s300_back/scan">
-  	<origin xyz="-0.360 0 0.223" rpy="3.14 0 -1.57" />
-  </xacro:sick_s300_laser_v0>
+<xacro:mpo_700_head_0 name="mpo_700_head_0" parent="base_link">
+    <origin xyz="0.24 0.18 0.25" rpy="3.14 0 -1.57" />
+  </xacro:mpo_700_head_0>
+<xacro:mpo_700_head_1 name="mpo_700_head_1" parent="base_link">
+    <origin xyz="0.24 -0.18 0.25" rpy="3.14 0 1.57" />
+  </xacro:mpo_700_head_1>
+<xacro:mpo_700_head_2 name="mpo_700_head_2" parent="base_link">
+    <origin xyz="-0.24 0.18 0.25" rpy="3.14 0 -1.57" />
+  </xacro:mpo_700_head_2>
+<xacro:mpo_700_head_3 name="mpo_700_head_3" parent="base_link">
+    <origin xyz="-0.24 -0.18 0.25" rpy="3.14 0 1.57" />
+  </xacro:mpo_700_head_3>
+<xacro:mpo_700_wheel name="wheel_0" parent="mpo_700_head_0_link">
+    <origin xyz="-0.05 0. 0.18" rpy="0 0 0" />
+  </xacro:mpo_700_wheel>
+<xacro:mpo_700_wheel name="wheel_1" parent="mpo_700_head_1_link">
+    <origin xyz="-0.05 0. 0.18" rpy="0 0 0" />
+  </xacro:mpo_700_wheel>
+<xacro:mpo_700_wheel name="wheel_2" parent="mpo_700_head_2_link">
+    <origin xyz="-0.05 0. 0.18" rpy="0 0 0" />
+  </xacro:mpo_700_wheel>
+<xacro:mpo_700_wheel name="wheel_3" parent="mpo_700_head_3_link">
+    <origin xyz="-0.05 0. 0.18" rpy="0 0 0" />
+  </xacro:mpo_700_wheel>
+<!-- Sensors -->
+<!-- Uncomment or comment it for sick s300 -->
+  <xacro:sick_v0 name="sick_s300_laser_front" parent="base_link" ros_topic="sick_s300_front/scan">
+  	<origin xyz="0.360 0 0.181" rpy="3.14 0 0 " />
+  </xacro:sick_v0>
+  <xacro:sick_v0 name="sick_s300_laser_back" parent="base_link" ros_topic="sick_s300_back/scan">
+  	<origin xyz="-0.360 0 0.181" rpy="3.14 0 3.14" />
+  </xacro:sick_v0>
+<!-- Uncomment or comment it for sick_microscan_3 -->
+<!--   <xacro:sick_v0 name="sick_microscan_3_front" parent="base_link" ros_topic="sick_s300_front/scan">
+    <origin xyz="0.360 0 0.28" rpy="3.14 3.14 0" />
+  </xacro:sick_v0>
+  <xacro:sick_v0 name="sick_microscan_3_back" parent="base_link" ros_topic="sick_s300_back/scan">
+    <origin xyz="-0.360 0 0.28" rpy="3.14 3.14 3.14" />
+  </xacro:sick_v0> -->
 </robot>

File: robots/mpo_700/xacros/mpo_700_body.xacro (robot description, xacro)
@@ -11,14 +11,13 @@
       </inertial>
       <visual>
-        <origin xyz="0.0 0.0 0.021" rpy="0 0 1.571" />
+        <origin xyz="0.0 0.0 0.0" rpy="0 0 -1.571" />
         <geometry>
-            <mesh filename="package://neo_simulation/robots/mpo_700/meshes/MPO-700.stl" scale="0.001 0.001 0.001"/>
+            <mesh filename="package://neo_simulation/robots/mpo_700/meshes/MPO-700-BODY.dae" scale="0.001 0.001 0.001"/>
         </geometry>
-        <material name="Neobotix/Grey" />
       </visual>
       <collision>
         <origin xyz="0. 0. 0.2" rpy="0 0 0" />
         <geometry>
-          <box size="0.610 0.515 0.360" />
+            <mesh filename="package://neo_simulation/robots/mpo_700/meshes/MPO-700-BODY.dae" scale="0.001 0.001 0.001"/>
         </geometry>
       </collision>

File: robots/mpo_700/xacros/mpo_700_gazebo.xacro (robot description, xacro)
@@ -1,11 +1,9 @@
 <?xml version="1.0"?>
-<robot name="mpo_500" xmlns:xacro="http://www.ros.org/wiki/xacro">
+<robot name="mpo_700" xmlns:xacro="http://www.ros.org/wiki/xacro">
    <gazebo reference="base_link">
     <gravity>true</gravity>
     <self_collide>false</self_collide>
-    <material value="Gazebo/Grey"/>
   </gazebo>
   <gazebo reference="sick_s300_laser_front_link">
-      <material value="Gazebo/Yellow"/>
       <sensor type="ray" name="sick_s300_laser_front_sensor">
           <pose>0 0 0 0 0 0</pose>
@@ -17,6 +15,6 @@
                 <samples>720</samples>
                 <resolution>1</resolution>
-                <min_angle>-0.174533</min_angle>
-                <max_angle>3.31613</max_angle>
+                <min_angle>-1.48</min_angle>
+                <max_angle>1.48</max_angle>
               </horizontal>
             </scan>
@@ -43,5 +41,4 @@
   </gazebo>
   <gazebo reference="sick_s300_laser_back_link">
-      <material value="Gazebo/Yellow"/>
       <sensor type="ray" name="sick_s300_laser_back_sensor">
           <pose>0 0 0 0 0 0</pose>
@@ -53,6 +50,6 @@
                 <samples>720</samples>
                 <resolution>1</resolution>
-                <min_angle>-0.174533</min_angle>
-                <max_angle>3.31613</max_angle>
+                <min_angle>-1.48</min_angle>
+                <max_angle>1.48</max_angle>
               </horizontal>
             </scan>
@@ -79,5 +76,5 @@
   </gazebo>
   <gazebo>
-    <plugin name="mpo_500_controller" filename="libgazebo_ros_planar_move.so">
+    <plugin name="mpo_700_controller" filename="libgazebo_ros_planar_move.so">
       <commandTopic>cmd_vel</commandTopic>
       <odometryTopic>odom</odometryTopic>

Commit message: MPO-500 is better with the wheels now changed from fixed to revolute joint

File: robots/mpo_500/mpo_500.urdf.xacro (robot description, xacro)
@@ -9,6 +9,4 @@
   <!-- SENSORS -->
   <xacro:include filename="$(find neo_simulation)/robots/mpo_500/xacros/sick_laser.xacro" />
-  <xacro:include filename="$(find neo_simulation)/robots/mpo_500/xacros/imu.xacro" />
-  <xacro:include filename="$(find neo_simulation)/robots/mpo_500/xacros/ultrasonic.xacro" />
   <!-- Base Macro-->
   <xacro:mpo_500_base name="base_link">
@@ -28,84 +26,9 @@
   </xacro:omni_wheel_250>
   <!-- Sensors -->
-  <xacro:sick_laser_v0 name="lidar_1" parent="base_link" ros_topic="lidar_1/scan_filtered">
+  <xacro:sick_laser_v0 name="lidar_1" parent="base_link" ros_topic="lidar_1/scan">
   	<origin xyz="0.442 0 0.372" rpy="0 0 0" />
   </xacro:sick_laser_v0>
-  <xacro:sick_laser_v0 name="lidar_2" parent="base_link" ros_topic="lidar_2/scan_filtered">
+  <xacro:sick_laser_v0 name="lidar_2" parent="base_link" ros_topic="lidar_2/scan">
   	<origin xyz="-0.442 0 0.372" rpy="0 0 3.14" />
   </xacro:sick_laser_v0>
-     <!--+++++++++++++++++++ IMU ++++++++++++++++++++++++-->
- <!-- Comment or uncomment based on your requirement -->
-<!--   <xacro:imu name="imu_1" parent="base_link">
-    <origin xyz="0.100 0 0.300" rpy="0 0 3.14" />
-  </xacro:imu> -->
-  <!--+++++++++++++++++++ Ultra Sonic ++++++++++++++++++++++++-->
-  <!-- Comment or uncomment based on your requirement -->
-  <!-- SENSOR 1 -->
-  <!-- xacro:us_sensor name="us_1" parent="base_link">
-    <origin xyz="0.100 0 0.300" rpy="0 3.14 3.14" />
-  </xacro:us_sensor-->
-  <!-- SENSOR 2 -->
-  <!-- xacro:us_sensor name="us_2" parent="base_link">
-    <origin xyz="0.110 0 0.300" rpy="0 3.14 3.14" />
-  </xacro:us_sensor-->
-  <!-- SENSOR 3 -->
-  <!-- xacro:us_sensor name="us_3" parent="base_link">
-    <origin xyz="0.120 0 0.300" rpy="0 3.14 3.14" />
-  </xacro:us_sensor-->
-  <!-- SENSOR 4 -->
-  <!-- xacro:us_sensor name="us_4" parent="base_link">
-    <origin xyz="0.130 0 0.300" rpy="0 3.14 3.14" />
-  </xacro:us_sensor-->
-  <!-- SENSOR 5 -->
-  <!-- xacro:us_sensor name="us_5" parent="base_link">
-    <origin xyz="0.140 0 0.300" rpy="0 3.14 3.14" />
-  </xacro:us_sensor-->
-  <!-- SENSOR 6 -->
-  <!-- xacro:us_sensor name="us_6" parent="base_link">
-    <origin xyz="0.150 0 0.300" rpy="0 3.14 3.14" />
-  </xacro:us_sensor-->
-  <!-- SENSOR 7 -->
-  <!-- xacro:us_sensor name="us_7" parent="base_link">
-    <origin xyz="0.160 0 0.300" rpy="0 3.14 3.14" />
-  </xacro:us_sensor-->
-  <!-- SENSOR 8 -->
-  <!-- xacro:us_sensor name="us_8" parent="base_link">
-    <origin xyz="0.170 0 0.300" rpy="0 3.14 3.14" />
-  </xacro:us_sensor-->
-  <!-- SENSOR 9 -->
-  <!-- xacro:us_sensor name="us_9" parent="base_link">
-    <origin xyz="0.180 0 0.300" rpy="0 3.14 3.14" />
-  </xacro:us_sensor-->
-  <!-- SENSOR 10 -->
-  <!-- xacro:us_sensor name="us_10" parent="base_link">
-    <origin xyz="0.100 0 0.300" rpy="0 3.14 3.14" />
-  </xacro:us_sensor-->
-  <!-- SENSOR 11 -->
-  <!-- xacro:us_sensor name="us_11" parent="base_link">
-    <origin xyz="0.100 0 0.300" rpy="0 3.14 3.14" />
-  </xacro:us_sensor-->
-  <!-- SENSOR 12 -->
-  <!-- xacro:us_sensor name="us_12" parent="base_link">
-    <origin xyz="0.190 0 0.300" rpy="0 3.14 3.14" />
-  </xacro:us_sensor-->
-  <!-- SENSOR 13 -->
-  <!-- xacro:us_sensor name="us_13" parent="base_link">
-    <origin xyz="0.200 0 0.300" rpy="0 3.14 3.14" />
-  </xacro:us_sensor-->
-  <!-- SENSOR 14 -->
-  <!-- xacro:us_sensor name="us_14" parent="base_link">
-    <origin xyz="0.210 0 0.300" rpy="0 3.14 3.14" />
-  </xacro:us_sensor-->
-  <!-- SENSOR 15 -->
-  <!-- xacro:us_sensor name="us_15" parent="base_link">
-    <origin xyz="0.220 0 0.300" rpy="0 3.14 3.14" />
-  </xacro:us_sensor-->
-  <!-- SENSOR 16 -->
-  <!-- xacro:us_sensor name="us_16" parent="base_link">
-    <origin xyz="0.230 0 0.300" rpy="0 3.14 3.14" />
-  </xacro:us_sensor-->
-    <!--Camera  -->
-<!-- <xacro:camera name="camera" parent="base_link">
-    <origin xyz="0 0 0.38" rpy="0 0 0" />
-  </xacro:camera> -->
 </robot>

File: robots/mpo_500/xacros/mpo_500_body.xacro (robot description, xacro)
@@ -4,5 +4,5 @@
     <link name="${name}">
       <inertial>
-        <mass value="30" />
+        <mass value="0.02" />
         <origin xyz="0 0 0" rpy="0 0 0"/>
         <inertia ixx="1.71402" ixy="0.0" ixz="0.0"

File: robots/mpo_500/xacros/mpo_500_gazebo.xacro (robot description, xacro)
@@ -86,102 +86,8 @@
           </ray>
           <plugin name="lidar_2" filename="libgazebo_ros_laser.so">
-            <topicName>lidar_2/scan_filtered</topicName>
+            <topicName>lidar_2/scan</topicName>
             <frameName>lidar_2_link</frameName>
           </plugin>
         </sensor>
-  </gazebo>
-    <gazebo reference="imu_1_link">
-    <gravity>true</gravity>
-    <sensor name="imu_sensor" type="imu">
-      <always_on>true</always_on>
-      <update_rate>100</update_rate>
-      <visualize>true</visualize>
-      <topic>__default_topic__</topic>
-      <plugin filename="libgazebo_ros_imu_sensor.so" name="imu_plugin">
-        <topicName>imu</topicName>
-        <bodyName>imu_link</bodyName>
-        <updateRateHZ>10.0</updateRateHZ>
-        <gaussianNoise>0.0</gaussianNoise>
-        <xyzOffset>0 0 0</xyzOffset>
-        <rpyOffset>0 0 0</rpyOffset>
-        <frameName>imu_link</frameName>
-      </plugin>
-      <pose>0 0 0 0 0 0</pose>
-    </sensor>
-  </gazebo>
-  <gazebo reference="us_1_link">
-  <!-- Visuals / Collisions omitted for this example -->
-  <sensor type="ray" name="range">
-    <ray>
-         <scan>
-            <horizontal>
-               <samples>1</samples>
-               <resolution>1.0</resolution>
-               <min_angle>-0.01</min_angle>
-               <max_angle>0.01</max_angle>
-            </horizontal>
-            <vertical>
-               <samples>1</samples>
-               <resolution>1</resolution>
-               <min_angle>-0.01</min_angle>
-               <max_angle>0.01</max_angle>
-            </vertical>
-         </scan>
-         <range>
-            <min>0.01</min>
-            <max>3.75</max>
-            <resolution>0.02</resolution>
-         </range>
-      </ray>
-    <plugin name="libgazebo_ros_range" filename="libgazebo_ros_range.so">
-         <gaussianNoise>0.005</gaussianNoise>
-         <alwaysOn>true</alwaysOn>
-         <updateRate>50</updateRate>
-         <topicName>us_sensor</topicName>
-         <frameName>us_1_link</frameName>
-         <radiation>SONAR</radiation>
-         <fov>0.2967</fov>
-    </plugin>
-  </sensor>
-  </gazebo>
-    <!-- camera -->
-  <gazebo reference="camera_link">
-    <sensor type="camera" name="camera1">
-      <update_rate>30.0</update_rate>
-      <camera name="head">
-        <horizontal_fov>1.3962634</horizontal_fov>
-        <image>
-          <width>800</width>
-          <height>800</height>
-          <format>R8G8B8</format>
-        </image>
-        <clip>
-          <near>0.02</near>
-          <far>300</far>
-        </clip>
-        <noise>
-          <type>gaussian</type>
-          <!-- Noise is sampled independently per pixel on each frame.
-               That pixel's noise value is added to each of its color
-               channels, which at that point lie in the range [0,1]. -->
-          <mean>0.0</mean>
-          <stddev>0.007</stddev>
-        </noise>
-      </camera>
-      <plugin name="camera_controller" filename="libgazebo_ros_camera.so">
-        <alwaysOn>true</alwaysOn>
-        <updateRate>0.0</updateRate>
-        <cameraName>camera1</cameraName>
-        <imageTopicName>image_raw</imageTopicName>
-        <cameraInfoTopicName>camera_info</cameraInfoTopicName>
-        <frameName>camera_link</frameName>
-        <hackBaseline>0.07</hackBaseline>
-        <distortionK1>0.0</distortionK1>
-        <distortionK2>0.0</distortionK2>
-        <distortionK3>0.0</distortionK3>
-        <distortionT1>0.0</distortionT1>
-        <distortionT2>0.0</distortionT2>
-      </plugin>
-    </sensor>
   </gazebo>
   <gazebo>

File: robots/mpo_500/xacros/omni_wheel.xacro (robot description, xacro)
@@ -2,8 +2,10 @@
 <robot xmlns:xacro="http://www.ros.org/wiki/xacro" name="mpo_500">
   <xacro:macro name="omni_wheel_250" params="name parent *origin">
-   <joint name="${name}_joint" type="fixed">
+   <joint name="${name}_joint" type="revolute">
     <insert_block name="origin" />
     <axis xyz="0 1 0" />
-    <joint_properties damping="1" friction="1" />
+    <joint_properties damping="100" friction="1000" />
+        <limit effort="1000.0" lower="-1e+16" upper="1e+16" velocity="3.5"/>
+    <joint_properties damping="1.0" friction="1" />
     <parent link="${parent}" />
     <child link="${name}_link" />
@@ -11,5 +13,5 @@
    <link name="${name}_link" type="wheel">
     <inertial>
-      <mass value="9" />
+      <mass value="1" />
       <origin xyz="0 0 0" rpy="0 0 0" />
       <inertia ixx="0.00044332" ixy="0" ixz="0" iyy="0.00044332" iyz="0" izz="0.00072" />
