Commit message: robot models updated for MMO-700, MPO-700, MMO-500, MPO-500

File: robots/mpo_500/mpo_500.urdf.xacro (robot description, xacro)
@@ -8,5 +8,10 @@
   <xacro:include filename="$(find neo_simulation)/robots/mpo_500/xacros/omni_wheel.xacro" />
   <!-- SENSORS -->
-  <xacro:include filename="$(find neo_simulation)/robots/mpo_500/xacros/sick_laser.xacro" />
+  <xacro:include filename="$(find neo_simulation)/robots/mpo_500/xacros/sick_S300.xacro" />
+  <!-- Microscan - Comment/Uncomment if required -->
+  <!-- <xacro:include filename="$(find neo_simulation)/robots/mpo_500/xacros/micro_scan.xacro" />  -->
+  <!--<xacro:include filename="$(find neo_simulation)/robots/mpo_500/xacros/imu.xacro" />
+  <xacro:include filename="$(find neo_simulation)/robots/mpo_500/xacros/ultrasonic.xacro" /> -->
+  <xacro:include filename="$(find neo_simulation)/robots/mpo_500/xacros/mpo_500_gazebo.xacro" />
   <!-- Base Macro-->
   <xacro:mpo_500_base name="base_link">

File: robots/mpo_700/mpo_700.urdf.xacro (robot description, xacro)
@@ -3,47 +3,52 @@
   <!-- BODY -->
   <xacro:include filename="$(find neo_simulation)/robots/mpo_700/xacros/mpo_700_body.xacro" />
-  <xacro:include filename="$(find neo_simulation)/robots/mpo_700/xacros/mpo_700_head.xacro" />
+  <!-- SENSORS -->
+  <!-- Sick S300 - Comment/Uncomment if required -->
+  <!-- <xacro:include filename="$(find neo_simulation)/robots/mpo_700/xacros/sick_S300.xacro" /> -->
+  <!-- Microscan - Comment/Uncomment if required -->
+  <xacro:include filename="$(find neo_simulation)/robots/mpo_700/xacros/micro_scan.xacro" />
+  <!--<xacro:include filename="$(find neo_simulation)/robots/mpo_700/xacros/imu.xacro" />
+  <xacro:include filename="$(find neo_simulation)/robots/mpo_700/xacros/ultrasonic.xacro" /> -->
+  <xacro:include filename="$(find neo_simulation)/robots/mpo_700/xacros/mpo_700_gazebo.xacro" />
+<!-- Caster and wheels -->
+  <xacro:include filename="$(find neo_simulation)/robots/mpo_700/xacros/mpo_700_caster.xacro" />
   <xacro:include filename="$(find neo_simulation)/robots/mpo_700/xacros/mpo_700_wheel.xacro" />
-  <!-- SENSORS -->
-  <xacro:include filename="$(find neo_simulation)/robots/mpo_700/xacros/sick_laser.xacro" />
-  <xacro:include filename="$(find neo_simulation)/robots/mpo_700/xacros/imu.xacro" />
-  <xacro:include filename="$(find neo_simulation)/robots/mpo_700/xacros/ultrasonic.xacro" />
-  <!-- <xacro:include filename="$(find neo_simulation)/robots/mpo_700/xacros/camera.xacro" /> -->
-  <xacro:include filename="$(find neo_simulation)/robots/mpo_700/xacros/mpo_700_gazebo.xacro" />
   <!-- Base Macro-->
   <xacro:mpo_700_base name="base_link">
   </xacro:mpo_700_base>
-<xacro:mpo_700_head_0 name="mpo_700_head_0" parent="base_link">
+<xacro:mpo_700_caster_0 name="mpo_700_caster_front_left" parent="base_link">
     <origin xyz="0.24 0.18 0.27" rpy="3.14 0 -1.57" />
-  </xacro:mpo_700_head_0>
-<xacro:mpo_700_head_1 name="mpo_700_head_1" parent="base_link">
+  </xacro:mpo_700_caster_0>
+<xacro:mpo_700_caster_1 name="mpo_700_caster_front_right" parent="base_link">
     <origin xyz="0.24 -0.18 0.27" rpy="3.14 0 1.57" />
-  </xacro:mpo_700_head_1>
-<xacro:mpo_700_head_2 name="mpo_700_head_2" parent="base_link">
+  </xacro:mpo_700_caster_1>
+<xacro:mpo_700_caster_2 name="mpo_700_caster_back_left" parent="base_link">
     <origin xyz="-0.24 0.18 0.27" rpy="3.14 0 -1.57" />
-  </xacro:mpo_700_head_2>
-<xacro:mpo_700_head_3 name="mpo_700_head_3" parent="base_link">
+  </xacro:mpo_700_caster_2>
+<xacro:mpo_700_caster_3 name="mpo_700_caster_back_right" parent="base_link">
     <origin xyz="-0.24 -0.18 0.27" rpy="3.14 0 1.57" />
-  </xacro:mpo_700_head_3>
-<xacro:mpo_700_wheel name="wheel_0" parent="mpo_700_head_0_link">
+  </xacro:mpo_700_caster_3>
+<xacro:mpo_700_wheel name="mpo_700_wheel_front_left" parent="mpo_700_caster_front_left_link">
     <origin xyz="-0.05 0. 0.18" rpy="0 0 0" />
   </xacro:mpo_700_wheel>
-<xacro:mpo_700_wheel name="wheel_1" parent="mpo_700_head_1_link">
+<xacro:mpo_700_wheel name="mpo_700_wheel_front_right" parent="mpo_700_caster_front_right_link">
     <origin xyz="-0.05 0. 0.18" rpy="0 0 0" />
   </xacro:mpo_700_wheel>
-<xacro:mpo_700_wheel name="wheel_2" parent="mpo_700_head_2_link">
+<xacro:mpo_700_wheel name="mpo_700_wheel_back_left" parent="mpo_700_caster_back_left_link">
     <origin xyz="-0.05 0. 0.18" rpy="0 0 0" />
   </xacro:mpo_700_wheel>
-<xacro:mpo_700_wheel name="wheel_3" parent="mpo_700_head_3_link">
+<xacro:mpo_700_wheel name="mpo_700_wheel_back_right" parent="mpo_700_caster_back_right_link">
     <origin xyz="-0.05 0. 0.18" rpy="0 0 0" />
   </xacro:mpo_700_wheel>
 <!-- Sensors -->
-  <xacro:sick_v0 name="lidar_1" parent="base_link" ros_topic="lidar_1/scan_filtered">
-  	<origin xyz="0.360 0 0.181" rpy="3.14 0 0 " />
-  </xacro:sick_v0>
-  <xacro:sick_v0 name="lidar_2" parent="base_link" ros_topic="lidar_2/scan_filtered">
-  	<origin xyz="-0.360 0 0.181" rpy="3.14 0 3.14" />
-  </xacro:sick_v0>
-   <!--+++++++++++++++++++ IMU ++++++++++++++++++++++++-->
+  <xacro:sick_laser_v0 name="lidar_1" parent="base_link" ros_topic="lidar_1/scan_filtered">
+  <!--<origin xyz="0.360 0 0.181" rpy="3.14 0 0" />-->
+    <origin xyz="0.338 0.288 0.223" rpy="3.14 0 0.79" /> <!-- Scanners on the side -->
+  </xacro:sick_laser_v0>
+  <xacro:sick_laser_v0 name="lidar_2" parent="base_link" ros_topic="lidar_2/scan_filtered">
+  <!--<origin xyz="-0.360 0 0.181" rpy="3.14 0 3.14" />-->
+    <origin xyz="-0.338 -0.288 0.223" rpy="3.14 0 3.93" /> <!-- Scanners on the side -->
+  </xacro:sick_laser_v0>
+     <!--+++++++++++++++++++ IMU ++++++++++++++++++++++++-->
  <!-- Comment or uncomment based on your requirement -->
 <!--   <xacro:imu name="imu_1" parent="base_link">
@@ -53,7 +58,7 @@
   <!-- Comment or uncomment based on your requirement -->
   <!-- SENSOR 1 -->
-<!--   <xacro:us_sensor name="us_1" parent="base_link">
-    <origin xyz="0.100 0 0.500" rpy="0 3.14 3.14"/>
-  </xacro:us_sensor> -->
+  <!-- xacro:us_sensor name="us_1" parent="base_link">
+    <origin xyz="0.100 0 0.300" rpy="0 3.14 3.14" />
+  </xacro:us_sensor-->
   <!-- SENSOR 2 -->
   <!-- xacro:us_sensor name="us_2" parent="base_link">
@@ -116,7 +121,8 @@
     <origin xyz="0.230 0 0.300" rpy="0 3.14 3.14" />
   </xacro:us_sensor-->
-    <!--Camera  -->
+      <!--Camera  -->
 <!-- <xacro:camera name="camera" parent="base_link">
     <origin xyz="0 0 0.38" rpy="0 0 0" />
-  </xacro:camera> -->
+  </xacro:camera>
+ -->
 </robot>

File: robots/mpo_700/xacros/mpo_700_gazebo.xacro (robot description, xacro)
@@ -75,5 +75,5 @@
         </sensor>
   </gazebo>
-    <gazebo reference="imu_1_link">
+    <gazebo reference="imu_link">
     <gravity>true</gravity>
     <sensor name="imu_sensor" type="imu">
@@ -97,6 +97,4 @@
   <gazebo reference="camera_link">
     <sensor type="camera" name="camera1">
-      <pose>0 0 0 0 0 0</pose>
-      <update_rate>50</update_rate>
       <update_rate>30.0</update_rate>
       <camera name="head">
@@ -136,39 +134,4 @@
     </sensor>
   </gazebo>
-  <gazebo reference="us_1_link">
-  <!-- Visuals / Collisions omitted for this example -->
-  <sensor type="ray" name="range">
-    <ray>
-         <scan>
-            <horizontal>
-               <samples>1</samples>
-               <resolution>1.0</resolution>
-               <min_angle>-0.01</min_angle>
-               <max_angle>0.01</max_angle>
-            </horizontal>
-            <vertical>
-               <samples>1</samples>
-               <resolution>1</resolution>
-               <min_angle>-0.01</min_angle>
-               <max_angle>0.01</max_angle>
-            </vertical>
-         </scan>
-         <range>
-            <min>0.01</min>
-            <max>3.75</max>
-            <resolution>0.02</resolution>
-         </range>
-      </ray>
-    <plugin name="libgazebo_ros_range" filename="libgazebo_ros_range.so">
-         <gaussianNoise>0.005</gaussianNoise>
-         <alwaysOn>true</alwaysOn>
-         <updateRate>50</updateRate>
-         <topicName>us_sensor</topicName>
-         <frameName>us_1_link</frameName>
-         <radiation>SONAR</radiation>
-         <fov>0.2967</fov>
-    </plugin>
-  </sensor>
-  </gazebo>
  <gazebo>
     <plugin name="mpo_700_controller" filename="libgazebo_ros_planar_move.so">

File: robots/mpo_700/xacros/ultrasonic.xacro (robot description, xacro)
@@ -1,4 +1,4 @@
 <?xml version="1.0"?>
-<robot xmlns:xacro="http://www.ros.org/wiki/xacro" name="mpo_700">
+<robot xmlns:xacro="http://www.ros.org/wiki/xacro" name="mp_400">
   <xacro:macro name="us_sensor" params="name parent *origin">
     <joint name="${name}_joint" type="fixed">

Commit message: mpo-500

File: robots/mpo_500/mpo_500.urdf.xacro (robot description, xacro)
@@ -8,5 +8,12 @@
   <xacro:include filename="$(find neo_simulation)/robots/mpo_500/xacros/omni_wheel.xacro" />
   <!-- SENSORS -->
-  <xacro:include filename="$(find neo_simulation)/robots/mpo_500/xacros/sick_laser.xacro" />
+  <!-- <xacro:include filename="$(find neo_simulation)/robots/mpo_500/xacros/sick_S300.xacro" /> -->
+  <!-- Microscan - Comment/Uncomment if required -->
+  <xacro:include filename="$(find neo_simulation)/robots/mpo_500/xacros/micro_scan.xacro" />
+  <!--<xacro:include filename="$(find neo_simulation)/robots/mpo_500/xacros/imu.xacro" />
+  <xacro:include filename="$(find neo_simulation)/robots/mpo_500/xacros/ultrasonic.xacro" /> -->
+  <xacro:include filename="$(find neo_simulation)/robots/mpo_500/xacros/mpo_500_gazebo.xacro" />
+  <xacro:include filename="$(find neo_simulation)/robots/mpo_500/xacros/mpo_500_caster.xacro" />
+  <xacro:include filename="$(find neo_simulation)/robots/mpo_500/xacros/mpo_500_wheel.xacro" />
   <!-- Base Macro-->
   <xacro:mpo_500_base name="base_link">
@@ -14,21 +21,21 @@
   <!-- Wheel Macro -->
   <xacro:omni_wheel_250 name="wheel_front_left" parent="base_link">
-  	<origin xyz="0.25 0.28 0.13" rpy="0 0 0" />
+    <origin xyz="0.25 0.28 0.13" rpy="0 0 0" />
   </xacro:omni_wheel_250>
   <xacro:omni_wheel_250 name="wheel_front_right" parent="base_link">
-  	<origin xyz="0.25 -0.28 0.13" rpy="0 0 3.14" />
+    <origin xyz="0.25 -0.28 0.13" rpy="0 0 3.14" />
   </xacro:omni_wheel_250>
   <xacro:omni_wheel_250 name="wheel_back_left" parent="base_link">
-  	<origin xyz="-0.25 0.28 0.13" rpy="0 0 0" />
+    <origin xyz="-0.25 0.28 0.13" rpy="0 0 0" />
   </xacro:omni_wheel_250>
   <xacro:omni_wheel_250 name="wheel_back_right" parent="base_link">
-  	<origin xyz="-0.25 -0.28 0.13" rpy="0 0 3.14" />
+    <origin xyz="-0.25 -0.28 0.13" rpy="0 0 3.14" />
   </xacro:omni_wheel_250>
   <!-- Sensors -->
   <xacro:sick_laser_v0 name="lidar_1" parent="base_link" ros_topic="lidar_1/scan">
-  	<origin xyz="0.442 0 0.372" rpy="0 0 0" />
+    <origin xyz="0.442 0 0.372" rpy="0 0 0" />
   </xacro:sick_laser_v0>
   <xacro:sick_laser_v0 name="lidar_2" parent="base_link" ros_topic="lidar_2/scan">
-  	<origin xyz="-0.442 0 0.372" rpy="0 0 3.14" />
+    <origin xyz="-0.442 0 0.372" rpy="0 0 3.14" />
   </xacro:sick_laser_v0>
 </robot>

Commit message: MPO-500 Kinematics integration2 : Adding virtual transmission elements for the virtual wheel controllers

File: robots/mpo_500/mpo_500.urdf.xacro (robot description, xacro)
@@ -119,3 +119,39 @@
     <origin xyz="0 0 0.38" rpy="0 0 0" />
   </xacro:camera> -->
+  <transmission name="mpo_500_omni_wheel_front_left">
+    <type>transmission_interface/SimpleTransmission</type>
+    <joint name="mpo_500_omni_wheel_front_left_joint">
+      <hardwareInterface>hardware_interface/VelocityJointInterface</hardwareInterface>
+    </joint>
+    <actuator name="mpo_500_omni_wheel_front_left_motor">
+      <mechanicalReduction>1</mechanicalReduction>
+    </actuator>
+  </transmission>
+  <transmission name="mpo_500_omni_wheel_front_right">
+    <type>transmission_interface/SimpleTransmission</type>
+    <joint name="mpo_500_omni_wheel_front_right_joint">
+      <hardwareInterface>hardware_interface/VelocityJointInterface</hardwareInterface>
+    </joint>
+    <actuator name="mpo_500_omni_wheel_front_right_motor">
+      <mechanicalReduction>30</mechanicalReduction>
+    </actuator>
+  </transmission>
+  <transmission name="mpo_500_omni_wheel_back_left">
+    <type>transmission_interface/SimpleTransmission</type>
+    <joint name="mpo_500_omni_wheel_back_left_joint">
+      <hardwareInterface>hardware_interface/VelocityJointInterface</hardwareInterface>
+    </joint>
+    <actuator name="mpo_500_omni_wheel_back_left_motor">
+      <mechanicalReduction>19</mechanicalReduction>
+    </actuator>
+  </transmission>
+  <transmission name="mpo_500_omni_wheel_back_right">
+    <type>transmission_interface/SimpleTransmission</type>
+    <joint name="mpo_500_omni_wheel_back_right_joint">
+      <hardwareInterface>hardware_interface/VelocityJointInterface</hardwareInterface>
+    </joint>
+    <actuator name="mpo_500_omni_wheel_back_right_motor">
+      <mechanicalReduction>30</mechanicalReduction>
+    </actuator>
+  </transmission>
 </robot>

Commit message: MPO-500 model updated - wheel simulation is better

File: robots/mpo_500/mpo_500.urdf.xacro (robot description, xacro)
@@ -17,18 +17,20 @@
   <-->
   <!-- <xacro:include filename="$(find neo_simulation)/robots/mpo_500/xacros/camera.xacro" />  -->
-  <!-- Base Macro-->
-  <xacro:mpo_500_base name="base_link">
+  <link name="base_link" />
+  <!-- Base link macro -->
+  <xacro:mpo_500_base name="base_footprint" parent="base_link">
+    <origin xyz="0 0 0" rpy="0 0 0" />
   </xacro:mpo_500_base>
   <!-- Wheel Macro -->
-  <xacro:omni_wheel_250 name="mpo_500_omni_wheel_front_left" parent="base_link">
+  <xacro:omni_wheel_250 name="mpo_500_omni_wheel_front_left" parent="base_footprint">
     <origin xyz="0.25 0.28 0.13" rpy="0 0 0" />
   </xacro:omni_wheel_250>
-  <xacro:omni_wheel_250 name="mpo_500_omni_wheel_front_right" parent="base_link">
+  <xacro:omni_wheel_250 name="mpo_500_omni_wheel_front_right" parent="base_footprint">
     <origin xyz="0.25 -0.28 0.13" rpy="0 0 3.14" />
   </xacro:omni_wheel_250>
-  <xacro:omni_wheel_250 name="mpo_500_omni_wheel_back_left" parent="base_link">
+  <xacro:omni_wheel_250 name="mpo_500_omni_wheel_back_left" parent="base_footprint">
     <origin xyz="-0.25 0.28 0.13" rpy="0 0 0" />
   </xacro:omni_wheel_250>
-  <xacro:omni_wheel_250 name="mpo_500_omni_wheel_back_right" parent="base_link">
+  <xacro:omni_wheel_250 name="mpo_500_omni_wheel_back_right" parent="base_footprint">
     <origin xyz="-0.25 -0.28 0.13" rpy="0 0 3.14" />
   </xacro:omni_wheel_250>
@@ -134,5 +136,5 @@
     </joint>
     <actuator name="mpo_500_omni_wheel_front_right_motor">
-      <mechanicalReduction>30</mechanicalReduction>
+      <mechanicalReduction>1</mechanicalReduction>
     </actuator>
   </transmission>
@@ -143,5 +145,5 @@
     </joint>
     <actuator name="mpo_500_omni_wheel_back_left_motor">
-      <mechanicalReduction>19</mechanicalReduction>
+      <mechanicalReduction>1</mechanicalReduction>
     </actuator>
   </transmission>
@@ -152,5 +154,5 @@
     </joint>
     <actuator name="mpo_500_omni_wheel_back_right_motor">
-      <mechanicalReduction>30</mechanicalReduction>
+      <mechanicalReduction>1</mechanicalReduction>
     </actuator>
   </transmission>

File: robots/mpo_500/xacros/mpo_500_body.xacro (robot description, xacro)
@@ -1,12 +1,20 @@
 <?xml version="1.0"?>
 <robot xmlns:xacro="http://www.ros.org/wiki/xacro" name="mpo_500">
-  <xacro:macro name="mpo_500_base" params="name">
+  <xacro:macro name="mpo_500_base" params="name parent *origin">
+    <joint name="${name}_joint" type="fixed">
+      <xacro:insert_block name="origin" />
+      <axis xyz="0 0 -1" />
+      <!-- <limit effort="1000.0" lower="-1e+16" upper="1e+16" velocity="3.5"/> -->
+      <joint_properties damping="1" friction="1" />
+      <parent link="${parent}" />
+      <child link="${name}" />
+   </joint>
     <link name="${name}">
       <inertial>
-        <mass value="0.02" />
-        <origin xyz="0 0 0" rpy="0 0 0"/>
-        <inertia ixx="1.71402" ixy="0.0" ixz="0.0"
-                 iyy="0.8856" iyz="0.0"
-                 izz="2.5725" />
+        <mass value="64"/>
+        <origin xyz="0 0.0 0.0" />
+         <inertia ixx="2.8" ixy="0.0" ixz="0.0"
+                 iyy="2.8" iyz="0.0"
+                 izz="2.8" />
       </inertial>
       <visual>

File: robots/mpo_500/xacros/mpo_500_gazebo.xacro (robot description, xacro)
@@ -164,10 +164,16 @@
       </sensor>
   </gazebo>
-  <gazebo>
+<gazebo>
+  <plugin name="ros_control" filename="libgazebo_ros_control.so">
+    <legacyModeNS>false</legacyModeNS>
+    <robotSimType>gazebo_ros_control/DefaultRobotHWSim</robotSimType>
+  </plugin>
+</gazebo>
+<gazebo>
     <plugin name="mpo_500_controller" filename="libgazebo_ros_planar_move.so">
       <commandTopic>cmd_vel</commandTopic>
       <odometryTopic>odom</odometryTopic>
       <odometryFrame>odom</odometryFrame>
-      <odometryRate>20.0</odometryRate>
+      <odometryRate>100.0</odometryRate>
       <robotBaseFrame>base_link</robotBaseFrame>
     </plugin>

File: robots/mpo_500/xacros/omni_wheel.xacro (robot description, xacro)
@@ -6,5 +6,5 @@
     <axis xyz="0 1 0" />
     <joint_properties damping="100" friction="1000" />
-        <limit effort="1000.0" lower="-1e+16" upper="1e+16" velocity="3.5"/>
+        <limit effort="1000.0" lower="-1e+16" upper="1e+16" velocity="15"/>
     <joint_properties damping="1.0" friction="1" />
     <parent link="${parent}" />
@@ -13,7 +13,9 @@
    <link name="${name}_link" type="wheel">
     <inertial>
-      <mass value="1" />
+      <mass value="2.2" />
       <origin xyz="0 0 0" rpy="0 0 0" />
-      <inertia ixx="0.00044332" ixy="0" ixz="0" iyy="0.00044332" iyz="0" izz="0.00072" />
+        <inertia  ixx="0.01" ixy="0.0" ixz="0.0"
+                  iyy="0.01" iyz="0.0"
+                  izz="0.01" />
     </inertial>
     <visual>
@@ -24,10 +26,19 @@
     </visual>
     <collision>
-     <origin xyz="0 0 0" rpy="0 0 0" />
+     <origin xyz="0 0 0" rpy="0 1.57 1.57" />
      <geometry>
-       <sphere radius="0.127"/>
+        <!-- <mesh filename="package://neo_simulation/robots/mpo_500/meshes/MPO-500-WHEEL.dae" scale="0.001 0.001 0.001"/> -->
+       <!-- <cylinder radius="0.126" length="0.110"/> -->
+      <sphere radius="0.117" />
      </geometry>
     </collision>
    </link>
+<gazebo reference="${name}_link">
+      <!-- <kp> 10000 </kp> -->
+      <!-- <fdir1>0 1 0</fdir1> -->
+      <!-- <slip1> 0.1 </slip1> -->
+      <mu1>0.0001</mu1>
+      <mu2>0.0001</mu2>
+</gazebo>
   </xacro:macro>
 </robot>
