Commit message: MPO's support custom kinematics in the simulation

File: robots/mpo_500/mpo_500.urdf.xacro (robot description, xacro)
@@ -15,18 +15,20 @@
   <xacro:include filename="$(find neo_simulation)/robots/mpo_500/xacros/ultrasonic.xacro" /> -->
   <!-- <xacro:include filename="$(find neo_simulation)/robots/mpo_500/xacros/camera.xacro" />  -->
-  <!-- Base Macro-->
-  <xacro:mpo_500_base name="base_link">
+  <link name="base_link" />
+  <!-- Base link macro -->
+  <xacro:mpo_500_base name="base_footprint" parent="base_link">
+    <origin xyz="0 0 0" rpy="0 0 0" />
   </xacro:mpo_500_base>
   <!-- Wheel Macro -->
-  <xacro:omni_wheel_250 name="wheel_front_left" parent="base_link">
+  <xacro:omni_wheel_250 name="mpo_500_omni_wheel_front_left" parent="base_footprint">
     <origin xyz="0.25 0.28 0.13" rpy="0 0 0" />
   </xacro:omni_wheel_250>
-  <xacro:omni_wheel_250 name="wheel_front_right" parent="base_link">
+  <xacro:omni_wheel_250 name="mpo_500_omni_wheel_front_right" parent="base_footprint">
     <origin xyz="0.25 -0.28 0.13" rpy="0 0 3.14" />
   </xacro:omni_wheel_250>
-  <xacro:omni_wheel_250 name="wheel_back_left" parent="base_link">
+  <xacro:omni_wheel_250 name="mpo_500_omni_wheel_back_left" parent="base_footprint">
     <origin xyz="-0.25 0.28 0.13" rpy="0 0 0" />
   </xacro:omni_wheel_250>
-  <xacro:omni_wheel_250 name="wheel_back_right" parent="base_link">
+  <xacro:omni_wheel_250 name="mpo_500_omni_wheel_back_right" parent="base_footprint">
     <origin xyz="-0.25 -0.28 0.13" rpy="0 0 3.14" />
   </xacro:omni_wheel_250>
@@ -38,15 +40,19 @@
     <origin xyz="-0.442 0 0.372" rpy="0 0 3.14" />
   </xacro:sick_laser_v0>
-      <!--+++++++++++++++++++ IMU ++++++++++++++++++++++++-->
- <!-- Comment or uncomment based on your requirement -->
-<!--   <xacro:imu name="imu_1" parent="base_link">
+  <!--+++++++++++++++++++ IMU ++++++++++++++++++++++++-->
+  <!-- Comment or uncomment based on your requirement -->
+  <!-->
+  <xacro:imu name="imu" parent="base_link">
     <origin xyz="0.100 0 0.300" rpy="0 0 3.14" />
-  </xacro:imu> -->
+  </xacro:imu>
+  <-->
   <!--+++++++++++++++++++ Ultra Sonic ++++++++++++++++++++++++-->
   <!-- Comment or uncomment based on your requirement -->
   <!-- SENSOR 1 -->
-  <!-- xacro:us_sensor name="us_1" parent="base_link">
-    <origin xyz="0.100 0 0.300" rpy="0 3.14 3.14" />
-  </xacro:us_sensor-->
+  <!-->
+  <xacro:us_sensor name="us_1" parent="base_link">
+    <origin xyz="0.100 0 0.500" rpy="0 3.14 3.14" />
+  </xacro:us_sensor>
+  <-->
   <!-- SENSOR 2 -->
   <!-- xacro:us_sensor name="us_2" parent="base_link">
@@ -109,7 +115,43 @@
     <origin xyz="0.230 0 0.300" rpy="0 3.14 3.14" />
   </xacro:us_sensor-->
-      <!--Camera  -->
+  <!--Camera  -->
 <!-- <xacro:camera name="camera" parent="base_link">
     <origin xyz="0 0 0.38" rpy="0 0 0" />
   </xacro:camera> -->
+  <transmission name="mpo_500_omni_wheel_front_left">
+    <type>transmission_interface/SimpleTransmission</type>
+    <joint name="mpo_500_omni_wheel_front_left_joint">
+      <hardwareInterface>hardware_interface/VelocityJointInterface</hardwareInterface>
+    </joint>
+    <actuator name="mpo_500_omni_wheel_front_left_motor">
+      <mechanicalReduction>1</mechanicalReduction>
+    </actuator>
+  </transmission>
+  <transmission name="mpo_500_omni_wheel_front_right">
+    <type>transmission_interface/SimpleTransmission</type>
+    <joint name="mpo_500_omni_wheel_front_right_joint">
+      <hardwareInterface>hardware_interface/VelocityJointInterface</hardwareInterface>
+    </joint>
+    <actuator name="mpo_500_omni_wheel_front_right_motor">
+      <mechanicalReduction>1</mechanicalReduction>
+    </actuator>
+  </transmission>
+  <transmission name="mpo_500_omni_wheel_back_left">
+    <type>transmission_interface/SimpleTransmission</type>
+    <joint name="mpo_500_omni_wheel_back_left_joint">
+      <hardwareInterface>hardware_interface/VelocityJointInterface</hardwareInterface>
+    </joint>
+    <actuator name="mpo_500_omni_wheel_back_left_motor">
+      <mechanicalReduction>1</mechanicalReduction>
+    </actuator>
+  </transmission>
+  <transmission name="mpo_500_omni_wheel_back_right">
+    <type>transmission_interface/SimpleTransmission</type>
+    <joint name="mpo_500_omni_wheel_back_right_joint">
+      <hardwareInterface>hardware_interface/VelocityJointInterface</hardwareInterface>
+    </joint>
+    <actuator name="mpo_500_omni_wheel_back_right_motor">
+      <mechanicalReduction>1</mechanicalReduction>
+    </actuator>
+  </transmission>
 </robot>

File: robots/mpo_500/xacros/mpo_500_gazebo.xacro (robot description, xacro)
@@ -1,24 +1,5 @@
 <?xml version="1.0"?>
 <robot name="mpo_500" xmlns:xacro="http://www.ros.org/wiki/xacro">
-   <gazebo reference="base_link">
-    <gravity>true</gravity>
-    <self_collide>false</self_collide>
-  </gazebo>
-   <gazebo reference="wheel_front_left_link">
-    <gravity>true</gravity>
-    <self_collide>false</self_collide>
-  </gazebo>
-  <gazebo reference="wheel_front_right_link">
-    <gravity>true</gravity>
-    <self_collide>false</self_collide>
-  </gazebo>
-  <gazebo reference="wheel_back_left_link">
-    <gravity>true</gravity>
-    <self_collide>false</self_collide>
-  </gazebo>
-  <gazebo reference="wheel_back_right_link">
-    <gravity>true</gravity>
-    <self_collide>false</self_collide>
-  </gazebo>
+  <!-- Lidar sensors -->
   <gazebo reference="lidar_1_link">
       <sensor type="ray" name="lidar_1_sensor">
@@ -91,5 +72,6 @@
         </sensor>
   </gazebo>
- <gazebo reference="camera_link">
+  <!-- Camera -->
+  <gazebo reference="camera_link">
     <sensor type="camera" name="camera1">
       <update_rate>30.0</update_rate>
@@ -126,6 +108,7 @@
       </plugin>
     </sensor>
-  </gazebo>
-      <gazebo reference="imu_1_link">
+   </gazebo>
+  <!-- IMU sensor -->
+  <gazebo reference="imu_link">
     <gravity>true</gravity>
     <sensor name="imu_sensor" type="imu">
@@ -146,4 +129,5 @@
     </sensor>
   </gazebo>
+  <!-- Ultrasonic sensors -->
   <gazebo reference="us_1_link">
   <sensor type="ray" name="range">
@@ -169,12 +153,27 @@
          </range>
       </ray>
+      <plugin filename="libgazebo_ros_range.so" name="gazebo_ros_range">
+	<gaussianNoise>0.005</gaussianNoise>
+	<alwaysOn>true</alwaysOn>
+	<updateRate>50</updateRate>
+	<topicName>ultrasonic/us1</topicName>
+	<frameName>us_1_link</frameName>
+	<radiation>INFRARED</radiation>
+	<fov>0.2967</fov>
+      </plugin>
       </sensor>
   </gazebo>
-  <gazebo>
+<gazebo>
+  <plugin name="ros_control" filename="libgazebo_ros_control.so">
+    <legacyModeNS>false</legacyModeNS>
+    <robotSimType>gazebo_ros_control/DefaultRobotHWSim</robotSimType>
+  </plugin>
+</gazebo>
+<gazebo>
     <plugin name="mpo_500_controller" filename="libgazebo_ros_planar_move.so">
       <commandTopic>cmd_vel</commandTopic>
       <odometryTopic>odom</odometryTopic>
       <odometryFrame>odom</odometryFrame>
-      <odometryRate>20.0</odometryRate>
+      <odometryRate>100.0</odometryRate>
       <robotBaseFrame>base_link</robotBaseFrame>
     </plugin>

File: robots/mpo_500/xacros/omni_wheel.xacro (robot description, xacro)
@@ -3,8 +3,8 @@
   <xacro:macro name="omni_wheel_250" params="name parent *origin">
    <joint name="${name}_joint" type="revolute">
-    <insert_block name="origin" />
+    <xacro:insert_block name="origin" />
     <axis xyz="0 1 0" />
     <joint_properties damping="100" friction="1000" />
-        <limit effort="1000.0" lower="-1e+16" upper="1e+16" velocity="3.5"/>
+        <limit effort="1000.0" lower="-1e+16" upper="1e+16" velocity="15"/>
     <joint_properties damping="1.0" friction="1" />
     <parent link="${parent}" />
@@ -13,7 +13,9 @@
    <link name="${name}_link" type="wheel">
     <inertial>
-      <mass value="1" />
+      <mass value="2.2" />
       <origin xyz="0 0 0" rpy="0 0 0" />
-      <inertia ixx="0.00044332" ixy="0" ixz="0" iyy="0.00044332" iyz="0" izz="0.00072" />
+        <inertia  ixx="0.01" ixy="0.0" ixz="0.0"
+                  iyy="0.01" iyz="0.0"
+                  izz="0.01" />
     </inertial>
     <visual>
@@ -24,10 +26,19 @@
     </visual>
     <collision>
-     <origin xyz="0 0 0" rpy="0 0 0" />
+     <origin xyz="0 0 0" rpy="0 1.57 1.57" />
      <geometry>
-        <mesh filename="package://neo_simulation/robots/mpo_500/meshes/MPO-500-WHEEL.dae" scale="0.001 0.001 0.001"/>
+        <!-- <mesh filename="package://neo_simulation/robots/mpo_500/meshes/MPO-500-WHEEL.dae" scale="0.001 0.001 0.001"/> -->
+       <!-- <cylinder radius="0.126" length="0.110"/> -->
+      <sphere radius="0.117" />
      </geometry>
     </collision>
    </link>
+<gazebo reference="${name}_link">
+      <!-- <kp> 10000 </kp> -->
+      <!-- <fdir1>0 1 0</fdir1> -->
+      <!-- <slip1> 0.1 </slip1> -->
+      <mu1>0.0001</mu1>
+      <mu2>0.0001</mu2>
+</gazebo>
   </xacro:macro>
 </robot>

File: robots/mpo_700/mpo_700.urdf.xacro (robot description, xacro)
@@ -16,39 +16,45 @@
   <!--Caster  -->
   <xacro:include filename="$(find neo_simulation)/robots/mpo_700/xacros/mpo_700_caster.xacro" />
+    <xacro:include filename="$(find neo_simulation)/robots/mpo_700/xacros/mpo_700_caster_left.xacro" />
+  <xacro:include filename="$(find neo_simulation)/robots/mpo_700/xacros/mpo_700_caster_right.xacro" />
   <!-- Wheels -->
   <xacro:include filename="$(find neo_simulation)/robots/mpo_700/xacros/mpo_700_wheel.xacro" />
   <!-- Base Macro-->
-  <xacro:mpo_700_base name="base_link">
+<link name="base_link" />
+  <!-- Base Macro-->
+  <xacro:mpo_700_base name="base_footprint" parent="base_link">
+    <origin xyz="0 0 0" rpy="0 0 0" />
   </xacro:mpo_700_base>
-<xacro:mpo_700_caster_0 name="mpo_700_caster_front_left" parent="base_link">
-    <origin xyz="0.24 0.18 0.27" rpy="3.14 0 -1.57" />
-  </xacro:mpo_700_caster_0>
-<xacro:mpo_700_caster_1 name="mpo_700_caster_front_right" parent="base_link">
-    <origin xyz="0.24 -0.18 0.27" rpy="3.14 0 1.57" />
-  </xacro:mpo_700_caster_1>
-<xacro:mpo_700_caster_2 name="mpo_700_caster_back_left" parent="base_link">
-    <origin xyz="-0.24 0.18 0.27" rpy="3.14 0 -1.57" />
-  </xacro:mpo_700_caster_2>
-<xacro:mpo_700_caster_3 name="mpo_700_caster_back_right" parent="base_link">
-    <origin xyz="-0.24 -0.18 0.27" rpy="3.14 0 1.57" />
-  </xacro:mpo_700_caster_3>
-<xacro:mpo_700_wheel name="mpo_700_wheel_front_left" parent="mpo_700_caster_front_left_link">
-    <origin xyz="-0.05 0. 0.18" rpy="0 0 0" />
-  </xacro:mpo_700_wheel>
-<xacro:mpo_700_wheel name="mpo_700_wheel_front_right" parent="mpo_700_caster_front_right_link">
-    <origin xyz="-0.05 0. 0.18" rpy="0 0 0" />
-  </xacro:mpo_700_wheel>
-<xacro:mpo_700_wheel name="mpo_700_wheel_back_left" parent="mpo_700_caster_back_left_link">
-    <origin xyz="-0.05 0. 0.18" rpy="0 0 0" />
-  </xacro:mpo_700_wheel>
-<xacro:mpo_700_wheel name="mpo_700_wheel_back_right" parent="mpo_700_caster_back_right_link">
-    <origin xyz="-0.05 0. 0.18" rpy="0 0 0" />
+ <xacro:mpo_700_caster_left name="mpo_700_caster_front_left" parent="base_footprint">
+    <origin xyz="0.24 0.18 0.22" rpy="0 0 3.14" />
+  </xacro:mpo_700_caster_left>
+  <xacro:mpo_700_caster_right name="mpo_700_caster_front_right" parent="base_footprint">
+    <origin xyz="0.24 -0.18 0.22" rpy="0 0 0" />
+  </xacro:mpo_700_caster_right>
+  <xacro:mpo_700_caster_left name="mpo_700_caster_back_left" parent="base_footprint">
+    <origin xyz="-0.24 0.18 0.22" rpy="0 0 3.14" />
+  </xacro:mpo_700_caster_left>
+  <xacro:mpo_700_caster_right name="mpo_700_caster_back_right" parent="base_footprint">
+    <origin xyz="-0.24 -0.18 0.22" rpy="0 0 0" />
+  </xacro:mpo_700_caster_right>
+  <!--Wheel Macro  -->
+  <xacro:mpo_700_wheel name="mpo_700_wheel_front_left" parent="mpo_700_caster_front_left_link">
+    <origin xyz="0.0 0.045 -0.12" rpy="0 0 0" />
+  </xacro:mpo_700_wheel>
+  <xacro:mpo_700_wheel name="mpo_700_wheel_front_right" parent="mpo_700_caster_front_right_link">
+    <origin xyz="0.0 -0.045 -0.12" rpy="0 0 3.14" />
+  </xacro:mpo_700_wheel>
+  <xacro:mpo_700_wheel name="mpo_700_wheel_back_left" parent="mpo_700_caster_back_left_link">
+      <origin xyz="0.0 0.045 -0.12" rpy="0 0 0" />
+  </xacro:mpo_700_wheel>
+  <xacro:mpo_700_wheel name="mpo_700_wheel_back_right" parent="mpo_700_caster_back_right_link">
+    <origin xyz="0.0 -0.045 -0.12" rpy="0 0 3.14" />
   </xacro:mpo_700_wheel>
 <!-- Sensors -->
-  <xacro:sick_laser_v0 name="lidar_1" parent="base_link" ros_topic="lidar_1/scan_filtered">
+  <xacro:sick_laser_v0 name="lidar_1" parent="base_footprint" ros_topic="lidar_1/scan_filtered">
   <!--<origin xyz="0.360 0 0.181" rpy="3.14 0 0" />-->
     <origin xyz="0.338 0.288 0.223" rpy="3.14 0 0.79" /> <!-- Scanners on the side -->
   </xacro:sick_laser_v0>
-  <xacro:sick_laser_v0 name="lidar_2" parent="base_link" ros_topic="lidar_2/scan_filtered">
+  <xacro:sick_laser_v0 name="lidar_2" parent="base_footprint" ros_topic="lidar_2/scan_filtered">
   <!--<origin xyz="-0.360 0 0.181" rpy="3.14 0 3.14" />-->
     <origin xyz="-0.338 -0.288 0.223" rpy="3.14 0 3.93" /> <!-- Scanners on the side -->
@@ -129,3 +135,75 @@
     <origin xyz="0 0 0.38" rpy="0 0 0" />
   </xacro:camera> -->
+   <transmission name="mpo_700_caster_front_left">
+    <type>transmission_interface/SimpleTransmission</type>
+    <joint name="mpo_700_caster_front_left_joint">
+      <hardwareInterface>hardware_interface/PositionJointInterface</hardwareInterface>
+    </joint>
+    <actuator name="mpo_700_caster_front_left_motor">
+      <mechanicalReduction>1</mechanicalReduction>
+    </actuator>
+  </transmission>
+  <transmission name="mpo_700_wheel_front_left">
+    <type>transmission_interface/SimpleTransmission</type>
+    <joint name="mpo_700_wheel_front_left_joint">
+      <hardwareInterface>hardware_interface/VelocityJointInterface</hardwareInterface>
+    </joint>
+    <actuator name="mpo_700_wheel_front_left_motor">
+      <mechanicalReduction>1</mechanicalReduction>
+    </actuator>
+  </transmission>
+  <transmission name="mpo_700_caster_back_left">
+    <type>transmission_interface/SimpleTransmission</type>
+    <joint name="mpo_700_caster_back_left_joint">
+      <hardwareInterface>hardware_interface/PositionJointInterface</hardwareInterface>
+    </joint>
+    <actuator name="mpo_700_caster_back_left_motor">
+      <mechanicalReduction>1</mechanicalReduction>
+    </actuator>
+  </transmission>
+  <transmission name="mpo_700_wheel_back_right">
+    <type>transmission_interface/SimpleTransmission</type>
+    <joint name="mpo_700_wheel_back_right_joint">
+      <hardwareInterface>hardware_interface/VelocityJointInterface</hardwareInterface>
+    </joint>
+    <actuator name="mpo_700_wheel_back_right_motor">
+      <mechanicalReduction>1</mechanicalReduction>
+    </actuator>
+  </transmission>
+  <transmission name="mpo_700_caster_back_right">
+    <type>transmission_interface/SimpleTransmission</type>
+    <joint name="mpo_700_caster_back_right_joint">
+      <hardwareInterface>hardware_interface/PositionJointInterface</hardwareInterface>
+    </joint>
+    <actuator name="mpo_700_caster_back_right_motor">
+      <mechanicalReduction>1</mechanicalReduction>
+    </actuator>
+  </transmission>
+  <transmission name="mpo_700_wheel_front_right">
+    <type>transmission_interface/SimpleTransmission</type>
+    <joint name="mpo_700_wheel_front_right_joint">
+      <hardwareInterface>hardware_interface/VelocityJointInterface</hardwareInterface>
+    </joint>
+    <actuator name="mpo_700_wheel_front_right_motor">
+      <mechanicalReduction>1</mechanicalReduction>
+    </actuator>
+  </transmission>
+  <transmission name="mpo_700_caster_front_right">
+    <type>transmission_interface/SimpleTransmission</type>
+    <joint name="mpo_700_caster_front_right_joint">
+      <hardwareInterface>hardware_interface/PositionJointInterface</hardwareInterface>
+    </joint>
+    <actuator name="mpo_700_caster_front_right_motor">
+      <mechanicalReduction>1</mechanicalReduction>
+    </actuator>
+  </transmission>
+  <transmission name="mpo_700_wheel_back_left">
+    <type>transmission_interface/SimpleTransmission</type>
+    <joint name="mpo_700_wheel_back_left_joint">
+      <hardwareInterface>hardware_interface/VelocityJointInterface</hardwareInterface>
+    </joint>
+    <actuator name="mpo_700_wheel_front_left_motor">
+      <mechanicalReduction>1</mechanicalReduction>
+    </actuator>
+  </transmission>
 </robot>

File: robots/mpo_700/xacros/camera.xacro (robot description, xacro)
@@ -1,31 +1,17 @@
 <?xml version="1.0"?>
-<robot xmlns:xacro="http://www.ros.org/wiki/xacro" name="mm_400">
+<robot xmlns:xacro="http://www.ros.org/wiki/xacro" name="mpo_700">
   <xacro:macro name="camera" params="name parent *origin">
-    <xacro:property name="camera_link" value="0.05" />
     <joint name="${name}_joint" type="fixed">
       <axis xyz="0 1 0" />
-      <insert_block name="origin" />
+      <xacro:insert_block name="origin" />
       <parent link="${parent}"/>
       <child link="${name}_link"/>
     </joint>
     <link name="${name}_link">
-    <collision>
-      <origin xyz="0 0 0" rpy="0 0 0"/>
-      <geometry>
-    <box size="${camera_link} ${camera_link} ${camera_link}"/>
-      </geometry>
-    </collision>
-    <visual>
-      <origin xyz="0 0 0" rpy="0 0 0"/>
-      <geometry>
-    <box size="${camera_link} ${camera_link} ${camera_link}"/>
-      </geometry>
-      <material name="red"/>
-    </visual>
-    <inertial>
-      <mass value="1e-5" />
-      <origin xyz="0 0 0" rpy="0 0 0"/>
-      <inertia ixx="1e-6" ixy="0" ixz="0" iyy="1e-6" iyz="0" izz="1e-6" />
-    </inertial>
+      <inertial>
+        <mass value="0.001" />
+        <origin xyz="0 0 0" rpy="0 0 0" />
+        <inertia ixx="0.0001" ixy="0" ixz="0" iyy="0.000001" iyz="0" izz="0.0001" />
+      </inertial>
     </link>
   </xacro:macro>

File: robots/mpo_700/xacros/mpo_700_body.xacro (robot description, xacro)
@@ -1,13 +1,21 @@
 <?xml version="1.0"?>
 <robot xmlns:xacro="http://www.ros.org/wiki/xacro" name="mpo_700">
-  <xacro:macro name="mpo_700_base" params="name">
+  <xacro:macro name="mpo_700_base" params="name parent *origin">
+   <joint name="${name}_joint" type="fixed">
+    <insert_block name="origin" />
+    <axis xyz="0 0 -1" />
+    <!-- <limit effort="1000.0" lower="-1e+16" upper="1e+16" velocity="3.5"/> -->
+    <joint_properties damping="1" friction="1" />
+    <parent link="${parent}" />
+    <child link="${name}" />
+   </joint>
     <link name="${name}">
-      <inertial>
-        <mass value="0.01" />
-        <origin xyz="0 0 0" rpy="0 0 0"/>
-        <inertia ixx="0.0008" ixy="0.0" ixz="0.0"
-                 iyy="0.0008" iyz="0.0"
-                 izz="0.0008" />
-      </inertial>
+    <inertial>
+      <mass value="90"/>
+      <origin xyz="0 0 0"/>
+      <inertia ixx="7.8" ixy="0.0" ixz="0"
+               iyy="7.8" iyz="0.0"
+               izz="7.8"/>
+    </inertial>
       <visual>
         <origin xyz="0.0 0.0 0.0" rpy="0 0 -1.571" />

File: robots/mpo_700/xacros/mpo_700_caster.xacro (robot description, xacro)
@@ -19,5 +19,5 @@
      <origin xyz="0 0 0.10" rpy="0 0 0"/>
      <geometry>
-        <mesh filename="package://neo_simulation/robots/mpo_700/meshes/MPO-700-HEAD.dae" scale="0.001 0.001 0.001"/>
+        <mesh filename="package://neo_simulation/robots/mpo_700/meshes/MPO-700-caster.dae" scale="0.001 0.001 0.001"/>
      </geometry>
     </visual>
@@ -25,5 +25,5 @@
      <origin xyz="0 0 0.10" rpy="0 0 0" />
      <geometry>
-        <mesh filename="package://neo_simulation/robots/mpo_700/meshes/MPO-700-HEAD.dae" scale="0.001 0.001 0.001"/>
+        <mesh filename="package://neo_simulation/robots/mpo_700/meshes/MPO-700-caster.dae" scale="0.001 0.001 0.001"/>
      </geometry>
     </collision>
@@ -47,5 +47,5 @@
      <origin xyz="0 0 0.10" rpy="0 0 0"/>
      <geometry>
-        <mesh filename="package://neo_simulation/robots/mpo_700/meshes/MPO-700-HEAD.dae" scale="0.001 0.001 0.001"/>
+        <mesh filename="package://neo_simulation/robots/mpo_700/meshes/MPO-700-caster.dae" scale="0.001 0.001 0.001"/>
      </geometry>
     </visual>
@@ -53,5 +53,5 @@
      <origin xyz="0 0 0.10" rpy="0 0 0" />
      <geometry>
-        <mesh filename="package://neo_simulation/robots/mpo_700/meshes/MPO-700-HEAD.dae" scale="0.001 0.001 0.001"/>
+        <mesh filename="package://neo_simulation/robots/mpo_700/meshes/MPO-700-caster.dae" scale="0.001 0.001 0.001"/>
      </geometry>
     </collision>
@@ -75,5 +75,5 @@
      <origin xyz="0 0 0.10" rpy="0 0 0"/>
      <geometry>
-        <mesh filename="package://neo_simulation/robots/mpo_700/meshes/MPO-700-HEAD.dae" scale="0.001 0.001 0.001"/>
+        <mesh filename="package://neo_simulation/robots/mpo_700/meshes/MPO-700-caster.dae" scale="0.001 0.001 0.001"/>
      </geometry>
     </visual>
@@ -81,5 +81,5 @@
      <origin xyz="0 0 0.10" rpy="0 0 0" />
      <geometry>
-        <mesh filename="package://neo_simulation/robots/mpo_700/meshes/MPO-700-HEAD.dae" scale="0.001 0.001 0.001"/>
+        <mesh filename="package://neo_simulation/robots/mpo_700/meshes/MPO-700-caster.dae" scale="0.001 0.001 0.001"/>
      </geometry>
     </collision>
@@ -103,5 +103,5 @@
      <origin xyz="0 0 0.10" rpy="0 0 0"/>
      <geometry>
-        <mesh filename="package://neo_simulation/robots/mpo_700/meshes/MPO-700-HEAD.dae" scale="0.001 0.001 0.001"/>
+        <mesh filename="package://neo_simulation/robots/mpo_700/meshes/MPO-700-caster.dae" scale="0.001 0.001 0.001"/>
      </geometry>
     </visual>
@@ -109,5 +109,5 @@
      <origin xyz="0 0 0.10" rpy="0 0 0" />
      <geometry>
-        <mesh filename="package://neo_simulation/robots/mpo_700/meshes/MPO-700-HEAD.dae" scale="0.001 0.001 0.001"/>
+        <mesh filename="package://neo_simulation/robots/mpo_700/meshes/MPO-700-caster.dae" scale="0.001 0.001 0.001"/>
      </geometry>
     </collision>
