Commit message: MPO's support custom kinematics in the simulation

File: robots/mpo_700/xacros/mpo_700_gazebo.xacro (robot description, xacro)
@@ -5,4 +5,10 @@
     <self_collide>false</self_collide>
   </gazebo>
+<gazebo>
+  <plugin name="ros_control" filename="libgazebo_ros_control.so">
+    <legacyModeNS>false</legacyModeNS>
+    <robotSimType>gazebo_ros_control/DefaultRobotHWSim</robotSimType>
+  </plugin>
+</gazebo>
   <gazebo reference="lidar_1_link">
       <sensor type="ray" name="lidar_1_sensor">
@@ -31,5 +37,5 @@
                    reading. -->
               <mean>0.0</mean>
-              <stddev>0.01</stddev>
+              <stddev>0.0</stddev>
             </noise>
           </ray>
@@ -66,5 +72,5 @@
                    reading. -->
               <mean>0.0</mean>
-              <stddev>0.01</stddev>
+              <stddev>0.0</stddev>
             </noise>
           </ray>
@@ -75,5 +81,5 @@
         </sensor>
   </gazebo>
-    <gazebo reference="imu_link">
+  <gazebo reference="imu_link">
     <gravity>true</gravity>
     <sensor name="imu_sensor" type="imu">
@@ -94,5 +100,4 @@
     </sensor>
   </gazebo>
-    <!-- camera -->
  <gazebo>
     <plugin name="mpo_700_controller" filename="libgazebo_ros_planar_move.so">
@@ -100,8 +105,9 @@
       <odometryTopic>odom</odometryTopic>
       <odometryFrame>odom</odometryFrame>
-      <odometryRate>20.0</odometryRate>
+      <odometryRate>100.0</odometryRate>
       <robotBaseFrame>base_link</robotBaseFrame>
     </plugin>
   </gazebo>
+  <!-- camera -->
   <gazebo reference="camera_link">
     <sensor type="camera" name="camera1">
@@ -109,9 +115,9 @@
       <camera name="head">
         <horizontal_fov>1.3962634</horizontal_fov>
-        <image>
-          <width>800</width>
-          <height>800</height>
-          <format>R8G8B8</format>
-        </image>
+	<image>
+	  <width>800</width>
+ 	  <height>800</height>
+	  <format>R8G8B8</format>
+	</image>
         <clip>
           <near>0.02</near>
@@ -130,5 +136,5 @@
         <alwaysOn>true</alwaysOn>
         <updateRate>0.0</updateRate>
-        <cameraName>camera1</cameraName>
+        <cameraName>robot/camera1</cameraName>
         <imageTopicName>image_raw</imageTopicName>
         <cameraInfoTopicName>camera_info</cameraInfoTopicName>
@@ -143,5 +149,6 @@
     </sensor>
   </gazebo>
-    <gazebo reference="us_1_link">
+  <!-- Sonar -->
+  <gazebo reference="us_1_link">
   <!-- Visuals / Collisions omitted for this example -->
   <sensor type="ray" name="range">
@@ -167,4 +174,13 @@
          </range>
       </ray>
+      <plugin filename="libgazebo_ros_range.so" name="gazebo_ros_range">
+	<gaussianNoise>0.005</gaussianNoise>
+	<alwaysOn>true</alwaysOn>
+	<updateRate>50</updateRate>
+	<topicName>ultrasonic/us1</topicName>
+	<frameName>us_1_link</frameName>
+	<radiation>INFRARED</radiation>
+	<fov>0.2967</fov>
+      </plugin>
       </sensor>
   </gazebo>
