Commit message: Collisions for MP-400 updated

File: robots/mp_400/xacros/mp_400_caster_wheel.xacro (robot description, xacro)
@@ -26,5 +26,5 @@
       <origin xyz="0 0. 0" rpy="0 0 0" />
       <geometry>
-            <mesh filename="package://neo_simulation/robots/mp_400/meshes/MP-400-CASTER-WHEEL.dae" scale="0.001 0.001 0.001"/>
+          <sphere radius="0.038"/>
       </geometry>
     </collision>

File: robots/mp_400/xacros/mp_400_fixed_wheel_left.xacro (robot description, xacro)
@@ -26,5 +26,5 @@
      <origin xyz="0. 0 0" rpy=" 0 0 0" />
       <geometry>
-            <mesh filename="package://neo_simulation/robots/mp_400/meshes/MP-400-FIXED-WHEEL-LEFT.dae" scale="0.001 0.001 0.001"/>
+         <sphere radius="0.0765"/>
       </geometry>
     </collision>

File: robots/mp_400/xacros/mp_400_fixed_wheel_right.xacro (robot description, xacro)
@@ -26,5 +26,5 @@
      <origin xyz="0. 0 0" rpy=" 0 0 0" />
       <geometry>
-            <mesh filename="package://neo_simulation/robots/mp_400/meshes/MP-400-FIXED-WHEEL-LEFT.dae" scale="0.001 0.001 0.001"/>
+        <sphere radius="0.0765"/>
       </geometry>
     </collision>

File: robots/mp_400/xacros/mp_400_gazebo.xacro (robot description, xacro)
@@ -163,5 +163,5 @@
         <publishWheelJointState>true</publishWheelJointState>
         <wheelAcceleration>0.0</wheelAcceleration>
-        <wheelTorque>2</wheelTorque>
+        <wheelTorque>20</wheelTorque>
         <odometrySource>world</odometrySource>
         <publishTf>1</publishTf>

Commit message: MP-400 models accomodates the gazebo 7 update

File: robots/mp_400/xacros/mp_400_caster_wheel.xacro (robot description, xacro)
@@ -13,8 +13,8 @@
    <inertial>
         <mass value="1.4"/>
-        <inertia ixx="0.00499743171" ixy="0.00000004464" ixz="-0.00000002245"
-                 iyy="0.00499741733" iyz="-0.00000000164"
+        <inertia ixx="0.00499743171" ixy="0.0" ixz="-0.0"
+                 iyy="0.00499741733" iyz="-0.0"
                  izz="0.00839239692"/>
-</inertial>
+  </inertial>
       <visual name='caster_wheel'>
     <origin xyz="0 0 0" rpy="0 0 0" />
@@ -26,5 +26,5 @@
       <origin xyz="0 0. 0" rpy="0 0 0" />
       <geometry>
-            <mesh filename="package://neo_simulation/robots/mp_400/meshes/MP-400-CASTER-WHEEL.dae" scale="0.001 0.001 0.001"/>
+          <sphere radius="0.040"/>
       </geometry>
     </collision>

File: robots/mp_400/xacros/mp_400_fixed_wheel_left.xacro (robot description, xacro)
@@ -12,9 +12,9 @@
    <link name="${name}_link" type="wheel">
    <inertial>
-        <mass value="1.82362"/>
-        <inertia ixx="0.00399743171" ixy="0.00000004464" ixz="-0.00000002245"
-                 iyy="0.00399741733" iyz="-0.00000000164"
+        <mass value="1.8"/>
+        <inertia ixx="0.00399743171" ixy="0.0" ixz="-0.0"
+                 iyy="0.00399741733" iyz="-0.0"
                  izz="0.00739239692"/>
-</inertial>
+    </inertial>
       <visual name='fixed_wheel_left'>
     <origin xyz="0 0 0.0" rpy="0 0 0" />
@@ -26,15 +26,13 @@
      <origin xyz="0. 0 0" rpy=" 0 0 0" />
       <geometry>
-            <mesh filename="package://neo_simulation/robots/mp_400/meshes/MP-400-FIXED-WHEEL-LEFT.dae" scale="0.001 0.001 0.001"/>
+        <sphere radius="0.079"/>
       </geometry>
     </collision>
 </link>
 <gazebo reference="${name}_link">
-      <kp>600.0</kp>
-      <kd>1465.0</kd>
-      <mu1>200</mu1>
+      <kp>100000.0</kp>
+      <kd>50.0</kd>
+      <mu1>100</mu1>
       <mu2>100</mu2>
-      <fdir1>.5 0 0</fdir1>
-      <maxVel>3.0</maxVel>
       <minDepth>0.00</minDepth>
       <implicitSpringDamper>1</implicitSpringDamper>

File: robots/mp_400/xacros/mp_400_fixed_wheel_right.xacro (robot description, xacro)
@@ -11,10 +11,10 @@
    </joint>
    <link name="${name}_link" type="wheel">
-   <inertial>
-        <mass value="1.82362"/>
-        <inertia ixx="0.00399743171" ixy="0.00000004464" ixz="-0.00000002245"
-                 iyy="0.00399741733" iyz="-0.00000000164"
+  <inertial>
+        <mass value="1.8"/>
+        <inertia ixx="0.00399743171" ixy="0.0" ixz="-0.0"
+                 iyy="0.00399741733" iyz="-0.0"
                  izz="0.00739239692"/>
-</inertial>
+  </inertial>
       <visual name='fixed_wheel_right'>
     <origin xyz="0 0 0.0" rpy="0 0 3.14" />
@@ -23,18 +23,16 @@
         </geometry>
       </visual>
-    <collision>
+  <collision>
      <origin xyz="0. 0 0" rpy=" 0 0 0" />
       <geometry>
-            <mesh filename="package://neo_simulation/robots/mp_400/meshes/MP-400-FIXED-WHEEL-LEFT.dae" scale="0.001 0.001 0.001"/>
+        <sphere radius="0.079"/>
       </geometry>
-    </collision>
+  </collision>
 </link>
 <gazebo reference="${name}_link">
-      <kp>600.0</kp> <!-- Partial Ziegler-Nichols method -->
-      <kd>1465.0</kd>
-      <mu1>200</mu1>
+      <kp>100000.0</kp>
+      <kd>50.0</kd>
+      <mu1>100</mu1>
       <mu2>100</mu2>
-      <fdir1>.5 0 0</fdir1>
-      <maxVel>3.0</maxVel>
       <minDepth>0.00</minDepth>
       <implicitSpringDamper>1</implicitSpringDamper>

File: robots/mp_400/xacros/mp_400_gazebo.xacro (robot description, xacro)
@@ -160,5 +160,5 @@
         <publishWheelJointState>true</publishWheelJointState>
         <wheelAcceleration>6.0</wheelAcceleration>
-        <wheelTorque>5</wheelTorque>
+        <wheelTorque>10</wheelTorque>
         <odometrySource>world</odometrySource>
         <publishTf>1</publishTf>
