Commit message: MP-500 laserscanner problem is fixed

File: robots/mp_400/xacros/mp_400_gazebo.xacro (robot description, xacro)
@@ -146,5 +146,5 @@
      <odometryTopic>odom</odometryTopic>
      <odometryFrame>odom</odometryFrame>
-     <robotBaseFrame>base_footprint</robotBaseFrame>
+     <robotBaseFrame>base_link</robotBaseFrame>
      <publishWheelTF>true</publishWheelTF>
      <publishWheelJointState>true</publishWheelJointState>

File: robots/mp_500/mp_500.urdf.xacro (robot description, xacro)
@@ -39,5 +39,5 @@
    <!-- SENSORS -->
   <xacro:sick_laser_v0 name="lidar_1" parent="base_link" ros_topic="lidar_1/scan_filtered">
-    <origin xyz="0.244 0 0.141" rpy="3.14 0 0" />
+    <origin xyz="0.244 0 0.141" rpy="0 0 0" />
   </xacro:sick_laser_v0>
      <!--+++++++++++++++++++ IMU ++++++++++++++++++++++++-->

File: robots/mp_500/xacros/sick_S300.xacro (robot description, xacro)
@@ -15,5 +15,5 @@
       </inertial>
       <visual>
-        <origin xyz="0 0 -0.12" rpy="-1.57 0 3.14" />
+        <origin xyz="0 0 0.12" rpy="-1.57 -3.14 0" />
         <geometry>
         <mesh filename="package://neo_simulation/robots/mp_500/meshes/SICK-S300.dae" scale="0.001 0.001 0.001" />
@@ -21,5 +21,5 @@
       </visual>
       <collision>
-        <origin xyz="0 0 -0.12" rpy="-1.57 0 3.14" />
+        <origin xyz="0 0 0.12" rpy="-1.57 0 3.14" />
         <geometry>
         <mesh filename="package://neo_simulation/robots/mp_500/meshes/SICK-S300.dae" scale="0.001 0.001 0.001" />
