Commit message: Readme updated

File: robots/mm_400/urdf/xacros/mp_400_body.xacro (robot description, xacro)
@@ -4,5 +4,5 @@
     <link name="${name}">
   <inertial>
-        <mass value="125" />
+        <mass value="30" />
         <origin xyz="0 0 0" rpy="0 0 0"/>
         <inertia ixx="1.71402" ixy="0.0" ixz="0.0"
@@ -13,5 +13,5 @@
       <origin xyz="0.0 0.0 0." rpy="0 0 1.57" />
         <geometry>
-            <mesh filename="package://neo_simulation/robots/mm_400/meshes/MP-400-BODY.dae" scale="0.001 0.001 0.001"/>
+            <mesh filename="package://neo_simulation/robots/mp_400/meshes/MP-400-BODY.dae" scale="0.001 0.001 0.001"/>
         <!--cylinder length="0.381" radius="0.2545"/-->
         <!--box size="0.445 0.277 0.17"/-->
@@ -21,5 +21,5 @@
         <origin xyz="0.0 0.0 0.0" rpy="0 0 1.57" />
         <geometry>
-          <mesh filename="package://neo_simulation/robots/mm_400/meshes/MP-400-BODY.dae" scale="0.001 0.001 0.001"/>
+          <mesh filename="package://neo_simulation/robots/mp_400/meshes/MP-400-BODY.dae" scale="0.001 0.001 0.001"/>
           <!--cylinder length="0.381" radius="0.2545"/-->
         </geometry>

File: robots/mm_400/urdf/xacros/mp_400_caster_wheel.xacro (robot description, xacro)
@@ -1,4 +1,4 @@
 <?xml version="1.0"?>
-<robot xmlns:xacro="http://www.ros.org/wiki/xacro" name="mm_400">
+<robot xmlns:xacro="http://www.ros.org/wiki/xacro" name="mp_400">
   <xacro:macro name="caster_wheel" params="name parent *origin">
    <joint name="${name}_joint" type="fixed">
@@ -11,14 +11,14 @@
    </joint>
    <link name="${name}_link" type="wheel">
-    <inertial>
-        <mass value="1.82362"/>
-        <inertia ixx="0.0000499743171" ixy="0.0000000004464" ixz="-0.0000000002245"
-                 iyy="0.00499741733" iyz="0.0000000000164"
-izz="0.0000839239692"/>
-</inertial>
+   <inertial>
+        <mass value="1.4"/>
+        <inertia ixx="0.00499743171" ixy="0.0" ixz="-0.0"
+                 iyy="0.00499741733" iyz="-0.0"
+                 izz="0.00839239692"/>
+  </inertial>
       <visual name='caster_wheel'>
     <origin xyz="0 0 0" rpy="0 0 0" />
     <geometry>
-            <mesh filename="package://neo_simulation/robots/mm_400/meshes/MP-400-CASTER-WHEEL.dae" scale="0.001 0.001 0.001"/>
+            <mesh filename="package://neo_simulation/robots/mp_400/meshes/MP-400-CASTER-WHEEL.dae" scale="0.001 0.001 0.001"/>
     </geometry>
     </visual>
@@ -26,8 +26,18 @@
       <origin xyz="0 0. 0" rpy="0 0 0" />
       <geometry>
-            <mesh filename="package://neo_simulation/robots/mm_400/meshes/MP-400-CASTER-WHEEL.dae" scale="0.001 0.001 0.001"/>
+          <sphere radius="0.040"/>
       </geometry>
     </collision>
     </link>
+<gazebo reference="${name}_link">
+      <kp>10000.0</kp>
+      <kd>10.0</kd>
+      <mu1>0.5</mu1>
+      <mu2>0.2</mu2>
+      <fdir1>.5 0 0</fdir1>
+      <maxVel>3.0</maxVel>
+      <minDepth>0.00</minDepth>
+      <implicitSpringDamper>3</implicitSpringDamper>
+</gazebo>
   </xacro:macro>
 </robot>

File: robots/mm_400/urdf/xacros/mp_400_fixed_wheel_left.xacro (robot description, xacro)
@@ -1,4 +1,4 @@
 <?xml version="1.0"?>
-<robot xmlns:xacro="http://www.ros.org/wiki/xacro" name="mm_400">
+<robot xmlns:xacro="http://www.ros.org/wiki/xacro" name="mp_400">
   <xacro:macro name="fixed_wheel_left" params="name parent *origin">
    <joint name="${name}_joint" type="revolute">
@@ -11,15 +11,14 @@
    </joint>
    <link name="${name}_link" type="wheel">
-<inertial>
-      <origin xyz="0 0 0" rpy="0 0 0"/>
-        <mass value="1.82362"/>
-        <inertia ixx="0.0399743171" ixy="0.00000004464" ixz="-0.00000002245"
-                 iyy="0.0399741733" iyz="-0.00000000164"
-                 izz="0.0739239692"/>
-</inertial>
+   <inertial>
+        <mass value="1.8"/>
+        <inertia ixx="0.00399743171" ixy="0.0" ixz="-0.0"
+                 iyy="0.00399741733" iyz="-0.0"
+                 izz="0.00739239692"/>
+    </inertial>
       <visual name='fixed_wheel_left'>
     <origin xyz="0 0 0.0" rpy="0 0 0" />
         <geometry>
-            <mesh filename="package://neo_simulation/robots/mm_400/meshes/MP-400-FIXED-WHEEL-LEFT.dae" scale="0.001 0.001 0.001"/>
+            <mesh filename="package://neo_simulation/robots/mp_400/meshes/MP-400-FIXED-WHEEL-LEFT.dae" scale="0.001 0.001 0.001"/>
         </geometry>
       </visual>
@@ -27,13 +26,12 @@
      <origin xyz="0. 0 0" rpy=" 0 0 0" />
       <geometry>
-            <mesh filename="package://neo_simulation/robots/mm_400/meshes/MP-400-FIXED-WHEEL-LEFT.dae" scale="0.001 0.001 0.001"/>
+        <sphere radius="0.079"/>
       </geometry>
     </collision>
 </link>
 <gazebo reference="${name}_link">
-      <kp>100000.0</kp>
+      <kp>200000.0</kp>
       <kd>50.0</kd>
       <mu1>100</mu1>
-      <gravity> 1 </gravity>
       <mu2>100</mu2>
       <minDepth>0.00</minDepth>

File: robots/mm_400/urdf/xacros/mp_400_fixed_wheel_right.xacro (robot description, xacro)
@@ -1,4 +1,4 @@
 <?xml version="1.0"?>
-<robot xmlns:xacro="http://www.ros.org/wiki/xacro" name="mm_400">
+<robot xmlns:xacro="http://www.ros.org/wiki/xacro" name="mp_400">
   <xacro:macro name="fixed_wheel_right" params="name parent *origin">
    <joint name="${name}_joint" type="revolute">
@@ -11,28 +11,26 @@
    </joint>
    <link name="${name}_link" type="wheel">
-      <inertial>
-      <origin xyz="0 0 0" rpy="0 0 0"/>
-        <mass value="1.82362"/>
-        <inertia ixx="0.0399743171" ixy="0.00000004464" ixz="-0.00000002245"
-                 iyy="0.0399741733" iyz="-0.00000000164"
-                 izz="0.0739239692"/>
-</inertial>
+  <inertial>
+        <mass value="1.8"/>
+        <inertia ixx="0.00399743171" ixy="0.0" ixz="-0.0"
+                 iyy="0.00399741733" iyz="-0.0"
+                 izz="0.00739239692"/>
+  </inertial>
       <visual name='fixed_wheel_right'>
     <origin xyz="0 0 0.0" rpy="0 0 3.14" />
         <geometry>
-            <mesh filename="package://neo_simulation/robots/mm_400/meshes/MP-400-FIXED-WHEEL-RIGHT.dae" scale="0.001 0.001 0.001"/>
+            <mesh filename="package://neo_simulation/robots/mp_400/meshes/MP-400-FIXED-WHEEL-RIGHT.dae" scale="0.001 0.001 0.001"/>
         </geometry>
       </visual>
-    <collision>
+  <collision>
      <origin xyz="0. 0 0" rpy=" 0 0 0" />
       <geometry>
-            <mesh filename="package://neo_simulation/robots/mm_400/meshes/MP-400-FIXED-WHEEL-LEFT.dae" scale="0.001 0.001 0.001"/>
+        <sphere radius="0.079"/>
       </geometry>
-    </collision>
+  </collision>
 </link>
 <gazebo reference="${name}_link">
-      <kp>100000.0</kp>
+      <kp>200000.0</kp>
       <kd>50.0</kd>
-      <gravity> 1 </gravity>
       <mu1>100</mu1>
       <mu2>100</mu2>

File: robots/mm_400/urdf/xacros/mp_400_gazebo.xacro (robot description, xacro)
@@ -13,44 +13,4 @@
     <self_collide>false</self_collide>
   </gazebo>
-<gazebo reference="wheel_front_right_link">
-      <kp>35000.0</kp>
-      <kd>1000.0</kd>
-      <mu1>0.051</mu1>
-      <mu2>0.051</mu2>
-      <fdir1>1 0 0</fdir1>
-    <maxVel>1.0</maxVel>
-    <minDepth>0.00</minDepth>
-      <implicitSpringDamper>1</implicitSpringDamper>
-</gazebo>
-<gazebo reference="wheel_front_left_link">
-      <kp>35000.0</kp>
-      <kd>1000.0</kd>
-      <mu1>0.051</mu1>
-      <mu2>0.051</mu2>
-          <fdir1>1 0 0</fdir1>
-    <maxVel>1.0</maxVel>
-    <minDepth>0.00</minDepth>
-      <implicitSpringDamper>1</implicitSpringDamper>
-</gazebo>
-<gazebo reference="wheel_back_left_link">
-      <kp>35000.0</kp>
-      <kd>1000.0</kd>
-      <mu1>0.051</mu1>
-      <mu2>0.051</mu2>
-          <fdir1>1 0 0</fdir1>
-    <maxVel>1.0</maxVel>
-    <minDepth>0.00</minDepth>
-      <implicitSpringDamper>1</implicitSpringDamper>
-</gazebo>
-<gazebo reference="wheel_back_right_link">
-      <kp>35000.0</kp>
-      <kd>1000.0</kd>
-      <mu1>0.051</mu1>
-      <mu2>0.051</mu2>
-          <fdir1>1 0 0</fdir1>
-    <maxVel>1.0</maxVel>
-    <minDepth>0.00</minDepth>
-      <implicitSpringDamper>1</implicitSpringDamper>
-</gazebo>
   <gazebo reference="lidar_1_link">
       <sensor type="ray" name="lidar_1_link">
