Commit message: IMU and USS Tested and updated

File: robots/mm_400/urdf/xacros/mp_400_gazebo.xacro (robot description, xacro)
@@ -72,5 +72,5 @@
     </plugin>
   </gazebo>
-    <gazebo reference="imu_link">
+    <gazebo reference="imu_1_link">
     <gravity>true</gravity>
     <sensor name="imu_sensor" type="imu">
@@ -90,4 +90,39 @@
       <pose>0 0 0 0 0 0</pose>
     </sensor>
+  </gazebo>
+  <gazebo reference="us_1_link">
+  <!-- Visuals / Collisions omitted for this example -->
+  <sensor type="ray" name="range">
+    <ray>
+         <scan>
+            <horizontal>
+               <samples>1</samples>
+               <resolution>1.0</resolution>
+               <min_angle>-0.01</min_angle>
+               <max_angle>0.01</max_angle>
+            </horizontal>
+            <vertical>
+               <samples>1</samples>
+               <resolution>1</resolution>
+               <min_angle>-0.01</min_angle>
+               <max_angle>0.01</max_angle>
+            </vertical>
+         </scan>
+         <range>
+            <min>0.01</min>
+            <max>3.75</max>
+            <resolution>0.02</resolution>
+         </range>
+      </ray>
+    <plugin name="libgazebo_ros_range" filename="libgazebo_ros_range.so">
+         <gaussianNoise>0.005</gaussianNoise>
+         <alwaysOn>true</alwaysOn>
+         <updateRate>50</updateRate>
+         <topicName>us_sensor</topicName>
+         <frameName>us_1_link</frameName>
+         <radiation>SONAR</radiation>
+         <fov>0.2967</fov>
+    </plugin>
+  </sensor>
   </gazebo>
     <!-- camera -->

File: robots/mmo_500/urdf/xacros/mpo_500_gazebo.xacro (robot description, xacro)
@@ -91,5 +91,5 @@
         </sensor>
   </gazebo>
-      <gazebo reference="imu_link">
+    <gazebo reference="imu_1_link">
     <gravity>true</gravity>
     <sensor name="imu_sensor" type="imu">
@@ -109,4 +109,39 @@
       <pose>0 0 0 0 0 0</pose>
     </sensor>
+  </gazebo>
+  <gazebo reference="us_1_link">
+  <!-- Visuals / Collisions omitted for this example -->
+  <sensor type="ray" name="range">
+    <ray>
+         <scan>
+            <horizontal>
+               <samples>1</samples>
+               <resolution>1.0</resolution>
+               <min_angle>-0.01</min_angle>
+               <max_angle>0.01</max_angle>
+            </horizontal>
+            <vertical>
+               <samples>1</samples>
+               <resolution>1</resolution>
+               <min_angle>-0.01</min_angle>
+               <max_angle>0.01</max_angle>
+            </vertical>
+         </scan>
+         <range>
+            <min>0.01</min>
+            <max>3.75</max>
+            <resolution>0.02</resolution>
+         </range>
+      </ray>
+    <plugin name="libgazebo_ros_range" filename="libgazebo_ros_range.so">
+         <gaussianNoise>0.005</gaussianNoise>
+         <alwaysOn>true</alwaysOn>
+         <updateRate>50</updateRate>
+         <topicName>us_sensor</topicName>
+         <frameName>us_1_link</frameName>
+         <radiation>SONAR</radiation>
+         <fov>0.2967</fov>
+    </plugin>
+  </sensor>
   </gazebo>
     <!-- camera -->

File: robots/mmo_700/urdf/xacros/mpo_700_gazebo.xacro (robot description, xacro)
@@ -134,5 +134,5 @@
     </sensor>
   </gazebo>
-  <gazebo>
+ <gazebo>
     <plugin name="mpo_700_controller" filename="libgazebo_ros_planar_move.so">
       <commandTopic>cmd_vel</commandTopic>

File: robots/mp_400/xacros/mp_400_gazebo.xacro (robot description, xacro)
@@ -48,5 +48,5 @@
         </sensor>
   </gazebo>
-    <gazebo reference="imu_link">
+    <gazebo reference="imu_1_link">
     <gravity>true</gravity>
     <sensor name="imu_sensor" type="imu">
@@ -66,4 +66,39 @@
       <pose>0 0 0 0 0 0</pose>
     </sensor>
+  </gazebo>
+  <gazebo reference="us_1_link">
+  <!-- Visuals / Collisions omitted for this example -->
+  <sensor type="ray" name="range">
+    <ray>
+         <scan>
+            <horizontal>
+               <samples>1</samples>
+               <resolution>1.0</resolution>
+               <min_angle>-0.01</min_angle>
+               <max_angle>0.01</max_angle>
+            </horizontal>
+            <vertical>
+               <samples>1</samples>
+               <resolution>1</resolution>
+               <min_angle>-0.01</min_angle>
+               <max_angle>0.01</max_angle>
+            </vertical>
+         </scan>
+         <range>
+            <min>0.01</min>
+            <max>3.75</max>
+            <resolution>0.02</resolution>
+         </range>
+      </ray>
+    <plugin name="libgazebo_ros_range" filename="libgazebo_ros_range.so">
+         <gaussianNoise>0.005</gaussianNoise>
+         <alwaysOn>true</alwaysOn>
+         <updateRate>50</updateRate>
+         <topicName>us_sensor</topicName>
+         <frameName>us_1_link</frameName>
+         <radiation>SONAR</radiation>
+         <fov>0.2967</fov>
+    </plugin>
+  </sensor>
   </gazebo>
     <!-- camera -->

File: robots/mp_500/xacros/mp_500_gazebo.xacro (robot description, xacro)
@@ -36,5 +36,5 @@
         </sensor>
   </gazebo>
-    <gazebo reference="imu_link">
+    <gazebo reference="imu_1_link">
     <gravity>true</gravity>
     <sensor name="imu_sensor" type="imu">
@@ -54,4 +54,39 @@
       <pose>0 0 0 0 0 0</pose>
     </sensor>
+  </gazebo>
+  <gazebo reference="us_1_link">
+  <!-- Visuals / Collisions omitted for this example -->
+  <sensor type="ray" name="range">
+    <ray>
+         <scan>
+            <horizontal>
+               <samples>1</samples>
+               <resolution>1.0</resolution>
+               <min_angle>-0.01</min_angle>
+               <max_angle>0.01</max_angle>
+            </horizontal>
+            <vertical>
+               <samples>1</samples>
+               <resolution>1</resolution>
+               <min_angle>-0.01</min_angle>
+               <max_angle>0.01</max_angle>
+            </vertical>
+         </scan>
+         <range>
+            <min>0.01</min>
+            <max>3.75</max>
+            <resolution>0.02</resolution>
+         </range>
+      </ray>
+    <plugin name="libgazebo_ros_range" filename="libgazebo_ros_range.so">
+         <gaussianNoise>0.005</gaussianNoise>
+         <alwaysOn>true</alwaysOn>
+         <updateRate>50</updateRate>
+         <topicName>us_sensor</topicName>
+         <frameName>us_1_link</frameName>
+         <radiation>SONAR</radiation>
+         <fov>0.2967</fov>
+    </plugin>
+  </sensor>
   </gazebo>
     <!-- camera -->

File: robots/mpo_500/xacros/mpo_500_gazebo.xacro (robot description, xacro)
@@ -91,5 +91,5 @@
         </sensor>
   </gazebo>
-    <gazebo reference="imu_link">
+    <gazebo reference="imu_1_link">
     <gravity>true</gravity>
     <sensor name="imu_sensor" type="imu">
@@ -109,4 +109,39 @@
       <pose>0 0 0 0 0 0</pose>
     </sensor>
+  </gazebo>
+  <gazebo reference="us_1_link">
+  <!-- Visuals / Collisions omitted for this example -->
+  <sensor type="ray" name="range">
+    <ray>
+         <scan>
+            <horizontal>
+               <samples>1</samples>
+               <resolution>1.0</resolution>
+               <min_angle>-0.01</min_angle>
+               <max_angle>0.01</max_angle>
+            </horizontal>
+            <vertical>
+               <samples>1</samples>
+               <resolution>1</resolution>
+               <min_angle>-0.01</min_angle>
+               <max_angle>0.01</max_angle>
+            </vertical>
+         </scan>
+         <range>
+            <min>0.01</min>
+            <max>3.75</max>
+            <resolution>0.02</resolution>
+         </range>
+      </ray>
+    <plugin name="libgazebo_ros_range" filename="libgazebo_ros_range.so">
+         <gaussianNoise>0.005</gaussianNoise>
+         <alwaysOn>true</alwaysOn>
+         <updateRate>50</updateRate>
+         <topicName>us_sensor</topicName>
+         <frameName>us_1_link</frameName>
+         <radiation>SONAR</radiation>
+         <fov>0.2967</fov>
+    </plugin>
+  </sensor>
   </gazebo>
     <!-- camera -->

File: robots/mpo_500/xacros/ultrasonic.xacro (robot description, xacro)
@@ -1,4 +1,4 @@
 <?xml version="1.0"?>
-<robot xmlns:xacro="http://www.ros.org/wiki/xacro" name="mp_400">
+<robot xmlns:xacro="http://www.ros.org/wiki/xacro" name="mpo_700">
   <xacro:macro name="us_sensor" params="name parent *origin">
     <joint name="${name}_joint" type="fixed">

File: robots/mpo_700/mpo_700.urdf.xacro (robot description, xacro)
@@ -7,6 +7,6 @@
   <!-- SENSORS -->
   <xacro:include filename="$(find neo_simulation)/robots/mpo_700/xacros/sick_laser.xacro" />
-<!--   <xacro:include filename="$(find neo_simulation)/robots/mpo_700/xacros/imu.xacro" />
-  <xacro:include filename="$(find neo_simulation)/robots/mpo_700/xacros/ultrasonic.xacro" /> -->
+  <xacro:include filename="$(find neo_simulation)/robots/mpo_700/xacros/imu.xacro" />
+  <xacro:include filename="$(find neo_simulation)/robots/mpo_700/xacros/ultrasonic.xacro" />
   <!-- <xacro:include filename="$(find neo_simulation)/robots/mpo_700/xacros/camera.xacro" /> -->
   <xacro:include filename="$(find neo_simulation)/robots/mpo_700/xacros/mpo_700_gazebo.xacro" />
@@ -53,7 +53,7 @@
   <!-- Comment or uncomment based on your requirement -->
   <!-- SENSOR 1 -->
-  <!-- xacro:us_sensor name="us_1" parent="base_link">
-    <origin xyz="0.100 0 0.300" rpy="0 3.14 3.14" />
-  </xacro:us_sensor-->
+<!--   <xacro:us_sensor name="us_1" parent="base_link">
+    <origin xyz="0.100 0 0.500" rpy="0 3.14 3.14"/>
+  </xacro:us_sensor> -->
   <!-- SENSOR 2 -->
   <!-- xacro:us_sensor name="us_2" parent="base_link">

File: robots/mpo_700/xacros/mpo_700_gazebo.xacro (robot description, xacro)
@@ -75,5 +75,5 @@
         </sensor>
   </gazebo>
-    <gazebo reference="imu_link">
+    <gazebo reference="imu_1_link">
     <gravity>true</gravity>
     <sensor name="imu_sensor" type="imu">
@@ -97,4 +97,6 @@
   <gazebo reference="camera_link">
     <sensor type="camera" name="camera1">
+      <pose>0 0 0 0 0 0</pose>
+      <update_rate>50</update_rate>
       <update_rate>30.0</update_rate>
       <camera name="head">
@@ -134,3 +136,47 @@
     </sensor>
   </gazebo>
+  <gazebo reference="us_1_link">
+  <!-- Visuals / Collisions omitted for this example -->
+  <sensor type="ray" name="range">
+    <ray>
+         <scan>
+            <horizontal>
+               <samples>1</samples>
+               <resolution>1.0</resolution>
+               <min_angle>-0.01</min_angle>
+               <max_angle>0.01</max_angle>
+            </horizontal>
+            <vertical>
+               <samples>1</samples>
+               <resolution>1</resolution>
+               <min_angle>-0.01</min_angle>
+               <max_angle>0.01</max_angle>
+            </vertical>
+         </scan>
+         <range>
+            <min>0.01</min>
+            <max>3.75</max>
+            <resolution>0.02</resolution>
+         </range>
+      </ray>
+    <plugin name="libgazebo_ros_range" filename="libgazebo_ros_range.so">
+         <gaussianNoise>0.005</gaussianNoise>
+         <alwaysOn>true</alwaysOn>
+         <updateRate>50</updateRate>
+         <topicName>us_sensor</topicName>
+         <frameName>us_1_link</frameName>
+         <radiation>SONAR</radiation>
+         <fov>0.2967</fov>
+    </plugin>
+  </sensor>
+  </gazebo>
+ <gazebo>
+    <plugin name="mpo_700_controller" filename="libgazebo_ros_planar_move.so">
+      <commandTopic>cmd_vel</commandTopic>
+      <odometryTopic>odom</odometryTopic>
+      <odometryFrame>odom</odometryFrame>
+      <odometryRate>20.0</odometryRate>
+      <robotBaseFrame>base_link</robotBaseFrame>
+    </plugin>
+  </gazebo>
 </robot>
