Commit message: Modified URDF, plugins for noetic

File: robots/mm_400/urdf/xacros/mp_400_gazebo.xacro (robot description, xacro)
@@ -1,16 +1,4 @@
 <?xml version="1.0"?>
 <robot name="mm_400" xmlns:xacro="http://www.ros.org/wiki/xacro">
-   <gazebo reference="base_link">
-    <gravity>true</gravity>
-    <self_collide>false</self_collide>
-  </gazebo>
-  <gazebo reference="castor_wheel_link">
-    <gravity>true</gravity>
-    <self_collide>false</self_collide>
-  </gazebo>
-  <gazebo reference="fixed_wheel_link">
-    <gravity>true</gravity>
-    <self_collide>false</self_collide>
-  </gazebo>
 <gazebo reference="mp_400_caster_wheel_front_right_link">
       <kp>35000.0</kp>

File: robots/mmo_500/urdf/xacros/mpo_500_gazebo.xacro (robot description, xacro)
@@ -1,24 +1,4 @@
 <?xml version="1.0"?>
 <robot name="mpo_500" xmlns:xacro="http://www.ros.org/wiki/xacro">
-   <gazebo reference="base_link">
-    <gravity>true</gravity>
-    <self_collide>false</self_collide>
-  </gazebo>
-   <gazebo reference="mpo_500_omni_wheel_front_left_link">
-    <gravity>true</gravity>
-    <self_collide>false</self_collide>
-  </gazebo>
-  <gazebo reference="mpo_500_omni_wheel_front_right_link">
-    <gravity>true</gravity>
-    <self_collide>false</self_collide>
-  </gazebo>
-  <gazebo reference="mpo_500_omni_wheel_back_left_link">
-    <gravity>true</gravity>
-    <self_collide>false</self_collide>
-  </gazebo>
-  <gazebo reference="mpo_500_omni_wheel_back_right_link">
-    <gravity>true</gravity>
-    <self_collide>false</self_collide>
-  </gazebo>
   <!-- Lidar sensors -->
   <gazebo reference="lidar_1_link">

File: robots/mmo_700/urdf/xacros/mpo_700_gazebo.xacro (robot description, xacro)
@@ -1,8 +1,4 @@
 <?xml version="1.0"?>
 <robot name="mpo_700" xmlns:xacro="http://www.ros.org/wiki/xacro">
-   <gazebo reference="base_link">
-    <gravity>true</gravity>
-    <self_collide>false</self_collide>
-  </gazebo>
   <!-- Lidar sensors -->
   <gazebo reference="lidar_1_link">
@@ -80,9 +76,9 @@
     <gravity>true</gravity>
     <sensor name="imu_sensor" type="imu">
-      <always_on>true</always_on>
-      <update_rate>100</update_rate>
-      <visualize>true</visualize>
-      <topic>__default_topic__</topic>
-      <plugin filename="libgazebo_ros_imu_sensor.so" name="imu_plugin">
+        <always_on>true</always_on>
+        <update_rate>100</update_rate>
+        <visualize>true</visualize>
+        <topic>__default_topic__</topic>
+        <plugin filename="libgazebo_ros_imu_sensor.so" name="imu_plugin">
         <topicName>imu</topicName>
         <bodyName>imu_link</bodyName>

File: robots/mp_400/mp_400.urdf.xacro (robot description, xacro)
@@ -22,17 +22,19 @@
   <xacro:include filename="$(find neo_simulation)/robots/mp_400/xacros/ultrasonic.xacro" />-->
 <!-- Base link macro -->
-  <xacro:mp_400_base name="base_link">
-  </xacro:mp_400_base>
-  <!-- Wheel Macro -->
-  <xacro:caster_wheel name="mp_400_caster_wheel_front_left" parent="base_link">
+  <link name="base_link" />
+  <xacro:mp_400_base name="base_footprint" parent="base_link">
+    <origin xyz="0 0 0" rpy="0 0 0" />
+   </xacro:mp_400_base>
+    <!-- Wheel Macro -->
+  <xacro:caster_wheel name="mp_400_caster_wheel_front_left" parent="base_footprint">
     <origin xyz="0.165 0.155 0.036" rpy="0 0 1.57" />
   </xacro:caster_wheel>
-  <xacro:caster_wheel name="mp_400_caster_wheel_back_left" parent="base_link">
+  <xacro:caster_wheel name="mp_400_caster_wheel_back_left" parent="base_footprint">
     <origin xyz="-0.220 0.155 0.036" rpy="0 0 1.57" />
   </xacro:caster_wheel>
-  <xacro:caster_wheel name="mp_400_caster_wheel_front_right" parent="base_link">
+  <xacro:caster_wheel name="mp_400_caster_wheel_front_right" parent="base_footprint">
     <origin xyz="0.165 -0.155 0.036" rpy="0 0 1.57" />
   </xacro:caster_wheel>
-   <xacro:caster_wheel name="mp_400_caster_wheel_back_right" parent="base_link">
+   <xacro:caster_wheel name="mp_400_caster_wheel_back_right" parent="base_footprint">
     <origin xyz="-0.220 -0.155 0.036" rpy="0 0 1.57" />
   </xacro:caster_wheel>

File: robots/mp_400/xacros/mp_400_body.xacro (robot description, xacro)
@@ -1,7 +1,15 @@
 <?xml version="1.0"?>
 <robot xmlns:xacro="http://www.ros.org/wiki/xacro" name="mp_400">
-  <xacro:macro name="mp_400_base" params="name">
+  <xacro:macro name="mp_400_base" params="name parent *origin">
+    <joint name="${name}_joint" type="fixed">
+      <xacro:insert_block name="origin" />
+      <axis xyz="0 0 -1" />
+      <!-- <limit effort="1000.0" lower="-1e+16" upper="1e+16" velocity="3.5"/> -->
+      <joint_properties damping="1" friction="1" />
+      <parent link="${parent}" />
+      <child link="${name}" />
+   </joint>
     <link name="${name}">
-  <inertial>
+    <inertial>
         <mass value="30" />
         <origin xyz="0 0 0" rpy="0 0 0"/>
@@ -9,5 +17,5 @@
                  iyy="0.8856" iyz="0.0"
                  izz="2.5725" />
-</inertial>
+    </inertial>
       <visual name='body'>
       <origin xyz="0.0 0.0 0." rpy="0 0 1.57" />

File: robots/mp_400/xacros/mp_400_gazebo.xacro (robot description, xacro)
@@ -1,16 +1,4 @@
 <?xml version="1.0"?>
 <robot name="mp_400" xmlns:xacro="http://www.ros.org/wiki/xacro">
-   <gazebo reference="base_link">
-    <gravity>true</gravity>
-    <self_collide>false</self_collide>
-  </gazebo>
-  <gazebo reference="castor_wheel_link">
-    <gravity>true</gravity>
-    <self_collide>false</self_collide>
-  </gazebo>
-  <gazebo reference="fixed_wheel_link">
-    <gravity>true</gravity>
-    <self_collide>false</self_collide>
-  </gazebo>
   <!-- Lidar sensor -->
   <gazebo reference="laser_1_link">
@@ -146,26 +134,26 @@
   </gazebo>
   <gazebo>
-    <plugin name="diff_dirve_controller" filename="libgazebo_ros_diff_drive.so">
-        <alwaysOn>true</alwaysOn>
-        <updateRate>40</updateRate>
-        <legacyMode>false</legacyMode>
-	<torque>2</torque>
-        <leftJoint>mp_400_fixed_wheel_left_joint</leftJoint>
-        <rightJoint>mp_400_fixed_wheel_right_joint</rightJoint>
-        <wheelSeparation>0.529</wheelSeparation>
-        <wheelDiameter>0.15</wheelDiameter>
-        <commandTopic>cmd_vel</commandTopic>
-        <rosDebugLevel>na</rosDebugLevel>
-        <odometryTopic>odom</odometryTopic>
-        <odometryFrame>odom</odometryFrame>
-        <robotBaseFrame>base_link</robotBaseFrame>
-        <publishWheelTF>true</publishWheelTF>
-        <publishWheelJointState>true</publishWheelJointState>
-        <wheelAcceleration>0.0</wheelAcceleration>
-        <wheelTorque>20</wheelTorque>
-        <odometrySource>world</odometrySource>
-        <publishTf>1</publishTf>
-        <publishOdomTF>true</publishOdomTF>
-    </plugin>
-  </gazebo>
+     <plugin name="differential_drive_controller" filename="libgazebo_ros_diff_drive.so">
+     <alwaysOn>true</alwaysOn>
+      <updateRate>60</updateRate>
+     <legacyMode>true</legacyMode>
+     <leftJoint>mp_400_fixed_wheel_left_joint</leftJoint>
+     <rightJoint>mp_400_fixed_wheel_right_joint</rightJoint>
+     <wheelSeparation>0.529</wheelSeparation>
+     <wheelDiameter>0.15</wheelDiameter>
+     <torque>2</torque>
+     <commandTopic>cmd_vel</commandTopic>
+     <odometryTopic>odom</odometryTopic>
+     <odometryFrame>odom</odometryFrame>
+     <robotBaseFrame>base_footprint</robotBaseFrame>
+     <publishWheelTF>true</publishWheelTF>
+     <publishWheelJointState>true</publishWheelJointState>
+     <rosDebugLevel>na</rosDebugLevel>
+     <wheelAcceleration>0</wheelAcceleration>
+     <wheelTorque>20</wheelTorque>
+     <odometrySource>world</odometrySource>
+     <publishTf>1</publishTf>
+     <publishOdomTF>true</publishOdomTF>
+  </plugin>
+   </gazebo>
 </robot>

File: robots/mp_500/mp_500.urdf.xacro (robot description, xacro)
@@ -21,14 +21,17 @@
   <xacro:include filename="$(find neo_simulation)/robots/mp_500/xacros/camera.xacro" />
   <-->
-  <xacro:mp_500_base name="base_link">
+<link name="base_link" />
+  <!-- Base link macro -->
+ <xacro:mp_500_base name="base_footprint" parent="base_link">
+    <origin xyz="0 0 0" rpy="0 0 0" />
   </xacro:mp_500_base>
   <!-- Wheel Macro -->
-  <xacro:caster_wheel name="mp_500_caster_wheel" parent="base_link">
+  <xacro:caster_wheel name="caster_wheel" parent="base_footprint">
     <origin xyz="-0.43 0. 0.176" rpy="-1.570796 0 1.570796 " />
   </xacro:caster_wheel>
-  <xacro:fixed_wheel_right name="mp_500_fixed_wheel_right" parent="base_link" number="1">
+  <xacro:fixed_wheel_right name="wheel_right" parent="base_footprint" number="1">
     <origin xyz="0. -0.25 0.13" rpy="0 0 -1.570796" />
   </xacro:fixed_wheel_right>
-  <xacro:fixed_wheel_left name="mp_500_fixed_wheel_left" parent="base_link" number="2">
+  <xacro:fixed_wheel_left name="wheel_left" parent="base_footprint" number="2">
     <origin xyz="0. 0.25 0.13" rpy="0 0 -1.570796" />
   </xacro:fixed_wheel_left>

File: robots/mp_500/xacros/mp_500_body.xacro (robot description, xacro)
@@ -1,5 +1,13 @@
 <?xml version="1.0"?>
 <robot xmlns:xacro="http://www.ros.org/wiki/xacro" name="mp_500">
-  <xacro:macro name="mp_500_base" params="name">
+<xacro:macro name="mp_500_base" params="name parent *origin">
+    <joint name="${name}_joint" type="fixed">
+      <xacro:insert_block name="origin" />
+      <axis xyz="0 0 -1" />
+      <!-- <limit effort="1000.0" lower="-1e+16" upper="1e+16" velocity="3.5"/> -->
+      <joint_properties damping="1" friction="1" />
+      <parent link="${parent}" />
+      <child link="${name}" />
+   </joint>
     <link name="${name}">
   <inertial>

File: robots/mp_500/xacros/mp_500_fixed_wheel_left.xacro (robot description, xacro)
@@ -10,15 +10,5 @@
     <child link="${name}_link" />
    </joint>
-   <transmission name="tran_${number}">
-    <type>transmission_interface/SimpleTransmission</type>
-    <joint name="${name}_joint" type="revolute">
-      <hardwareInterface>hardware_interface/VelocityJointInterface</hardwareInterface>
-        </joint>
-      <actuator name="left_wheel_actuator">
-      <mechanicalReduction>7</mechanicalReduction>
-            <hardwareInterface>hardware_interface/VelocityJointInterface</hardwareInterface>
-      </actuator>
-  </transmission>
-   <link name="${name}_link" type="wheel">
+    <link name="${name}_link" type="wheel">
     <inertial>
       <origin xyz="0 0 0" rpy="0 0 0"/>
@@ -41,11 +31,4 @@
     </collision>
 </link>
-  <gazebo reference="${name}_link">
-      <mu1 value = "300.0"/>
-      <mu2 value = "100.0"/>
-      <kp value="8000.0" />
-      <kd value="1460.0" />
-      <fdir1 value="0.5 0 0"/>
-</gazebo>
   </xacro:macro>
 </robot>

File: robots/mp_500/xacros/mp_500_fixed_wheel_right.xacro (robot description, xacro)
@@ -10,14 +10,4 @@
     <child link="${name}_link" />
    </joint>
-   <transmission name="tran_${number}">
-    <type>transmission_interface/SimpleTransmission</type>
-    <joint name="${name}_joint" type="revolute">
-      <hardwareInterface>hardware_interface/VelocityJointInterface</hardwareInterface>
-        </joint>
-      <actuator name="right_wheel_actuator">
-      <mechanicalReduction>7</mechanicalReduction>
-            <hardwareInterface>hardware_interface/VelocityJointInterface</hardwareInterface>
-      </actuator>
-  </transmission>
    <link name="${name}_link" type="wheel">
     <inertial>
@@ -41,11 +31,4 @@
     </collision>
 </link>
-  <gazebo reference="${name}_link">
-      <mu1 value = "300.0"/>
-      <mu2 value = "100.0"/>
-      <kp value="8000.0" />
-      <kd value="1460.0" />
-      <fdir1 value="0.5 0 0"/>
-</gazebo>
   </xacro:macro>
 </robot>

File: robots/mp_500/xacros/mp_500_gazebo.xacro (robot description, xacro)
@@ -1,4 +1,28 @@
 <?xml version="1.0"?>
 <robot name="mp_500" xmlns:xacro="http://www.ros.org/wiki/xacro">
+  <gazebo>
+     <plugin name="differential_drive_controller" filename="libgazebo_ros_diff_drive.so">
+     <alwaysOn>true</alwaysOn>
+      <updateRate>60</updateRate>
+     <legacyMode>true</legacyMode>
+     <leftJoint>wheel_left_joint</leftJoint>
+     <rightJoint>wheel_right_joint</rightJoint>
+     <wheelSeparation>0.592</wheelSeparation>
+     <wheelDiameter>0.260</wheelDiameter>
+     <torque>20</torque>
+     <commandTopic>cmd_vel</commandTopic>
+     <odometryTopic>odom</odometryTopic>
+     <odometryFrame>odom</odometryFrame>
+     <robotBaseFrame>base_link</robotBaseFrame>
+     <publishWheelTF>false</publishWheelTF>
+     <publishWheelJointState>false</publishWheelJointState>
+     <rosDebugLevel>na</rosDebugLevel>
+     <wheelAcceleration>0</wheelAcceleration>
+     <wheelTorque>5</wheelTorque>
+     <odometrySource>world</odometrySource>
+     <publishTf>1</publishTf>
+     <publishOdomTF>True</publishOdomTF>>
+  </plugin>
+  </gazebo>
   <gazebo reference="lidar_1_link">
       <sensor type="ray" name="lidar_1_link">
@@ -132,28 +156,4 @@
     </sensor>
   </gazebo>
-  <gazebo>
-    <plugin name="diff_dirve_controller" filename="libgazebo_ros_diff_drive.so">
-        <alwaysOn>true</alwaysOn>
-        <updateRate>100</updateRate>
-        <legacyMode>false</legacyMode>
-        <torque>2.5</torque>
-        <leftJoint>mp_500_fixed_wheel_left_joint</leftJoint>
-        <rightJoint>mp_500_fixed_wheel_right_joint</rightJoint>
-        <wheelSeparation>0.592</wheelSeparation>
-        <wheelDiameter>0.260</wheelDiameter>
-        <commandTopic>cmd_vel</commandTopic>
-        <rosDebugLevel>na</rosDebugLevel>
-        <odometryTopic>odom</odometryTopic>
-        <odometryFrame>odom</odometryFrame>
-        <robotBaseFrame>base_link</robotBaseFrame>
-        <publishWheelTF>true</publishWheelTF>
-        <publishWheelJointState>true</publishWheelJointState>
-        <wheelAcceleration>0</wheelAcceleration>
-        <wheelTorque>200</wheelTorque>
-        <odometrySource>world</odometrySource>
-        <publishTf>1</publishTf>
-        <publishOdomTF>true</publishOdomTF>
-    </plugin>
-  </gazebo>
 <!-- <gazebo>
   <plugin name="gazebo_ros_control" filename="libgazebo_ros_control.so">

File: robots/mpo_700/xacros/mpo_700_gazebo.xacro (robot description, xacro)
@@ -1,8 +1,4 @@
 <?xml version="1.0"?>
 <robot name="mpo_700" xmlns:xacro="http://www.ros.org/wiki/xacro">
-   <gazebo reference="base_link">
-    <gravity>true</gravity>
-    <self_collide>false</self_collide>
-  </gazebo>
   <gazebo reference="lidar_1_link">
       <sensor type="ray" name="lidar_1_sensor">
@@ -105,5 +101,5 @@
       <odometryTopic>odom</odometryTopic>
       <odometryFrame>odom</odometryFrame>
-      <odometryRate>150.0</odometryRate>
+      <odometryRate>100.0</odometryRate>
       <robotBaseFrame>base_link</robotBaseFrame>
     </plugin>
