Commit message: Microscan position for mpo_700 is repositioned

File: robots/mpo_700/mpo_700.urdf.xacro (robot description, xacro)
@@ -37,16 +37,17 @@
 <!-- Sensors -->
 <!-- Uncomment or comment it for sick s300 -->
-  <xacro:sick_v0 name="sick_s300_laser_front" parent="base_link" ros_topic="sick_s300_front/scan">
+  <xacro:sick_v0 name="sick_laser_front" parent="base_link" ros_topic="sick_front/scan">
   	<origin xyz="0.360 0 0.181" rpy="3.14 0 0 " />
   </xacro:sick_v0>
-  <xacro:sick_v0 name="sick_s300_laser_back" parent="base_link" ros_topic="sick_s300_back/scan">
+  <xacro:sick_v0 name="sick_laser_back" parent="base_link" ros_topic="sick_back/scan">
   	<origin xyz="-0.360 0 0.181" rpy="3.14 0 3.14" />
   </xacro:sick_v0>
 <!-- Uncomment or comment it for sick_microscan_3 -->
-<!--   <xacro:sick_v0 name="sick_microscan_3_front" parent="base_link" ros_topic="sick_s300_front/scan">
-    <origin xyz="0.360 0 0.28" rpy="3.14 3.14 0" />
+<!--   <xacro:sick_v0 name="sick_laser_front" parent="base_link" ros_topic="sick_front/scan">
+    <origin xyz="0.360 0 0.181" rpy="3.14 3.14 3.14" />
   </xacro:sick_v0>
-  <xacro:sick_v0 name="sick_microscan_3_back" parent="base_link" ros_topic="sick_s300_back/scan">
-    <origin xyz="-0.360 0 0.28" rpy="3.14 3.14 3.14" />
-  </xacro:sick_v0> -->
+  <xacro:sick_v0 name="sick_laser_back" parent="base_link" ros_topic="sick_back/scan">
+    <origin xyz="-0.360 0 0.181" rpy="3.14 3.14 0" />
+  </xacro:sick_v0>
+ -->
 </robot>

File: robots/mpo_700/xacros/mpo_700_body.xacro (robot description, xacro)
@@ -17,5 +17,5 @@
       </visual>
       <collision>
-        <origin xyz="0. 0. 0.2" rpy="0 0 0" />
+        <origin xyz="0. 0. 0." rpy="0 0 -1.571" />
         <geometry>
             <mesh filename="package://neo_simulation/robots/mpo_700/meshes/MPO-700-BODY.dae" scale="0.001 0.001 0.001"/>

File: robots/mpo_700/xacros/mpo_700_gazebo.xacro (robot description, xacro)
@@ -5,6 +5,41 @@
     <self_collide>false</self_collide>
   </gazebo>
-  <gazebo reference="sick_s300_laser_front_link">
-      <sensor type="ray" name="sick_s300_laser_front_sensor">
+  <gazebo reference="sick_laser_front_link">
+      <sensor type="ray" name="sick_laser_front_sensor">
+          <pose>0 0 0 0 0 0</pose>
+          <visualize>true</visualize>
+          <update_rate>40</update_rate>
+          <ray>
+            <scan>
+              <horizontal>
+                <samples>720</samples>
+                <resolution>1</resolution>
+                <min_angle>-1.48</min_angle>
+                <max_angle>1.48</max_angle>
+              </horizontal>
+            </scan>
+            <range>
+              <min>0.10</min>
+              <max>30.0</max>
+              <resolution>0.05</resolution>
+            </range>
+            <noise>
+              <type>gaussian</type>
+              <!-- Noise parameters based on published spec for Hokuyo laser
+                   achieving "+-30mm" accuracy at range < 10m.  A mean of 0.0m and
+                   stddev of 0.01m will put 99.7% of samples within 0.03m of the true
+                   reading. -->
+              <mean>0.0</mean>
+              <stddev>0.01</stddev>
+            </noise>
+          </ray>
+          <plugin name="sick_laser_front" filename="libgazebo_ros_laser.so">
+            <topicName>sick_front/scan</topicName>
+            <frameName>sick_laser_front_link</frameName>
+          </plugin>
+        </sensor>
+  </gazebo>
+  <gazebo reference="sick_laser_back_link">
+      <sensor type="ray" name="sick_laser_back_sensor">
           <pose>0 0 0 0 0 0</pose>
           <visualize>false</visualize>
@@ -34,42 +69,7 @@
             </noise>
           </ray>
-          <plugin name="sick_s300_laser_front" filename="libgazebo_ros_laser.so">
-            <topicName>sick_s300_front/scan</topicName>
-            <frameName>sick_s300_laser_front_link</frameName>
-          </plugin>
-        </sensor>
-  </gazebo>
-  <gazebo reference="sick_s300_laser_back_link">
-      <sensor type="ray" name="sick_s300_laser_back_sensor">
-          <pose>0 0 0 0 0 0</pose>
-          <visualize>false</visualize>
-          <update_rate>40</update_rate>
-          <ray>
-            <scan>
-              <horizontal>
-                <samples>720</samples>
-                <resolution>1</resolution>
-                <min_angle>-1.48</min_angle>
-                <max_angle>1.48</max_angle>
-              </horizontal>
-            </scan>
-            <range>
-              <min>0.10</min>
-              <max>30.0</max>
-              <resolution>0.05</resolution>
-            </range>
-            <noise>
-              <type>gaussian</type>
-              <!-- Noise parameters based on published spec for Hokuyo laser
-                   achieving "+-30mm" accuracy at range < 10m.  A mean of 0.0m and
-                   stddev of 0.01m will put 99.7% of samples within 0.03m of the true
-                   reading. -->
-              <mean>0.0</mean>
-              <stddev>0.01</stddev>
-            </noise>
-          </ray>
-          <plugin name="sick_s300_laser_back" filename="libgazebo_ros_laser.so">
-            <topicName>sick_s300_back/scan</topicName>
-            <frameName>sick_s300_laser_back_link</frameName>
+          <plugin name="sick_laser_back" filename="libgazebo_ros_laser.so">
+            <topicName>sick_back/scan</topicName>
+            <frameName>sick_laser_back_link</frameName>
           </plugin>
         </sensor>

File: robots/mpo_700/xacros/sick_laser.xacro (robot description, xacro)
@@ -22,5 +22,5 @@
       </visual>
       <collision>
-        <origin xyz="0 0 0." rpy="-1.57 0 3.14" />
+        <origin xyz="0 0 -0.12" rpy="-1.57 0 3.14" />
         <geometry>
         <mesh filename="package://neo_simulation/robots/mpo_700/meshes/SICK-S300.dae" scale="0.001 0.001 0.001" />
@@ -44,5 +44,5 @@
       </inertial>
       <visual>
-        <origin xyz="0 0 0.0" rpy="-1.57 0 3.14" />
+        <origin xyz="0 0 0.08" rpy="-1.57 0 0" />
         <geometry>
           <mesh filename="package://neo_simulation/robots/mpo_700/meshes/SICK-MICROSCAN3.dae" scale="0.001 0.001 0.001" />
@@ -50,5 +50,5 @@
       </visual>
       <collision>
-        <origin xyz="0 0 0" rpy="0 0 0" />
+        <origin xyz="0 0 0.08" rpy="-1.57 0 0" />
         <geometry>
           <mesh filename="package://neo_simulation/robots/mpo_700/meshes/SICK-MICROSCAN3.dae" scale="0.001 0.001 0.001" />
@@ -56,4 +56,5 @@
       </collision>
     </link>
-  </xacro:macro> -->
+  </xacro:macro>
+ -->
 </robot>

Commit message: Robot model for mpo-700 is updated

File: robots/mpo_700/mpo_700.urdf.xacro (robot description, xacro)
@@ -12,14 +12,14 @@
   </xacro:mpo_700_base>
 <xacro:mpo_700_head_0 name="mpo_700_head_0" parent="base_link">
-    <origin xyz="0.24 0.18 0.25" rpy="3.14 0 -1.57" />
+    <origin xyz="0.24 0.18 0.27" rpy="3.14 0 -1.57" />
   </xacro:mpo_700_head_0>
 <xacro:mpo_700_head_1 name="mpo_700_head_1" parent="base_link">
-    <origin xyz="0.24 -0.18 0.25" rpy="3.14 0 1.57" />
+    <origin xyz="0.24 -0.18 0.27" rpy="3.14 0 1.57" />
   </xacro:mpo_700_head_1>
 <xacro:mpo_700_head_2 name="mpo_700_head_2" parent="base_link">
-    <origin xyz="-0.24 0.18 0.25" rpy="3.14 0 -1.57" />
+    <origin xyz="-0.24 0.18 0.27" rpy="3.14 0 -1.57" />
   </xacro:mpo_700_head_2>
 <xacro:mpo_700_head_3 name="mpo_700_head_3" parent="base_link">
-    <origin xyz="-0.24 -0.18 0.25" rpy="3.14 0 1.57" />
+    <origin xyz="-0.24 -0.18 0.27" rpy="3.14 0 1.57" />
   </xacro:mpo_700_head_3>
 <xacro:mpo_700_wheel name="wheel_0" parent="mpo_700_head_0_link">
@@ -36,5 +36,4 @@
   </xacro:mpo_700_wheel>
 <!-- Sensors -->
-<!-- Uncomment or comment it for sick s300 -->
   <xacro:sick_v0 name="sick_laser_front" parent="base_link" ros_topic="sick_front/scan">
   	<origin xyz="0.360 0 0.181" rpy="3.14 0 0 " />
@@ -43,11 +42,3 @@
   	<origin xyz="-0.360 0 0.181" rpy="3.14 0 3.14" />
   </xacro:sick_v0>
-<!-- Uncomment or comment it for sick_microscan_3 -->
-<!--   <xacro:sick_v0 name="sick_laser_front" parent="base_link" ros_topic="sick_front/scan">
-    <origin xyz="0.360 0 0.181" rpy="3.14 3.14 3.14" />
-  </xacro:sick_v0>
-  <xacro:sick_v0 name="sick_laser_back" parent="base_link" ros_topic="sick_back/scan">
-    <origin xyz="-0.360 0 0.181" rpy="3.14 3.14 0" />
-  </xacro:sick_v0>
- -->
 </robot>

File: robots/mpo_700/xacros/mpo_700_head.xacro (robot description, xacro)
@@ -17,5 +17,5 @@
     </inertial>
     <visual>
-     <origin xyz="0 0 0.05" rpy="0 0 0"/>
+     <origin xyz="0 0 0.10" rpy="0 0 0"/>
      <geometry>
         <mesh filename="package://neo_simulation/robots/mpo_700/meshes/MPO-700-HEAD.dae" scale="0.001 0.001 0.001"/>
@@ -23,5 +23,5 @@
     </visual>
     <collision>
-     <origin xyz="0 0 0.05" rpy="0 0 0" />
+     <origin xyz="0 0 0.10" rpy="0 0 0" />
      <geometry>
         <mesh filename="package://neo_simulation/robots/mpo_700/meshes/MPO-700-HEAD.dae" scale="0.001 0.001 0.001"/>
@@ -45,5 +45,5 @@
     </inertial>
     <visual>
-     <origin xyz="0 0 0.05" rpy="0 0 0"/>
+     <origin xyz="0 0 0.10" rpy="0 0 0"/>
      <geometry>
         <mesh filename="package://neo_simulation/robots/mpo_700/meshes/MPO-700-HEAD.dae" scale="0.001 0.001 0.001"/>
@@ -51,5 +51,5 @@
     </visual>
     <collision>
-     <origin xyz="0 0 0.05" rpy="0 0 0" />
+     <origin xyz="0 0 0.10" rpy="0 0 0" />
      <geometry>
         <mesh filename="package://neo_simulation/robots/mpo_700/meshes/MPO-700-HEAD.dae" scale="0.001 0.001 0.001"/>
@@ -73,5 +73,5 @@
     </inertial>
     <visual>
-     <origin xyz="0 0 0.05" rpy="0 0 0"/>
+     <origin xyz="0 0 0.10" rpy="0 0 0"/>
      <geometry>
         <mesh filename="package://neo_simulation/robots/mpo_700/meshes/MPO-700-HEAD.dae" scale="0.001 0.001 0.001"/>
@@ -79,5 +79,5 @@
     </visual>
     <collision>
-     <origin xyz="0 0 0.05" rpy="0 0 0" />
+     <origin xyz="0 0 0.10" rpy="0 0 0" />
      <geometry>
         <mesh filename="package://neo_simulation/robots/mpo_700/meshes/MPO-700-HEAD.dae" scale="0.001 0.001 0.001"/>
@@ -101,5 +101,5 @@
     </inertial>
     <visual>
-     <origin xyz="0 0 0.05" rpy="0 0 0"/>
+     <origin xyz="0 0 0.10" rpy="0 0 0"/>
      <geometry>
         <mesh filename="package://neo_simulation/robots/mpo_700/meshes/MPO-700-HEAD.dae" scale="0.001 0.001 0.001"/>
@@ -107,5 +107,5 @@
     </visual>
     <collision>
-     <origin xyz="0 0 0.05" rpy="0 0 0" />
+     <origin xyz="0 0 0.10" rpy="0 0 0" />
      <geometry>
         <mesh filename="package://neo_simulation/robots/mpo_700/meshes/MPO-700-HEAD.dae" scale="0.001 0.001 0.001"/>

File: robots/mpo_700/xacros/sick_laser.xacro (robot description, xacro)
@@ -44,5 +44,5 @@
       </inertial>
       <visual>
-        <origin xyz="0 0 0.08" rpy="-1.57 0 0" />
+        <origin xyz="0 0 -0.06" rpy="1.57 0 0" />
         <geometry>
           <mesh filename="package://neo_simulation/robots/mpo_700/meshes/SICK-MICROSCAN3.dae" scale="0.001 0.001 0.001" />
@@ -50,5 +50,5 @@
       </visual>
       <collision>
-        <origin xyz="0 0 0.08" rpy="-1.57 0 0" />
+        <origin xyz="0 0 -0.06" rpy="1.57 0 0" />
         <geometry>
           <mesh filename="package://neo_simulation/robots/mpo_700/meshes/SICK-MICROSCAN3.dae" scale="0.001 0.001 0.001" />
@@ -56,5 +56,4 @@
       </collision>
     </link>
-  </xacro:macro>
- -->
+  </xacro:macro> -->
 </robot>

Commit message: mpo-700: Naming modified and Sensors added - Usage is ready

File: robots/mpo_700/mpo_700.urdf.xacro (robot description, xacro)
@@ -3,9 +3,11 @@
   <!-- BODY -->
   <xacro:include filename="$(find neo_simulation)/robots/mpo_700/xacros/mpo_700_body.xacro" />
+  <xacro:include filename="$(find neo_simulation)/robots/mpo_700/xacros/mpo_700_head.xacro" />
+  <xacro:include filename="$(find neo_simulation)/robots/mpo_700/xacros/mpo_700_wheel.xacro" />
   <!-- SENSORS -->
   <xacro:include filename="$(find neo_simulation)/robots/mpo_700/xacros/sick_laser.xacro" />
+  <xacro:include filename="$(find neo_simulation)/robots/mpo_700/xacros/imu.xacro" />
   <xacro:include filename="$(find neo_simulation)/robots/mpo_700/xacros/mpo_700_gazebo.xacro" />
-  <xacro:include filename="$(find neo_simulation)/robots/mpo_700/xacros/mpo_700_head.xacro" />
-  <xacro:include filename="$(find neo_simulation)/robots/mpo_700/xacros/mpo_700_wheel.xacro" />
+  <xacro:include filename="$(find neo_simulation)/robots/mpo_700/xacros/ultrasonic.xacro" />
   <!-- Base Macro-->
   <xacro:mpo_700_base name="base_link">
@@ -36,9 +38,80 @@
   </xacro:mpo_700_wheel>
 <!-- Sensors -->
-  <xacro:sick_v0 name="lidar_1" parent="base_link" ros_topic="lidar_1/scan">
+  <xacro:sick_v0 name="lidar_1" parent="base_link" ros_topic="lidar_1/scan_filtered">
   	<origin xyz="0.360 0 0.181" rpy="3.14 0 0 " />
   </xacro:sick_v0>
-  <xacro:sick_v0 name="lidar_2" parent="base_link" ros_topic="lidar_2/scan">
+  <xacro:sick_v0 name="lidar_2" parent="base_link" ros_topic="lidar_2/scan_filtered">
   	<origin xyz="-0.360 0 0.181" rpy="3.14 0 3.14" />
   </xacro:sick_v0>
+   <!--+++++++++++++++++++ IMU ++++++++++++++++++++++++-->
+ <!-- Comment or uncomment based on your requirement -->
+  <xacro:imu name="imu_1" parent="base_link">
+    <origin xyz="0.100 0 0.300" rpy="0 0 3.14" />
+  </xacro:imu>
+  <!--+++++++++++++++++++ Ultra Sonic ++++++++++++++++++++++++-->
+  <!-- Comment or uncomment based on your requirement -->
+  <!-- SENSOR 1 -->
+  <!-- xacro:us_sensor name="us_1" parent="base_link">
+    <origin xyz="0.100 0 0.300" rpy="0 3.14 3.14" />
+  </xacro:us_sensor-->
+  <!-- SENSOR 2 -->
+  <!-- xacro:us_sensor name="us_2" parent="base_link">
+    <origin xyz="0.110 0 0.300" rpy="0 3.14 3.14" />
+  </xacro:us_sensor-->
+  <!-- SENSOR 3 -->
+  <!-- xacro:us_sensor name="us_3" parent="base_link">
+    <origin xyz="0.120 0 0.300" rpy="0 3.14 3.14" />
+  </xacro:us_sensor-->
+  <!-- SENSOR 4 -->
+  <!-- xacro:us_sensor name="us_4" parent="base_link">
+    <origin xyz="0.130 0 0.300" rpy="0 3.14 3.14" />
+  </xacro:us_sensor-->
+  <!-- SENSOR 5 -->
+  <!-- xacro:us_sensor name="us_5" parent="base_link">
+    <origin xyz="0.140 0 0.300" rpy="0 3.14 3.14" />
+  </xacro:us_sensor-->
+  <!-- SENSOR 6 -->
+  <!-- xacro:us_sensor name="us_6" parent="base_link">
+    <origin xyz="0.150 0 0.300" rpy="0 3.14 3.14" />
+  </xacro:us_sensor-->
+  <!-- SENSOR 7 -->
+  <!-- xacro:us_sensor name="us_7" parent="base_link">
+    <origin xyz="0.160 0 0.300" rpy="0 3.14 3.14" />
+  </xacro:us_sensor-->
+  <!-- SENSOR 8 -->
+  <!-- xacro:us_sensor name="us_8" parent="base_link">
+    <origin xyz="0.170 0 0.300" rpy="0 3.14 3.14" />
+  </xacro:us_sensor-->
+  <!-- SENSOR 9 -->
+  <!-- xacro:us_sensor name="us_9" parent="base_link">
+    <origin xyz="0.180 0 0.300" rpy="0 3.14 3.14" />
+  </xacro:us_sensor-->
+  <!-- SENSOR 10 -->
+  <!-- xacro:us_sensor name="us_10" parent="base_link">
+    <origin xyz="0.100 0 0.300" rpy="0 3.14 3.14" />
+  </xacro:us_sensor-->
+  <!-- SENSOR 11 -->
+  <!-- xacro:us_sensor name="us_11" parent="base_link">
+    <origin xyz="0.100 0 0.300" rpy="0 3.14 3.14" />
+  </xacro:us_sensor-->
+  <!-- SENSOR 12 -->
+  <!-- xacro:us_sensor name="us_12" parent="base_link">
+    <origin xyz="0.190 0 0.300" rpy="0 3.14 3.14" />
+  </xacro:us_sensor-->
+  <!-- SENSOR 13 -->
+  <!-- xacro:us_sensor name="us_13" parent="base_link">
+    <origin xyz="0.200 0 0.300" rpy="0 3.14 3.14" />
+  </xacro:us_sensor-->
+  <!-- SENSOR 14 -->
+  <!-- xacro:us_sensor name="us_14" parent="base_link">
+    <origin xyz="0.210 0 0.300" rpy="0 3.14 3.14" />
+  </xacro:us_sensor-->
+  <!-- SENSOR 15 -->
+  <!-- xacro:us_sensor name="us_15" parent="base_link">
+    <origin xyz="0.220 0 0.300" rpy="0 3.14 3.14" />
+  </xacro:us_sensor-->
+  <!-- SENSOR 16 -->
+  <!-- xacro:us_sensor name="us_16" parent="base_link">
+    <origin xyz="0.230 0 0.300" rpy="0 3.14 3.14" />
+  </xacro:us_sensor-->
 </robot>

File: robots/mpo_700/xacros/mpo_700_gazebo.xacro (robot description, xacro)
@@ -5,6 +5,6 @@
     <self_collide>false</self_collide>
   </gazebo>
-  <gazebo reference="sick_laser_front_link">
-      <sensor type="ray" name="sick_laser_front_sensor">
+  <gazebo reference="lidar_1_link">
+      <sensor type="ray" name="lidar_1_sensor">
           <pose>0 0 0 0 0 0</pose>
           <visualize>false</visualize>
@@ -34,12 +34,12 @@
             </noise>
           </ray>
-          <plugin name="sick_laser_front" filename="libgazebo_ros_laser.so">
-            <topicName>lidar_1/scan</topicName>
-            <frameName>sick_laser_front_link</frameName>
+          <plugin name="lidar_1" filename="libgazebo_ros_laser.so">
+            <topicName>lidar_1/scan_filtered</topicName>
+            <frameName>lidar_1_link</frameName>
           </plugin>
         </sensor>
   </gazebo>
-  <gazebo reference="sick_laser_back_link">
-      <sensor type="ray" name="sick_laser_back_sensor">
+  <gazebo reference="lidar_2_link">
+      <sensor type="ray" name="lidar_2_sensor">
           <pose>0 0 0 0 0 0</pose>
           <visualize>false</visualize>
@@ -69,7 +69,7 @@
             </noise>
           </ray>
-          <plugin name="sick_laser_back" filename="libgazebo_ros_laser.so">
-            <topicName>lidar_2/scan</topicName>
-            <frameName>sick_laser_back_link</frameName>
+          <plugin name="lidar_2" filename="libgazebo_ros_laser.so">
+            <topicName>lidar_2/scan_filtered</topicName>
+            <frameName>lidar_2_link</frameName>
           </plugin>
         </sensor>

Commit message: MPO-700 main xacro updated with the co-ordinates for the laser scanners in the corners

File: robots/mpo_700/mpo_700.urdf.xacro (robot description, xacro)
@@ -4,5 +4,10 @@
   <xacro:include filename="$(find neo_simulation)/robots/mpo_700/xacros/mpo_700_body.xacro" />
   <!-- SENSORS -->
-  <xacro:include filename="$(find neo_simulation)/robots/mpo_700/xacros/sick_laser.xacro" />
+  <!-- Sick S300 - Comment/Uncomment if required -->
+  <!-- <xacro:include filename="$(find neo_simulation)/robots/mpo_700/xacros/sick_S300.xacro" /> -->
+  <!-- Microscan - Comment/Uncomment if required -->
+  <xacro:include filename="$(find neo_simulation)/robots/mpo_700/xacros/micro_scan.xacro" />
+  <!--<xacro:include filename="$(find neo_simulation)/robots/mpo_700/xacros/imu.xacro" />
+  <xacro:include filename="$(find neo_simulation)/robots/mpo_700/xacros/ultrasonic.xacro" /> -->
   <xacro:include filename="$(find neo_simulation)/robots/mpo_700/xacros/mpo_700_gazebo.xacro" />
   <xacro:include filename="$(find neo_simulation)/robots/mpo_700/xacros/mpo_700_head.xacro" />
@@ -36,9 +41,87 @@
   </xacro:mpo_700_wheel>
 <!-- Sensors -->
-  <xacro:sick_v0 name="lidar_1" parent="base_link" ros_topic="lidar_1/scan">
-  	<origin xyz="0.360 0 0.181" rpy="3.14 0 0 " />
-  </xacro:sick_v0>
-  <xacro:sick_v0 name="lidar_2" parent="base_link" ros_topic="lidar_2/scan">
-  	<origin xyz="-0.360 0 0.181" rpy="3.14 0 3.14" />
-  </xacro:sick_v0>
+  <xacro:sick_laser_v0 name="lidar_1" parent="base_link" ros_topic="lidar_1/scan_filtered">
+  <!--<origin xyz="0.360 0 0.181" rpy="3.14 0 0" />-->
+    <origin xyz="0.338 0.288 0.223" rpy="3.14 0 0.79" /> <!-- Scanners on the side -->
+  </xacro:sick_laser_v0>
+  <xacro:sick_laser_v0 name="lidar_2" parent="base_link" ros_topic="lidar_2/scan_filtered">
+  <!--<origin xyz="-0.360 0 0.181" rpy="3.14 0 3.14" />-->
+    <origin xyz="-0.338 -0.288 0.223" rpy="3.14 0 3.93" /> <!-- Scanners on the side -->
+  </xacro:sick_laser_v0>
+     <!--+++++++++++++++++++ IMU ++++++++++++++++++++++++-->
+ <!-- Comment or uncomment based on your requirement -->
+<!--   <xacro:imu name="imu_1" parent="base_link">
+    <origin xyz="0.100 0 0.300" rpy="0 0 3.14" />
+  </xacro:imu> -->
+  <!--+++++++++++++++++++ Ultra Sonic ++++++++++++++++++++++++-->
+  <!-- Comment or uncomment based on your requirement -->
+  <!-- SENSOR 1 -->
+  <!-- xacro:us_sensor name="us_1" parent="base_link">
+    <origin xyz="0.100 0 0.300" rpy="0 3.14 3.14" />
+  </xacro:us_sensor-->
+  <!-- SENSOR 2 -->
+  <!-- xacro:us_sensor name="us_2" parent="base_link">
+    <origin xyz="0.110 0 0.300" rpy="0 3.14 3.14" />
+  </xacro:us_sensor-->
+  <!-- SENSOR 3 -->
+  <!-- xacro:us_sensor name="us_3" parent="base_link">
+    <origin xyz="0.120 0 0.300" rpy="0 3.14 3.14" />
+  </xacro:us_sensor-->
+  <!-- SENSOR 4 -->
+  <!-- xacro:us_sensor name="us_4" parent="base_link">
+    <origin xyz="0.130 0 0.300" rpy="0 3.14 3.14" />
+  </xacro:us_sensor-->
+  <!-- SENSOR 5 -->
+  <!-- xacro:us_sensor name="us_5" parent="base_link">
+    <origin xyz="0.140 0 0.300" rpy="0 3.14 3.14" />
+  </xacro:us_sensor-->
+  <!-- SENSOR 6 -->
+  <!-- xacro:us_sensor name="us_6" parent="base_link">
+    <origin xyz="0.150 0 0.300" rpy="0 3.14 3.14" />
+  </xacro:us_sensor-->
+  <!-- SENSOR 7 -->
+  <!-- xacro:us_sensor name="us_7" parent="base_link">
+    <origin xyz="0.160 0 0.300" rpy="0 3.14 3.14" />
+  </xacro:us_sensor-->
+  <!-- SENSOR 8 -->
+  <!-- xacro:us_sensor name="us_8" parent="base_link">
+    <origin xyz="0.170 0 0.300" rpy="0 3.14 3.14" />
+  </xacro:us_sensor-->
+  <!-- SENSOR 9 -->
+  <!-- xacro:us_sensor name="us_9" parent="base_link">
+    <origin xyz="0.180 0 0.300" rpy="0 3.14 3.14" />
+  </xacro:us_sensor-->
+  <!-- SENSOR 10 -->
+  <!-- xacro:us_sensor name="us_10" parent="base_link">
+    <origin xyz="0.100 0 0.300" rpy="0 3.14 3.14" />
+  </xacro:us_sensor-->
+  <!-- SENSOR 11 -->
+  <!-- xacro:us_sensor name="us_11" parent="base_link">
+    <origin xyz="0.100 0 0.300" rpy="0 3.14 3.14" />
+  </xacro:us_sensor-->
+  <!-- SENSOR 12 -->
+  <!-- xacro:us_sensor name="us_12" parent="base_link">
+    <origin xyz="0.190 0 0.300" rpy="0 3.14 3.14" />
+  </xacro:us_sensor-->
+  <!-- SENSOR 13 -->
+  <!-- xacro:us_sensor name="us_13" parent="base_link">
+    <origin xyz="0.200 0 0.300" rpy="0 3.14 3.14" />
+  </xacro:us_sensor-->
+  <!-- SENSOR 14 -->
+  <!-- xacro:us_sensor name="us_14" parent="base_link">
+    <origin xyz="0.210 0 0.300" rpy="0 3.14 3.14" />
+  </xacro:us_sensor-->
+  <!-- SENSOR 15 -->
+  <!-- xacro:us_sensor name="us_15" parent="base_link">
+    <origin xyz="0.220 0 0.300" rpy="0 3.14 3.14" />
+  </xacro:us_sensor-->
+  <!-- SENSOR 16 -->
+  <!-- xacro:us_sensor name="us_16" parent="base_link">
+    <origin xyz="0.230 0 0.300" rpy="0 3.14 3.14" />
+  </xacro:us_sensor-->
+      <!--Camera  -->
+<!-- <xacro:camera name="camera" parent="base_link">
+    <origin xyz="0 0 0.38" rpy="0 0 0" />
+  </xacro:camera>
+ -->
 </robot>
