Commit message: Dummy link issue resolved and neo local planners updated

File: robots/mpo_700/mpo_700.urdf.xacro (robot description, xacro)
@@ -20,6 +20,8 @@
   <!-- Wheels -->
   <xacro:include filename="$(find neo_simulation)/robots/mpo_700/xacros/mpo_700_wheel.xacro" />
+  <link name="dummy_link" />
   <!-- Base Macro-->
-  <xacro:mpo_700_base name="base_link">
+  <xacro:mpo_700_base name="base_link" parent="dummy_link">
+    <origin xyz="0 0 0" rpy="0 0 0" />
   </xacro:mpo_700_base>
 <xacro:mpo_700_caster_0 name="mpo_700_caster_front_left" parent="base_link">

File: robots/mpo_700/xacros/camera.xacro (robot description, xacro)
@@ -4,5 +4,5 @@
     <joint name="${name}_joint" type="fixed">
       <axis xyz="0 1 0" />
-      <xacro:insert_block name="origin" />
+      <insert_block name="origin" />
       <parent link="${parent}"/>
       <child link="${name}_link"/>

File: robots/mpo_700/xacros/imu.xacro (robot description, xacro)
@@ -4,5 +4,5 @@
     <joint name="${name}_joint" type="fixed">
       <axis xyz="0 1 0" />
-      <xacro:insert_block name="origin" />
+      <insert_block name="origin" />
       <parent link="${parent}"/>
       <child link="${name}_link"/>

File: robots/mpo_700/xacros/micro_scan.xacro (robot description, xacro)
@@ -4,5 +4,5 @@
     <joint name="${name}_joint" type="fixed">
       <axis xyz="0 1 0" />
-      <xacro:insert_block name="origin" />
+      <insert_block name="origin" />
       <parent link="${parent}"/>
       <child link="${name}_link"/>

File: robots/mpo_700/xacros/mpo_700_body.xacro (robot description, xacro)
@@ -1,5 +1,13 @@
 <?xml version="1.0"?>
 <robot xmlns:xacro="http://www.ros.org/wiki/xacro" name="mpo_700">
-  <xacro:macro name="mpo_700_base" params="name">
+  <xacro:macro name="mpo_700_base" params="name parent *origin">
+   <joint name="${name}_joint" type="fixed">
+    <insert_block name="origin" />
+    <axis xyz="0 0 -1" />
+    <!-- <limit effort="1000.0" lower="-1e+16" upper="1e+16" velocity="3.5"/> -->
+    <joint_properties damping="1" friction="1" />
+    <parent link="${parent}" />
+    <child link="${name}" />
+   </joint>
     <link name="${name}">
       <inertial>

File: robots/mpo_700/xacros/mpo_700_caster.xacro (robot description, xacro)
@@ -3,5 +3,5 @@
   <xacro:macro name="mpo_700_caster_0" params="name parent *origin">
    <joint name="${name}_joint" type="fixed">
-    <xacro:insert_block name="origin" />
+    <insert_block name="origin" />
     <axis xyz="0 0 -1" />
     <!-- <limit effort="1000.0" lower="-1e+16" upper="1e+16" velocity="3.5"/> -->
@@ -32,5 +32,5 @@
   <xacro:macro name="mpo_700_caster_1" params="name parent *origin">
    <joint name="${name}_joint" type="fixed">
-    <xacro:insert_block name="origin" />
+    <insert_block name="origin" />
     <axis xyz="0 0 -1" />
     <joint_properties damping="1" friction="1" />
@@ -60,5 +60,5 @@
   <xacro:macro name="mpo_700_caster_2" params="name parent *origin">
    <joint name="${name}_joint" type="fixed">
-    <xacro:insert_block name="origin" />
+    <insert_block name="origin" />
     <axis xyz="0 0 -1" />
     <joint_properties damping="1" friction="1" />
@@ -88,5 +88,5 @@
   <xacro:macro name="mpo_700_caster_3" params="name parent *origin">
    <joint name="${name}_joint" type="fixed">
-    <xacro:insert_block name="origin" />
+    <insert_block name="origin" />
     <axis xyz="0 0 -1" />
     <joint_properties damping="1" friction="1" />

File: robots/mpo_700/xacros/mpo_700_wheel.xacro (robot description, xacro)
@@ -3,5 +3,5 @@
   <xacro:macro name="mpo_700_wheel" params="name parent *origin">
    <joint name="${name}_joint" type="fixed">
-    <xacro:insert_block name="origin" />
+    <insert_block name="origin" />
     <limit effort="1000.0" lower="-1e+16" upper="1e+16" velocity="3.5"/>
     <axis xyz="1 0 0" />

File: robots/mpo_700/xacros/sick_S300.xacro (robot description, xacro)
@@ -4,5 +4,5 @@
     <joint name="${name}_joint" type="fixed">
       <axis xyz="0 1 0" />
-      <xacro:insert_block name="origin" />
+      <insert_block name="origin" />
       <parent link="${parent}"/>
       <child link="${name}_link"/>

File: robots/mpo_700/xacros/ultrasonic.xacro (robot description, xacro)
@@ -4,5 +4,5 @@
     <joint name="${name}_joint" type="fixed">
       <axis xyz="0 1 0" />
-      <xacro:insert_block name="origin" />
+      <insert_block name="origin" />
       <parent link="${parent}"/>
       <child link="${name}_link"/>

Commit message: Missing camera xacros added

File: robots/mpo_700/mpo_700.urdf.xacro (robot description, xacro)
@@ -8,4 +8,6 @@
   <!-- Microscan - Comment/Uncomment if required -->
   <xacro:include filename="$(find neo_simulation)/robots/mpo_700/xacros/micro_scan.xacro" />
+  <!-- Depth camera -->
+  <!-- <xacro:include filename="$(find neo_simulation)/robots/mpo_700/xacros/depth_camera.xacro" />  -->
   <!--Ultrasonics, cameras and IMU's  -->
   <!-->
@@ -20,19 +22,19 @@
   <!-- Wheels -->
   <xacro:include filename="$(find neo_simulation)/robots/mpo_700/xacros/mpo_700_wheel.xacro" />
-  <link name="dummy_link" />
+  <link name="base_link" />
   <!-- Base Macro-->
-  <xacro:mpo_700_base name="base_link" parent="dummy_link">
+  <xacro:mpo_700_base name="base_footprint" parent="base_link">
     <origin xyz="0 0 0" rpy="0 0 0" />
   </xacro:mpo_700_base>
-<xacro:mpo_700_caster_0 name="mpo_700_caster_front_left" parent="base_link">
+<xacro:mpo_700_caster_0 name="mpo_700_caster_front_left" parent="base_footprint">
     <origin xyz="0.24 0.18 0.27" rpy="3.14 0 -1.57" />
   </xacro:mpo_700_caster_0>
-<xacro:mpo_700_caster_1 name="mpo_700_caster_front_right" parent="base_link">
+<xacro:mpo_700_caster_1 name="mpo_700_caster_front_right" parent="base_footprint">
     <origin xyz="0.24 -0.18 0.27" rpy="3.14 0 1.57" />
   </xacro:mpo_700_caster_1>
-<xacro:mpo_700_caster_2 name="mpo_700_caster_back_left" parent="base_link">
+<xacro:mpo_700_caster_2 name="mpo_700_caster_back_left" parent="base_footprint">
     <origin xyz="-0.24 0.18 0.27" rpy="3.14 0 -1.57" />
   </xacro:mpo_700_caster_2>
-<xacro:mpo_700_caster_3 name="mpo_700_caster_back_right" parent="base_link">
+<xacro:mpo_700_caster_3 name="mpo_700_caster_back_right" parent="base_footprint">
     <origin xyz="-0.24 -0.18 0.27" rpy="3.14 0 1.57" />
   </xacro:mpo_700_caster_3>
@@ -139,3 +141,7 @@
   </xacro:camera>
   <-->
+  <!-- Depth Camera -->
+<!--   <xacro:depth_camera name="camera" parent="base_link">
+    <origin xyz="0.228 0 0.461" rpy="0 0 0" />
+  </xacro:depth_camera> -->
 </robot>

File: robots/mpo_700/xacros/mpo_700_gazebo.xacro (robot description, xacro)
@@ -99,5 +99,5 @@
       <odometryTopic>odom</odometryTopic>
       <odometryFrame>odom</odometryFrame>
-      <odometryRate>20.0</odometryRate>
+      <odometryRate>100.0</odometryRate>
       <robotBaseFrame>base_link</robotBaseFrame>
     </plugin>

Commit message: Virtual wheel controller and the kinematics for MPO-700 are available

File: robots/mpo_700/mpo_700.urdf.xacro (robot description, xacro)
@@ -19,5 +19,6 @@
   <xacro:include filename="$(find neo_simulation)/robots/mpo_700/xacros/mpo_700_gazebo.xacro" />
   <!--Caster  -->
-  <xacro:include filename="$(find neo_simulation)/robots/mpo_700/xacros/mpo_700_caster.xacro" />
+  <xacro:include filename="$(find neo_simulation)/robots/mpo_700/xacros/mpo_700_caster_left.xacro" />
+  <xacro:include filename="$(find neo_simulation)/robots/mpo_700/xacros/mpo_700_caster_right.xacro" />
   <!-- Wheels -->
   <xacro:include filename="$(find neo_simulation)/robots/mpo_700/xacros/mpo_700_wheel.xacro" />
@@ -27,36 +28,38 @@
     <origin xyz="0 0 0" rpy="0 0 0" />
   </xacro:mpo_700_base>
-<xacro:mpo_700_caster_0 name="mpo_700_caster_front_left" parent="base_footprint">
-    <origin xyz="0.24 0.18 0.27" rpy="3.14 0 -1.57" />
-  </xacro:mpo_700_caster_0>
-<xacro:mpo_700_caster_1 name="mpo_700_caster_front_right" parent="base_footprint">
-    <origin xyz="0.24 -0.18 0.27" rpy="3.14 0 1.57" />
-  </xacro:mpo_700_caster_1>
-<xacro:mpo_700_caster_2 name="mpo_700_caster_back_left" parent="base_footprint">
-    <origin xyz="-0.24 0.18 0.27" rpy="3.14 0 -1.57" />
-  </xacro:mpo_700_caster_2>
-<xacro:mpo_700_caster_3 name="mpo_700_caster_back_right" parent="base_footprint">
-    <origin xyz="-0.24 -0.18 0.27" rpy="3.14 0 1.57" />
-  </xacro:mpo_700_caster_3>
-<xacro:mpo_700_wheel name="mpo_700_wheel_front_left" parent="mpo_700_caster_front_left_link">
-    <origin xyz="-0.05 0. 0.18" rpy="0 0 0" />
-  </xacro:mpo_700_wheel>
-<xacro:mpo_700_wheel name="mpo_700_wheel_front_right" parent="mpo_700_caster_front_right_link">
-    <origin xyz="-0.05 0. 0.18" rpy="0 0 0" />
-  </xacro:mpo_700_wheel>
-<xacro:mpo_700_wheel name="mpo_700_wheel_back_left" parent="mpo_700_caster_back_left_link">
-    <origin xyz="-0.05 0. 0.18" rpy="0 0 0" />
-  </xacro:mpo_700_wheel>
-<xacro:mpo_700_wheel name="mpo_700_wheel_back_right" parent="mpo_700_caster_back_right_link">
-    <origin xyz="-0.05 0. 0.18" rpy="0 0 0" />
+  <!--Caster Macro  -->
+  <xacro:mpo_700_caster_left name="mpo_700_caster_front_left" parent="base_footprint">
+    <origin xyz="0.24 0.18 0.22" rpy="0 0 3.14" />
+  </xacro:mpo_700_caster_left>
+  <xacro:mpo_700_caster_right name="mpo_700_caster_front_right" parent="base_footprint">
+    <origin xyz="0.24 -0.18 0.22" rpy="0 0 0" />
+  </xacro:mpo_700_caster_right>
+  <xacro:mpo_700_caster_left name="mpo_700_caster_back_left" parent="base_footprint">
+    <origin xyz="-0.24 0.18 0.22" rpy="0 0 3.14" />
+  </xacro:mpo_700_caster_left>
+  <xacro:mpo_700_caster_right name="mpo_700_caster_back_right" parent="base_footprint">
+    <origin xyz="-0.24 -0.18 0.22" rpy="0 0 0" />
+  </xacro:mpo_700_caster_right>
+  <!--Wheel Macro  -->
+  <xacro:mpo_700_wheel name="mpo_700_wheel_front_left" parent="mpo_700_caster_front_left_link">
+    <origin xyz="0.0 0.045 -0.12" rpy="0 0 0" />
+  </xacro:mpo_700_wheel>
+  <xacro:mpo_700_wheel name="mpo_700_wheel_front_right" parent="mpo_700_caster_front_right_link">
+    <origin xyz="0.0 -0.045 -0.12" rpy="0 0 3.14" />
+  </xacro:mpo_700_wheel>
+  <xacro:mpo_700_wheel name="mpo_700_wheel_back_left" parent="mpo_700_caster_back_left_link">
+      <origin xyz="0.0 0.045 -0.12" rpy="0 0 0" />
+  </xacro:mpo_700_wheel>
+  <xacro:mpo_700_wheel name="mpo_700_wheel_back_right" parent="mpo_700_caster_back_right_link">
+    <origin xyz="0.0 -0.045 -0.12" rpy="0 0 3.14" />
   </xacro:mpo_700_wheel>
 <!-- Sensors -->
   <!-- Lidar sensors -->
   <xacro:sick_laser_v0 name="lidar_1" parent="base_link" ros_topic="lidar_1/scan_filtered">
-  <!--<origin xyz="0.360 0 0.181" rpy="3.14 0 0" />-->
+  <!--<origin xyz="0.360 0 0.181" rpy="3.14 0 0" />--> <!-- Scanners on the front  -->
     <origin xyz="0.338 0.288 0.223" rpy="3.14 0 0.79" /> <!-- Scanners on the side -->
   </xacro:sick_laser_v0>
   <xacro:sick_laser_v0 name="lidar_2" parent="base_link" ros_topic="lidar_2/scan_filtered">
-  <!--<origin xyz="-0.360 0 0.181" rpy="3.14 0 3.14" />-->
+  <!--<origin xyz="-0.360 0 0.181" rpy="3.14 0 3.14" />--> <!-- Scanners on the rear -->
     <origin xyz="-0.338 -0.288 0.223" rpy="3.14 0 3.93" /> <!-- Scanners on the side -->
   </xacro:sick_laser_v0>
@@ -145,3 +148,75 @@
     <origin xyz="0.228 0 0.461" rpy="0 0 0" />
   </xacro:depth_camera> -->
+  <transmission name="mpo_700_caster_front_left">
+    <type>transmission_interface/SimpleTransmission</type>
+    <joint name="mpo_700_caster_front_left_joint">
+      <hardwareInterface>hardware_interface/PositionJointInterface</hardwareInterface>
+    </joint>
+    <actuator name="mpo_700_caster_front_left_motor">
+      <mechanicalReduction>1</mechanicalReduction>
+    </actuator>
+  </transmission>
+  <transmission name="mpo_700_wheel_front_left">
+    <type>transmission_interface/SimpleTransmission</type>
+    <joint name="mpo_700_wheel_front_left_joint">
+      <hardwareInterface>hardware_interface/VelocityJointInterface</hardwareInterface>
+    </joint>
+    <actuator name="mpo_700_wheel_front_left_motor">
+      <mechanicalReduction>1</mechanicalReduction>
+    </actuator>
+  </transmission>
+  <transmission name="mpo_700_caster_back_left">
+    <type>transmission_interface/SimpleTransmission</type>
+    <joint name="mpo_700_caster_back_left_joint">
+      <hardwareInterface>hardware_interface/PositionJointInterface</hardwareInterface>
+    </joint>
+    <actuator name="mpo_700_caster_back_left_motor">
+      <mechanicalReduction>1</mechanicalReduction>
+    </actuator>
+  </transmission>
+  <transmission name="mpo_700_wheel_back_right">
+    <type>transmission_interface/SimpleTransmission</type>
+    <joint name="mpo_700_wheel_back_right_joint">
+      <hardwareInterface>hardware_interface/VelocityJointInterface</hardwareInterface>
+    </joint>
+    <actuator name="mpo_700_wheel_back_right_motor">
+      <mechanicalReduction>1</mechanicalReduction>
+    </actuator>
+  </transmission>
+  <transmission name="mpo_700_caster_back_right">
+    <type>transmission_interface/SimpleTransmission</type>
+    <joint name="mpo_700_caster_back_right_joint">
+      <hardwareInterface>hardware_interface/PositionJointInterface</hardwareInterface>
+    </joint>
+    <actuator name="mpo_700_caster_back_right_motor">
+      <mechanicalReduction>1</mechanicalReduction>
+    </actuator>
+  </transmission>
+  <transmission name="mpo_700_wheel_front_right">
+    <type>transmission_interface/SimpleTransmission</type>
+    <joint name="mpo_700_wheel_front_right_joint">
+      <hardwareInterface>hardware_interface/VelocityJointInterface</hardwareInterface>
+    </joint>
+    <actuator name="mpo_700_wheel_front_right_motor">
+      <mechanicalReduction>1</mechanicalReduction>
+    </actuator>
+  </transmission>
+  <transmission name="mpo_700_caster_front_right">
+    <type>transmission_interface/SimpleTransmission</type>
+    <joint name="mpo_700_caster_front_right_joint">
+      <hardwareInterface>hardware_interface/PositionJointInterface</hardwareInterface>
+    </joint>
+    <actuator name="mpo_700_caster_front_right_motor">
+      <mechanicalReduction>1</mechanicalReduction>
+    </actuator>
+  </transmission>
+  <transmission name="mpo_700_wheel_back_left">
+    <type>transmission_interface/SimpleTransmission</type>
+    <joint name="mpo_700_wheel_back_left_joint">
+      <hardwareInterface>hardware_interface/VelocityJointInterface</hardwareInterface>
+    </joint>
+    <actuator name="mpo_700_wheel_front_left_motor">
+      <mechanicalReduction>1</mechanicalReduction>
+    </actuator>
+  </transmission>
 </robot>

File: robots/mpo_700/xacros/mpo_700_body.xacro (robot description, xacro)
@@ -11,11 +11,11 @@
    </joint>
     <link name="${name}">
-      <inertial>
-        <mass value="0.01" />
-        <origin xyz="0 0 0" rpy="0 0 0"/>
-        <inertia ixx="0.0008" ixy="0.0" ixz="0.0"
-                 iyy="0.0008" iyz="0.0"
-                 izz="0.0008" />
-      </inertial>
+    <inertial>
+      <mass value="90"/>
+      <origin xyz="0 0 0"/>
+      <inertia ixx="7.8" ixy="0.0" ixz="0"
+               iyy="7.8" iyz="0.0"
+               izz="7.8"/>
+    </inertial>
       <visual>
         <origin xyz="0.0 0.0 0.0" rpy="0 0 -1.571" />

File: robots/mpo_700/xacros/mpo_700_gazebo.xacro (robot description, xacro)
@@ -5,4 +5,10 @@
     <self_collide>false</self_collide>
   </gazebo>
+<gazebo>
+  <plugin name="ros_control" filename="libgazebo_ros_control.so">
+    <legacyModeNS>false</legacyModeNS>
+    <robotSimType>gazebo_ros_control/DefaultRobotHWSim</robotSimType>
+  </plugin>
+</gazebo>
   <gazebo reference="lidar_1_link">
       <sensor type="ray" name="lidar_1_sensor">

File: robots/mpo_700/xacros/mpo_700_wheel.xacro (robot description, xacro)
@@ -2,9 +2,9 @@
 <robot xmlns:xacro="http://www.ros.org/wiki/xacro" name="mpo_700">
   <xacro:macro name="mpo_700_wheel" params="name parent *origin">
-   <joint name="${name}_joint" type="fixed">
+   <joint name="${name}_joint" type="revolute">
     <insert_block name="origin" />
-    <limit effort="1000.0" lower="-1e+16" upper="1e+16" velocity="3.5"/>
-    <axis xyz="1 0 0" />
-    <joint_properties damping="1" friction="1" />
+    <limit effort="1000.0" lower="-1e+16" upper="1e+16" velocity="20.5"/>
+    <axis xyz="0 -1 0" />
+    <joint_properties damping="30" friction="110"/>
     <parent link="${parent}" />
     <child link="${name}_link" />
@@ -12,12 +12,12 @@
    <link name="${name}_link" type="wheel">
     <inertial>
-      <mass value="0.0006" />
-      <origin xyz="0 0 0" rpy="0 0 0" />
-        <inertia  ixx="0.04" ixy="0.000" ixz="0.0"
-                  iyy="0.02" iyz="0.00"
-                  izz="0.05" />
+      <mass value="1.2"/>
+      <origin rpy="0 0 0" xyz="0 0 0"/>
+      <inertia ixx="0.11042056" ixy="0.0" ixz="0.0"
+               iyy="0.11042056" iyz="0.0"
+               izz="0.11042056"/>
     </inertial>
     <visual>
-     <origin xyz="0 0 0" rpy="0 0 0"/>
+     <origin xyz="0 0 0" rpy="0 0 3.14"/>
      <geometry>
         <mesh filename="package://neo_simulation/robots/mpo_700/meshes/MPO-700-WHEEL.dae" scale="0.001 0.001 0.001"/>

Commit message: Added docking adapter to the MPO-700 simulation model

File: robots/mpo_700/mpo_700.urdf.xacro (robot description, xacro)
@@ -16,4 +16,5 @@
   <xacro:include filename="$(find neo_simulation)/robots/mpo_700/xacros/ultrasonic.xacro" />
   <-->
+  <xacro:include filename="$(find neo_simulation)/robots/mpo_700/xacros/docking_adapter.xacro" />
   <!--Gazebo  -->
   <xacro:include filename="$(find neo_simulation)/robots/mpo_700/xacros/mpo_700_gazebo.xacro" />
@@ -64,4 +65,7 @@
     <origin xyz="-0.338 -0.288 0.223" rpy="3.14 0 3.93" /> <!-- Scanners on the side -->
   </xacro:sick_laser_v0>
+  <xacro:docking_adapter name="docking_adapter" parent="base_link">
+    <origin xyz="0.300 0 0.320" rpy="0 0 1.57" />
+  </xacro:docking_adapter>
      <!--+++++++++++++++++++ IMU ++++++++++++++++++++++++-->
   <!-- Comment or uncomment based on your requirement -->
