Commit message: Changes are updated for a perfect docking

File: robots/mpo_700/mpo_700.urdf.xacro (robot description, xacro)
@@ -66,5 +66,5 @@
   </xacro:sick_laser_v0>
   <xacro:docking_adapter name="docking_adapter" parent="base_link">
-    <origin xyz="0.300 0 0.320" rpy="0 0 1.57" />
+    <origin xyz="-0.300 0 0.320" rpy="0 0 -1.57" />
   </xacro:docking_adapter>
      <!--+++++++++++++++++++ IMU ++++++++++++++++++++++++-->
@@ -150,5 +150,5 @@
   <!-- Depth Camera -->
   <xacro:depth_camera name="camera" parent="base_link">
-    <origin xyz="0.228 0 0.461" rpy="0 0 0" />
+    <origin xyz="-0.228 0.015 0.461" rpy="0 0 3.14159" />
   </xacro:depth_camera>
   <transmission name="mpo_700_caster_front_left">

File: robots/mpo_700/xacros/depth_camera.xacro (robot description, xacro)
@@ -5,12 +5,17 @@
 		    <joint name="${name}_joint" type="fixed">
 		      <axis xyz="0 1 0" />
-		      <xacro:insert_block name="origin" />
+		      <insert_block name="origin" />
 		      <parent link="${parent}"/>
 		      <child link="${name}_link"/>
 		    </joint>
 		    <joint name="${name}_optical_joint" type="fixed">
-		    	<origin xyz="0 0 0" rpy="${-pi/2} 0 ${-pi/2}"/>
+		    	<origin xyz="0 0.015 0" rpy="${-pi/2} 0 ${-pi/2}"/>
 		    	<parent link="${name}_link"/>
 		    	<child link="${name}_link_optical"/>
+		    </joint>
+		    <joint name="${name}_gazebo_joint" type="fixed">
+		    	<origin xyz="0 0.015 0" rpy="0 0 0"/>
+		    	<parent link="${name}_link"/>
+		    	<child link="${name}_link_gazebo"/>
 		    </joint>
 		    <link name="${name}_link">
@@ -24,5 +29,5 @@
 			      <origin xyz="0 -0.0175 0" rpy="1.570796 0 1.570796"/>
 			      <geometry>
-			      	<mesh filename="package://neo_simulation/robots/mpo_700/meshes/d435.dae"/>
+			      	<mesh filename="package://neo_mpo_700/robot_model/mpo_700/meshes/d435.dae"/>
 			      </geometry>
 			      <material name="red">
@@ -38,4 +43,5 @@
 		    <link  name="${name}_link_optical">
 		    </link>
+		    <link name="${name}_link_gazebo" />
 	</xacro:macro>
 </robot>

File: robots/mpo_700/xacros/mpo_700_body.xacro (robot description, xacro)
@@ -12,5 +12,5 @@
     <link name="${name}">
     <inertial>
-      <mass value="90"/>
+      <mass value="140"/>
       <origin xyz="0 0 0"/>
       <inertia ixx="7.8" ixy="0.0" ixz="0"

File: robots/mpo_700/xacros/mpo_700_gazebo.xacro (robot description, xacro)
@@ -5,10 +5,4 @@
     <self_collide>false</self_collide>
   </gazebo>
-<gazebo>
-  <plugin name="ros_control" filename="libgazebo_ros_control.so">
-    <legacyModeNS>false</legacyModeNS>
-    <robotSimType>gazebo_ros_control/DefaultRobotHWSim</robotSimType>
-  </plugin>
-</gazebo>
   <gazebo reference="lidar_1_link">
       <sensor type="ray" name="lidar_1_sensor">
@@ -37,5 +31,5 @@
                    reading. -->
               <mean>0.0</mean>
-              <stddev>0.0</stddev>
+              <stddev>0.01</stddev>
             </noise>
           </ray>
@@ -46,4 +40,10 @@
         </sensor>
   </gazebo>
+<gazebo>
+  <plugin name="ros_control" filename="libgazebo_ros_control.so">
+    <legacyModeNS>false</legacyModeNS>
+    <robotSimType>gazebo_ros_control/DefaultRobotHWSim</robotSimType>
+  </plugin>
+</gazebo>
   <gazebo reference="lidar_2_link">
       <sensor type="ray" name="lidar_2_sensor">
@@ -72,5 +72,5 @@
                    reading. -->
               <mean>0.0</mean>
-              <stddev>0.0</stddev>
+              <stddev>0.01</stddev>
             </noise>
           </ray>
@@ -105,47 +105,52 @@
       <odometryTopic>odom</odometryTopic>
       <odometryFrame>odom</odometryFrame>
-      <odometryRate>100.0</odometryRate>
+      <odometryRate>150.0</odometryRate>
       <robotBaseFrame>base_link</robotBaseFrame>
     </plugin>
   </gazebo>
   <!-- camera -->
-  <!-- Sonar -->
-  <gazebo reference="us_1_link">
-  <!-- Visuals / Collisions omitted for this example -->
-  <sensor type="ray" name="range">
-    <ray>
-         <scan>
-            <horizontal>
-               <samples>1</samples>
-               <resolution>1.0</resolution>
-               <min_angle>-0.01</min_angle>
-               <max_angle>0.01</max_angle>
-            </horizontal>
-            <vertical>
-               <samples>1</samples>
-               <resolution>1</resolution>
-               <min_angle>-0.01</min_angle>
-               <max_angle>0.01</max_angle>
-            </vertical>
-         </scan>
-         <range>
-            <min>0.01</min>
-            <max>3.75</max>
-            <resolution>0.02</resolution>
-         </range>
-      </ray>
-      <plugin filename="libgazebo_ros_range.so" name="gazebo_ros_range">
-	<gaussianNoise>0.005</gaussianNoise>
-	<alwaysOn>true</alwaysOn>
-	<updateRate>50</updateRate>
-	<topicName>ultrasonic/us1</topicName>
-	<frameName>us_1_link</frameName>
-	<radiation>INFRARED</radiation>
-	<fov>0.2967</fov>
-      </plugin>
-      </sensor>
-  </gazebo>
+  <!-->
   <gazebo reference="camera_link">
-    <sensor name="camera" type="depth">
+    <sensor type="camera" name="camera1">
+      <update_rate>30.0</update_rate>
+      <camera name="head">
+        <horizontal_fov>1.3962634</horizontal_fov>
+  <image>
+    <width>800</width>
+    <height>800</height>
+    <format>R8G8B8</format>
+  </image>
+        <clip>
+          <near>0.02</near>
+          <far>300</far>
+        </clip>
+        <noise>
+          <type>gaussian</type>
+           Noise is sampled independently per pixel on each frame.
+               That pixel's noise value is added to each of its color
+               channels, which at that point lie in the range [0,1].
+          <mean>0.0</mean>
+          <stddev>0.007</stddev>
+        </noise>
+      </camera>
+      <plugin name="camera_controller" filename="libgazebo_ros_camera.so">
+        <alwaysOn>true</alwaysOn>
+        <updateRate>0.0</updateRate>
+        <cameraName>robot/camera1</cameraName>
+        <imageTopicName>image_raw</imageTopicName>
+        <cameraInfoTopicName>camera_info</cameraInfoTopicName>
+        <frameName>camera_link</frameName>
+        <hackBaseline>0.07</hackBaseline>
+        <distortionK1>0.0</distortionK1>
+        <distortionK2>0.0</distortionK2>
+        <distortionK3>0.0</distortionK3>
+        <distortionT1>0.0</distortionT1>
+        <distortionT2>0.0</distortionT2>
+      </plugin>
+    </sensor>
+  </gazebo>
+  <-->
+  <gazebo reference="camera_link_gazebo">
+    <sensor name="camera1" type="depth">
       <update_rate>15</update_rate>
       <hfov>70</hfov>
@@ -195,3 +200,39 @@
     </sensor>
   </gazebo>
+  <!-- Sonar -->
+  <gazebo reference="us_1_link">
+  <!-- Visuals / Collisions omitted for this example -->
+  <sensor type="ray" name="range">
+    <ray>
+         <scan>
+            <horizontal>
+               <samples>1</samples>
+               <resolution>1.0</resolution>
+               <min_angle>-0.01</min_angle>
+               <max_angle>0.01</max_angle>
+            </horizontal>
+            <vertical>
+               <samples>1</samples>
+               <resolution>1</resolution>
+               <min_angle>-0.01</min_angle>
+               <max_angle>0.01</max_angle>
+            </vertical>
+         </scan>
+         <range>
+            <min>0.01</min>
+            <max>3.75</max>
+            <resolution>0.02</resolution>
+         </range>
+      </ray>
+      <plugin filename="libgazebo_ros_range.so" name="gazebo_ros_range">
+  <gaussianNoise>0.005</gaussianNoise>
+  <alwaysOn>true</alwaysOn>
+  <updateRate>50</updateRate>
+  <topicName>ultrasonic/us1</topicName>
+  <frameName>us_1_link</frameName>
+  <radiation>INFRARED</radiation>
+  <fov>0.2967</fov>
+      </plugin>
+      </sensor>
+  </gazebo>
 </robot>

File: robots/mpo_700/xacros/mpo_700_wheel.xacro (robot description, xacro)
@@ -4,5 +4,5 @@
    <joint name="${name}_joint" type="revolute">
     <insert_block name="origin" />
-    <limit effort="1000.0" lower="-1e+16" upper="1e+16" velocity="30.5"/>
+    <limit effort="1000.0" lower="-1e+16" upper="1e+16" velocity="20.5"/>
     <axis xyz="0 -1 0" />
     <joint_properties damping="30" friction="110"/>

Commit message: Docking adapter added

File: robots/mpo_700/mpo_700.urdf.xacro (robot description, xacro)
@@ -8,23 +8,27 @@
   <!-- Microscan - Comment/Uncomment if required -->
   <xacro:include filename="$(find neo_simulation)/robots/mpo_700/xacros/micro_scan.xacro" />
+  <!-- Depth camera -->
+  <xacro:include filename="$(find neo_simulation)/robots/mpo_700/xacros/depth_camera.xacro" />
   <!--Ultrasonics, cameras and IMU's  -->
-  <!-- <xacro:include filename="$(find neo_simulation)/robots/mpo_700/xacros/camera.xacro" /> -->
-  <!--<xacro:include filename="$(find neo_simulation)/robots/mpo_700/xacros/imu.xacro" />
-  <xacro:include filename="$(find neo_simulation)/robots/mpo_700/xacros/ultrasonic.xacro" /> -->
+  <!-->
+  <xacro:include filename="$(find neo_simulation)/robots/mpo_700/xacros/camera.xacro" />
+  <xacro:include filename="$(find neo_simulation)/robots/mpo_700/xacros/imu.xacro" />
+  <xacro:include filename="$(find neo_simulation)/robots/mpo_700/xacros/ultrasonic.xacro" />
+  <-->
+  <xacro:include filename="$(find neo_simulation)/robots/mpo_700/xacros/docking_adapter.xacro" />
   <!--Gazebo  -->
   <xacro:include filename="$(find neo_simulation)/robots/mpo_700/xacros/mpo_700_gazebo.xacro" />
   <!--Caster  -->
-  <xacro:include filename="$(find neo_simulation)/robots/mpo_700/xacros/mpo_700_caster.xacro" />
-    <xacro:include filename="$(find neo_simulation)/robots/mpo_700/xacros/mpo_700_caster_left.xacro" />
+  <xacro:include filename="$(find neo_simulation)/robots/mpo_700/xacros/mpo_700_caster_left.xacro" />
   <xacro:include filename="$(find neo_simulation)/robots/mpo_700/xacros/mpo_700_caster_right.xacro" />
   <!-- Wheels -->
   <xacro:include filename="$(find neo_simulation)/robots/mpo_700/xacros/mpo_700_wheel.xacro" />
-  <!-- Base Macro-->
-<link name="base_link" />
+  <link name="base_link" />
   <!-- Base Macro-->
   <xacro:mpo_700_base name="base_footprint" parent="base_link">
     <origin xyz="0 0 0" rpy="0 0 0" />
   </xacro:mpo_700_base>
- <xacro:mpo_700_caster_left name="mpo_700_caster_front_left" parent="base_footprint">
+  <!--Caster Macro  -->
+  <xacro:mpo_700_caster_left name="mpo_700_caster_front_left" parent="base_footprint">
     <origin xyz="0.24 0.18 0.22" rpy="0 0 3.14" />
   </xacro:mpo_700_caster_left>
@@ -52,23 +56,31 @@
   </xacro:mpo_700_wheel>
 <!-- Sensors -->
-  <xacro:sick_laser_v0 name="lidar_1" parent="base_footprint" ros_topic="lidar_1/scan_filtered">
-  <!--<origin xyz="0.360 0 0.181" rpy="3.14 0 0" />-->
+  <!-- Lidar sensors -->
+  <xacro:sick_laser_v0 name="lidar_1" parent="base_link" ros_topic="lidar_1/scan_filtered">
+  <!--<origin xyz="0.360 0 0.181" rpy="3.14 0 0" />--> <!-- Scanners on the front  -->
     <origin xyz="0.338 0.288 0.223" rpy="3.14 0 0.79" /> <!-- Scanners on the side -->
   </xacro:sick_laser_v0>
-  <xacro:sick_laser_v0 name="lidar_2" parent="base_footprint" ros_topic="lidar_2/scan_filtered">
-  <!--<origin xyz="-0.360 0 0.181" rpy="3.14 0 3.14" />-->
+  <xacro:sick_laser_v0 name="lidar_2" parent="base_link" ros_topic="lidar_2/scan_filtered">
+  <!--<origin xyz="-0.360 0 0.181" rpy="3.14 0 3.14" />--> <!-- Scanners on the rear -->
     <origin xyz="-0.338 -0.288 0.223" rpy="3.14 0 3.93" /> <!-- Scanners on the side -->
   </xacro:sick_laser_v0>
+  <xacro:docking_adapter name="docking_adapter" parent="base_link">
+    <origin xyz="-0.300 0 0.320" rpy="0 0 -1.57" />
+  </xacro:docking_adapter>
      <!--+++++++++++++++++++ IMU ++++++++++++++++++++++++-->
- <!-- Comment or uncomment based on your requirement -->
-<!--   <xacro:imu name="imu_1" parent="base_link">
-    <origin xyz="0.100 0 0.300" rpy="0 0 3.14" />
-  </xacro:imu> -->
+  <!-- Comment or uncomment based on your requirement -->
+  <!-->
+  <xacro:imu name="imu" parent="base_link">
+    <origin xyz="0.100 0 0.500" rpy="0 0 3.14" />
+  </xacro:imu>
+  <-->
   <!--+++++++++++++++++++ Ultra Sonic ++++++++++++++++++++++++-->
   <!-- Comment or uncomment based on your requirement -->
   <!-- SENSOR 1 -->
-  <!-- xacro:us_sensor name="us_1" parent="base_link">
-    <origin xyz="0.100 0 0.300" rpy="0 3.14 3.14" />
-  </xacro:us_sensor-->
+  <!-->
+  <xacro:us_sensor name="us_1" parent="base_link">
+    <origin xyz="0.100 0 0.500" rpy="0 3.14 3.14" />
+  </xacro:us_sensor>
+  <-->
   <!-- SENSOR 2 -->
   <!-- xacro:us_sensor name="us_2" parent="base_link">
@@ -131,9 +143,14 @@
     <origin xyz="0.230 0 0.300" rpy="0 3.14 3.14" />
   </xacro:us_sensor-->
-      <!--Camera  -->
-<!-- <xacro:camera name="camera" parent="base_link">
+  <!--Camera  -->
+  <!--><xacro:camera name="camera" parent="base_link">
     <origin xyz="0 0 0.38" rpy="0 0 0" />
-  </xacro:camera> -->
-   <transmission name="mpo_700_caster_front_left">
+  </xacro:camera>
+  <-->
+  <!-- Depth Camera -->
+  <xacro:depth_camera name="camera" parent="base_link">
+    <origin xyz="-0.228 0.015 0.461" rpy="0 0 3.14159" />
+  </xacro:depth_camera>
+  <transmission name="mpo_700_caster_front_left">
     <type>transmission_interface/SimpleTransmission</type>
     <joint name="mpo_700_caster_front_left_joint">

File: robots/mpo_700/xacros/depth_camera.xacro (robot description, xacro)
@@ -5,12 +5,17 @@
 		    <joint name="${name}_joint" type="fixed">
 		      <axis xyz="0 1 0" />
-		      <xacro:insert_block name="origin" />
+		      <insert_block name="origin" />
 		      <parent link="${parent}"/>
 		      <child link="${name}_link"/>
 		    </joint>
 		    <joint name="${name}_optical_joint" type="fixed">
-		    	<origin xyz="0 0 0" rpy="${-pi/2} 0 ${-pi/2}"/>
+		    	<origin xyz="0 0.015 0" rpy="${-pi/2} 0 ${-pi/2}"/>
 		    	<parent link="${name}_link"/>
 		    	<child link="${name}_link_optical"/>
+		    </joint>
+		    <joint name="${name}_gazebo_joint" type="fixed">
+		    	<origin xyz="0 0.015 0" rpy="0 0 0"/>
+		    	<parent link="${name}_link"/>
+		    	<child link="${name}_link_gazebo"/>
 		    </joint>
 		    <link name="${name}_link">
@@ -38,4 +43,5 @@
 		    <link  name="${name}_link_optical">
 		    </link>
+		    <link name="${name}_link_gazebo" />
 	</xacro:macro>
 </robot>

File: robots/mpo_700/xacros/mpo_700_gazebo.xacro (robot description, xacro)
@@ -5,10 +5,4 @@
     <self_collide>false</self_collide>
   </gazebo>
-<gazebo>
-  <plugin name="ros_control" filename="libgazebo_ros_control.so">
-    <legacyModeNS>false</legacyModeNS>
-    <robotSimType>gazebo_ros_control/DefaultRobotHWSim</robotSimType>
-  </plugin>
-</gazebo>
   <gazebo reference="lidar_1_link">
       <sensor type="ray" name="lidar_1_sensor">
@@ -37,5 +31,5 @@
                    reading. -->
               <mean>0.0</mean>
-              <stddev>0.0</stddev>
+              <stddev>0.01</stddev>
             </noise>
           </ray>
@@ -46,4 +40,10 @@
         </sensor>
   </gazebo>
+<gazebo>
+  <plugin name="ros_control" filename="libgazebo_ros_control.so">
+    <legacyModeNS>false</legacyModeNS>
+    <robotSimType>gazebo_ros_control/DefaultRobotHWSim</robotSimType>
+  </plugin>
+</gazebo>
   <gazebo reference="lidar_2_link">
       <sensor type="ray" name="lidar_2_sensor">
@@ -72,5 +72,5 @@
                    reading. -->
               <mean>0.0</mean>
-              <stddev>0.0</stddev>
+              <stddev>0.01</stddev>
             </noise>
           </ray>
@@ -105,9 +105,10 @@
       <odometryTopic>odom</odometryTopic>
       <odometryFrame>odom</odometryFrame>
-      <odometryRate>100.0</odometryRate>
+      <odometryRate>150.0</odometryRate>
       <robotBaseFrame>base_link</robotBaseFrame>
     </plugin>
   </gazebo>
   <!-- camera -->
+  <!-->
   <gazebo reference="camera_link">
     <sensor type="camera" name="camera1">
@@ -115,9 +116,9 @@
       <camera name="head">
         <horizontal_fov>1.3962634</horizontal_fov>
-	<image>
-	  <width>800</width>
- 	  <height>800</height>
-	  <format>R8G8B8</format>
-	</image>
+  <image>
+    <width>800</width>
+    <height>800</height>
+    <format>R8G8B8</format>
+  </image>
         <clip>
           <near>0.02</near>
@@ -126,7 +127,7 @@
         <noise>
           <type>gaussian</type>
-          <!-- Noise is sampled independently per pixel on each frame.
+           Noise is sampled independently per pixel on each frame.
                That pixel's noise value is added to each of its color
-               channels, which at that point lie in the range [0,1]. -->
+               channels, which at that point lie in the range [0,1].
           <mean>0.0</mean>
           <stddev>0.007</stddev>
@@ -146,4 +147,54 @@
         <distortionT1>0.0</distortionT1>
         <distortionT2>0.0</distortionT2>
+      </plugin>
+    </sensor>
+  </gazebo>
+  <-->
+  <gazebo reference="camera_link_gazebo">
+    <sensor name="camera1" type="depth">
+      <update_rate>15</update_rate>
+      <hfov>70</hfov>
+      <camera name="head">
+        <image>
+          <width>320</width>
+          <height>240</height>
+          <format>R8G8B8</format>
+        </image>
+        <clip>
+          <near>0.02</near>
+          <far>300</far>
+        </clip>
+        <noise>
+          <type>gaussian</type>
+          <!-- Noise is sampled independently per pixel on each frame.
+               That pixel's noise value is added to each of its color
+               channels, which at that point lie in the range [0,1]. -->
+          <mean>0.0</mean>
+          <stddev>0.03</stddev>
+        </noise>
+      </camera>
+      <plugin name="camera1_controller" filename="libgazebo_ros_openni_kinect.so">
+        <!--<baseline>0.2</baseline>-->
+        <alwaysOn>true</alwaysOn>
+        <updateRate>0.0</updateRate>
+        <cameraName>camera_ir</cameraName>
+        <imageTopicName>/camera/depth/image_raw</imageTopicName>
+        <cameraInfoTopicName>/camera/depth/camera_info</cameraInfoTopicName>
+        <depthImageTopicName>/camera/depth/depth_raw</depthImageTopicName>
+        <depthImageInfoTopicName>/camera/depth/camera_info</depthImageInfoTopicName>
+        <pointCloudTopicName>/camera/depth_registered/points</pointCloudTopicName>
+        <frameName>camera_link_optical</frameName>
+        <pointCloudCutoff>0.12</pointCloudCutoff>
+        <pointCloudCutoffMax>3.0</pointCloudCutoffMax>
+        <distortionK1>0.00000001</distortionK1>
+        <distortionK2>0.00000001</distortionK2>
+        <distortionK3>0.00000001</distortionK3>
+        <distortionT1>0.00000001</distortionT1>
+        <distortionT2>0.00000001</distortionT2>
+        <CxPrime>0</CxPrime>
+        <Cx>0</Cx>
+        <Cy>0</Cy>
+        <focalLength>0</focalLength>
+        <hackBaseline>0</hackBaseline>
       </plugin>
     </sensor>
@@ -175,11 +226,11 @@
       </ray>
       <plugin filename="libgazebo_ros_range.so" name="gazebo_ros_range">
-	<gaussianNoise>0.005</gaussianNoise>
-	<alwaysOn>true</alwaysOn>
-	<updateRate>50</updateRate>
-	<topicName>ultrasonic/us1</topicName>
-	<frameName>us_1_link</frameName>
-	<radiation>INFRARED</radiation>
-	<fov>0.2967</fov>
+  <gaussianNoise>0.005</gaussianNoise>
+  <alwaysOn>true</alwaysOn>
+  <updateRate>50</updateRate>
+  <topicName>ultrasonic/us1</topicName>
+  <frameName>us_1_link</frameName>
+  <radiation>INFRARED</radiation>
+  <fov>0.2967</fov>
       </plugin>
       </sensor>

File: robots/mpo_700/xacros/mpo_700_wheel.xacro (robot description, xacro)
@@ -27,5 +27,6 @@
      <origin xyz="0 0 0" rpy="0 0 0" />
      <geometry>
-        <mesh filename="package://neo_simulation/robots/mpo_700/meshes/MPO-700-WHEEL.dae" scale="0.001 0.001 0.001"/>
+      <sphere radius="0.09" />
+        <!-- <mesh filename="package://neo_simulation/robots/mpo_700/meshes/MPO-700-WHEEL.dae" scale="0.001 0.001 0.001"/> -->
      </geometry>
     </collision>
