Commit message: Depth camera model changed

File: robots/mpo_700/mpo_700.urdf.xacro (robot description, xacro)
@@ -8,27 +8,25 @@
   <!-- Microscan - Comment/Uncomment if required -->
   <xacro:include filename="$(find neo_simulation)/robots/mpo_700/xacros/micro_scan.xacro" />
-  <!-- Depth camera -->
-  <xacro:include filename="$(find neo_simulation)/robots/mpo_700/xacros/depth_camera.xacro" />
   <!--Ultrasonics, cameras and IMU's  -->
-  <!-->
-  <xacro:include filename="$(find neo_simulation)/robots/mpo_700/xacros/camera.xacro" />
-  <xacro:include filename="$(find neo_simulation)/robots/mpo_700/xacros/imu.xacro" />
-  <xacro:include filename="$(find neo_simulation)/robots/mpo_700/xacros/ultrasonic.xacro" />
-  <-->
-  <xacro:include filename="$(find neo_simulation)/robots/mpo_700/xacros/docking_adapter.xacro" />
+  <!-- <xacro:include filename="$(find neo_simulation)/robots/mpo_700/xacros/camera.xacro" /> -->
+  <!--<xacro:include filename="$(find neo_simulation)/robots/mpo_700/xacros/imu.xacro" />
+  <xacro:include filename="$(find neo_simulation)/robots/mpo_700/xacros/ultrasonic.xacro" /> -->
   <!--Gazebo  -->
   <xacro:include filename="$(find neo_simulation)/robots/mpo_700/xacros/mpo_700_gazebo.xacro" />
   <!--Caster  -->
-  <xacro:include filename="$(find neo_simulation)/robots/mpo_700/xacros/mpo_700_caster_left.xacro" />
+  <xacro:include filename="$(find neo_simulation)/robots/mpo_700/xacros/mpo_700_caster.xacro" />
+    <xacro:include filename="$(find neo_simulation)/robots/mpo_700/xacros/mpo_700_caster_left.xacro" />
   <xacro:include filename="$(find neo_simulation)/robots/mpo_700/xacros/mpo_700_caster_right.xacro" />
   <!-- Wheels -->
   <xacro:include filename="$(find neo_simulation)/robots/mpo_700/xacros/mpo_700_wheel.xacro" />
-  <link name="base_link" />
+  <!-- Depth camera -->
+  <xacro:include filename="$(find neo_simulation)/robots/mpo_700/xacros/depth_camera.xacro" />
+  <!-- Base Macro-->
+<link name="base_link" />
   <!-- Base Macro-->
   <xacro:mpo_700_base name="base_footprint" parent="base_link">
     <origin xyz="0 0 0" rpy="0 0 0" />
   </xacro:mpo_700_base>
-  <!--Caster Macro  -->
-  <xacro:mpo_700_caster_left name="mpo_700_caster_front_left" parent="base_footprint">
+ <xacro:mpo_700_caster_left name="mpo_700_caster_front_left" parent="base_footprint">
     <origin xyz="0.24 0.18 0.22" rpy="0 0 3.14" />
   </xacro:mpo_700_caster_left>
@@ -56,31 +54,23 @@
   </xacro:mpo_700_wheel>
 <!-- Sensors -->
-  <!-- Lidar sensors -->
-  <xacro:sick_laser_v0 name="lidar_1" parent="base_link" ros_topic="lidar_1/scan_filtered">
-  <!--<origin xyz="0.360 0 0.181" rpy="3.14 0 0" />--> <!-- Scanners on the front  -->
+  <xacro:sick_laser_v0 name="lidar_1" parent="base_footprint" ros_topic="lidar_1/scan_filtered">
+  <!--<origin xyz="0.360 0 0.181" rpy="3.14 0 0" />-->
     <origin xyz="0.338 0.288 0.223" rpy="3.14 0 0.79" /> <!-- Scanners on the side -->
   </xacro:sick_laser_v0>
-  <xacro:sick_laser_v0 name="lidar_2" parent="base_link" ros_topic="lidar_2/scan_filtered">
-  <!--<origin xyz="-0.360 0 0.181" rpy="3.14 0 3.14" />--> <!-- Scanners on the rear -->
+  <xacro:sick_laser_v0 name="lidar_2" parent="base_footprint" ros_topic="lidar_2/scan_filtered">
+  <!--<origin xyz="-0.360 0 0.181" rpy="3.14 0 3.14" />-->
     <origin xyz="-0.338 -0.288 0.223" rpy="3.14 0 3.93" /> <!-- Scanners on the side -->
   </xacro:sick_laser_v0>
-  <xacro:docking_adapter name="docking_adapter" parent="base_link">
-    <origin xyz="-0.300 0 0.320" rpy="0 0 -1.57" />
-  </xacro:docking_adapter>
      <!--+++++++++++++++++++ IMU ++++++++++++++++++++++++-->
-  <!-- Comment or uncomment based on your requirement -->
-  <!-->
-  <xacro:imu name="imu" parent="base_link">
-    <origin xyz="0.100 0 0.500" rpy="0 0 3.14" />
-  </xacro:imu>
-  <-->
+ <!-- Comment or uncomment based on your requirement -->
+<!--   <xacro:imu name="imu_1" parent="base_link">
+    <origin xyz="0.100 0 0.300" rpy="0 0 3.14" />
+  </xacro:imu> -->
   <!--+++++++++++++++++++ Ultra Sonic ++++++++++++++++++++++++-->
   <!-- Comment or uncomment based on your requirement -->
   <!-- SENSOR 1 -->
-  <!-->
-  <xacro:us_sensor name="us_1" parent="base_link">
-    <origin xyz="0.100 0 0.500" rpy="0 3.14 3.14" />
-  </xacro:us_sensor>
-  <-->
+  <!-- xacro:us_sensor name="us_1" parent="base_link">
+    <origin xyz="0.100 0 0.300" rpy="0 3.14 3.14" />
+  </xacro:us_sensor-->
   <!-- SENSOR 2 -->
   <!-- xacro:us_sensor name="us_2" parent="base_link">
@@ -143,14 +133,9 @@
     <origin xyz="0.230 0 0.300" rpy="0 3.14 3.14" />
   </xacro:us_sensor-->
-  <!--Camera  -->
-  <!--><xacro:camera name="camera" parent="base_link">
-    <origin xyz="0 0 0.38" rpy="0 0 0" />
-  </xacro:camera>
-  <-->
   <!-- Depth Camera -->
   <xacro:depth_camera name="camera" parent="base_link">
     <origin xyz="-0.228 0.015 0.461" rpy="0 0 3.14159" />
   </xacro:depth_camera>
-  <transmission name="mpo_700_caster_front_left">
+   <transmission name="mpo_700_caster_front_left">
     <type>transmission_interface/SimpleTransmission</type>
     <joint name="mpo_700_caster_front_left_joint">

File: robots/mpo_700/xacros/mpo_700_body.xacro (robot description, xacro)
@@ -12,5 +12,5 @@
     <link name="${name}">
     <inertial>
-      <mass value="140"/>
+      <mass value="90"/>
       <origin xyz="0 0 0"/>
       <inertia ixx="7.8" ixy="0.0" ixz="0"

File: robots/mpo_700/xacros/mpo_700_gazebo.xacro (robot description, xacro)
@@ -5,4 +5,10 @@
     <self_collide>false</self_collide>
   </gazebo>
+<gazebo>
+  <plugin name="ros_control" filename="libgazebo_ros_control.so">
+    <legacyModeNS>false</legacyModeNS>
+    <robotSimType>gazebo_ros_control/DefaultRobotHWSim</robotSimType>
+  </plugin>
+</gazebo>
   <gazebo reference="lidar_1_link">
       <sensor type="ray" name="lidar_1_sensor">
@@ -31,5 +37,5 @@
                    reading. -->
               <mean>0.0</mean>
-              <stddev>0.01</stddev>
+              <stddev>0.0</stddev>
             </noise>
           </ray>
@@ -40,10 +46,4 @@
         </sensor>
   </gazebo>
-<gazebo>
-  <plugin name="ros_control" filename="libgazebo_ros_control.so">
-    <legacyModeNS>false</legacyModeNS>
-    <robotSimType>gazebo_ros_control/DefaultRobotHWSim</robotSimType>
-  </plugin>
-</gazebo>
   <gazebo reference="lidar_2_link">
       <sensor type="ray" name="lidar_2_sensor">
@@ -72,5 +72,5 @@
                    reading. -->
               <mean>0.0</mean>
-              <stddev>0.01</stddev>
+              <stddev>0.0</stddev>
             </noise>
           </ray>
@@ -105,51 +105,10 @@
       <odometryTopic>odom</odometryTopic>
       <odometryFrame>odom</odometryFrame>
-      <odometryRate>150.0</odometryRate>
+      <odometryRate>100.0</odometryRate>
       <robotBaseFrame>base_link</robotBaseFrame>
     </plugin>
   </gazebo>
   <!-- camera -->
-  <!-->
-  <gazebo reference="camera_link">
-    <sensor type="camera" name="camera1">
-      <update_rate>30.0</update_rate>
-      <camera name="head">
-        <horizontal_fov>1.3962634</horizontal_fov>
-  <image>
-    <width>800</width>
-    <height>800</height>
-    <format>R8G8B8</format>
-  </image>
-        <clip>
-          <near>0.02</near>
-          <far>300</far>
-        </clip>
-        <noise>
-          <type>gaussian</type>
-           Noise is sampled independently per pixel on each frame.
-               That pixel's noise value is added to each of its color
-               channels, which at that point lie in the range [0,1].
-          <mean>0.0</mean>
-          <stddev>0.007</stddev>
-        </noise>
-      </camera>
-      <plugin name="camera_controller" filename="libgazebo_ros_camera.so">
-        <alwaysOn>true</alwaysOn>
-        <updateRate>0.0</updateRate>
-        <cameraName>robot/camera1</cameraName>
-        <imageTopicName>image_raw</imageTopicName>
-        <cameraInfoTopicName>camera_info</cameraInfoTopicName>
-        <frameName>camera_link</frameName>
-        <hackBaseline>0.07</hackBaseline>
-        <distortionK1>0.0</distortionK1>
-        <distortionK2>0.0</distortionK2>
-        <distortionK3>0.0</distortionK3>
-        <distortionT1>0.0</distortionT1>
-        <distortionT2>0.0</distortionT2>
-      </plugin>
-    </sensor>
-  </gazebo>
-  <-->
-  <gazebo reference="camera_link_gazebo">
+ <gazebo reference="camera_link_gazebo">
     <sensor name="camera1" type="depth">
       <update_rate>15</update_rate>
@@ -226,11 +185,11 @@
       </ray>
       <plugin filename="libgazebo_ros_range.so" name="gazebo_ros_range">
-  <gaussianNoise>0.005</gaussianNoise>
-  <alwaysOn>true</alwaysOn>
-  <updateRate>50</updateRate>
-  <topicName>ultrasonic/us1</topicName>
-  <frameName>us_1_link</frameName>
-  <radiation>INFRARED</radiation>
-  <fov>0.2967</fov>
+	<gaussianNoise>0.005</gaussianNoise>
+	<alwaysOn>true</alwaysOn>
+	<updateRate>50</updateRate>
+	<topicName>ultrasonic/us1</topicName>
+	<frameName>us_1_link</frameName>
+	<radiation>INFRARED</radiation>
+	<fov>0.2967</fov>
       </plugin>
       </sensor>

File: robots/mpo_700/xacros/mpo_700_wheel.xacro (robot description, xacro)
@@ -27,6 +27,5 @@
      <origin xyz="0 0 0" rpy="0 0 0" />
      <geometry>
-      <sphere radius="0.09" />
-        <!-- <mesh filename="package://neo_simulation/robots/mpo_700/meshes/MPO-700-WHEEL.dae" scale="0.001 0.001 0.001"/> -->
+        <mesh filename="package://neo_simulation/robots/mpo_700/meshes/MPO-700-WHEEL.dae" scale="0.001 0.001 0.001"/>
      </geometry>
     </collision>

Commit message: Added the missing adapter

File: robots/mpo_700/mpo_700.urdf.xacro (robot description, xacro)
@@ -22,4 +22,5 @@
   <!-- Depth camera -->
   <xacro:include filename="$(find neo_simulation)/robots/mpo_700/xacros/depth_camera.xacro" />
+  <xacro:include filename="$(find neo_simulation)/robots/mpo_700/xacros/docking_adapter.xacro" />
   <!-- Base Macro-->
 <link name="base_link" />
@@ -137,4 +138,8 @@
     <origin xyz="-0.228 0.015 0.461" rpy="0 0 3.14159" />
   </xacro:depth_camera>
+  <!-- Docking station -->
+    <xacro:docking_adapter name="docking_adapter" parent="base_link">
+    <origin xyz="-0.300 0 0.320" rpy="0 0 -1.57" />
+  </xacro:docking_adapter>
    <transmission name="mpo_700_caster_front_left">
     <type>transmission_interface/SimpleTransmission</type>

Commit message: Updated the mpo-700 robot model to avoid problem of contact solution

File: robots/mpo_700/mpo_700.urdf.xacro (robot description, xacro)
@@ -15,6 +15,5 @@
   <xacro:include filename="$(find neo_simulation)/robots/mpo_700/xacros/mpo_700_gazebo.xacro" />
   <!--Caster  -->
-  <xacro:include filename="$(find neo_simulation)/robots/mpo_700/xacros/mpo_700_caster.xacro" />
-    <xacro:include filename="$(find neo_simulation)/robots/mpo_700/xacros/mpo_700_caster_left.xacro" />
+  <xacro:include filename="$(find neo_simulation)/robots/mpo_700/xacros/mpo_700_caster_left.xacro" />
   <xacro:include filename="$(find neo_simulation)/robots/mpo_700/xacros/mpo_700_caster_right.xacro" />
   <!-- Wheels -->
@@ -22,4 +21,5 @@
   <!-- Depth camera -->
   <xacro:include filename="$(find neo_simulation)/robots/mpo_700/xacros/depth_camera.xacro" />
+  <!-- Docking station -->
   <xacro:include filename="$(find neo_simulation)/robots/mpo_700/xacros/docking_adapter.xacro" />
   <!-- Base Macro-->

File: robots/mpo_700/xacros/mpo_700_wheel.xacro (robot description, xacro)
@@ -12,5 +12,5 @@
    <link name="${name}_link" type="wheel">
     <inertial>
-      <mass value="1.2"/>
+      <mass value="3"/>
       <origin rpy="0 0 0" xyz="0 0 0"/>
       <inertia ixx="0.11042056" ixy="0.0" ixz="0.0"
@@ -27,8 +27,16 @@
      <origin xyz="0 0 0" rpy="0 0 0" />
      <geometry>
-        <mesh filename="package://neo_simulation/robots/mpo_700/meshes/MPO-700-WHEEL.dae" scale="0.001 0.001 0.001"/>
+      <sphere radius="0.087"/>
+        <!-- <mesh filename="package://neo_simulation/robots/mpo_700/meshes/MPO-700-WHEEL.dae" scale="0.001 0.001 0.001"/> -->
      </geometry>
     </collision>
    </link>
+     <gazebo reference="${name}_link">
+      <!-- <kp> 10000 </kp> -->
+      <!-- <fdir1>0 1 0</fdir1> -->
+      <!-- <slip1> 0.1 </slip1> -->
+      <mu1>0.0001</mu1>
+      <mu2>0.0001</mu2>
+</gazebo>
   </xacro:macro>
 </robot>
