Commit message: fix: Cabinet visual and collision fix
The cabinet visual and collision were not aligned.

File: robots/mmo_700/urdf/xacros/cabinet.xacro (robot description, xacro)
@@ -23,5 +23,5 @@
       </visual>
       <collision>
-        <origin xyz="0. 0. 0" rpy="0 0 0" />
+        <origin xyz="0 0 0" rpy="0 0 -1.5708" />
         <geometry>
             <mesh filename="package://neo_simulation/robots/mmo_500/meshes/cabin.dae" scale="0.001 0.001 0.001"/>
