Commit message: mp-500 is updated

File: robots/mp_500/mp_500.urdf.xacro (robot description, xacro)
@@ -13,18 +13,18 @@
   </xacro:mp_500_base>
   <!-- Wheel Macro -->
-  <xacro:caster_wheel name="wheel_front" parent="base_link">
-    <origin xyz="-0.37 0. 0.06" rpy="-1.570796 0 1.57" />
+  <xacro:caster_wheel name="caster_wheel" parent="base_link">
+    <origin xyz="-0.43 0. 0.171" rpy="-1.570796 0 1.570796 " />
   </xacro:caster_wheel>
-  <xacro:fixed_wheel name="fixed_wheel_right" parent="base_link">
-    <origin xyz="0. -0.25 0.12" rpy="0 0 -1.570796" />
+  <xacro:fixed_wheel name="wheel_right" parent="base_link">
+    <origin xyz="0. -0.25 0.125" rpy="0 0 1.570796" />
   </xacro:fixed_wheel>
-  <xacro:fixed_wheel name="fixed_wheel_left" parent="base_link">
-    <origin xyz="0. 0.25 0.12" rpy="0 0 -1.570796" />
+  <xacro:fixed_wheel name="wheel_left" parent="base_link">
+    <origin xyz="0. 0.25 0.125" rpy="0 0 -1.570796" />
   </xacro:fixed_wheel>
  <!--+++++++++++++++++++laserscanner_front_link++++++++++++++++++++++++-->
    <!-- SENSORS -->
   <xacro:include filename="$(find neo_simulation)/robots/mp_500/xacros/sick_laser.xacro" />
-  <xacro:sick_laser_v0 name="laserscanner" parent="base_link" ros_topic="sick_300/scan">
-    <origin xyz="0.244 0 0.141" rpy="0 0 0" />
+  <xacro:sick_laser_v0 name="laserscanner_1" parent="base_link" ros_topic="sick/scan">
+    <origin xyz="0.244 0 0.141" rpy="3.14 0 0" />
   </xacro:sick_laser_v0>
 </robot>

File: robots/mp_500/xacros/mp_500_body.xacro (robot description, xacro)
@@ -11,7 +11,7 @@
   </inertial>
   <visual name='body'>
-  <origin xyz="0.0 0.0 -0.06" rpy="0 0 1.570796" /><!-- for STL -->
+  <origin xyz="0.0 0.0 0" rpy="0 0 1.570796" />
   <geometry>
-      <mesh filename="package://neo_mp_500/robot_model/mp_500/meshes/MP-500-BODY.dae" scale="0.001 0.001 0.001"/>
+      <mesh filename="package://neo_simulation/robots/mp_500/meshes/MP-500-BODY.dae" scale="0.001 0.001 0.001"/>
   </geometry>
   </visual>
@@ -19,5 +19,5 @@
   <origin xyz="0.0 0.0 0.0" rpy=" 0 0. 1.570796" />
   <geometry>
-    <mesh filename="package://neo_mp_500/robot_model/mp_500/meshes/MP-500-BODY.dae" scale="0.001 0.001 0.001"/>
+    <mesh filename="package://neo_simulation/robots/mp_500/meshes/MP-500-BODY.dae" scale="0.001 0.001 0.001"/>
   </geometry>
   </collision>

File: robots/mp_500/xacros/mp_500_caster_wheel.xacro (robot description, xacro)
@@ -16,7 +16,7 @@
     </inertial>
       <visual name='castor_wheel'>
-    <origin xyz="0.0 -0.06 0.06" rpy="0 0 0" />
+    <origin xyz="0 0 0" rpy="0 0 0" />
         <geometry>
-            <mesh filename="package://neo_mp_500/robot_model/mp_500/meshes/MP-500-WHEEL.dae" scale="0.001 0.001 0.001"/>
+            <mesh filename="package://neo_simulation/robots/mp_500/meshes/MP-500-WHEEL.dae" scale="0.001 0.001 0.001"/>
         </geometry>
       </visual>
@@ -24,5 +24,5 @@
       <origin xyz="0 0 0" rpy="0 0 0" />
       <geometry>
-            <mesh filename="package://neo_mp_500/robot_model/mp_500/meshes/MP-500-WHEEL.STL" scale="0.001 0.001 0.001"/>
+            <mesh filename="package://neo_simulation/robots/mp_500/meshes/MP-500-WHEEL.dae" scale="0.001 0.001 0.001"/>
       </geometry>
     </collision>

File: robots/mp_500/xacros/mp_500_fixed_wheel.xacro (robot description, xacro)
@@ -16,5 +16,5 @@
     </inertial>
       <visual>
-    <origin xyz="0 0. -0.04" rpy=" 0 0 0" />
+    <origin xyz="0 0 0" rpy="0 0 0" />
         <geometry>
             <mesh filename="package://neo_simulation/robots/mp_500/meshes/MP-500-FIXED-WHEEL.dae" scale="0.001 0.001 0.001"/>
@@ -24,5 +24,5 @@
      <origin xyz="0 0 0" rpy="0 0 0" />
       <geometry>
-            <mesh filename="package://neo_simulation/robots/mp_500/meshes/MP-500-WHEEL.STL" scale="0.001 0.001 0.001"/>
+            <mesh filename="package://neo_simulation/robots/mp_500/meshes/MP-500-FIXED-WHEEL.dae" scale="0.001 0.001 0.001"/>
       </geometry>
     </collision>

File: robots/mp_500/xacros/sick_laser.xacro (robot description, xacro)
@@ -16,5 +16,5 @@
       <visual>
       <!-- SICK S3 sensor: Uncomment/Comment it out if required  -->
-      <origin xyz="0 0 0.12" rpy="1.57 0 3.14" />
+      <origin xyz="0 0 -0.12" rpy="-1.57 0 3.14" />
         <geometry>
         <mesh filename="package://neo_simulation/robots/mp_500/meshes/SICK-S300.dae" scale="0.001 0.001 0.001" />
@@ -22,5 +22,5 @@
       </visual>
       <collision>
-        <origin xyz="0 0 0" rpy="1.57 0 3.14" />
+        <origin xyz="0 0 -0.13" rpy="-1.57 0 3.14" />
         <geometry>
         <mesh filename="package://neo_simulation/robots/mp_500/meshes/SICK-S300.dae" scale="0.001 0.001 0.001" />
@@ -28,5 +28,5 @@
       </collision>
       <!-- Microscan 3 sensor: Uncomment/Comment it out if required  -->
-<!--  <origin xyz="-0.0 0 0.06" rpy="-1.57 0 0" />
+<!--  <origin xyz="-0.0 0 -0.06" rpy="1.57 0 0" />
       <geometry>
       <mesh filename="package://neo_simulation/robots/mp_500/meshes/SICK-MICROSCAN3.dae" scale="0.001 0.001 0.001" />
@@ -34,5 +34,5 @@
       </visual>
       <collision>
- <origin xyz="-0.0 0 0.06" rpy="-1.57 0 0" />
+ <origin xyz="-0.0 0 -0.06" rpy="1.57 0 0" />
       <geometry>
         <mesh filename="package://neo_simulation/robots/mp_500/meshes/SICK-MICROSCAN3.dae" scale="0.001 0.001 0.001" />

Commit message: mp_500 urdf update

File: robots/mp_500/mp_500.urdf.xacro (robot description, xacro)
@@ -9,5 +9,6 @@
 <xacro:include filename="$(find neo_simulation)/robots/mp_500/xacros/mp_500_caster_wheel.xacro" />
 <!--+++++++++++++++++++left_wheel_link++++++++++++++++++++++++-->
-<xacro:include filename="$(find neo_simulation)/robots/mp_500/xacros/mp_500_fixed_wheel.xacro" />
+<xacro:include filename="$(find neo_simulation)/robots/mp_500/xacros/mp_500_fixed_wheel_left.xacro" />
+<xacro:include filename="$(find neo_simulation)/robots/mp_500/xacros/mp_500_fixed_wheel_right.xacro" />
   <xacro:mp_500_base name="base_link">
   </xacro:mp_500_base>
@@ -16,10 +17,10 @@
     <origin xyz="-0.43 0. 0.176" rpy="-1.570796 0 1.570796 " />
   </xacro:caster_wheel>
-  <xacro:fixed_wheel name="wheel_right" parent="base_link">
+  <xacro:fixed_wheel_right name="wheel_right" parent="base_link" number="1">
     <origin xyz="0. -0.25 0.13" rpy="0 0 -1.570796" />
-  </xacro:fixed_wheel>
-  <xacro:fixed_wheel name="wheel_left" parent="base_link">
+  </xacro:fixed_wheel_right>
+  <xacro:fixed_wheel_left name="wheel_left" parent="base_link" number="2">
     <origin xyz="0. 0.25 0.13" rpy="0 0 -1.570796" />
-  </xacro:fixed_wheel>
+  </xacro:fixed_wheel_left>
  <!--+++++++++++++++++++laserscanner_front_link++++++++++++++++++++++++-->
    <!-- SENSORS -->

File: robots/mp_500/xacros/mp_500_fixed_wheel_right.xacro (robot description, xacro)
@@ -1,15 +1,26 @@
 <?xml version="1.0"?>
 <robot xmlns:xacro="http://www.ros.org/wiki/xacro" name="mp_500">
-  <xacro:macro name="fixed_wheel" params="name parent *origin">
-   <joint name="${name}_joint" type="revolute">
+  <xacro:macro name="fixed_wheel_right" params="name parent number *origin">
+    <joint name="${name}_joint" type="revolute">
     <insert_block name="origin" />
     <limit effort="1000.0" lower="-1e+16" upper="1e+16" velocity="3.5"/>
     <axis xyz="-1 0 0" />
     <joint_properties damping="0" friction="0.0" />
-    <parent link="${parent}" />
+    <parent link="base_link" />
     <child link="${name}_link" />
    </joint>
+   <transmission name="tran_${number}">
+    <type>transmission_interface/SimpleTransmission</type>
+    <joint name="${name}_joint" type="revolute">
+      <hardwareInterface>hardware_interface/VelocityJointInterface</hardwareInterface>
+        </joint>
+      <actuator name="right_wheel_actuator">
+      <mechanicalReduction>7</mechanicalReduction>
+            <hardwareInterface>hardware_interface/VelocityJointInterface</hardwareInterface>
+      </actuator>
+  </transmission>
    <link name="${name}_link" type="wheel">
     <inertial>
+      <origin xyz="0 0 0" rpy="0 0 0"/>
         <mass value="1.82362"/>
         <inertia ixx="0.00399743171" ixy="0.00000004464" ixz="-0.00000002245"
@@ -20,5 +31,5 @@
     <origin xyz="0 0 0" rpy="0 0 0" />
         <geometry>
-            <mesh filename="package://neo_simulation/robots/mp_500/meshes/MP-500-FIXED-WHEEL.dae" scale="0.001 0.001 0.001"/>
+            <mesh filename="package://neo_simulation/robots/mp_500/meshes/MP-500-WHEEL-RIGHT.dae" scale="0.001 0.001 0.001"/>
         </geometry>
       </visual>
@@ -26,5 +37,5 @@
      <origin xyz="0 0 0" rpy="0 0 0" />
       <geometry>
-            <mesh filename="package://neo_simulation/robots/mp_500/meshes/MP-500-FIXED-WHEEL.dae" scale="0.001 0.001 0.001"/>
+            <mesh filename="package://neo_simulation/robots/mp_500/meshes/MP-500-WHEEL-RIGHT.dae" scale="0.001 0.001 0.001"/>
       </geometry>
     </collision>

File: robots/mp_500/xacros/mp_500_gazebo.xacro (robot description, xacro)
@@ -1,12 +1,4 @@
 <?xml version="1.0"?>
 <robot name="mp_500" xmlns:xacro="http://www.ros.org/wiki/xacro">
-   <gazebo reference="base_link">
-    <gravity>true</gravity>
-    <self_collide>false</self_collide>
-  </gazebo>
-  <gazebo reference="castor_wheel_link">
-    <gravity>true</gravity>
-    <self_collide>false</self_collide>
-  </gazebo>
   <gazebo reference="laserscanner_1_link">
       <sensor type="ray" name="laserscanner_1_link">
@@ -68,3 +60,10 @@
     </plugin>
   </gazebo>
+<!-- <gazebo>
+  <plugin name="gazebo_ros_control" filename="libgazebo_ros_control.so">
+ <legacyModeNS> false </legacyModeNS>
+  <robotParam>/robot_description</robotParam>
+       <robotSimType>gazebo_ros_control/DefaultRobotHWSim</robotSimType>
+  </plugin>
+</gazebo> -->
 </robot>

Commit message: Mp-500 now have seperate Xacro and Macro

File: robots/mp_500/mp_500.urdf.xacro (robot description, xacro)
@@ -12,6 +12,11 @@
 <xacro:include filename="$(find neo_simulation)/robots/mp_500/xacros/mp_500_fixed_wheel_right.xacro" />
  <!-- SENSORS -->
-<xacro:include filename="$(find neo_simulation)/robots/mp_500/xacros/sick_laser.xacro" />
+ <!-- Sick laser S300 -->
+<xacro:include filename="$(find neo_simulation)/robots/mp_500/xacros/sick_laser_s300.xacro" />
+<!-- Sick laser Microscan -->
+<!-- <xacro:include filename="$(find neo_simulation)/robots/mp_500/xacros/sick_laser_microscan.xacro" /> -->
+<!-- IMU -->
 <xacro:include filename="$(find neo_simulation)/robots/mp_500/xacros/imu.xacro" />
+<!-- UltraSonic Sensor -->
 <xacro:include filename="$(find neo_simulation)/robots/mp_500/xacros/ultrasonic.xacro" />
   <xacro:mp_500_base name="base_link">
@@ -29,8 +34,14 @@
  <!--+++++++++++++++++++laserscanner_front_link++++++++++++++++++++++++-->
    <!-- SENSORS -->
-  <xacro:include filename="$(find neo_simulation)/robots/mp_500/xacros/sick_laser.xacro" />
-  <xacro:sick_laser_v0 name="lidar_1" parent="base_link" ros_topic="lidar_1/scan_filtered">
+   <!-- Sick S300 -->
+  <xacro:include filename="$(find neo_simulation)/robots/mp_500/xacros/sick_laser_s300.xacro" />
+  <xacro:sick_laser_s300 name="lidar_1" parent="base_link" ros_topic="lidar_1/scan_filtered">
     <origin xyz="0.244 0 0.141" rpy="3.14 0 0" />
-  </xacro:sick_laser_v0>
+  </xacro:sick_laser_s300>
+  <!-- Sick Microscan -->
+<!-- <xacro:include filename="$(find neo_simulation)/robots/mp_500/xacros/sick_laser_microscan.xacro" />
+  <xacro:sick_laser_microscan name="lidar_1" parent="base_link" ros_topic="lidar_1/scan_filtered">
+    <origin xyz="0.244 0 0.141" rpy="3.14 0 0" />
+  </xacro:sick_laser_microscan> -->
      <!--+++++++++++++++++++ IMU ++++++++++++++++++++++++-->
  <!-- Comment or uncomment based on your requirement -->

File: robots/mp_500/xacros/sick_laser_s300.xacro (robot description, xacro)
@@ -15,5 +15,4 @@
       </inertial>
       <visual>
-      <!-- SICK S3 sensor: Uncomment/Comment it out if required  -->
       <origin xyz="0 0 -0.12" rpy="-1.57 0 3.14" />
         <geometry>
@@ -27,16 +26,4 @@
         </geometry>
       </collision>
-      <!-- Microscan 3 sensor: Uncomment/Comment it out if required  -->
-<!--  <origin xyz="-0.0 0 -0.06" rpy="1.57 0 0" />
-      <geometry>
-      <mesh filename="package://neo_simulation/robots/mp_500/meshes/SICK-MICROSCAN3.dae" scale="0.001 0.001 0.001" />
-      </geometry>
-      </visual>
-      <collision>
- <origin xyz="-0.0 0 -0.06" rpy="1.57 0 0" />
-      <geometry>
-        <mesh filename="package://neo_simulation/robots/mp_500/meshes/SICK-MICROSCAN3.dae" scale="0.001 0.001 0.001" />
-        </geometry>
-      </collision> -->
     </link>
   </xacro:macro>

Commit message: Models for MP-500, MPO-500 and MP-500 updated with cameras, IMU and USS

File: robots/mp_500/mp_500.urdf.xacro (robot description, xacro)
@@ -1,23 +1,21 @@
 <?xml version="1.0"?>
-<!-- Materials -->
 <robot xmlns:xacro="http://www.ros.org/wiki/xacro" name="mp_500">
-<xacro:include filename="$(find neo_simulation)/robots/mp_500/xacros/mp_500_gazebo.xacro" />
-<!--++++++++++++++++++++++++++++++base_link++++++++++++++++++++++++++++++++++++++++++++++++++++-->
-<!--++++++++++++++++++++body++++++++++++++++++++++++++++-->
-<xacro:include filename="$(find neo_simulation)/robots/mp_500/xacros/mp_500_body.xacro" />
-<!--+++++++++++++++++++castor_wheel_link++++++++++++++++++++++++-->
-<xacro:include filename="$(find neo_simulation)/robots/mp_500/xacros/mp_500_caster_wheel.xacro" />
-<!--+++++++++++++++++++left_wheel_link++++++++++++++++++++++++-->
-<xacro:include filename="$(find neo_simulation)/robots/mp_500/xacros/mp_500_fixed_wheel_left.xacro" />
-<xacro:include filename="$(find neo_simulation)/robots/mp_500/xacros/mp_500_fixed_wheel_right.xacro" />
- <!-- SENSORS -->
- <!-- Sick laser S300 -->
-<xacro:include filename="$(find neo_simulation)/robots/mp_500/xacros/sick_laser_s300.xacro" />
-<!-- Sick laser Microscan -->
-<!-- <xacro:include filename="$(find neo_simulation)/robots/mp_500/xacros/sick_laser_microscan.xacro" /> -->
-<!-- IMU -->
-<xacro:include filename="$(find neo_simulation)/robots/mp_500/xacros/imu.xacro" />
-<!-- UltraSonic Sensor -->
-<xacro:include filename="$(find neo_simulation)/robots/mp_500/xacros/ultrasonic.xacro" />
+  <xacro:include filename="$(find neo_simulation)/robots/mp_500/xacros/mp_500_gazebo.xacro" />
+  <!--++++++++++++++++++++++++++++++base_link++++++++++++++++++++++++++++++++++++++++++++++++++++-->
+  <!--++++++++++++++++++++body++++++++++++++++++++++++++++-->
+  <xacro:include filename="$(find neo_simulation)/robots/mp_500/xacros/mp_500_body.xacro" />
+  <!--+++++++++++++++++++castor_wheel_link++++++++++++++++++++++++-->
+  <xacro:include filename="$(find neo_simulation)/robots/mp_500/xacros/mp_500_caster_wheel.xacro" />
+  <!--+++++++++++++++++++left_wheel_link++++++++++++++++++++++++-->
+  <xacro:include filename="$(find neo_simulation)/robots/mp_500/xacros/mp_500_fixed_wheel_left.xacro" />
+  <xacro:include filename="$(find neo_simulation)/robots/mp_500/xacros/mp_500_fixed_wheel_right.xacro" />
+  <!-- SENSORS -->
+  <!-- Sick S300 - Comment/Uncomment if required  -->
+  <xacro:include filename="$(find neo_simulation)/robots/mp_500/xacros/sick_S300.xacro" />
+  <!-- Microscan - Comment/Uncomment if required -->
+  <!-- <xacro:include filename="$(find neo_simulation)/robots/mp_500/xacros/micro_scan.xacro" /> -->
+  <!-- USS and IMU - Comment/Uncomment if required  -->
+  <!-- <xacro:include filename="$(find neo_simulation)/robots/mp_500/xacros/imu.xacro" />
+  <xacro:include filename="$(find neo_simulation)/robots/mp_500/xacros/ultrasonic.xacro" /> -->
   <xacro:mp_500_base name="base_link">
   </xacro:mp_500_base>
@@ -34,14 +32,7 @@
  <!--+++++++++++++++++++laserscanner_front_link++++++++++++++++++++++++-->
    <!-- SENSORS -->
-   <!-- Sick S300 -->
-  <xacro:include filename="$(find neo_simulation)/robots/mp_500/xacros/sick_laser_s300.xacro" />
-  <xacro:sick_laser_s300 name="lidar_1" parent="base_link" ros_topic="lidar_1/scan_filtered">
+  <xacro:sick_laser_v0 name="lidar_1" parent="base_link" ros_topic="lidar_1/scan_filtered">
     <origin xyz="0.244 0 0.141" rpy="3.14 0 0" />
-  </xacro:sick_laser_s300>
-  <!-- Sick Microscan -->
-<!-- <xacro:include filename="$(find neo_simulation)/robots/mp_500/xacros/sick_laser_microscan.xacro" />
-  <xacro:sick_laser_microscan name="lidar_1" parent="base_link" ros_topic="lidar_1/scan_filtered">
-    <origin xyz="0.244 0 0.141" rpy="3.14 0 0" />
-  </xacro:sick_laser_microscan> -->
+  </xacro:sick_laser_v0>
      <!--+++++++++++++++++++ IMU ++++++++++++++++++++++++-->
  <!-- Comment or uncomment based on your requirement -->

File: robots/mp_500/xacros/imu.xacro (robot description, xacro)
@@ -1,5 +1,5 @@
 <?xml version="1.0"?>
-<robot xmlns:xacro="http://www.ros.org/wiki/xacro" name="mp_400">
-  <xacro:macro name="us_sensor" params="name parent *origin">
+<robot xmlns:xacro="http://www.ros.org/wiki/xacro" name="mp_500">
+  <xacro:macro name="imu" params="name parent *origin">
     <joint name="${name}_joint" type="fixed">
       <axis xyz="0 1 0" />

Commit message: Depth camera and additional laser scanner is added to the robot model

File: robots/mp_500/mp_500.urdf.xacro (robot description, xacro)
@@ -21,4 +21,6 @@
   <xacro:include filename="$(find neo_simulation)/robots/mp_500/xacros/camera.xacro" />
   <-->
+  <!-- Depth camera -->
+  <xacro:include filename="$(find neo_simulation)/robots/mp_500/xacros/depth_camera.xacro" />
   <xacro:mp_500_base name="base_link">
   </xacro:mp_500_base>
@@ -38,4 +40,9 @@
     <origin xyz="0.244 0 0.141" rpy="3.14 0 0" />
   </xacro:sick_laser_v0>
+<!-- If extra laser scanner is needed -->
+<!--   <xacro:sick_laser_v0 name="lidar_2" parent="base_link" ros_topic="lidar_2/scan_filtered">
+    <origin xyz="0.244 0.1 0.141" rpy="3.14 0 0" />
+  </xacro:sick_laser_v0>
+ -->
      <!--+++++++++++++++++++ IMU ++++++++++++++++++++++++-->
   <!-- Comment or uncomment based on your requirement -->
@@ -109,8 +116,7 @@
     <origin xyz="0.230 0 0.300" rpy="0 3.14 3.14" />
   </xacro:us_sensor-->
-  <!--Camera  -->
-<!-- <xacro:camera name="camera" parent="base_link">
-    <origin xyz="0 0 0.38" rpy="0 0 0" />
-  </xacro:camera>
- -->
+  <!-- depth Camera  -->
+<!--   <xacro:depth_camera name="camera" parent="base_link">
+    <origin xyz="0.0 0.0 0.371" rpy="0 0 3.14159" />
+  </xacro:depth_camera> -->
 </robot>

File: robots/mp_500/xacros/mp_500_gazebo.xacro (robot description, xacro)
@@ -33,4 +33,39 @@
             <topicName>lidar_1/scan_filtered</topicName>
             <frameName>lidar_1_link</frameName>
+          </plugin>
+        </sensor>
+  </gazebo>
+  <gazebo reference="lidar_2_link">
+      <sensor type="ray" name="lidar_2_link">
+          <pose>0 0 0 0 0 0</pose>
+          <visualize>false</visualize>
+          <update_rate>40</update_rate>
+          <ray>
+            <scan>
+              <horizontal>
+                <samples>720</samples>
+                <resolution>1</resolution>
+                <min_angle>-1.48353</min_angle>
+                <max_angle>1.48353</max_angle>
+              </horizontal>
+            </scan>
+            <range>
+              <min>0.10</min>
+              <max>30.0</max>
+              <resolution>0.05</resolution>
+            </range>
+            <noise>
+              <type>gaussian</type>
+              <!-- Noise parameters based on published spec for Hokuyo laser
+                   achieving "+-30mm" accuracy at range < 10m.  A mean of 0.0m and
+                   stddev of 0.01m will put 99.7% of samples within 0.03m of the true
+                   reading. -->
+              <mean>0.0</mean>
+              <stddev>0.01</stddev>
+            </noise>
+          </ray>
+          <plugin name="lidar_2_link" filename="libgazebo_ros_laser.so">
+            <topicName>lidar_2/scan_filtered</topicName>
+            <frameName>lidar_2_link</frameName>
           </plugin>
         </sensor>
@@ -156,4 +191,53 @@
     </plugin>
   </gazebo>
+  <gazebo reference="camera_link_gazebo">
+    <sensor name="camera1" type="depth">
+      <update_rate>15</update_rate>
+      <hfov>70</hfov>
+      <camera name="head">
+        <image>
+          <width>320</width>
+          <height>240</height>
+          <format>R8G8B8</format>
+        </image>
+        <clip>
+          <near>0.02</near>
+          <far>300</far>
+        </clip>
+        <noise>
+          <type>gaussian</type>
+          <!-- Noise is sampled independently per pixel on each frame.
+               That pixel's noise value is added to each of its color
+               channels, which at that point lie in the range [0,1]. -->
+          <mean>0.0</mean>
+          <stddev>0.03</stddev>
+        </noise>
+      </camera>
+      <plugin name="camera1_controller" filename="libgazebo_ros_openni_kinect.so">
+        <!--<baseline>0.2</baseline>-->
+        <alwaysOn>true</alwaysOn>
+        <updateRate>0.0</updateRate>
+        <cameraName>camera_ir</cameraName>
+        <imageTopicName>/camera/depth/image_raw</imageTopicName>
+        <cameraInfoTopicName>/camera/depth/camera_info</cameraInfoTopicName>
+        <depthImageTopicName>/camera/depth/depth_raw</depthImageTopicName>
+        <depthImageInfoTopicName>/camera/depth/camera_info</depthImageInfoTopicName>
+        <pointCloudTopicName>/camera/depth_registered/points</pointCloudTopicName>
+        <frameName>camera_link_optical</frameName>
+        <pointCloudCutoff>0.12</pointCloudCutoff>
+        <pointCloudCutoffMax>3.0</pointCloudCutoffMax>
+        <distortionK1>0.00000001</distortionK1>
+        <distortionK2>0.00000001</distortionK2>
+        <distortionK3>0.00000001</distortionK3>
+        <distortionT1>0.00000001</distortionT1>
+        <distortionT2>0.00000001</distortionT2>
+        <CxPrime>0</CxPrime>
+        <Cx>0</Cx>
+        <Cy>0</Cy>
+        <focalLength>0</focalLength>
+        <hackBaseline>0</hackBaseline>
+      </plugin>
+    </sensor>
+  </gazebo>
 <!-- <gazebo>
   <plugin name="gazebo_ros_control" filename="libgazebo_ros_control.so">

Commit message: Changed the angle convention to accommodate the light_scan on mp_599

File: robots/mp_500/mp_500.urdf.xacro (robot description, xacro)
@@ -38,5 +38,5 @@
    <!-- SENSORS -->
   <xacro:sick_laser_v0 name="lidar_1" parent="base_link" ros_topic="lidar_1/scan_filtered">
-    <origin xyz="0.244 0 0.141" rpy="3.14 0 0" />
+    <origin xyz="0.244 0 0.141" rpy="0 0 0" />
   </xacro:sick_laser_v0>
 <!-- If extra laser scanner is needed -->
