Commit message: New maps has been added

File: robots/mm_400/mm_400.urdf.xacro (robot description, xacro)
@@ -17,4 +17,6 @@
  <!-- SENSORS -->
 <xacro:include filename="$(find neo_simulation)/robots/mm_400/urdf/xacros/sick_laser.xacro" />
+<!-- Gripper -->
+<xacro:include filename="$(find schunk_description)/pg70.urdf.xacro" />
   <xacro:mp_400_base name="base_link">
   </xacro:mp_400_base>
@@ -45,4 +47,7 @@
     <origin xyz="0 0 0." rpy="0 0 0" />
   </xacro:prbt>
+  <xacro:pg70 parent="pilztool0">
+    <origin xyz="0 0 0." rpy="0 0 0" />
+  </xacro:pg70>
   <!--+++++++++++++++++++laserscanner_link++++++++++++++++++++++++-->
   <xacro:sick_laser_v0 name="laser_1" parent="base_link" ros_topic="laser_1/scan">

Commit message: Kinetic branch updated with the laser scanner names, coorected wheel alignment for mpo 500

File: robots/mm_400/mm_400.urdf.xacro (robot description, xacro)
@@ -17,4 +17,6 @@
  <!-- SENSORS -->
 <xacro:include filename="$(find neo_simulation)/robots/mm_400/urdf/xacros/sick_laser.xacro" />
+<!-- Gripper -->
+<xacro:include filename="$(find schunk_description)/pg70.urdf.xacro" />
   <xacro:mp_400_base name="base_link">
   </xacro:mp_400_base>
@@ -45,6 +47,9 @@
     <origin xyz="0 0 0." rpy="0 0 0" />
   </xacro:prbt>
+  <xacro:pg70 parent="pilztool0">
+    <origin xyz="0 0 0." rpy="0 0 0" />
+  </xacro:pg70>
   <!--+++++++++++++++++++laserscanner_link++++++++++++++++++++++++-->
-  <xacro:sick_laser_v0 name="laser_1" parent="base_link" ros_topic="laser_1/scan">
+  <xacro:sick_laser_v0 name="laser_1" parent="base_link" ros_topic="lidar_1/scan">
     <origin xyz="0.230 0 0.110" rpy="0 3.14 3.14" />
   </xacro:sick_laser_v0>

File: robots/mmo_500/mmo_500.urdf.xacro (robot description, xacro)
@@ -25,18 +25,18 @@
   	<origin xyz="0.25 0.28 0.13" rpy="0 0 0" />
   </xacro:omni_wheel_250>
-  <xacro:omni_wheel_250 name="wheel_front_right" parent="base_link" >
-  	<origin xyz="0.25 -0.28 0.13" rpy="0 0 0" />
+  <xacro:omni_wheel_250 name="wheel_front_right" parent="base_link">
+  	<origin xyz="0.25 -0.28 0.13" rpy="0 0 3.14" />
   </xacro:omni_wheel_250>
   <xacro:omni_wheel_250 name="wheel_back_left" parent="base_link">
   	<origin xyz="-0.25 0.28 0.13" rpy="0 0 0" />
   </xacro:omni_wheel_250>
-  <xacro:omni_wheel_250 name="wheel_back_right" parent="base_link" >
-  	<origin xyz="-0.25 -0.28 0.13" rpy="0 0 0" />
+  <xacro:omni_wheel_250 name="wheel_back_right" parent="base_link">
+  	<origin xyz="-0.25 -0.28 0.13" rpy="0 0 3.14" />
   </xacro:omni_wheel_250>
   <!-- Sensors -->
-  <xacro:sick_laser_v0 name="sick_laser_front" parent="base_link" ros_topic="sick_front/scan">
+  <xacro:sick_laser_v0 name="sick_laser_front" parent="base_link" ros_topic="lidar_1/scan">
     <origin xyz="0.442 0 0.372" rpy="0 0 0" />
   </xacro:sick_laser_v0>
-  <xacro:sick_laser_v0 name="sick_laser_back" parent="base_link" ros_topic="sick_back/scan">
+  <xacro:sick_laser_v0 name="sick_laser_back" parent="base_link" ros_topic="lidar_2/scan">
     <origin xyz="-0.442 0 0.372" rpy="0 0 3.14" />
   </xacro:sick_laser_v0>

File: robots/mpo_500/mpo_500.urdf.xacro (robot description, xacro)
@@ -17,5 +17,5 @@
   </xacro:omni_wheel_250>
   <xacro:omni_wheel_250 name="wheel_front_right" parent="base_link">
-  	<origin xyz="0.25 -0.28 0.13" rpy="0 0 0" />
+  	<origin xyz="0.25 -0.28 0.13" rpy="0 0 3.14" />
   </xacro:omni_wheel_250>
   <xacro:omni_wheel_250 name="wheel_back_left" parent="base_link">
@@ -23,11 +23,11 @@
   </xacro:omni_wheel_250>
   <xacro:omni_wheel_250 name="wheel_back_right" parent="base_link">
-  	<origin xyz="-0.25 -0.28 0.13" rpy="0 0 0" />
+  	<origin xyz="-0.25 -0.28 0.13" rpy="0 0 3.14" />
   </xacro:omni_wheel_250>
   <!-- Sensors -->
-  <xacro:sick_laser_v0 name="sick_laser_front" parent="base_link" ros_topic="sick_front/scan">
+  <xacro:sick_laser_v0 name="sick_laser_front" parent="base_link" ros_topic="lidar_1/scan">
   	<origin xyz="0.442 0 0.372" rpy="0 0 0" />
   </xacro:sick_laser_v0>
-  <xacro:sick_laser_v0 name="sick_laser_back" parent="base_link" ros_topic="sick_back/scan">
+  <xacro:sick_laser_v0 name="sick_laser_back" parent="base_link" ros_topic="lidar_2/scan">
   	<origin xyz="-0.442 0 0.372" rpy="0 0 3.14" />
   </xacro:sick_laser_v0>

Commit message: MM-400 with both Pilz and Frank emika arm is working

File: robots/mm_400/mm_400.urdf.xacro (robot description, xacro)
@@ -14,9 +14,11 @@
 <!--+++++++++++++++++++cabinet++++++++++++++++++++++++-->
 <xacro:include filename="$(find neo_simulation)/robots/mm_400/urdf/xacros/cabinet.xacro" />
+<!-- PRBT -->
 <xacro:include filename="$(find neo_simulation)/robots/mm_400/urdf/prbt_macro.xacro" />
+<!-- Panda -->
+  <xacro:include filename="$(find neo_simulation)/robots/mm_400/urdf/panda_arm.xacro" />
  <!-- SENSORS -->
 <xacro:include filename="$(find neo_simulation)/robots/mm_400/urdf/xacros/sick_laser.xacro" />
 <!-- Gripper -->
-<xacro:include filename="$(find schunk_description)/pg70.urdf.xacro" />
   <xacro:mp_400_base name="base_link">
   </xacro:mp_400_base>
@@ -47,7 +49,8 @@
     <origin xyz="0 0 0." rpy="0 0 0" />
   </xacro:prbt>
-  <xacro:pg70 parent="pilztool0">
+<!-- Panda -->
+<!--   <xacro:panda_arm parent="base_link" prefix="panda">
     <origin xyz="0 0 0." rpy="0 0 0" />
-  </xacro:pg70>
+  </xacro:panda_arm> -->
   <!--+++++++++++++++++++laserscanner_link++++++++++++++++++++++++-->
   <xacro:sick_laser_v0 name="laser_1" parent="base_link" ros_topic="lidar_1/scan">

File: robots/mm_400/urdf/xacros/mp_400_caster_wheel.xacro (robot description, xacro)
@@ -11,8 +11,9 @@
    </joint>
    <link name="${name}_link" type="wheel">
- <inertial>
-      <origin rpy="0 0 0" xyz="0 0 0" />
-      <mass value="0.08" />
-      <inertia ixx="0.00000045" ixy="0" ixz="0" iyy="0.0000005" iyz="0" izz="0.00000045" />
+    <inertial>
+        <mass value="1.82362"/>
+        <inertia ixx="0.0000499743171" ixy="0.0000000004464" ixz="-0.0000000002245"
+                 iyy="0.00499741733" iyz="0.0000000000164"
+izz="0.0000839239692"/>
 </inertial>
       <visual name='caster_wheel'>
@@ -29,11 +30,4 @@
     </collision>
     </link>
-<gazebo reference="${name}_link">
-      <kp>50000.0</kp>
-      <kd>500.0</kd>
-      <mu1>0.02</mu1>
-      <mu2>0.01</mu2>
-      <implicitSpringDamper>1</implicitSpringDamper>
-</gazebo>
   </xacro:macro>
 </robot>

File: robots/mm_400/urdf/xacros/mp_400_fixed_wheel_left.xacro (robot description, xacro)
@@ -11,9 +11,10 @@
    </joint>
    <link name="${name}_link" type="wheel">
-   <inertial>
-        <mass value="1."/>
-        <inertia ixx="0.000399743171" ixy="0.000000004464" ixz="-0.000000002245"
-                 iyy="0.000399741733" iyz="-0.000000000164"
-                 izz="0.000739239692"/>
+<inertial>
+      <origin xyz="0 0 0" rpy="0 0 0"/>
+        <mass value="1.82362"/>
+        <inertia ixx="0.0399743171" ixy="0.00000004464" ixz="-0.00000002245"
+                 iyy="0.0399741733" iyz="-0.00000000164"
+                 izz="0.0739239692"/>
 </inertial>
       <visual name='fixed_wheel_left'>
@@ -33,7 +34,8 @@
       <kp>100000.0</kp>
       <kd>50.0</kd>
-      <mu1>20</mu1>
-      <mu2>10</mu2>
-      <fdir1>1 0 0</fdir1>
+      <mu1>100</mu1>
+      <gravity> 1 </gravity>
+      <mu2>100</mu2>
+      <minDepth>0.00</minDepth>
       <implicitSpringDamper>1</implicitSpringDamper>
 </gazebo>

File: robots/mm_400/urdf/xacros/mp_400_fixed_wheel_right.xacro (robot description, xacro)
@@ -11,9 +11,10 @@
    </joint>
    <link name="${name}_link" type="wheel">
-   <inertial>
-        <mass value="1."/>
-        <inertia ixx="0.000399743171" ixy="0.00000004464" ixz="-0.00000002245"
-                 iyy="0.000399741733" iyz="-0.00000000164"
-                 izz="0.000739239692"/>
+      <inertial>
+      <origin xyz="0 0 0" rpy="0 0 0"/>
+        <mass value="1.82362"/>
+        <inertia ixx="0.0399743171" ixy="0.00000004464" ixz="-0.00000002245"
+                 iyy="0.0399741733" iyz="-0.00000000164"
+                 izz="0.0739239692"/>
 </inertial>
       <visual name='fixed_wheel_right'>
@@ -33,7 +34,8 @@
       <kp>100000.0</kp>
       <kd>50.0</kd>
-      <mu1>20</mu1>
-      <mu2>10</mu2>
-      <fdir1>1 0 0</fdir1>
+      <gravity> 1 </gravity>
+      <mu1>100</mu1>
+      <mu2>100</mu2>
+      <minDepth>0.00</minDepth>
       <implicitSpringDamper>1</implicitSpringDamper>
 </gazebo>

File: robots/mm_400/urdf/xacros/mp_400_gazebo.xacro (robot description, xacro)
@@ -13,4 +13,44 @@
     <self_collide>false</self_collide>
   </gazebo>
+<gazebo reference="wheel_front_right_link">
+      <kp>35000.0</kp>
+      <kd>1000.0</kd>
+      <mu1>0.051</mu1>
+      <mu2>0.051</mu2>
+      <fdir1>1 0 0</fdir1>
+    <maxVel>1.0</maxVel>
+    <minDepth>0.00</minDepth>
+      <implicitSpringDamper>1</implicitSpringDamper>
+</gazebo>
+<gazebo reference="wheel_front_left_link">
+      <kp>35000.0</kp>
+      <kd>1000.0</kd>
+      <mu1>0.051</mu1>
+      <mu2>0.051</mu2>
+          <fdir1>1 0 0</fdir1>
+    <maxVel>1.0</maxVel>
+    <minDepth>0.00</minDepth>
+      <implicitSpringDamper>1</implicitSpringDamper>
+</gazebo>
+<gazebo reference="wheel_back_left_link">
+      <kp>35000.0</kp>
+      <kd>1000.0</kd>
+      <mu1>0.051</mu1>
+      <mu2>0.051</mu2>
+          <fdir1>1 0 0</fdir1>
+    <maxVel>1.0</maxVel>
+    <minDepth>0.00</minDepth>
+      <implicitSpringDamper>1</implicitSpringDamper>
+</gazebo>
+<gazebo reference="wheel_back_right_link">
+      <kp>35000.0</kp>
+      <kd>1000.0</kd>
+      <mu1>0.051</mu1>
+      <mu2>0.051</mu2>
+          <fdir1>1 0 0</fdir1>
+    <maxVel>1.0</maxVel>
+    <minDepth>0.00</minDepth>
+      <implicitSpringDamper>1</implicitSpringDamper>
+</gazebo>
   <gazebo reference="laser_1_link">
       <sensor type="ray" name="laser_1_link">
@@ -43,5 +83,5 @@
           </ray>
           <plugin name="laser_1_link" filename="libgazebo_ros_laser.so">
-            <topicName>lidar_1/scan</topicName>
+            <topicName>laser_1/scan</topicName>
             <frameName>laser_1_link</frameName>
           </plugin>
@@ -53,5 +93,5 @@
         <updateRate>40</updateRate>
         <legacyMode>false</legacyMode>
-        <torque>5</torque>
+        <torque>0.05</torque>
         <leftJoint>fixed_wheel_left_joint</leftJoint>
         <rightJoint>fixed_wheel_right_joint</rightJoint>
@@ -66,5 +106,5 @@
         <publishWheelJointState>true</publishWheelJointState>
         <wheelAcceleration>6.0</wheelAcceleration>
-        <wheelTorque>5</wheelTorque>
+        <wheelTorque>200</wheelTorque>
         <odometrySource>world</odometrySource>
         <publishTf>1</publishTf>
