Commit message: MM-400 updated

File: robots/mm_400/mm_400.urdf.xacro (robot description, xacro)
@@ -14,11 +14,17 @@
 <!--+++++++++++++++++++cabinet++++++++++++++++++++++++-->
 <xacro:include filename="$(find neo_simulation)/robots/mm_400/urdf/xacros/cabinet.xacro" />
+<!-- PRBT -->
 <xacro:include filename="$(find neo_simulation)/robots/mm_400/urdf/prbt_macro.xacro" />
+<!-- Panda -->
+  <xacro:include filename="$(find neo_simulation)/robots/mm_400/urdf/panda_arm.xacro" />
  <!-- SENSORS -->
-<xacro:include filename="$(find neo_simulation)/robots/mm_400/urdf/xacros/sick_laser.xacro" />
-<xacro:include filename="$(find neo_simulation)/robots/mm_400/urdf/xacros/imu.xacro" />
+<!-- SENSORS -->
+<!-- <xacro:include filename="$(find neo_simulation)/robots/mm_400/urdf/xacros/sick_S300.xacro" /> -->
+<!-- Microscan - Comment/Uncomment if required -->
+<xacro:include filename="$(find neo_simulation)/robots/mm_400/urdf/xacros/micro_scan.xacro" />
+<!-- Additional sensors if required -->
+<!-- <xacro:include filename="$(find neo_simulation)/robots/mm_400/urdf/xacros/imu.xacro" />
 <xacro:include filename="$(find neo_simulation)/robots/mm_400/urdf/xacros/ultrasonic.xacro" />
-<!-- Gripper -->
-<xacro:include filename="$(find schunk_description)/pg70.urdf.xacro" />
+<xacro:include filename="$(find neo_simulation)/robots/mm_400/urdf/xacros/camera.xacro" />-->
   <xacro:mp_400_base name="base_link">
   </xacro:mp_400_base>
@@ -49,85 +55,11 @@
     <origin xyz="0 0 0." rpy="0 0 0" />
   </xacro:prbt>
-  <xacro:pg70 parent="pilztool0">
+<!-- Panda -->
+<!--   <xacro:panda_arm parent="base_link" prefix="panda">
     <origin xyz="0 0 0." rpy="0 0 0" />
-  </xacro:pg70>
+  </xacro:panda_arm> -->
   <!--+++++++++++++++++++laserscanner_link++++++++++++++++++++++++-->
   <xacro:sick_laser_v0 name="lidar_1" parent="base_link" ros_topic="lidar_1/scan_filtered">
     <origin xyz="0.230 0 0.110" rpy="0 3.14 3.14" />
   </xacro:sick_laser_v0>
-   <!--+++++++++++++++++++ IMU ++++++++++++++++++++++++-->
- <!-- Comment or uncomment based on your requirement -->
-<!--   <xacro:imu name="imu_1" parent="base_link">
-    <origin xyz="0.100 0 0.300" rpy="0 0 3.14" />
-  </xacro:imu> -->
-  <!--+++++++++++++++++++ Ultra Sonic ++++++++++++++++++++++++-->
-  <!-- Comment or uncomment based on your requirement -->
-  <!-- SENSOR 1 -->
-  <!-- xacro:us_sensor name="us_1" parent="base_link">
-    <origin xyz="0.100 0 0.300" rpy="0 3.14 3.14" />
-  </xacro:us_sensor-->
-  <!-- SENSOR 2 -->
-  <!-- xacro:us_sensor name="us_2" parent="base_link">
-    <origin xyz="0.110 0 0.300" rpy="0 3.14 3.14" />
-  </xacro:us_sensor-->
-  <!-- SENSOR 3 -->
-  <!-- xacro:us_sensor name="us_3" parent="base_link">
-    <origin xyz="0.120 0 0.300" rpy="0 3.14 3.14" />
-  </xacro:us_sensor-->
-  <!-- SENSOR 4 -->
-  <!-- xacro:us_sensor name="us_4" parent="base_link">
-    <origin xyz="0.130 0 0.300" rpy="0 3.14 3.14" />
-  </xacro:us_sensor-->
-  <!-- SENSOR 5 -->
-  <!-- xacro:us_sensor name="us_5" parent="base_link">
-    <origin xyz="0.140 0 0.300" rpy="0 3.14 3.14" />
-  </xacro:us_sensor-->
-  <!-- SENSOR 6 -->
-  <!-- xacro:us_sensor name="us_6" parent="base_link">
-    <origin xyz="0.150 0 0.300" rpy="0 3.14 3.14" />
-  </xacro:us_sensor-->
-  <!-- SENSOR 7 -->
-  <!-- xacro:us_sensor name="us_7" parent="base_link">
-    <origin xyz="0.160 0 0.300" rpy="0 3.14 3.14" />
-  </xacro:us_sensor-->
-  <!-- SENSOR 8 -->
-  <!-- xacro:us_sensor name="us_8" parent="base_link">
-    <origin xyz="0.170 0 0.300" rpy="0 3.14 3.14" />
-  </xacro:us_sensor-->
-  <!-- SENSOR 9 -->
-  <!-- xacro:us_sensor name="us_9" parent="base_link">
-    <origin xyz="0.180 0 0.300" rpy="0 3.14 3.14" />
-  </xacro:us_sensor-->
-  <!-- SENSOR 10 -->
-  <!-- xacro:us_sensor name="us_10" parent="base_link">
-    <origin xyz="0.100 0 0.300" rpy="0 3.14 3.14" />
-  </xacro:us_sensor-->
-  <!-- SENSOR 11 -->
-  <!-- xacro:us_sensor name="us_11" parent="base_link">
-    <origin xyz="0.100 0 0.300" rpy="0 3.14 3.14" />
-  </xacro:us_sensor-->
-  <!-- SENSOR 12 -->
-  <!-- xacro:us_sensor name="us_12" parent="base_link">
-    <origin xyz="0.190 0 0.300" rpy="0 3.14 3.14" />
-  </xacro:us_sensor-->
-  <!-- SENSOR 13 -->
-  <!-- xacro:us_sensor name="us_13" parent="base_link">
-    <origin xyz="0.200 0 0.300" rpy="0 3.14 3.14" />
-  </xacro:us_sensor-->
-  <!-- SENSOR 14 -->
-  <!-- xacro:us_sensor name="us_14" parent="base_link">
-    <origin xyz="0.210 0 0.300" rpy="0 3.14 3.14" />
-  </xacro:us_sensor-->
-  <!-- SENSOR 15 -->
-  <!-- xacro:us_sensor name="us_15" parent="base_link">
-    <origin xyz="0.220 0 0.300" rpy="0 3.14 3.14" />
-  </xacro:us_sensor-->
-  <!-- SENSOR 16 -->
-  <!-- xacro:us_sensor name="us_16" parent="base_link">
-    <origin xyz="0.230 0 0.300" rpy="0 3.14 3.14" />
-  </xacro:us_sensor-->
-    <!--Camera  -->
-<!-- <xacro:camera name="camera" parent="base_link">
-    <origin xyz="0 0 0.38" rpy="0 0 0" />
-  </xacro:camera> -->
 </robot>

File: robots/mm_400/urdf/xacros/camera.xacro (robot description, xacro)
@@ -2,5 +2,5 @@
 <robot xmlns:xacro="http://www.ros.org/wiki/xacro" name="mm_400">
   <xacro:macro name="camera" params="name parent *origin">
-      <xacro:property name="camera_link" value="0.05" />
+    <xacro:property name="camera_link" value="0.05" />
     <joint name="${name}_joint" type="fixed">
       <axis xyz="0 1 0" />

File: robots/mm_400/urdf/xacros/mp_400_gazebo.xacro (robot description, xacro)
@@ -13,4 +13,44 @@
     <self_collide>false</self_collide>
   </gazebo>
+<gazebo reference="wheel_front_right_link">
+      <kp>35000.0</kp>
+      <kd>1000.0</kd>
+      <mu1>0.051</mu1>
+      <mu2>0.051</mu2>
+      <fdir1>1 0 0</fdir1>
+    <maxVel>1.0</maxVel>
+    <minDepth>0.00</minDepth>
+      <implicitSpringDamper>1</implicitSpringDamper>
+</gazebo>
+<gazebo reference="wheel_front_left_link">
+      <kp>35000.0</kp>
+      <kd>1000.0</kd>
+      <mu1>0.051</mu1>
+      <mu2>0.051</mu2>
+          <fdir1>1 0 0</fdir1>
+    <maxVel>1.0</maxVel>
+    <minDepth>0.00</minDepth>
+      <implicitSpringDamper>1</implicitSpringDamper>
+</gazebo>
+<gazebo reference="wheel_back_left_link">
+      <kp>35000.0</kp>
+      <kd>1000.0</kd>
+      <mu1>0.051</mu1>
+      <mu2>0.051</mu2>
+          <fdir1>1 0 0</fdir1>
+    <maxVel>1.0</maxVel>
+    <minDepth>0.00</minDepth>
+      <implicitSpringDamper>1</implicitSpringDamper>
+</gazebo>
+<gazebo reference="wheel_back_right_link">
+      <kp>35000.0</kp>
+      <kd>1000.0</kd>
+      <mu1>0.051</mu1>
+      <mu2>0.051</mu2>
+          <fdir1>1 0 0</fdir1>
+    <maxVel>1.0</maxVel>
+    <minDepth>0.00</minDepth>
+      <implicitSpringDamper>1</implicitSpringDamper>
+</gazebo>
   <gazebo reference="lidar_1_link">
       <sensor type="ray" name="lidar_1_link">
@@ -53,5 +93,5 @@
         <updateRate>40</updateRate>
         <legacyMode>false</legacyMode>
-        <torque>5</torque>
+        <torque>0.05</torque>
         <leftJoint>fixed_wheel_left_joint</leftJoint>
         <rightJoint>fixed_wheel_right_joint</rightJoint>
@@ -66,5 +106,5 @@
         <publishWheelJointState>true</publishWheelJointState>
         <wheelAcceleration>6.0</wheelAcceleration>
-        <wheelTorque>5</wheelTorque>
+        <wheelTorque>200</wheelTorque>
         <odometrySource>world</odometrySource>
         <publishTf>1</publishTf>
@@ -72,23 +112,10 @@
     </plugin>
   </gazebo>
-    <gazebo reference="imu_1_link">
-    <gravity>true</gravity>
-    <sensor name="imu_sensor" type="imu">
-      <always_on>true</always_on>
-      <update_rate>100</update_rate>
-      <visualize>true</visualize>
-      <topic>__default_topic__</topic>
-      <plugin filename="libgazebo_ros_imu_sensor.so" name="imu_plugin">
-        <topicName>imu</topicName>
-        <bodyName>imu_link</bodyName>
-        <updateRateHZ>10.0</updateRateHZ>
-        <gaussianNoise>0.0</gaussianNoise>
-        <xyzOffset>0 0 0</xyzOffset>
-        <rpyOffset>0 0 0</rpyOffset>
-        <frameName>imu_link</frameName>
-      </plugin>
-      <pose>0 0 0 0 0 0</pose>
-    </sensor>
-  </gazebo>
+<gazebo>
+  <plugin name="ros_control" filename="libgazebo_ros_control.so">
+    <legacyModeNS>false</legacyModeNS>
+    <robotSimType>gazebo_ros_control/DefaultRobotHWSim</robotSimType>
+  </plugin>
+</gazebo>
   <gazebo reference="us_1_link">
   <!-- Visuals / Collisions omitted for this example -->
@@ -166,9 +193,3 @@
     </sensor>
   </gazebo>
-<gazebo>
-  <plugin name="ros_control" filename="libgazebo_ros_control.so">
-    <legacyModeNS>false</legacyModeNS>
-    <robotSimType>gazebo_ros_control/DefaultRobotHWSim</robotSimType>
-  </plugin>
-</gazebo>
 </robot>

File: robots/mm_400/urdf/xacros/ultrasonic.xacro (robot description, xacro)
@@ -1,4 +1,4 @@
 <?xml version="1.0"?>
-<robot xmlns:xacro="http://www.ros.org/wiki/xacro" name="mm_400">
+<robot xmlns:xacro="http://www.ros.org/wiki/xacro" name="mp_400">
   <xacro:macro name="us_sensor" params="name parent *origin">
     <joint name="${name}_joint" type="fixed">

File: robots/mp_400/xacros/mp_400_gazebo.xacro (robot description, xacro)
@@ -166,8 +166,3 @@
     </plugin>
   </gazebo>
-<!-- <gazebo>
-  <plugin name="gazebo_ros_control" filename="libgazebo_ros_control.so">
-    <robotNamespace>/mp_400</robotNamespace>
-  </plugin>
-</gazebo> -->
 </robot>

Commit message: MM-400 updated

File: robots/mm_400/mm_400.urdf.xacro (robot description, xacro)
@@ -14,11 +14,17 @@
 <!--+++++++++++++++++++cabinet++++++++++++++++++++++++-->
 <xacro:include filename="$(find neo_simulation)/robots/mm_400/urdf/xacros/cabinet.xacro" />
+<!-- PRBT -->
 <xacro:include filename="$(find neo_simulation)/robots/mm_400/urdf/prbt_macro.xacro" />
+<!-- Panda -->
+  <xacro:include filename="$(find neo_simulation)/robots/mm_400/urdf/panda_arm.xacro" />
  <!-- SENSORS -->
-<xacro:include filename="$(find neo_simulation)/robots/mm_400/urdf/xacros/sick_laser.xacro" />
-<xacro:include filename="$(find neo_simulation)/robots/mm_400/urdf/xacros/imu.xacro" />
+<!-- SENSORS -->
+<!-- <xacro:include filename="$(find neo_simulation)/robots/mm_400/urdf/xacros/sick_S300.xacro" /> -->
+<!-- Microscan - Comment/Uncomment if required -->
+<xacro:include filename="$(find neo_simulation)/robots/mm_400/urdf/xacros/micro_scan.xacro" />
+<!-- Additional sensors if required -->
+<!-- <xacro:include filename="$(find neo_simulation)/robots/mm_400/urdf/xacros/imu.xacro" />
 <xacro:include filename="$(find neo_simulation)/robots/mm_400/urdf/xacros/ultrasonic.xacro" />
-<!-- Gripper -->
-<xacro:include filename="$(find schunk_description)/pg70.urdf.xacro" />
+<xacro:include filename="$(find neo_simulation)/robots/mm_400/urdf/xacros/camera.xacro" />-->
   <xacro:mp_400_base name="base_link">
   </xacro:mp_400_base>
@@ -42,92 +48,19 @@
     <origin xyz="-0. 0.26 0.074" rpy="0 0 1.57" />
   </xacro:fixed_wheel_left>
-  <xacro:mm_400_cabinet name="cabinet" parent="base_link">
+<!--   <xacro:mm_400_cabinet name="cabinet" parent="base_link">
     <origin xyz="0.02 0 0.551" rpy="0 0 3.14" />
-  </xacro:mm_400_cabinet>
+  </xacro:mm_400_cabinet> -->
    <!-- Robot arm -->
-  <xacro:prbt parent="cabinet_link" prefix="pilz">
+<!--   <xacro:prbt parent="cabinet_link" prefix="pilz">
     <origin xyz="0 0 0." rpy="0 0 0" />
   </xacro:prbt>
-  <xacro:pg70 parent="pilztool0">
+ -->
+<!-- Panda -->
+  <xacro:panda_arm parent="base_link" prefix="panda">
     <origin xyz="0 0 0." rpy="0 0 0" />
-  </xacro:pg70>
+  </xacro:panda_arm>
   <!--+++++++++++++++++++laserscanner_link++++++++++++++++++++++++-->
   <xacro:sick_laser_v0 name="lidar_1" parent="base_link" ros_topic="lidar_1/scan_filtered">
     <origin xyz="0.230 0 0.110" rpy="0 3.14 3.14" />
   </xacro:sick_laser_v0>
-   <!--+++++++++++++++++++ IMU ++++++++++++++++++++++++-->
- <!-- Comment or uncomment based on your requirement -->
-<!--   <xacro:imu name="imu_1" parent="base_link">
-    <origin xyz="0.100 0 0.300" rpy="0 0 3.14" />
-  </xacro:imu> -->
-  <!--+++++++++++++++++++ Ultra Sonic ++++++++++++++++++++++++-->
-  <!-- Comment or uncomment based on your requirement -->
-  <!-- SENSOR 1 -->
-  <!-- xacro:us_sensor name="us_1" parent="base_link">
-    <origin xyz="0.100 0 0.300" rpy="0 3.14 3.14" />
-  </xacro:us_sensor-->
-  <!-- SENSOR 2 -->
-  <!-- xacro:us_sensor name="us_2" parent="base_link">
-    <origin xyz="0.110 0 0.300" rpy="0 3.14 3.14" />
-  </xacro:us_sensor-->
-  <!-- SENSOR 3 -->
-  <!-- xacro:us_sensor name="us_3" parent="base_link">
-    <origin xyz="0.120 0 0.300" rpy="0 3.14 3.14" />
-  </xacro:us_sensor-->
-  <!-- SENSOR 4 -->
-  <!-- xacro:us_sensor name="us_4" parent="base_link">
-    <origin xyz="0.130 0 0.300" rpy="0 3.14 3.14" />
-  </xacro:us_sensor-->
-  <!-- SENSOR 5 -->
-  <!-- xacro:us_sensor name="us_5" parent="base_link">
-    <origin xyz="0.140 0 0.300" rpy="0 3.14 3.14" />
-  </xacro:us_sensor-->
-  <!-- SENSOR 6 -->
-  <!-- xacro:us_sensor name="us_6" parent="base_link">
-    <origin xyz="0.150 0 0.300" rpy="0 3.14 3.14" />
-  </xacro:us_sensor-->
-  <!-- SENSOR 7 -->
-  <!-- xacro:us_sensor name="us_7" parent="base_link">
-    <origin xyz="0.160 0 0.300" rpy="0 3.14 3.14" />
-  </xacro:us_sensor-->
-  <!-- SENSOR 8 -->
-  <!-- xacro:us_sensor name="us_8" parent="base_link">
-    <origin xyz="0.170 0 0.300" rpy="0 3.14 3.14" />
-  </xacro:us_sensor-->
-  <!-- SENSOR 9 -->
-  <!-- xacro:us_sensor name="us_9" parent="base_link">
-    <origin xyz="0.180 0 0.300" rpy="0 3.14 3.14" />
-  </xacro:us_sensor-->
-  <!-- SENSOR 10 -->
-  <!-- xacro:us_sensor name="us_10" parent="base_link">
-    <origin xyz="0.100 0 0.300" rpy="0 3.14 3.14" />
-  </xacro:us_sensor-->
-  <!-- SENSOR 11 -->
-  <!-- xacro:us_sensor name="us_11" parent="base_link">
-    <origin xyz="0.100 0 0.300" rpy="0 3.14 3.14" />
-  </xacro:us_sensor-->
-  <!-- SENSOR 12 -->
-  <!-- xacro:us_sensor name="us_12" parent="base_link">
-    <origin xyz="0.190 0 0.300" rpy="0 3.14 3.14" />
-  </xacro:us_sensor-->
-  <!-- SENSOR 13 -->
-  <!-- xacro:us_sensor name="us_13" parent="base_link">
-    <origin xyz="0.200 0 0.300" rpy="0 3.14 3.14" />
-  </xacro:us_sensor-->
-  <!-- SENSOR 14 -->
-  <!-- xacro:us_sensor name="us_14" parent="base_link">
-    <origin xyz="0.210 0 0.300" rpy="0 3.14 3.14" />
-  </xacro:us_sensor-->
-  <!-- SENSOR 15 -->
-  <!-- xacro:us_sensor name="us_15" parent="base_link">
-    <origin xyz="0.220 0 0.300" rpy="0 3.14 3.14" />
-  </xacro:us_sensor-->
-  <!-- SENSOR 16 -->
-  <!-- xacro:us_sensor name="us_16" parent="base_link">
-    <origin xyz="0.230 0 0.300" rpy="0 3.14 3.14" />
-  </xacro:us_sensor-->
-    <!--Camera  -->
-<!-- <xacro:camera name="camera" parent="base_link">
-    <origin xyz="0 0 0.38" rpy="0 0 0" />
-  </xacro:camera> -->
 </robot>

File: robots/mpo_700/xacros/mpo_700_caster.xacro (robot description, xacro)
@@ -19,5 +19,5 @@
      <origin xyz="0 0 0.10" rpy="0 0 0"/>
      <geometry>
-        <mesh filename="package://neo_simulation/robots/mpo_700/meshes/MPO-700-caster.dae" scale="0.001 0.001 0.001"/>
+        <mesh filename="package://neo_simulation/robots/mpo_700/meshes/MPO-700-HEAD.dae" scale="0.001 0.001 0.001"/>
      </geometry>
     </visual>
@@ -25,5 +25,5 @@
      <origin xyz="0 0 0.10" rpy="0 0 0" />
      <geometry>
-        <mesh filename="package://neo_simulation/robots/mpo_700/meshes/MPO-700-caster.dae" scale="0.001 0.001 0.001"/>
+        <mesh filename="package://neo_simulation/robots/mpo_700/meshes/MPO-700-HEAD.dae" scale="0.001 0.001 0.001"/>
      </geometry>
     </collision>
@@ -47,5 +47,5 @@
      <origin xyz="0 0 0.10" rpy="0 0 0"/>
      <geometry>
-        <mesh filename="package://neo_simulation/robots/mpo_700/meshes/MPO-700-caster.dae" scale="0.001 0.001 0.001"/>
+        <mesh filename="package://neo_simulation/robots/mpo_700/meshes/MPO-700-HEAD.dae" scale="0.001 0.001 0.001"/>
      </geometry>
     </visual>
@@ -53,5 +53,5 @@
      <origin xyz="0 0 0.10" rpy="0 0 0" />
      <geometry>
-        <mesh filename="package://neo_simulation/robots/mpo_700/meshes/MPO-700-caster.dae" scale="0.001 0.001 0.001"/>
+        <mesh filename="package://neo_simulation/robots/mpo_700/meshes/MPO-700-HEAD.dae" scale="0.001 0.001 0.001"/>
      </geometry>
     </collision>
@@ -75,5 +75,5 @@
      <origin xyz="0 0 0.10" rpy="0 0 0"/>
      <geometry>
-        <mesh filename="package://neo_simulation/robots/mpo_700/meshes/MPO-700-caster.dae" scale="0.001 0.001 0.001"/>
+        <mesh filename="package://neo_simulation/robots/mpo_700/meshes/MPO-700-HEAD.dae" scale="0.001 0.001 0.001"/>
      </geometry>
     </visual>
@@ -81,5 +81,5 @@
      <origin xyz="0 0 0.10" rpy="0 0 0" />
      <geometry>
-        <mesh filename="package://neo_simulation/robots/mpo_700/meshes/MPO-700-caster.dae" scale="0.001 0.001 0.001"/>
+        <mesh filename="package://neo_simulation/robots/mpo_700/meshes/MPO-700-HEAD.dae" scale="0.001 0.001 0.001"/>
      </geometry>
     </collision>
@@ -103,5 +103,5 @@
      <origin xyz="0 0 0.10" rpy="0 0 0"/>
      <geometry>
-        <mesh filename="package://neo_simulation/robots/mpo_700/meshes/MPO-700-caster.dae" scale="0.001 0.001 0.001"/>
+        <mesh filename="package://neo_simulation/robots/mpo_700/meshes/MPO-700-HEAD.dae" scale="0.001 0.001 0.001"/>
      </geometry>
     </visual>
@@ -109,5 +109,5 @@
      <origin xyz="0 0 0.10" rpy="0 0 0" />
      <geometry>
-        <mesh filename="package://neo_simulation/robots/mpo_700/meshes/MPO-700-caster.dae" scale="0.001 0.001 0.001"/>
+        <mesh filename="package://neo_simulation/robots/mpo_700/meshes/MPO-700-HEAD.dae" scale="0.001 0.001 0.001"/>
      </geometry>
     </collision>
