Commit message: Updated the missing xacros

File: robots/mm_400/mm_400.urdf.xacro (robot description, xacro)
@@ -48,19 +48,93 @@
     <origin xyz="-0. 0.26 0.074" rpy="0 0 1.57" />
   </xacro:fixed_wheel_left>
-<!--   <xacro:mm_400_cabinet name="cabinet" parent="base_link">
+  <xacro:mm_400_cabinet name="cabinet" parent="base_link">
     <origin xyz="0.02 0 0.551" rpy="0 0 3.14" />
-  </xacro:mm_400_cabinet> -->
+  </xacro:mm_400_cabinet>
    <!-- Robot arm -->
-<!--   <xacro:prbt parent="cabinet_link" prefix="pilz">
+  <xacro:prbt parent="cabinet_link" prefix="pilz">
     <origin xyz="0 0 0." rpy="0 0 0" />
   </xacro:prbt>
- -->
 <!-- Panda -->
-  <xacro:panda_arm parent="base_link" prefix="panda">
+<!--   <xacro:panda_arm parent="base_link" prefix="panda">
     <origin xyz="0 0 0." rpy="0 0 0" />
-  </xacro:panda_arm>
+  </xacro:panda_arm> -->
   <!--+++++++++++++++++++laserscanner_link++++++++++++++++++++++++-->
   <xacro:sick_laser_v0 name="lidar_1" parent="base_link" ros_topic="lidar_1/scan_filtered">
     <origin xyz="0.230 0 0.110" rpy="0 3.14 3.14" />
   </xacro:sick_laser_v0>
+       <!--+++++++++++++++++++ IMU ++++++++++++++++++++++++-->
+ <!-- Comment or uncomment based on your requirement -->
+<!--   <xacro:imu name="imu_1" parent="base_link">
+    <origin xyz="0.100 0 0.300" rpy="0 0 3.14" />
+  </xacro:imu> -->
+  <!--+++++++++++++++++++ Ultra Sonic ++++++++++++++++++++++++-->
+  <!-- Comment or uncomment based on your requirement -->
+  <!-- SENSOR 1 -->
+  <!-- xacro:us_sensor name="us_1" parent="base_link">
+    <origin xyz="0.100 0 0.300" rpy="0 3.14 3.14" />
+  </xacro:us_sensor-->
+  <!-- SENSOR 2 -->
+  <!-- xacro:us_sensor name="us_2" parent="base_link">
+    <origin xyz="0.110 0 0.300" rpy="0 3.14 3.14" />
+  </xacro:us_sensor-->
+  <!-- SENSOR 3 -->
+  <!-- xacro:us_sensor name="us_3" parent="base_link">
+    <origin xyz="0.120 0 0.300" rpy="0 3.14 3.14" />
+  </xacro:us_sensor-->
+  <!-- SENSOR 4 -->
+  <!-- xacro:us_sensor name="us_4" parent="base_link">
+    <origin xyz="0.130 0 0.300" rpy="0 3.14 3.14" />
+  </xacro:us_sensor-->
+  <!-- SENSOR 5 -->
+  <!-- xacro:us_sensor name="us_5" parent="base_link">
+    <origin xyz="0.140 0 0.300" rpy="0 3.14 3.14" />
+  </xacro:us_sensor-->
+  <!-- SENSOR 6 -->
+  <!-- xacro:us_sensor name="us_6" parent="base_link">
+    <origin xyz="0.150 0 0.300" rpy="0 3.14 3.14" />
+  </xacro:us_sensor-->
+  <!-- SENSOR 7 -->
+  <!-- xacro:us_sensor name="us_7" parent="base_link">
+    <origin xyz="0.160 0 0.300" rpy="0 3.14 3.14" />
+  </xacro:us_sensor-->
+  <!-- SENSOR 8 -->
+  <!-- xacro:us_sensor name="us_8" parent="base_link">
+    <origin xyz="0.170 0 0.300" rpy="0 3.14 3.14" />
+  </xacro:us_sensor-->
+  <!-- SENSOR 9 -->
+  <!-- xacro:us_sensor name="us_9" parent="base_link">
+    <origin xyz="0.180 0 0.300" rpy="0 3.14 3.14" />
+  </xacro:us_sensor-->
+  <!-- SENSOR 10 -->
+  <!-- xacro:us_sensor name="us_10" parent="base_link">
+    <origin xyz="0.100 0 0.300" rpy="0 3.14 3.14" />
+  </xacro:us_sensor-->
+  <!-- SENSOR 11 -->
+  <!-- xacro:us_sensor name="us_11" parent="base_link">
+    <origin xyz="0.100 0 0.300" rpy="0 3.14 3.14" />
+  </xacro:us_sensor-->
+  <!-- SENSOR 12 -->
+  <!-- xacro:us_sensor name="us_12" parent="base_link">
+    <origin xyz="0.190 0 0.300" rpy="0 3.14 3.14" />
+  </xacro:us_sensor-->
+  <!-- SENSOR 13 -->
+  <!-- xacro:us_sensor name="us_13" parent="base_link">
+    <origin xyz="0.200 0 0.300" rpy="0 3.14 3.14" />
+  </xacro:us_sensor-->
+  <!-- SENSOR 14 -->
+  <!-- xacro:us_sensor name="us_14" parent="base_link">
+    <origin xyz="0.210 0 0.300" rpy="0 3.14 3.14" />
+  </xacro:us_sensor-->
+  <!-- SENSOR 15 -->
+  <!-- xacro:us_sensor name="us_15" parent="base_link">
+    <origin xyz="0.220 0 0.300" rpy="0 3.14 3.14" />
+  </xacro:us_sensor-->
+  <!-- SENSOR 16 -->
+  <!-- xacro:us_sensor name="us_16" parent="base_link">
+    <origin xyz="0.230 0 0.300" rpy="0 3.14 3.14" />
+  </xacro:us_sensor-->
+    <!--Camera  -->
+<!-- <xacro:camera name="camera" parent="base_link">
+    <origin xyz="0 0 0.38" rpy="0 0 0" />
+  </xacro:camera> -->
 </robot>

File: robots/mm_400/urdf/xacros/mp_400_gazebo.xacro (robot description, xacro)
@@ -193,3 +193,22 @@
     </sensor>
   </gazebo>
+    <gazebo reference="imu_1_link">
+    <gravity>true</gravity>
+    <sensor name="imu_sensor" type="imu">
+      <always_on>true</always_on>
+      <update_rate>100</update_rate>
+      <visualize>true</visualize>
+      <topic>__default_topic__</topic>
+      <plugin filename="libgazebo_ros_imu_sensor.so" name="imu_plugin">
+        <topicName>imu</topicName>
+        <bodyName>imu_link</bodyName>
+        <updateRateHZ>10.0</updateRateHZ>
+        <gaussianNoise>0.0</gaussianNoise>
+        <xyzOffset>0 0 0</xyzOffset>
+        <rpyOffset>0 0 0</rpyOffset>
+        <frameName>imu_link</frameName>
+      </plugin>
+      <pose>0 0 0 0 0 0</pose>
+    </sensor>
+  </gazebo>
 </robot>

File: robots/mmo_500/mmo_500.urdf.xacro (robot description, xacro)
@@ -16,5 +16,6 @@
   <xacro:include filename="$(find neo_simulation)/robots/mmo_500/urdf/xacros/micro_scan.xacro" />
   <!-- <xacro:include filename="$(find neo_simulation)/robots/mmo_500/urdf/xacros/imu.xacro" />
-  <xacro:include filename="$(find neo_simulation)/robots/mmo_500/urdf/xacros/ultrasonic.xacro" /> -->
+  <xacro:include filename="$(find neo_simulation)/robots/mmo_500/urdf/xacros/ultrasonic.xacro" />
+   <xacro:include filename="$(find neo_simulation)/robots/mmo_500/urdf/xacros/camera.xacro" />-->
   <!-- CABINET -->
   <xacro:include filename="$(find neo_simulation)/robots/mmo_500/urdf/xacros/cabinet.xacro" />

File: robots/mmo_700/mmo_700.urdf.xacro (robot description, xacro)
@@ -15,5 +15,6 @@
   <xacro:include filename="$(find neo_simulation)/robots/mmo_700/urdf/xacros/micro_scan.xacro" />
   <!--   <xacro:include filename="$(find neo_simulation)/robots/mmo_700/urdf/xacros/imu.xacro" />
-  <xacro:include filename="$(find neo_simulation)/robots/mmo_700/urdf/xacros/ultrasonic.xacro" /> -->
+  <xacro:include filename="$(find neo_simulation)/robots/mmo_700/urdf/xacros/ultrasonic.xacro" />
+ <xacro:include filename="$(find neo_simulation)/robots/mmo_700/urdf/xacros/camera.xacro" -->
   <!-- Gazebo -->
   <xacro:include filename="$(find neo_simulation)/robots/mmo_700/urdf/xacros/mpo_700_gazebo.xacro" />

File: robots/mp_400/mp_400.urdf.xacro (robot description, xacro)
@@ -13,7 +13,12 @@
 <xacro:include filename="$(find neo_simulation)/robots/mp_400/xacros/mp_400_fixed_wheel_right.xacro" />
 <!-- SENSORS -->
-<xacro:include filename="$(find neo_simulation)/robots/mp_400/xacros/sick_laser.xacro" />
+<!-- Micro_scan -->
+<xacro:include filename="$(find neo_simulation)/robots/mp_400/xacros/micro_scan.xacro" />
+<!-- Sick s300 -->
+<!-- <xacro:include filename="$(find neo_simulation)/robots/mp_400/xacros/sick_S300.xacro" /> -->
+<!-- USS, IMU and Camera, UNcomment if required -->
+<!-- <xacro:include filename="$(find neo_simulation)/robots/mp_400/xacros/camera.xacro" />
 <xacro:include filename="$(find neo_simulation)/robots/mp_400/xacros/imu.xacro" />
-<xacro:include filename="$(find neo_simulation)/robots/mp_400/xacros/ultrasonic.xacro" />
+<xacro:include filename="$(find neo_simulation)/robots/mp_400/xacros/ultrasonic.xacro" /> -->
 <!-- Base link macro -->
   <xacro:mp_400_base name="base_link">

File: robots/mp_500/mp_500.urdf.xacro (robot description, xacro)
@@ -17,5 +17,6 @@
   <!-- USS and IMU - Comment/Uncomment if required  -->
   <!-- <xacro:include filename="$(find neo_simulation)/robots/mp_500/xacros/imu.xacro" />
-  <xacro:include filename="$(find neo_simulation)/robots/mp_500/xacros/ultrasonic.xacro" /> -->
+  <xacro:include filename="$(find neo_simulation)/robots/mp_500/xacros/ultrasonic.xacro" />
+  <xacro:include filename="$(find neo_simulation)/robots/mp_500/xacros/camera.xacro" /> -->-->
   <xacro:mp_500_base name="base_link">
   </xacro:mp_500_base>

File: robots/mpo_500/mpo_500.urdf.xacro (robot description, xacro)
@@ -8,10 +8,11 @@
   <xacro:include filename="$(find neo_simulation)/robots/mpo_500/xacros/omni_wheel.xacro" />
   <!-- SENSORS -->
-  <xacro:include filename="$(find neo_simulation)/robots/mpo_500/xacros/sick_S300.xacro" />
+  <!-- <xacro:include filename="$(find neo_simulation)/robots/mpo_500/xacros/sick_S300.xacro" /> -->
   <!-- Microscan - Comment/Uncomment if required -->
-  <!-- <xacro:include filename="$(find neo_simulation)/robots/mpo_500/xacros/micro_scan.xacro" />  -->
+  <xacro:include filename="$(find neo_simulation)/robots/mpo_500/xacros/micro_scan.xacro" />
+  <!--Ultrasonics, cameras and IMU's  -->
   <!--<xacro:include filename="$(find neo_simulation)/robots/mpo_500/xacros/imu.xacro" />
   <xacro:include filename="$(find neo_simulation)/robots/mpo_500/xacros/ultrasonic.xacro" /> -->
-  <xacro:include filename="$(find neo_simulation)/robots/mpo_500/xacros/mpo_500_gazebo.xacro" />
+  <!-- <xacro:include filename="$(find neo_simulation)/robots/mpo_500/xacros/camera.xacro" />  -->
   <!-- Base Macro-->
   <xacro:mpo_500_base name="base_link">
@@ -19,21 +20,96 @@
   <!-- Wheel Macro -->
   <xacro:omni_wheel_250 name="wheel_front_left" parent="base_link">
-  	<origin xyz="0.25 0.28 0.13" rpy="0 0 0" />
+    <origin xyz="0.25 0.28 0.13" rpy="0 0 0" />
   </xacro:omni_wheel_250>
   <xacro:omni_wheel_250 name="wheel_front_right" parent="base_link">
-  	<origin xyz="0.25 -0.28 0.13" rpy="0 0 3.14" />
+    <origin xyz="0.25 -0.28 0.13" rpy="0 0 3.14" />
   </xacro:omni_wheel_250>
   <xacro:omni_wheel_250 name="wheel_back_left" parent="base_link">
-  	<origin xyz="-0.25 0.28 0.13" rpy="0 0 0" />
+    <origin xyz="-0.25 0.28 0.13" rpy="0 0 0" />
   </xacro:omni_wheel_250>
   <xacro:omni_wheel_250 name="wheel_back_right" parent="base_link">
-  	<origin xyz="-0.25 -0.28 0.13" rpy="0 0 3.14" />
+    <origin xyz="-0.25 -0.28 0.13" rpy="0 0 3.14" />
   </xacro:omni_wheel_250>
   <!-- Sensors -->
-  <xacro:sick_laser_v0 name="lidar_1" parent="base_link" ros_topic="lidar_1/scan">
-  	<origin xyz="0.442 0 0.372" rpy="0 0 0" />
+  <xacro:sick_laser_v0 name="lidar_1" parent="base_link" ros_topic="lidar_1/scan_filtered">
+    <origin xyz="0.442 0 0.372" rpy="0 0 0" />
   </xacro:sick_laser_v0>
-  <xacro:sick_laser_v0 name="lidar_2" parent="base_link" ros_topic="lidar_2/scan">
-  	<origin xyz="-0.442 0 0.372" rpy="0 0 3.14" />
+  <xacro:sick_laser_v0 name="lidar_2" parent="base_link" ros_topic="lidar_2/scan_filtered">
+    <origin xyz="-0.442 0 0.372" rpy="0 0 3.14" />
   </xacro:sick_laser_v0>
+      <!--+++++++++++++++++++ IMU ++++++++++++++++++++++++-->
+ <!-- Comment or uncomment based on your requirement -->
+<!--   <xacro:imu name="imu_1" parent="base_link">
+    <origin xyz="0.100 0 0.300" rpy="0 0 3.14" />
+  </xacro:imu> -->
+  <!--+++++++++++++++++++ Ultra Sonic ++++++++++++++++++++++++-->
+  <!-- Comment or uncomment based on your requirement -->
+  <!-- SENSOR 1 -->
+  <!-- xacro:us_sensor name="us_1" parent="base_link">
+    <origin xyz="0.100 0 0.300" rpy="0 3.14 3.14" />
+  </xacro:us_sensor-->
+  <!-- SENSOR 2 -->
+  <!-- xacro:us_sensor name="us_2" parent="base_link">
+    <origin xyz="0.110 0 0.300" rpy="0 3.14 3.14" />
+  </xacro:us_sensor-->
+  <!-- SENSOR 3 -->
+  <!-- xacro:us_sensor name="us_3" parent="base_link">
+    <origin xyz="0.120 0 0.300" rpy="0 3.14 3.14" />
+  </xacro:us_sensor-->
+  <!-- SENSOR 4 -->
+  <!-- xacro:us_sensor name="us_4" parent="base_link">
+    <origin xyz="0.130 0 0.300" rpy="0 3.14 3.14" />
+  </xacro:us_sensor-->
+  <!-- SENSOR 5 -->
+  <!-- xacro:us_sensor name="us_5" parent="base_link">
+    <origin xyz="0.140 0 0.300" rpy="0 3.14 3.14" />
+  </xacro:us_sensor-->
+  <!-- SENSOR 6 -->
+  <!-- xacro:us_sensor name="us_6" parent="base_link">
+    <origin xyz="0.150 0 0.300" rpy="0 3.14 3.14" />
+  </xacro:us_sensor-->
+  <!-- SENSOR 7 -->
+  <!-- xacro:us_sensor name="us_7" parent="base_link">
+    <origin xyz="0.160 0 0.300" rpy="0 3.14 3.14" />
+  </xacro:us_sensor-->
+  <!-- SENSOR 8 -->
+  <!-- xacro:us_sensor name="us_8" parent="base_link">
+    <origin xyz="0.170 0 0.300" rpy="0 3.14 3.14" />
+  </xacro:us_sensor-->
+  <!-- SENSOR 9 -->
+  <!-- xacro:us_sensor name="us_9" parent="base_link">
+    <origin xyz="0.180 0 0.300" rpy="0 3.14 3.14" />
+  </xacro:us_sensor-->
+  <!-- SENSOR 10 -->
+  <!-- xacro:us_sensor name="us_10" parent="base_link">
+    <origin xyz="0.100 0 0.300" rpy="0 3.14 3.14" />
+  </xacro:us_sensor-->
+  <!-- SENSOR 11 -->
+  <!-- xacro:us_sensor name="us_11" parent="base_link">
+    <origin xyz="0.100 0 0.300" rpy="0 3.14 3.14" />
+  </xacro:us_sensor-->
+  <!-- SENSOR 12 -->
+  <!-- xacro:us_sensor name="us_12" parent="base_link">
+    <origin xyz="0.190 0 0.300" rpy="0 3.14 3.14" />
+  </xacro:us_sensor-->
+  <!-- SENSOR 13 -->
+  <!-- xacro:us_sensor name="us_13" parent="base_link">
+    <origin xyz="0.200 0 0.300" rpy="0 3.14 3.14" />
+  </xacro:us_sensor-->
+  <!-- SENSOR 14 -->
+  <!-- xacro:us_sensor name="us_14" parent="base_link">
+    <origin xyz="0.210 0 0.300" rpy="0 3.14 3.14" />
+  </xacro:us_sensor-->
+  <!-- SENSOR 15 -->
+  <!-- xacro:us_sensor name="us_15" parent="base_link">
+    <origin xyz="0.220 0 0.300" rpy="0 3.14 3.14" />
+  </xacro:us_sensor-->
+  <!-- SENSOR 16 -->
+  <!-- xacro:us_sensor name="us_16" parent="base_link">
+    <origin xyz="0.230 0 0.300" rpy="0 3.14 3.14" />
+  </xacro:us_sensor-->
+      <!--Camera  -->
+<!-- <xacro:camera name="camera" parent="base_link">
+    <origin xyz="0 0 0.38" rpy="0 0 0" />
+  </xacro:camera> -->
 </robot>

File: robots/mpo_500/xacros/mpo_500_gazebo.xacro (robot description, xacro)
@@ -86,8 +86,88 @@
           </ray>
           <plugin name="lidar_2" filename="libgazebo_ros_laser.so">
-            <topicName>lidar_2/scan</topicName>
+            <topicName>lidar_2/scan_filtered</topicName>
             <frameName>lidar_2_link</frameName>
           </plugin>
         </sensor>
+  </gazebo>
+ <gazebo reference="camera_link">
+    <sensor type="camera" name="camera1">
+      <update_rate>30.0</update_rate>
+      <camera name="head">
+        <horizontal_fov>1.3962634</horizontal_fov>
+        <image>
+          <width>800</width>
+          <height>800</height>
+          <format>R8G8B8</format>
+        </image>
+        <clip>
+          <near>0.02</near>
+          <far>300</far>
+        </clip>
+        <noise>
+          <type>gaussian</type>
+          <mean>0.0</mean>
+          <stddev>0.007</stddev>
+        </noise>
+      </camera>
+      <plugin name="camera_controller" filename="libgazebo_ros_camera.so">
+        <alwaysOn>true</alwaysOn>
+        <updateRate>0.0</updateRate>
+        <cameraName>camera1</cameraName>
+        <imageTopicName>image_raw</imageTopicName>
+        <cameraInfoTopicName>camera_info</cameraInfoTopicName>
+        <frameName>camera_link</frameName>
+        <hackBaseline>0.07</hackBaseline>
+        <distortionK1>0.0</distortionK1>
+        <distortionK2>0.0</distortionK2>
+        <distortionK3>0.0</distortionK3>
+        <distortionT1>0.0</distortionT1>
+        <distortionT2>0.0</distortionT2>
+      </plugin>
+    </sensor>
+  </gazebo>
+      <gazebo reference="imu_1_link">
+    <gravity>true</gravity>
+    <sensor name="imu_sensor" type="imu">
+      <always_on>true</always_on>
+      <update_rate>100</update_rate>
+      <visualize>true</visualize>
+      <topic>__default_topic__</topic>
+      <plugin filename="libgazebo_ros_imu_sensor.so" name="imu_plugin">
+        <topicName>imu</topicName>
+        <bodyName>imu_link</bodyName>
+        <updateRateHZ>10.0</updateRateHZ>
+        <gaussianNoise>0.0</gaussianNoise>
+        <xyzOffset>0 0 0</xyzOffset>
+        <rpyOffset>0 0 0</rpyOffset>
+        <frameName>imu_link</frameName>
+      </plugin>
+      <pose>0 0 0 0 0 0</pose>
+    </sensor>
+  </gazebo>
+  <gazebo reference="us_1_link">
+  <sensor type="ray" name="range">
+    <ray>
+         <scan>
+            <horizontal>
+               <samples>1</samples>
+               <resolution>1.0</resolution>
+               <min_angle>-0.01</min_angle>
+               <max_angle>0.01</max_angle>
+            </horizontal>
+            <vertical>
+               <samples>1</samples>
+               <resolution>1</resolution>
+               <min_angle>-0.01</min_angle>
+               <max_angle>0.01</max_angle>
+            </vertical>
+         </scan>
+         <range>
+            <min>0.01</min>
+            <max>3.75</max>
+            <resolution>0.02</resolution>
+         </range>
+      </ray>
+      </sensor>
   </gazebo>
   <gazebo>

File: robots/mpo_700/mpo_700.urdf.xacro (robot description, xacro)
@@ -8,9 +8,13 @@
   <!-- Microscan - Comment/Uncomment if required -->
   <xacro:include filename="$(find neo_simulation)/robots/mpo_700/xacros/micro_scan.xacro" />
+  <!--Ultrasonics, cameras and IMU's  -->
+  <!-- <xacro:include filename="$(find neo_simulation)/robots/mpo_700/xacros/camera.xacro" /> -->
   <!--<xacro:include filename="$(find neo_simulation)/robots/mpo_700/xacros/imu.xacro" />
   <xacro:include filename="$(find neo_simulation)/robots/mpo_700/xacros/ultrasonic.xacro" /> -->
+  <!--Gazebo  -->
   <xacro:include filename="$(find neo_simulation)/robots/mpo_700/xacros/mpo_700_gazebo.xacro" />
-<!-- Caster and wheels -->
+  <!--Caster  -->
   <xacro:include filename="$(find neo_simulation)/robots/mpo_700/xacros/mpo_700_caster.xacro" />
+  <!-- Wheels -->
   <xacro:include filename="$(find neo_simulation)/robots/mpo_700/xacros/mpo_700_wheel.xacro" />
   <!-- Base Macro-->
@@ -124,5 +128,4 @@
 <!-- <xacro:camera name="camera" parent="base_link">
     <origin xyz="0 0 0.38" rpy="0 0 0" />
-  </xacro:camera>
- -->
+  </xacro:camera> -->
 </robot>

File: robots/mpo_700/xacros/mpo_700_gazebo.xacro (robot description, xacro)
@@ -95,4 +95,13 @@
   </gazebo>
     <!-- camera -->
+ <gazebo>
+    <plugin name="mpo_700_controller" filename="libgazebo_ros_planar_move.so">
+      <commandTopic>cmd_vel</commandTopic>
+      <odometryTopic>odom</odometryTopic>
+      <odometryFrame>odom</odometryFrame>
+      <odometryRate>20.0</odometryRate>
+      <robotBaseFrame>base_link</robotBaseFrame>
+    </plugin>
+  </gazebo>
   <gazebo reference="camera_link">
     <sensor type="camera" name="camera1">
@@ -134,12 +143,29 @@
     </sensor>
   </gazebo>
- <gazebo>
-    <plugin name="mpo_700_controller" filename="libgazebo_ros_planar_move.so">
-      <commandTopic>cmd_vel</commandTopic>
-      <odometryTopic>odom</odometryTopic>
-      <odometryFrame>odom</odometryFrame>
-      <odometryRate>20.0</odometryRate>
-      <robotBaseFrame>base_link</robotBaseFrame>
-    </plugin>
+    <gazebo reference="us_1_link">
+  <!-- Visuals / Collisions omitted for this example -->
+  <sensor type="ray" name="range">
+    <ray>
+         <scan>
+            <horizontal>
+               <samples>1</samples>
+               <resolution>1.0</resolution>
+               <min_angle>-0.01</min_angle>
+               <max_angle>0.01</max_angle>
+            </horizontal>
+            <vertical>
+               <samples>1</samples>
+               <resolution>1</resolution>
+               <min_angle>-0.01</min_angle>
+               <max_angle>0.01</max_angle>
+            </vertical>
+         </scan>
+         <range>
+            <min>0.01</min>
+            <max>3.75</max>
+            <resolution>0.02</resolution>
+         </range>
+      </ray>
+      </sensor>
   </gazebo>
 </robot>
