Commit message: Sensors fixed, comments added.

File: robots/mm_400/mm_400.urdf.xacro (robot description, xacro)
@@ -23,8 +23,7 @@
 <!-- Microscan - Comment/Uncomment if required -->
 <xacro:include filename="$(find neo_simulation)/robots/mm_400/urdf/xacros/micro_scan.xacro" />
-<!-- Additional sensors if required -->
-<!-- <xacro:include filename="$(find neo_simulation)/robots/mm_400/urdf/xacros/imu.xacro" />
-<xacro:include filename="$(find neo_simulation)/robots/mm_400/urdf/xacros/ultrasonic.xacro" />
-<xacro:include filename="$(find neo_simulation)/robots/mm_400/urdf/xacros/camera.xacro" />-->
+<!-- Additional sensors if required
+<xacro:include filename="$(find neo_simulation)/robots/mm_400/urdf/xacros/imu.xacro" />
+<xacro:include filename="$(find neo_simulation)/robots/mm_400/urdf/xacros/ultrasonic.xacro" /> <xacro:include filename="$(find neo_simulation)/robots/mm_400/urdf/xacros/camera.xacro" />-->
   <xacro:mp_400_base name="base_link">
   </xacro:mp_400_base>
@@ -48,13 +47,14 @@
     <origin xyz="-0. 0.26 0.074" rpy="0 0 1.57" />
   </xacro:fixed_wheel_left>
+<!--  -->
   <xacro:mm_400_cabinet name="cabinet" parent="base_link">
     <origin xyz="0.02 0 0.551" rpy="0 0 3.14" />
   </xacro:mm_400_cabinet>
-   <!-- Robot arm -->
+   <!-- Robot arm  -->
   <xacro:prbt parent="cabinet_link" prefix="pilz">
     <origin xyz="0 0 0." rpy="0 0 0" />
   </xacro:prbt>
 <!-- Panda -->
-<!--   <xacro:panda_arm parent="base_link" prefix="panda">
+<!--  <xacro:panda_arm parent="base_link" prefix="panda">
     <origin xyz="0 0 0." rpy="0 0 0" />
   </xacro:panda_arm> -->
@@ -63,15 +63,15 @@
     <origin xyz="0.230 0 0.110" rpy="0 3.14 3.14" />
   </xacro:sick_laser_v0>
-       <!--+++++++++++++++++++ IMU ++++++++++++++++++++++++-->
- <!-- Comment or uncomment based on your requirement -->
-<!--   <xacro:imu name="imu_1" parent="base_link">
+  <!--+++++++++++++++++++ IMU ++++++++++++++++++++++++-->
+  <!-- Comment or uncomment based on your requirement
+  <xacro:imu name="imu_1" parent="base_link">
     <origin xyz="0.100 0 0.300" rpy="0 0 3.14" />
-  </xacro:imu> -->
+  </xacro:imu>-->
   <!--+++++++++++++++++++ Ultra Sonic ++++++++++++++++++++++++-->
   <!-- Comment or uncomment based on your requirement -->
-  <!-- SENSOR 1 -->
-  <!-- xacro:us_sensor name="us_1" parent="base_link">
-    <origin xyz="0.100 0 0.300" rpy="0 3.14 3.14" />
-  </xacro:us_sensor-->
+  <!-- SENSOR 1
+  <xacro:us_sensor name="us_1" parent="base_link">
+    <origin xyz="0.300 0 0.500" rpy="0 3.14 3.14" />
+  </xacro:us_sensor>-->
   <!-- SENSOR 2 -->
   <!-- xacro:us_sensor name="us_2" parent="base_link">

File: robots/mm_400/urdf/xacros/mp_400_gazebo.xacro (robot description, xacro)
@@ -53,4 +53,5 @@
       <implicitSpringDamper>1</implicitSpringDamper>
 </gazebo>
+  <!-- Lidar -->
   <gazebo reference="lidar_1_link">
       <sensor type="ray" name="lidar_1_link">
@@ -112,5 +113,6 @@
     </plugin>
   </gazebo>
-  <gazebo reference="imu_1_link">
+  <!-- IMU sensor -->
+  <gazebo reference="imu_link">
     <gravity>true</gravity>
     <sensor name="imu_sensor" type="imu">
@@ -137,4 +139,5 @@
   </plugin>
 </gazebo>
+  <!-- Ultrasonic sensors -->
   <gazebo reference="us_1_link">
   <!-- Visuals / Collisions omitted for this example -->
@@ -165,5 +168,5 @@
          <alwaysOn>true</alwaysOn>
          <updateRate>50</updateRate>
-         <topicName>us_sensor</topicName>
+         <topicName>ultrasonic/us1</topicName>
          <frameName>us_1_link</frameName>
          <radiation>SONAR</radiation>
@@ -172,5 +175,5 @@
   </sensor>
   </gazebo>
-    <!-- camera -->
+  <!-- camera -->
   <gazebo reference="camera_link">
     <sensor type="camera" name="camera1">

File: robots/mmo_500/urdf/xacros/mpo_500_gazebo.xacro (robot description, xacro)
@@ -21,4 +21,5 @@
     <self_collide>false</self_collide>
   </gazebo>
+  <!-- Lidar sensors -->
   <gazebo reference="lidar_1_link">
       <sensor type="ray" name="lidar_1_sensor">
@@ -91,5 +92,6 @@
         </sensor>
   </gazebo>
-    <gazebo reference="imu_1_link">
+  <!-- IMU sensor -->
+  <gazebo reference="imu_link">
     <gravity>true</gravity>
     <sensor name="imu_sensor" type="imu">
@@ -110,4 +112,5 @@
     </sensor>
   </gazebo>
+  <!-- Ultrasonic sensors -->
   <gazebo reference="us_1_link">
   <!-- Visuals / Collisions omitted for this example -->
@@ -145,5 +148,5 @@
   </sensor>
   </gazebo>
-    <!-- camera -->
+  <!-- camera -->
   <gazebo reference="camera_link">
     <sensor type="camera" name="camera1">

File: robots/mmo_700/mmo_700.urdf.xacro (robot description, xacro)
@@ -15,6 +15,8 @@
   <xacro:include filename="$(find neo_simulation)/robots/mmo_700/urdf/xacros/micro_scan.xacro" />
   <!--Ultrasonics, cameras and IMU's  -->
-  <!--   <xacro:include filename="$(find neo_simulation)/robots/mmo_700/urdf/xacros/imu.xacro" />
-  <xacro:include filename="$(find neo_simulation)/robots/mmo_700/urdf/xacros/ultrasonic.xacro" /> -->
+  <!-->
+  <xacro:include filename="$(find neo_simulation)/robots/mmo_700/urdf/xacros/imu.xacro" />
+  <xacro:include filename="$(find neo_simulation)/robots/mmo_700/urdf/xacros/ultrasonic.xacro" />
+  <-->
   <!-- <xacro:include filename="$(find neo_simulation)/robots/mmo_700/urdf/xacros/camera.xacro" />  -->
   <!-- Gazebo -->
@@ -63,14 +65,18 @@
   </xacro:sick_laser_v0>
      <!--+++++++++++++++++++ IMU ++++++++++++++++++++++++-->
- <!-- Comment or uncomment based on your requirement -->
-<!--   <xacro:imu name="imu_1" parent="base_link">
+  <!-- Comment or uncomment based on your requirement -->
+  <!-->
+  <xacro:imu name="imu" parent="base_link">
     <origin xyz="0.100 0 0.300" rpy="0 0 3.14" />
-  </xacro:imu> -->
+  </xacro:imu>
+  <-->
   <!--+++++++++++++++++++ Ultra Sonic ++++++++++++++++++++++++-->
   <!-- Comment or uncomment based on your requirement -->
   <!-- SENSOR 1 -->
-  <!-- xacro:us_sensor name="us_1" parent="base_link">
-    <origin xyz="0.100 0 0.300" rpy="0 3.14 3.14" />
-  </xacro:us_sensor-->
+  <!-->
+  <xacro:us_sensor name="us_1" parent="base_link">
+    <origin xyz="0.400 0 0.500" rpy="0 3.14 3.14" />
+  </xacro:us_sensor>
+  <-->
   <!-- SENSOR 2 -->
   <!-- xacro:us_sensor name="us_2" parent="base_link">
@@ -133,4 +139,9 @@
     <origin xyz="0.230 0 0.300" rpy="0 3.14 3.14" />
   </xacro:us_sensor-->
+  <!--Camera  -->
+  <!--><xacro:camera name="camera" parent="base_link">
+    <origin xyz="0 0 0.38" rpy="0 0 0" />
+  </xacro:camera>
+  <-->
   <!--cabinet-->
   <xacro:mmo_700_cabinet name="cabinet" parent="base_link">

File: robots/mmo_700/urdf/xacros/mpo_700_gazebo.xacro (robot description, xacro)
@@ -5,4 +5,5 @@
     <self_collide>false</self_collide>
   </gazebo>
+  <!-- Lidar sensors -->
   <gazebo reference="lidar_1_link">
       <sensor type="ray" name="lidar_1_sensor">
@@ -75,4 +76,5 @@
         </sensor>
   </gazebo>
+   <!-- IMU sensor -->
     <gazebo reference="imu_link">
     <gravity>true</gravity>
@@ -93,4 +95,40 @@
       <pose>0 0 0 0 0 0</pose>
     </sensor>
+  </gazebo>
+  <!-- Sonar -->
+  <gazebo reference="us_1_link">
+  <!-- Visuals / Collisions omitted for this example -->
+  <sensor type="ray" name="range">
+    <ray>
+         <scan>
+            <horizontal>
+               <samples>1</samples>
+               <resolution>1.0</resolution>
+               <min_angle>-0.01</min_angle>
+               <max_angle>0.01</max_angle>
+            </horizontal>
+            <vertical>
+               <samples>1</samples>
+               <resolution>1</resolution>
+               <min_angle>-0.01</min_angle>
+               <max_angle>0.01</max_angle>
+            </vertical>
+         </scan>
+         <range>
+            <min>0.01</min>
+            <max>3.75</max>
+            <resolution>0.02</resolution>
+         </range>
+      </ray>
+      <plugin filename="libgazebo_ros_range.so" name="gazebo_ros_range">
+	<gaussianNoise>0.005</gaussianNoise>
+	<alwaysOn>true</alwaysOn>
+	<updateRate>50</updateRate>
+	<topicName>ultrasonic/us1</topicName>
+	<frameName>us_1_link</frameName>
+	<radiation>INFRARED</radiation>
+	<fov>0.2967</fov>
+      </plugin>
+      </sensor>
   </gazebo>
     <!-- camera -->

File: robots/mp_400/mp_400.urdf.xacro (robot description, xacro)
@@ -17,8 +17,8 @@
   <!--Sick Micro-scan  -->
   <xacro:include filename="$(find neo_simulation)/robots/mp_400/xacros/micro_scan.xacro" />
-    <!--Ultrasonics, cameras and IMU's  -->
-<!-- <xacro:include filename="$(find neo_simulation)/robots/mp_400/xacros/camera.xacro" /> -->
-<!-- <xacro:include filename="$(find neo_simulation)/robots/mp_400/xacros/imu.xacro" /> -->
-<!-- <xacro:include filename="$(find neo_simulation)/robots/mp_400/xacros/ultrasonic.xacro" /> -->
+  <!--Ultrasonics, cameras and IMU's  -->
+<!-- <xacro:include filename="$(find neo_simulation)/robots/mp_400/xacros/camera.xacro" />
+  <xacro:include filename="$(find neo_simulation)/robots/mp_400/xacros/imu.xacro" />
+  <xacro:include filename="$(find neo_simulation)/robots/mp_400/xacros/ultrasonic.xacro" />-->
 <!-- Base link macro -->
   <xacro:mp_400_base name="base_link">
@@ -47,15 +47,15 @@
     <origin xyz="0.230 0 0.110" rpy="0 3.14 3.14" />
   </xacro:sick_laser_v0>
-     <!--+++++++++++++++++++ IMU ++++++++++++++++++++++++-->
- <!-- Comment or uncomment based on your requirement -->
-<!--   <xacro:imu name="imu_1" parent="base_link">
+  <!--+++++++++++++++++++ IMU ++++++++++++++++++++++++-->
+  <!-- Comment or uncomment based on your requirement -->
+  <!--><xacro:imu name="imu" parent="base_link">
     <origin xyz="0.100 0 0.300" rpy="0 0 3.14" />
-  </xacro:imu> -->
+  </xacro:imu><-->
   <!--+++++++++++++++++++ Ultra Sonic ++++++++++++++++++++++++-->
   <!-- Comment or uncomment based on your requirement -->
   <!-- SENSOR 1 -->
-  <!-- xacro:us_sensor name="us_1" parent="base_link">
-    <origin xyz="0.100 0 0.300" rpy="0 3.14 3.14" />
-  </xacro:us_sensor-->
+  <!--><xacro:us_sensor name="us_1" parent="base_link">
+    <origin xyz="0.100 0 0.500" rpy="0 3.14 3.14" />
+  </xacro:us_sensor><-->
   <!-- SENSOR 2 -->
   <!-- xacro:us_sensor name="us_2" parent="base_link">

File: robots/mp_400/xacros/mp_400_fixed_wheel_left.xacro (robot description, xacro)
@@ -31,10 +31,9 @@
 </link>
 <gazebo reference="${name}_link">
-      <kp>600.0</kp>
-      <kd>1465.0</kd>
-      <mu1>200</mu1>
+      <kp>100000.0</kp>
+      <kd>50.0</kd>
+      <gravity> 1 </gravity>
+      <mu1>100</mu1>
       <mu2>100</mu2>
-      <fdir1>.5 0 0</fdir1>
-      <maxVel>3.0</maxVel>
       <minDepth>0.00</minDepth>
       <implicitSpringDamper>1</implicitSpringDamper>

File: robots/mp_400/xacros/mp_400_fixed_wheel_right.xacro (robot description, xacro)
@@ -30,14 +30,13 @@
     </collision>
 </link>
-<gazebo reference="${name}_link">
-      <kp>600.0</kp> <!-- Partial Ziegler-Nichols method -->
-      <kd>1465.0</kd>
-      <mu1>200</mu1>
+  <gazebo reference="${name}_link">
+      <kp>100000.0</kp>
+      <kd>50.0</kd>
+      <gravity> 1 </gravity>
+      <mu1>100</mu1>
       <mu2>100</mu2>
-      <fdir1>.5 0 0</fdir1>
-      <maxVel>3.0</maxVel>
       <minDepth>0.00</minDepth>
       <implicitSpringDamper>1</implicitSpringDamper>
-</gazebo>
+  </gazebo>
   </xacro:macro>
 </robot>

File: robots/mp_400/xacros/mp_400_gazebo.xacro (robot description, xacro)
@@ -13,4 +13,5 @@
     <self_collide>false</self_collide>
   </gazebo>
+  <!-- Lidar sensor -->
   <gazebo reference="laser_1_link">
       <sensor type="ray" name="laser_1_link">
@@ -48,5 +49,6 @@
         </sensor>
   </gazebo>
-    <gazebo reference="imu_1_link">
+  <!-- IMU sensor -->
+  <gazebo reference="imu_link">
     <gravity>true</gravity>
     <sensor name="imu_sensor" type="imu">
@@ -67,4 +69,5 @@
     </sensor>
   </gazebo>
+  <!-- Ultrasonic sensor -->
   <gazebo reference="us_1_link">
   <!-- Visuals / Collisions omitted for this example -->
@@ -91,16 +94,16 @@
          </range>
       </ray>
-      </sensor>
-    <plugin name="libgazebo_ros_range" filename="libgazebo_ros_range.so">
+      <plugin name="libgazebo_ros_range" filename="libgazebo_ros_range.so">
          <gaussianNoise>0.005</gaussianNoise>
          <alwaysOn>true</alwaysOn>
          <updateRate>50</updateRate>
-         <topicName>us_sensor</topicName>
+         <topicName>ultrasonic/us1</topicName>
          <frameName>us_1_link</frameName>
          <radiation>SONAR</radiation>
          <fov>0.2967</fov>
-    </plugin>
+      </plugin>
+  </sensor>
   </gazebo>
-    <!-- camera -->
+  <!-- camera -->
   <gazebo reference="camera_link">
     <sensor type="camera" name="camera1">
@@ -147,5 +150,5 @@
         <updateRate>40</updateRate>
         <legacyMode>false</legacyMode>
-        <torque>5</torque>
+	<torque>2</torque>
         <leftJoint>fixed_wheel_left_joint</leftJoint>
         <rightJoint>fixed_wheel_right_joint</rightJoint>
@@ -159,6 +162,6 @@
         <publishWheelTF>true</publishWheelTF>
         <publishWheelJointState>true</publishWheelJointState>
-        <wheelAcceleration>6.0</wheelAcceleration>
-        <wheelTorque>5</wheelTorque>
+        <wheelAcceleration>0.0</wheelAcceleration>
+        <wheelTorque>2</wheelTorque>
         <odometrySource>world</odometrySource>
         <publishTf>1</publishTf>

File: robots/mp_500/mp_500.urdf.xacro (robot description, xacro)
@@ -16,7 +16,9 @@
   <!-- <xacro:include filename="$(find neo_simulation)/robots/mp_500/xacros/micro_scan.xacro" /> -->
   <!-- USS, IMU and Camera- Comment/Uncomment if required  -->
-  <!-- <xacro:include filename="$(find neo_simulation)/robots/mp_500/xacros/imu.xacro" />
-  <xacro:include filename="$(find neo_simulation)/robots/mp_500/xacros/ultrasonic.xacro" /> -->
-    <!-- <xacro:include filename="$(find neo_simulation)/robots/mp_500/xacros/camera.xacro" />  -->
+  <!-->
+  <xacro:include filename="$(find neo_simulation)/robots/mp_500/xacros/imu.xacro" />
+  <xacro:include filename="$(find neo_simulation)/robots/mp_500/xacros/ultrasonic.xacro" />
+  <xacro:include filename="$(find neo_simulation)/robots/mp_500/xacros/camera.xacro" />
+  <-->
   <xacro:mp_500_base name="base_link">
   </xacro:mp_500_base>
@@ -37,14 +39,14 @@
   </xacro:sick_laser_v0>
      <!--+++++++++++++++++++ IMU ++++++++++++++++++++++++-->
- <!-- Comment or uncomment based on your requirement -->
-<!--   <xacro:imu name="imu_1" parent="base_link">
+  <!-- Comment or uncomment based on your requirement -->
+  <!--><xacro:imu name="imu" parent="base_link">
     <origin xyz="0.100 0 0.300" rpy="0 0 3.14" />
-  </xacro:imu> -->
+  </xacro:imu><-->
   <!--+++++++++++++++++++ Ultra Sonic ++++++++++++++++++++++++-->
   <!-- Comment or uncomment based on your requirement -->
   <!-- SENSOR 1 -->
-  <!-- xacro:us_sensor name="us_1" parent="base_link">
-    <origin xyz="0.100 0 0.300" rpy="0 3.14 3.14" />
-  </xacro:us_sensor-->
+  <!--><xacro:us_sensor name="us_1" parent="base_link">
+    <origin xyz="0.100 0 0.500" rpy="0 3.14 3.14" />
+  </xacro:us_sensor><-->
   <!-- SENSOR 2 -->
   <!-- xacro:us_sensor name="us_2" parent="base_link">
@@ -107,5 +109,5 @@
     <origin xyz="0.230 0 0.300" rpy="0 3.14 3.14" />
   </xacro:us_sensor-->
-      <!--Camera  -->
+  <!--Camera  -->
 <!-- <xacro:camera name="camera" parent="base_link">
     <origin xyz="0 0 0.38" rpy="0 0 0" />

File: robots/mp_500/xacros/mp_500_gazebo.xacro (robot description, xacro)
@@ -36,5 +36,6 @@
         </sensor>
   </gazebo>
-    <gazebo reference="imu_1_link">
+  <!-- IMU sensor -->
+  <gazebo reference="imu_link">
     <gravity>true</gravity>
     <sensor name="imu_sensor" type="imu">
@@ -55,4 +56,5 @@
     </sensor>
   </gazebo>
+  <!-- Ultrasonic sensors -->
   <gazebo reference="us_1_link">
   <!-- Visuals / Collisions omitted for this example -->
@@ -83,5 +85,5 @@
          <alwaysOn>true</alwaysOn>
          <updateRate>50</updateRate>
-         <topicName>us_sensor</topicName>
+         <topicName>ultrasonic/us1</topicName>
          <frameName>us_1_link</frameName>
          <radiation>SONAR</radiation>
@@ -90,5 +92,5 @@
   </sensor>
   </gazebo>
-    <!-- camera -->
+  <!-- camera -->
   <gazebo reference="camera_link">
     <sensor type="camera" name="camera1">

File: robots/mpo_500/mpo_500.urdf.xacro (robot description, xacro)
@@ -12,6 +12,8 @@
   <xacro:include filename="$(find neo_simulation)/robots/mpo_500/xacros/micro_scan.xacro" />
   <!--Ultrasonics, cameras and IMU's  -->
-  <!--<xacro:include filename="$(find neo_simulation)/robots/mpo_500/xacros/imu.xacro" />
-  <xacro:include filename="$(find neo_simulation)/robots/mpo_500/xacros/ultrasonic.xacro" /> -->
+  <!-->
+  <xacro:include filename="$(find neo_simulation)/robots/mpo_500/xacros/imu.xacro" />
+  <xacro:include filename="$(find neo_simulation)/robots/mpo_500/xacros/ultrasonic.xacro" />
+  <-->
   <!-- <xacro:include filename="$(find neo_simulation)/robots/mpo_500/xacros/camera.xacro" />  -->
   <!-- Base Macro-->
@@ -38,15 +40,19 @@
     <origin xyz="-0.442 0 0.372" rpy="0 0 3.14" />
   </xacro:sick_laser_v0>
-      <!--+++++++++++++++++++ IMU ++++++++++++++++++++++++-->
- <!-- Comment or uncomment based on your requirement -->
-<!--   <xacro:imu name="imu_1" parent="base_link">
+  <!--+++++++++++++++++++ IMU ++++++++++++++++++++++++-->
+  <!-- Comment or uncomment based on your requirement -->
+  <!-->
+  <xacro:imu name="imu" parent="base_link">
     <origin xyz="0.100 0 0.300" rpy="0 0 3.14" />
-  </xacro:imu> -->
+  </xacro:imu>
+  <-->
   <!--+++++++++++++++++++ Ultra Sonic ++++++++++++++++++++++++-->
   <!-- Comment or uncomment based on your requirement -->
   <!-- SENSOR 1 -->
-  <!-- xacro:us_sensor name="us_1" parent="base_link">
-    <origin xyz="0.100 0 0.300" rpy="0 3.14 3.14" />
-  </xacro:us_sensor-->
+  <!-->
+  <xacro:us_sensor name="us_1" parent="base_link">
+    <origin xyz="0.100 0 0.500" rpy="0 3.14 3.14" />
+  </xacro:us_sensor>
+  <-->
   <!-- SENSOR 2 -->
   <!-- xacro:us_sensor name="us_2" parent="base_link">
@@ -109,5 +115,5 @@
     <origin xyz="0.230 0 0.300" rpy="0 3.14 3.14" />
   </xacro:us_sensor-->
-      <!--Camera  -->
+  <!--Camera  -->
 <!-- <xacro:camera name="camera" parent="base_link">
     <origin xyz="0 0 0.38" rpy="0 0 0" />

File: robots/mpo_500/xacros/mpo_500_gazebo.xacro (robot description, xacro)
@@ -21,4 +21,5 @@
     <self_collide>false</self_collide>
   </gazebo>
+  <!-- Lidar sensors -->
   <gazebo reference="lidar_1_link">
       <sensor type="ray" name="lidar_1_sensor">
@@ -91,5 +92,6 @@
         </sensor>
   </gazebo>
- <gazebo reference="camera_link">
+  <!-- Camera -->
+  <gazebo reference="camera_link">
     <sensor type="camera" name="camera1">
       <update_rate>30.0</update_rate>
@@ -126,6 +128,7 @@
       </plugin>
     </sensor>
-  </gazebo>
-      <gazebo reference="imu_1_link">
+   </gazebo>
+  <!-- IMU sensor -->
+  <gazebo reference="imu_link">
     <gravity>true</gravity>
     <sensor name="imu_sensor" type="imu">
@@ -146,4 +149,5 @@
     </sensor>
   </gazebo>
+  <!-- Ultrasonic sensors -->
   <gazebo reference="us_1_link">
   <sensor type="ray" name="range">
@@ -169,4 +173,13 @@
          </range>
       </ray>
+      <plugin filename="libgazebo_ros_range.so" name="gazebo_ros_range">
+	<gaussianNoise>0.005</gaussianNoise>
+	<alwaysOn>true</alwaysOn>
+	<updateRate>50</updateRate>
+	<topicName>ultrasonic/us1</topicName>
+	<frameName>us_1_link</frameName>
+	<radiation>INFRARED</radiation>
+	<fov>0.2967</fov>
+      </plugin>
       </sensor>
   </gazebo>

File: robots/mpo_700/mpo_700.urdf.xacro (robot description, xacro)
@@ -9,7 +9,9 @@
   <xacro:include filename="$(find neo_simulation)/robots/mpo_700/xacros/micro_scan.xacro" />
   <!--Ultrasonics, cameras and IMU's  -->
-  <!-- <xacro:include filename="$(find neo_simulation)/robots/mpo_700/xacros/camera.xacro" /> -->
-  <!--<xacro:include filename="$(find neo_simulation)/robots/mpo_700/xacros/imu.xacro" />
-  <xacro:include filename="$(find neo_simulation)/robots/mpo_700/xacros/ultrasonic.xacro" /> -->
+  <!-->
+  <xacro:include filename="$(find neo_simulation)/robots/mpo_700/xacros/camera.xacro" />
+  <xacro:include filename="$(find neo_simulation)/robots/mpo_700/xacros/imu.xacro" />
+  <xacro:include filename="$(find neo_simulation)/robots/mpo_700/xacros/ultrasonic.xacro" />
+  <-->
   <!--Gazebo  -->
   <xacro:include filename="$(find neo_simulation)/robots/mpo_700/xacros/mpo_700_gazebo.xacro" />
@@ -46,4 +48,5 @@
   </xacro:mpo_700_wheel>
 <!-- Sensors -->
+  <!-- Lidar sensors -->
   <xacro:sick_laser_v0 name="lidar_1" parent="base_link" ros_topic="lidar_1/scan_filtered">
   <!--<origin xyz="0.360 0 0.181" rpy="3.14 0 0" />-->
@@ -55,14 +58,18 @@
   </xacro:sick_laser_v0>
      <!--+++++++++++++++++++ IMU ++++++++++++++++++++++++-->
- <!-- Comment or uncomment based on your requirement -->
-<!--   <xacro:imu name="imu_1" parent="base_link">
-    <origin xyz="0.100 0 0.300" rpy="0 0 3.14" />
-  </xacro:imu> -->
+  <!-- Comment or uncomment based on your requirement -->
+  <!-->
+  <xacro:imu name="imu" parent="base_link">
+    <origin xyz="0.100 0 0.500" rpy="0 0 3.14" />
+  </xacro:imu>
+  <-->
   <!--+++++++++++++++++++ Ultra Sonic ++++++++++++++++++++++++-->
   <!-- Comment or uncomment based on your requirement -->
   <!-- SENSOR 1 -->
-  <!-- xacro:us_sensor name="us_1" parent="base_link">
-    <origin xyz="0.100 0 0.300" rpy="0 3.14 3.14" />
-  </xacro:us_sensor-->
+  <!-->
+  <xacro:us_sensor name="us_1" parent="base_link">
+    <origin xyz="0.100 0 0.500" rpy="0 3.14 3.14" />
+  </xacro:us_sensor>
+  <-->
   <!-- SENSOR 2 -->
   <!-- xacro:us_sensor name="us_2" parent="base_link">
@@ -125,7 +132,8 @@
     <origin xyz="0.230 0 0.300" rpy="0 3.14 3.14" />
   </xacro:us_sensor-->
-      <!--Camera  -->
-<!-- <xacro:camera name="camera" parent="base_link">
+  <!--Camera  -->
+  <!--><xacro:camera name="camera" parent="base_link">
     <origin xyz="0 0 0.38" rpy="0 0 0" />
-  </xacro:camera> -->
+  </xacro:camera>
+  <-->
 </robot>
