Commit message: Sensors fixed, comments added.

File: robots/mpo_700/xacros/mpo_700_gazebo.xacro (robot description, xacro)
@@ -75,5 +75,5 @@
         </sensor>
   </gazebo>
-    <gazebo reference="imu_link">
+  <gazebo reference="imu_link">
     <gravity>true</gravity>
     <sensor name="imu_sensor" type="imu">
@@ -94,5 +94,4 @@
     </sensor>
   </gazebo>
-    <!-- camera -->
  <gazebo>
     <plugin name="mpo_700_controller" filename="libgazebo_ros_planar_move.so">
@@ -104,4 +103,5 @@
     </plugin>
   </gazebo>
+  <!-- camera -->
   <gazebo reference="camera_link">
     <sensor type="camera" name="camera1">
@@ -109,9 +109,9 @@
       <camera name="head">
         <horizontal_fov>1.3962634</horizontal_fov>
-        <image>
-          <width>800</width>
-          <height>800</height>
-          <format>R8G8B8</format>
-        </image>
+	<image>
+	  <width>800</width>
+ 	  <height>800</height>
+	  <format>R8G8B8</format>
+	</image>
         <clip>
           <near>0.02</near>
@@ -130,5 +130,5 @@
         <alwaysOn>true</alwaysOn>
         <updateRate>0.0</updateRate>
-        <cameraName>camera1</cameraName>
+        <cameraName>robot/camera1</cameraName>
         <imageTopicName>image_raw</imageTopicName>
         <cameraInfoTopicName>camera_info</cameraInfoTopicName>
@@ -143,5 +143,6 @@
     </sensor>
   </gazebo>
-    <gazebo reference="us_1_link">
+  <!-- Sonar -->
+  <gazebo reference="us_1_link">
   <!-- Visuals / Collisions omitted for this example -->
   <sensor type="ray" name="range">
@@ -167,4 +168,13 @@
          </range>
       </ray>
+      <plugin filename="libgazebo_ros_range.so" name="gazebo_ros_range">
+	<gaussianNoise>0.005</gaussianNoise>
+	<alwaysOn>true</alwaysOn>
+	<updateRate>50</updateRate>
+	<topicName>ultrasonic/us1</topicName>
+	<frameName>us_1_link</frameName>
+	<radiation>INFRARED</radiation>
+	<fov>0.2967</fov>
+      </plugin>
       </sensor>
   </gazebo>

Commit message: removing pilz arm from MM-400

File: robots/mm_400/mm_400.urdf.xacro (robot description, xacro)
@@ -14,9 +14,6 @@
 <!--+++++++++++++++++++cabinet++++++++++++++++++++++++-->
 <xacro:include filename="$(find neo_simulation)/robots/mm_400/urdf/xacros/cabinet.xacro" />
-<!-- PRBT -->
-<xacro:include filename="$(find neo_simulation)/robots/mm_400/urdf/prbt_macro.xacro" />
 <!-- Panda -->
-  <xacro:include filename="$(find neo_simulation)/robots/mm_400/urdf/panda_arm.xacro" />
- <!-- SENSORS -->
+<xacro:include filename="$(find neo_simulation)/robots/mm_400/urdf/panda_arm.xacro" />
 <!-- SENSORS -->
 <!-- <xacro:include filename="$(find neo_simulation)/robots/mm_400/urdf/xacros/sick_S300.xacro" /> -->
@@ -47,16 +44,9 @@
     <origin xyz="-0. 0.26 0.074" rpy="0 0 1.57" />
   </xacro:fixed_wheel_left>
-<!--  -->
-  <xacro:mm_400_cabinet name="cabinet" parent="base_link">
-    <origin xyz="0.02 0 0.551" rpy="0 0 3.14" />
-  </xacro:mm_400_cabinet>
-   <!-- Robot arm  -->
-  <xacro:prbt parent="cabinet_link" prefix="pilz">
+  <!-- Robot arm  -->
+  <!-- Panda -->
+  <xacro:panda_arm parent="base_link" prefix="panda">
     <origin xyz="0 0 0." rpy="0 0 0" />
-  </xacro:prbt>
-<!-- Panda -->
-<!--  <xacro:panda_arm parent="base_link" prefix="panda">
-    <origin xyz="0 0 0." rpy="0 0 0" />
-  </xacro:panda_arm> -->
+  </xacro:panda_arm>
   <!--+++++++++++++++++++laserscanner_link++++++++++++++++++++++++-->
   <xacro:sick_laser_v0 name="lidar_1" parent="base_link" ros_topic="lidar_1/scan_filtered">
